File: 10106052 PowerPack/3V_reference_voltage.sch (KiCad schematic (older format))
At the start: 0 parts

Commit message: +3V ref schematic block added
Parts:
- added C5, C7: 100n, symbol Device:C
- added C6: 1u, symbol Device:C
- added U2: LM4120AIM5-3.0, Package_TO_SOT_SMD:SOT-23-5_HandSoldering, symbol 10106052_PowerPack:LM4120AIM5-3.0
Connections:
- new net +3.0VREF: C5.1, C6.1, U2.5 (VOUT)
- new net +5V: C7.1, U2.3 (EN), U2.4 (VIN)
- new net GND: U2.2 (GND)
- new net GNDA: C5.2, C6.2, C7.2
Changed lines of the file:
@@
 Comment4 ""
 $EndDescr
+$Comp
+L 10106052_PowerPack:LM4120AIM5-3.0 U2
+U 1 1 5E88FB21
+P 6175 3725
+F 0 "U2" H 6175 4090 50  0000 C CNN
+F 1 "LM4120AIM5-3.0" H 6175 3999 50  0000 C CNN
+F 2 "Package_TO_SOT_SMD:SOT-23-5_HandSoldering" H 6175 3725 50  0001 C CNN
+F 3 "" H 6175 3725 50  0001 C CNN
+	1    6175 3725
+	1    0    0    -1
+$EndComp
+Wire Wire Line
+	6575 3725 6650 3725
+Wire Wire Line
+	6650 3725 6650 3775
+$Comp
+L power:GND #PWR?
+U 1 1 5E88FF57
+P 6650 3775
+F 0 "#PWR?" H 6650 3525 50  0001 C CNN
+F 1 "GND" H 6650 3625 50  0000 C CNN
+F 2 "" H 6650 3775 50  0001 C CNN
+F 3 "" H 6650 3775 50  0001 C CNN
+	1    6650 3775
+	1    0    0    -1
+$EndComp
+$Comp
+L Device:C C7
+U 1 1 5E8911E8
+P 5550 4025
+F 0 "C7" H 5665 4071 50  0000 L CNN
+F 1 "100n" H 5665 3980 50  0000 L CNN
+F 2 "" H 5588 3875 50  0001 C CNN
+F 3 "~" H 5550 4025 50  0001 C CNN
+	1    5550 4025
+	1    0    0    -1
+$EndComp
+$Comp
+L Device:C C6
+U 1 1 5E891DE6
+P 5125 4025
+F 0 "C6" H 5240 4071 50  0000 L CNN
+F 1 "1u" H 5240 3980 50  0000 L CNN
+F 2 "" H 5163 3875 50  0001 C CNN
+F 3 "~" H 5125 4025 50  0001 C CNN
+	1    5125 4025
+	1    0    0    -1
+$EndComp
+$Comp
+L Device:C C5
+U 1 1 5E89226C
+P 4725 4025
+F 0 "C5" H 4840 4071 50  0000 L CNN
+F 1 "100n" H 4840 3980 50  0000 L CNN
+F 2 "" H 4763 3875 50  0001 C CNN
+F 3 "~" H 4725 4025 50  0001 C CNN
+	1    4725 4025
+	1    0    0    -1
+$EndComp
+Wire Wire Line
+	5550 3875 5550 3725
+Wire Wire Line
+	4525 3825 4725 3825
+Wire Wire Line
+	5125 3875 5125 3825
+Connection ~ 5125 3825
+Wire Wire Line
+	5125 3825 5775 3825
+Wire Wire Line
+	4725 3875 4725 3825
+Connection ~ 4725 3825
+Wire Wire Line
+	4725 3825 5125 3825
+Wire Wire Line
+	4725 4175 4725 4225
+Wire Wire Line
+	4725 4225 5125 4225
+Wire Wire Line
+	5550 4225 5550 4175
+Wire Wire Line
+	5125 4175 5125 4225
+Connection ~ 5125 4225
+Wire Wire Line
+	5125 4225 5550 4225
+$Comp
+L power:GNDA #PWR?
+U 1 1 5E894D35
+P 5125 4225
+F 0 "#PWR?" H 5125 3975 50  0001 C CNN
+F 1 "GNDA" H 5130 4052 50  0000 C CNN
+F 2 "" H 5125 4225 50  0001 C CNN
+F 3 "" H 5125 4225 50  0001 C CNN
+	1    5125 4225
+	1    0    0    -1
+$EndComp
+Wire Wire Line
+	5550 3725 5775 3725
+Connection ~ 5550 3725
+Wire Wire Line
+	5550 3725 5550 3625
+Wire Wire Line
+	5775 3625 5550 3625
+Connection ~ 5550 3625
+Wire Wire Line
+	5550 3625 5550 3375
+$Comp
+L power:+5V #PWR?
+U 1 1 5E89588F
+P 5550 3375
+F 0 "#PWR?" H 5550 3225 50  0001 C CNN
+F 1 "+5V" H 5565 3548 50  0000 C CNN
+F 2 "" H 5550 3375 50  0001 C CNN
+F 3 "" H 5550 3375 50  0001 C CNN
+	1    5550 3375
+	1    0    0    -1
+$EndComp
+Text HLabel 4525 3825 0    50   Output ~ 0
++3.0VREF
 $EndSCHEMATC
