File: 10106052 PowerPack/5V_power_supply.sch (KiCad schematic (older format))
At the start: 9 parts, among them T3 SI2309CDS-T1-GE3, T5 SI2300DS-T1-GE3, U1 NCV87722DT50RKG

Commit message: Initial Microntroller Work
Created the PIC symbol
Started the initial schematic page
Parts:
- D5: symbol dk_Diodes-Rectifiers-Arrays:BAT54C-7-F -> 10106052-PowerPack-rescue:BAT54C-7-F-dk_Diodes-Rectifiers-Arrays
- U1: symbol 10106052~PowerPack:NCV87722DT50RKG -> 10106052-PowerPack-rescue:NCV87722DT50RKG-10106052~PowerPack
Changed lines of the file:
@@
 $EndDescr
 $Comp
-L 10106052~PowerPack:NCV87722DT50RKG U1
+L 10106052-PowerPack-rescue:NCV87722DT50RKG-10106052~PowerPack U1
 U 1 1 5E87972E
 P 6900 3600
+AR Path="/5E87972E" Ref="U1"  Part="1"
+AR Path="/5E87819A/5E87972E" Ref="U1"  Part="1"
 F 0 "U1" H 6900 4015 50  0000 C CNN
 F 1 "NCV87722DT50RKG" H 6900 3924 50  0000 C CNN
@@
 	4825 3700 4575 3700
 $Comp
-L dk_Diodes-Rectifiers-Arrays:BAT54C-7-F D5
+L 10106052-PowerPack-rescue:BAT54C-7-F-dk_Diodes-Rectifiers-Arrays D5
 U 1 1 5E884331
 P 4025 5000

Commit message: Cleanup extra pro files and rescue library
Parts:
- D5: symbol 10106052-PowerPack-rescue:BAT54C-7-F-dk_Diodes-Rectifiers-Arrays -> 10106052_PowerPack:BAT54C-7-F-dk_Diodes-Rectifiers-Arrays
- U1: symbol 10106052-PowerPack-rescue:NCV87722DT50RKG-10106052~PowerPack -> 10106052_PowerPack:NCV87722DT50RKG-10106052_PowerPack
Changed lines of the file:
@@
-EESchema Schematic File Version 4
-EELAYER 30 0
+EESchema Schematic File Version 5
+EELAYER 33 0
 EELAYER END
 $Descr A4 11693 8268
@@
 Comment3 ""
 Comment4 ""
+Comment5 ""
+Comment6 ""
+Comment7 ""
+Comment8 ""
+Comment9 ""
 $EndDescr
-$Comp
-L 10106052-PowerPack-rescue:NCV87722DT50RKG-10106052~PowerPack U1
-U 1 1 5E87972E
-P 6900 3600
-AR Path="/5E87972E" Ref="U1"  Part="1"
-AR Path="/5E87819A/5E87972E" Ref="U1"  Part="1"
-F 0 "U1" H 6900 4015 50  0000 C CNN
-F 1 "NCV87722DT50RKG" H 6900 3924 50  0000 C CNN
-F 2 "" H 6900 3450 50  0001 C CNN
-F 3 "" H 6900 3450 50  0001 C CNN
-	1    6900 3600
-	1    0    0    -1
-$EndComp
-$Comp
-L Device:C C2
-U 1 1 5E879983
-P 7650 3800
-F 0 "C2" H 7765 3846 50  0000 L CNN
-F 1 "C" H 7765 3755 50  0000 L CNN
-F 2 "" H 7688 3650 50  0001 C CNN
-F 3 "~" H 7650 3800 50  0001 C CNN
-	1    7650 3800
-	1    0    0    -1
-$EndComp
+Connection ~ 6900 4250
+Connection ~ 7650 3500
+Connection ~ 3825 3200
+Connection ~ 4575 2750
+Connection ~ 5075 2750
+Connection ~ 3250 3950
+Connection ~ 3825 4275
+Connection ~ 5550 3500
+Connection ~ 5550 4275
+Connection ~ 4825 3700
+NoConn ~ 7300 3700
+Wire Wire Line
+	3150 3950 3250 3950
+Wire Wire Line
+	3250 3950 3525 3950
+Wire Wire Line
+	3250 4275 3250 3950
+Wire Wire Line
+	3250 4275 3375 4275
+Wire Wire Line
+	3675 4275 3825 4275
+Wire Wire Line
+	3675 4900 3825 4900
+Wire Wire Line
+	3675 5100 3825 5100
+Wire Wire Line
+	3825 2750 3825 3200
+Wire Wire Line
+	3825 3200 4275 3200
+Wire Wire Line
+	3825 3325 3825 3200
+Wire Wire Line
+	3825 3750 3825 3625
+Wire Wire Line
+	3825 4275 3825 4150
+Wire Wire Line
+	3825 4275 5550 4275
+Wire Wire Line
+	4050 2750 3825 2750
+Wire Wire Line
+	4350 2750 4575 2750
+Wire Wire Line
+	4575 2750 4575 3000
+Wire Wire Line
+	4575 2750 5075 2750
+Wire Wire Line
+	4575 3700 4575 3400
+Wire Wire Line
+	4825 3700 4575 3700
+Wire Wire Line
+	4825 3700 4825 5000
+Wire Wire Line
+	4825 5000 4325 5000
+Wire Wire Line
+	5075 2750 5075 2625
+Wire Wire Line
+	5075 2750 5550 2750
+Wire Wire Line
+	5550 2750 5550 3500
+Wire Wire Line
+	5550 3500 6500 3500
+Wire Wire Line
+	5550 3825 5550 3500
+Wire Wire Line
+	5550 4275 5550 4125
+Wire Wire Line
+	5550 4300 5550 4275
+Wire Wire Line
+	6500 3700 4825 3700
+Wire Wire Line
+	6900 4250 6900 3950
+Wire Wire Line
+	7650 3325 7650 3500
+Wire Wire Line
+	7650 3500 7300 3500
 Wire Wire Line
 	7650 3650 7650 3500
 Wire Wire Line
-	7650 3500 7300 3500
-Wire Wire Line
 	7650 3950 7650 4250
 Wire Wire Line
 	7650 4250 6900 4250
-Wire Wire Line
-	6900 4250 6900 3950
+Text GLabel 5075 2625 1    50   Input ~ 0
++VDC_PERM
+Text HLabel 3150 3950 0    50   Input ~ 0
+V_EN
+Text HLabel 3675 4900 0    50   Input ~ 0
+BP
+Text HLabel 3675 5100 0    50   Input ~ 0
+V_DC_CHARGER
+$Comp
+L power:+5V #PWR?
+U 1 1 5E87AC0C
+P 7650 3325
+F 0 "#PWR?" H 7650 3175 50  0001 C CNN
+F 1 "+5V" H 7665 3498 50  0000 C CNN
+F 2 "" H 7650 3325 50  0001 C CNN
+F 3 "" H 7650 3325 50  0001 C CNN
+	1    7650 3325
+	1    0    0    -1
+$EndComp
+$Comp
+L power:GND #PWR?
+U 1 1 5E8825AC
+P 5550 4300
+F 0 "#PWR?" H 5550 4050 50  0001 C CNN
+F 1 "GND" H 5555 4127 50  0000 C CNN
+F 2 "" H 5550 4300 50  0001 C CNN
+F 3 "" H 5550 4300 50  0001 C CNN
+	1    5550 4300
+	1    0    0    -1
+$EndComp
 $Comp
 L power:GND #PWR?
@@
 	1    0    0    -1
 $EndComp
-Connection ~ 6900 4250
-$Comp
-L power:+5V #PWR?
-U 1 1 5E87AC0C
-P 7650 3325
-F 0 "#PWR?" H 7650 3175 50  0001 C CNN
-F 1 "+5V" H 7665 3498 50  0000 C CNN
-F 2 "" H 7650 3325 50  0001 C CNN
-F 3 "" H 7650 3325 50  0001 C CNN
-	1    7650 3325
-	1    0    0    -1
-$EndComp
-Wire Wire Line
-	7650 3325 7650 3500
-Connection ~ 7650 3500
-NoConn ~ 7300 3700
-$Comp
-L Device:Q_NMOS_GSD T3
-U 1 1 5E87B529
-P 4475 3200
-F 0 "T3" H 4681 3246 50  0000 L CNN
-F 1 "SI2309CDS-T1-GE3" H 4681 3155 50  0000 L CNN
-F 2 "" H 4675 3300 50  0001 C CNN
-F 3 "~" H 4475 3200 50  0001 C CNN
-	1    4475 3200
-	1    0    0    -1
-$EndComp
-$Comp
-L Device:Q_NMOS_GSD T5
-U 1 1 5E87BE5D
-P 3725 3950
-F 0 "T5" H 3931 3996 50  0000 L CNN
-F 1 "SI2300DS-T1-GE3" H 3931 3905 50  0000 L CNN
-F 2 "" H 3925 4050 50  0001 C CNN
-F 3 "~" H 3725 3950 50  0001 C CNN
-	1    3725 3950
-	1    0    0    -1
+$Comp
+L Device:R R11
+U 1 1 5E87F3FA
+P 3525 4275
+F 0 "R11" V 3425 4250 50  0000 C CNN
+F 1 "10k" V 3325 4275 50  0000 C CNN
+F 2 "" V 3455 4275 50  0001 C CNN
+F 3 "~" H 3525 4275 50  0001 C CNN
+	1    3525 4275
+	0    1    -1   0
 $EndComp
 $Comp
@@
 	1    0    0    -1
 $EndComp
-Wire Wire Line
-	3825 3750 3825 3625
-Wire Wire Line
-	3825 3325 3825 3200
-Wire Wire Line
-	3825 3200 4275 3200
 $Comp
 L Device:R R6
@@
 	0    1    1    0
 $EndComp
-Wire Wire Line
-	4050 2750 3825 2750
-Wire Wire Line
-	3825 2750 3825 3200
-Connection ~ 3825 3200
-Wire Wire Line
-	4350 2750 4575 2750
-Wire Wire Line
-	4575 2750 4575 3000
-Wire Wire Line
-	4575 2750 5075 2750
-Wire Wire Line
-	5075 2750 5075 2625
-Connection ~ 4575 2750
-Wire Wire Line
-	5075 2750 5550 2750
-Wire Wire Line
-	5550 2750 5550 3500
-Wire Wire Line
-	5550 3500 6500 3500
-Connection ~ 5075 2750
-Text GLabel 5075 2625 1    50   Input ~ 0
-+VDC_PERM
-Wire Wire Line
-	3150 3950 3250 3950
-Text HLabel 3150 3950 0    50   Input ~ 0
-V_EN
-$Comp
-L Device:R R11
-U 1 1 5E87F3FA
-P 3525 4275
-F 0 "R11" V 3425 4250 50  0000 C CNN
-F 1 "10k" V 3325 4275 50  0000 C CNN
-F 2 "" V 3455 4275 50  0001 C CNN
-F 3 "~" H 3525 4275 50  0001 C CNN
-	1    3525 4275
-	0    1    -1   0
-$EndComp
-Wire Wire Line
-	3675 4275 3825 4275
-Wire Wire Line
-	3825 4275 3825 4150
-Wire Wire Line
-	3250 4275 3250 3950
-Wire Wire Line
-	3250 4275 3375 4275
-Connection ~ 3250 3950
-Wire Wire Line
-	3250 3950 3525 3950
-Wire Wire Line
-	3825 4275 5550 4275
-Wire Wire Line
-	5550 4275 5550 4125
-Connection ~ 3825 4275
 $Comp
 L Device:C C3
@@
 	1    0    0    -1
 $EndComp
-Wire Wire Line
-	5550 3825 5550 3500
-Connection ~ 5550 3500
-$Comp
-L power:GND #PWR?
-U 1 1 5E8825AC
-P 5550 4300
-F 0 "#PWR?" H 5550 4050 50  0001 C CNN
-F 1 "GND" H 5555 4127 50  0000 C CNN
-F 2 "" H 5550 4300 50  0001 C CNN
-F 3 "" H 5550 4300 50  0001 C CNN
-	1    5550 4300
-	1    0    0    -1
-$EndComp
-Wire Wire Line
-	5550 4300 5550 4275
-Connection ~ 5550 4275
-Wire Wire Line
-	6500 3700 4825 3700
-Wire Wire Line
-	4575 3700 4575 3400
-Wire Wire Line
-	4825 3700 4825 5000
-Wire Wire Line
-	4825 5000 4325 5000
-Connection ~ 4825 3700
-Wire Wire Line
-	4825 3700 4575 3700
-$Comp
-L 10106052-PowerPack-rescue:BAT54C-7-F-dk_Diodes-Rectifiers-Arrays D5
+$Comp
+L Device:C C2
+U 1 1 5E879983
+P 7650 3800
+F 0 "C2" H 7765 3846 50  0000 L CNN
+F 1 "C" H 7765 3755 50  0000 L CNN
+F 2 "" H 7688 3650 50  0001 C CNN
+F 3 "~" H 7650 3800 50  0001 C CNN
+	1    7650 3800
+	1    0    0    -1
+$EndComp
+$Comp
+L 10106052_PowerPack:BAT54C-7-F-dk_Diodes-Rectifiers-Arrays D5
 U 1 1 5E884331
 P 4025 5000
@@
 	1    0    0    -1
 $EndComp
-Text HLabel 3675 4900 0    50   Input ~ 0
-BP
-Wire Wire Line
-	3675 4900 3825 4900
-Text HLabel 3675 5100 0    50   Input ~ 0
-V_DC_CHARGER
-Wire Wire Line
-	3675 5100 3825 5100
+$Comp
+L Device:Q_NMOS_GSD T5
+U 1 1 5E87BE5D
+P 3725 3950
+F 0 "T5" H 3931 3996 50  0000 L CNN
+F 1 "SI2300DS-T1-GE3" H 3931 3905 50  0000 L CNN
+F 2 "" H 3925 4050 50  0001 C CNN
+F 3 "~" H 3725 3950 50  0001 C CNN
+	1    3725 3950
+	1    0    0    -1
+$EndComp
+$Comp
+L Device:Q_NMOS_GSD T3
+U 1 1 5E87B529
+P 4475 3200
+F 0 "T3" H 4681 3246 50  0000 L CNN
+F 1 "SI2309CDS-T1-GE3" H 4681 3155 50  0000 L CNN
+F 2 "" H 4675 3300 50  0001 C CNN
+F 3 "~" H 4475 3200 50  0001 C CNN
+	1    4475 3200
+	1    0    0    -1
+$EndComp
+$Comp
+L 10106052_PowerPack:NCV87722DT50RKG-10106052_PowerPack U1
+U 1 1 5E87972E
+P 6900 3600
+AR Path="/5E87972E" Ref="U1"  Part="1"
+AR Path="/5E87819A/5E87972E" Ref="U1"  Part="1"
+F 0 "U1" H 6900 4015 50  0000 C CNN
+F 1 "NCV87722DT50RKG" H 6900 3924 50  0000 C CNN
+F 2 "" H 6900 3450 50  0001 C CNN
+F 3 "" H 6900 3450 50  0001 C CNN
+	1    6900 3600
+	1    0    0    -1
+$EndComp
 $EndSCHEMATC

Commit message: start to create switching block
Parts:
- D5: symbol 10106052_PowerPack:BAT54C-7-F-dk_Diodes-Rectifiers-Arrays -> 10106052-PowerPack-rescue:BAT54C-7-F-dk_Diodes-Rectifiers-Arrays
- U1: symbol 10106052_PowerPack:NCV87722DT50RKG-10106052_PowerPack -> 10106052-PowerPack-rescue:NCV87722DT50RKG-10106052_PowerPack
Changed lines of the file:
@@
-EESchema Schematic File Version 5
-EELAYER 33 0
+EESchema Schematic File Version 4
+EELAYER 30 0
 EELAYER END
 $Descr A4 11693 8268
@@
 Comment3 ""
 Comment4 ""
-Comment5 ""
-Comment6 ""
-Comment7 ""
-Comment8 ""
-Comment9 ""
 $EndDescr
+$Comp
+L 10106052-PowerPack-rescue:NCV87722DT50RKG-10106052_PowerPack U1
+U 1 1 5E87972E
+P 6900 3600
+AR Path="/5E87972E" Ref="U1"  Part="1"
+AR Path="/5E87819A/5E87972E" Ref="U1"  Part="1"
+F 0 "U1" H 6900 4015 50  0000 C CNN
+F 1 "NCV87722DT50RKG" H 6900 3924 50  0000 C CNN
+F 2 "" H 6900 3450 50  0001 C CNN
+F 3 "" H 6900 3450 50  0001 C CNN
+	1    6900 3600
+	1    0    0    -1
+$EndComp
+$Comp
+L Device:C C2
+U 1 1 5E879983
+P 7650 3800
+F 0 "C2" H 7765 3846 50  0000 L CNN
+F 1 "C" H 7765 3755 50  0000 L CNN
+F 2 "" H 7688 3650 50  0001 C CNN
+F 3 "~" H 7650 3800 50  0001 C CNN
+	1    7650 3800
+	1    0    0    -1
+$EndComp
+Wire Wire Line
+	7650 3650 7650 3500
+Wire Wire Line
+	7650 3500 7300 3500
+Wire Wire Line
+	7650 3950 7650 4250
+Wire Wire Line
+	7650 4250 6900 4250
+Wire Wire Line
+	6900 4250 6900 3950
+$Comp
+L power:GND #PWR?
+U 1 1 5E87A940
+P 6900 4250
+F 0 "#PWR?" H 6900 4000 50  0001 C CNN
+F 1 "GND" H 6905 4077 50  0000 C CNN
+F 2 "" H 6900 4250 50  0001 C CNN
+F 3 "" H 6900 4250 50  0001 C CNN
+	1    6900 4250
+	1    0    0    -1
+$EndComp
 Connection ~ 6900 4250
-Connection ~ 7650 3500
-Connection ~ 3825 3200
-Connection ~ 4575 2750
-Connection ~ 5075 2750
-Connection ~ 3250 3950
-Connection ~ 3825 4275
-Connection ~ 5550 3500
-Connection ~ 5550 4275
-Connection ~ 4825 3700
-NoConn ~ 7300 3700
-Wire Wire Line
-	3150 3950 3250 3950
-Wire Wire Line
-	3250 3950 3525 3950
-Wire Wire Line
-	3250 4275 3250 3950
-Wire Wire Line
-	3250 4275 3375 4275
-Wire Wire Line
-	3675 4275 3825 4275
-Wire Wire Line
-	3675 4900 3825 4900
-Wire Wire Line
-	3675 5100 3825 5100
-Wire Wire Line
-	3825 2750 3825 3200
-Wire Wire Line
-	3825 3200 4275 3200
-Wire Wire Line
-	3825 3325 3825 3200
-Wire Wire Line
-	3825 3750 3825 3625
-Wire Wire Line
-	3825 4275 3825 4150
-Wire Wire Line
-	3825 4275 5550 4275
-Wire Wire Line
-	4050 2750 3825 2750
-Wire Wire Line
-	4350 2750 4575 2750
-Wire Wire Line
-	4575 2750 4575 3000
-Wire Wire Line
-	4575 2750 5075 2750
-Wire Wire Line
-	4575 3700 4575 3400
-Wire Wire Line
-	4825 3700 4575 3700
-Wire Wire Line
-	4825 3700 4825 5000
-Wire Wire Line
-	4825 5000 4325 5000
-Wire Wire Line
-	5075 2750 5075 2625
-Wire Wire Line
-	5075 2750 5550 2750
-Wire Wire Line
-	5550 2750 5550 3500
-Wire Wire Line
-	5550 3500 6500 3500
-Wire Wire Line
-	5550 3825 5550 3500
-Wire Wire Line
-	5550 4275 5550 4125
-Wire Wire Line
-	5550 4300 5550 4275
-Wire Wire Line
-	6500 3700 4825 3700
-Wire Wire Line
-	6900 4250 6900 3950
-Wire Wire Line
-	7650 3325 7650 3500
-Wire Wire Line
-	7650 3500 7300 3500
-Wire Wire Line
-	7650 3650 7650 3500
-Wire Wire Line
-	7650 3950 7650 4250
-Wire Wire Line
-	7650 4250 6900 4250
-Text GLabel 5075 2625 1    50   Input ~ 0
-+VDC_PERM
-Text HLabel 3150 3950 0    50   Input ~ 0
-V_EN
-Text HLabel 3675 4900 0    50   Input ~ 0
-BP
-Text HLabel 3675 5100 0    50   Input ~ 0
-V_DC_CHARGER
 $Comp
 L power:+5V #PWR?
@@
 	1    0    0    -1
 $EndComp
-$Comp
-L power:GND #PWR?
-U 1 1 5E8825AC
-P 5550 4300
-F 0 "#PWR?" H 5550 4050 50  0001 C CNN
-F 1 "GND" H 5555 4127 50  0000 C CNN
-F 2 "" H 5550 4300 50  0001 C CNN
-F 3 "" H 5550 4300 50  0001 C CNN
-	1    5550 4300
-	1    0    0    -1
-$EndComp
-$Comp
-L power:GND #PWR?
-U 1 1 5E87A940
-P 6900 4250
-F 0 "#PWR?" H 6900 4000 50  0001 C CNN
-F 1 "GND" H 6905 4077 50  0000 C CNN
-F 2 "" H 6900 4250 50  0001 C CNN
-F 3 "" H 6900 4250 50  0001 C CNN
-	1    6900 4250
-	1    0    0    -1
-$EndComp
+Wire Wire Line
+	7650 3325 7650 3500
+Connection ~ 7650 3500
+NoConn ~ 7300 3700
+$Comp
+L Device:Q_NMOS_GSD T3
+U 1 1 5E87B529
+P 4475 3200
+F 0 "T3" H 4681 3246 50  0000 L CNN
+F 1 "SI2309CDS-T1-GE3" H 4681 3155 50  0000 L CNN
+F 2 "" H 4675 3300 50  0001 C CNN
+F 3 "~" H 4475 3200 50  0001 C CNN
+	1    4475 3200
+	1    0    0    -1
+$EndComp
+$Comp
+L Device:Q_NMOS_GSD T5
+U 1 1 5E87BE5D
+P 3725 3950
+F 0 "T5" H 3931 3996 50  0000 L CNN
+F 1 "SI2300DS-T1-GE3" H 3931 3905 50  0000 L CNN
+F 2 "" H 3925 4050 50  0001 C CNN
+F 3 "~" H 3725 3950 50  0001 C CNN
+	1    3725 3950
+	1    0    0    -1
+$EndComp
+$Comp
+L Device:R R9
+U 1 1 5E87D4E3
+P 3825 3475
+F 0 "R9" H 3895 3521 50  0000 L CNN
+F 1 "10k" H 3895 3430 50  0000 L CNN
+F 2 "" V 3755 3475 50  0001 C CNN
+F 3 "~" H 3825 3475 50  0001 C CNN
+	1    3825 3475
+	1    0    0    -1
+$EndComp
+Wire Wire Line
+	3825 3750 3825 3625
+Wire Wire Line
+	3825 3325 3825 3200
+Wire Wire Line
+	3825 3200 4275 3200
+$Comp
+L Device:R R6
+U 1 1 5E87DA14
+P 4200 2750
+F 0 "R6" V 3993 2750 50  0000 C CNN
+F 1 "10k" V 4084 2750 50  0000 C CNN
+F 2 "" V 4130 2750 50  0001 C CNN
+F 3 "~" H 4200 2750 50  0001 C CNN
+	1    4200 2750
+	0    1    1    0
+$EndComp
+Wire Wire Line
+	4050 2750 3825 2750
+Wire Wire Line
+	3825 2750 3825 3200
+Connection ~ 3825 3200
+Wire Wire Line
+	4350 2750 4575 2750
+Wire Wire Line
+	4575 2750 4575 3000
+Wire Wire Line
+	4575 2750 5075 2750
+Wire Wire Line
+	5075 2750 5075 2625
+Connection ~ 4575 2750
+Wire Wire Line
+	5075 2750 5550 2750
+Wire Wire Line
+	5550 2750 5550 3500
+Wire Wire Line
+	5550 3500 6500 3500
+Connection ~ 5075 2750
+Text GLabel 5075 2625 1    50   Input ~ 0
++VDC_PERM
+Wire Wire Line
+	3150 3950 3250 3950
+Text HLabel 3150 3950 0    50   Input ~ 0
+V_EN
 $Comp
 L Device:R R11
@@
 	0    1    -1   0
 $EndComp
-$Comp
-L Device:R R9
-U 1 1 5E87D4E3
-P 3825 3475
-F 0 "R9" H 3895 3521 50  0000 L CNN
-F 1 "10k" H 3895 3430 50  0000 L CNN
-F 2 "" V 3755 3475 50  0001 C CNN
-F 3 "~" H 3825 3475 50  0001 C CNN
-	1    3825 3475
-	1    0    0    -1
-$EndComp
-$Comp
-L Device:R R6
-U 1 1 5E87DA14
-P 4200 2750
-F 0 "R6" V 3993 2750 50  0000 C CNN
-F 1 "10k" V 4084 2750 50  0000 C CNN
-F 2 "" V 4130 2750 50  0001 C CNN
-F 3 "~" H 4200 2750 50  0001 C CNN
-	1    4200 2750
-	0    1    1    0
-$EndComp
+Wire Wire Line
+	3675 4275 3825 4275
+Wire Wire Line
+	3825 4275 3825 4150
+Wire Wire Line
+	3250 4275 3250 3950
+Wire Wire Line
+	3250 4275 3375 4275
+Connection ~ 3250 3950
+Wire Wire Line
+	3250 3950 3525 3950
+Wire Wire Line
+	3825 4275 5550 4275
+Wire Wire Line
+	5550 4275 5550 4125
+Connection ~ 3825 4275
 $Comp
 L Device:C C3
@@
 	1    0    0    -1
 $EndComp
-$Comp
-L Device:C C2
-U 1 1 5E879983
-P 7650 3800
-F 0 "C2" H 7765 3846 50  0000 L CNN
-F 1 "C" H 7765 3755 50  0000 L CNN
-F 2 "" H 7688 3650 50  0001 C CNN
-F 3 "~" H 7650 3800 50  0001 C CNN
-	1    7650 3800
-	1    0    0    -1
-$EndComp
-$Comp
-L 10106052_PowerPack:BAT54C-7-F-dk_Diodes-Rectifiers-Arrays D5
+Wire Wire Line
+	5550 3825 5550 3500
+Connection ~ 5550 3500
+$Comp
+L power:GND #PWR?
+U 1 1 5E8825AC
+P 5550 4300
+F 0 "#PWR?" H 5550 4050 50  0001 C CNN
+F 1 "GND" H 5555 4127 50  0000 C CNN
+F 2 "" H 5550 4300 50  0001 C CNN
+F 3 "" H 5550 4300 50  0001 C CNN
+	1    5550 4300
+	1    0    0    -1
+$EndComp
+Wire Wire Line
+	5550 4300 5550 4275
+Connection ~ 5550 4275
+Wire Wire Line
+	6500 3700 4825 3700
+Wire Wire Line
+	4575 3700 4575 3400
+Wire Wire Line
+	4825 3700 4825 5000
+Wire Wire Line
+	4825 5000 4325 5000
+Connection ~ 4825 3700
+Wire Wire Line
+	4825 3700 4575 3700
+$Comp
+L 10106052-PowerPack-rescue:BAT54C-7-F-dk_Diodes-Rectifiers-Arrays D5
 U 1 1 5E884331
 P 4025 5000
@@
 	1    0    0    -1
 $EndComp
-$Comp
-L Device:Q_NMOS_GSD T5
-U 1 1 5E87BE5D
-P 3725 3950
-F 0 "T5" H 3931 3996 50  0000 L CNN
-F 1 "SI2300DS-T1-GE3" H 3931 3905 50  0000 L CNN
-F 2 "" H 3925 4050 50  0001 C CNN
-F 3 "~" H 3725 3950 50  0001 C CNN
-	1    3725 3950
-	1    0    0    -1
-$EndComp
-$Comp
-L Device:Q_NMOS_GSD T3
-U 1 1 5E87B529
-P 4475 3200
-F 0 "T3" H 4681 3246 50  0000 L CNN
-F 1 "SI2309CDS-T1-GE3" H 4681 3155 50  0000 L CNN
-F 2 "" H 4675 3300 50  0001 C CNN
-F 3 "~" H 4475 3200 50  0001 C CNN
-	1    4475 3200
-	1    0    0    -1
-$EndComp
-$Comp
-L 10106052_PowerPack:NCV87722DT50RKG-10106052_PowerPack U1
-U 1 1 5E87972E
-P 6900 3600
-AR Path="/5E87972E" Ref="U1"  Part="1"
-AR Path="/5E87819A/5E87972E" Ref="U1"  Part="1"
-F 0 "U1" H 6900 4015 50  0000 C CNN
-F 1 "NCV87722DT50RKG" H 6900 3924 50  0000 C CNN
-F 2 "" H 6900 3450 50  0001 C CNN
-F 3 "" H 6900 3450 50  0001 C CNN
-	1    6900 3600
-	1    0    0    -1
-$EndComp
+Text HLabel 3675 4900 0    50   Input ~ 0
+BP
+Wire Wire Line
+	3675 4900 3825 4900
+Text HLabel 3675 5100 0    50   Input ~ 0
+V_DC_CHARGER
+Wire Wire Line
+	3675 5100 3825 5100
 $EndSCHEMATC

Commit message: micro block schematic done
Parts:
- D5: symbol 10106052-PowerPack-rescue:BAT54C-7-F-dk_Diodes-Rectifiers-Arrays -> 10106052-PowerPack-rescue:BAT54C-7-F-dk_Diodes-Rectifiers-Arrays-10106052-PowerPack-rescue
- U1: symbol 10106052-PowerPack-rescue:NCV87722DT50RKG-10106052_PowerPack -> 10106052-PowerPack-rescue:NCV87722DT50RKG-10106052_PowerPack-10106052-PowerPack-rescue
Changed lines of the file:
@@
 $EndDescr
 $Comp
-L 10106052-PowerPack-rescue:NCV87722DT50RKG-10106052_PowerPack U1
+L 10106052-PowerPack-rescue:NCV87722DT50RKG-10106052_PowerPack-10106052-PowerPack-rescue U1
 U 1 1 5E87972E
 P 6900 3600
@@
 	4825 3700 4575 3700
 $Comp
-L 10106052-PowerPack-rescue:BAT54C-7-F-dk_Diodes-Rectifiers-Arrays D5
+L 10106052-PowerPack-rescue:BAT54C-7-F-dk_Diodes-Rectifiers-Arrays-10106052-PowerPack-rescue D5
 U 1 1 5E884331
 P 4025 5000
