File: 10106052 PowerPack/switching_block.sch (KiCad schematic (older format))
At the start: 80 parts, among them J1 811-S1-002-10-015101, J11 43650-0229, J2 811-S1-002-10-015101, J3 811-S1-002-10-015101, J4 GKS 913 305 230 A 15 02 S, J5 811-S1-002-10-015101, J6 811-S1-002-10-015101, J7 811-S1-002-10-015101, J8 GKS 913 305 230 A 15 02 S, J9 26-61-4020, T1 2N7002TA, T10 2N7002TA, T12 2N7002TA, T13 2N7002TA, T14 SUD50P06-15, T15 2N7002TA, T2 SUD50P06-15, T4 SUD50P06-15, T6 2N7002TA, T7 2N7002TA, T8 SUD50P06-15, T9 SUD50P06-15, U3 INA170

Commit message: Added parameters to components
Parts:
- C1, C14, C4: Description (none) -> CAPACITOR CERAMIC 100NF 50V 10% X7R 0603; Item Number (none) -> 10021386; Manufacturer (none) -> Kemet; Manufacturer_No (none) -> C0603C104K5RACTU
- C10, C11, C12: Description (none) -> CAPACITOR CERAMIC,10NF,+/-10%,50V,0603; Item Number (none) -> 10022508; Manufacturer (none) -> Yageo; Manufacturer_No (none) -> CC0603KRX7R9BB103; Note (none) -> BOM lists 223858615636, this is the same
- C8, C9: Description (none) -> CAP EL 100UF 20% 50V LOW ESR; Item Number (none) -> 10107886; Manufacturer (none) -> Kemet; Manufacturer_No (none) -> ESW107M050AG3AA
- D1, D7, D9: Description (none) -> DIODE TRANSIL 33V, SMA; Item Number (none) -> 10060347; Manufacturer (none) -> STMicroelectronics; Manufacturer_No (none) -> SMA6J28A-TR
- D15: Description (none) -> DIODE ARRAY SCHOTTKY 30V SOT323; Manufacturer (none) -> ON Semiconductor; Manufacturer_No (none) -> BAT54CWT1G; Note (none) -> DNP
- D2, D8: Description (none) -> TVS AVAL DIODE ARRAY 2CH SC70-3; Item Number (none) -> GR101899; Manufacturer (none) -> Littelfuse Inc.; Manufacturer_No (none) -> SP0502BAJTG
- D3, D4, D6: Description (none) -> DIODE SCHOTTKY, 500MA,40V,SOD323; Item Number (none) -> 10022515; Manufacturer (none) -> Nexperia USA Inc.; Manufacturer_No (none) -> PMEG4005AEA,115
- F1: Description (none) -> PTC RESETTABLE 33V 1.1A 2016 SMD; Item Number (none) -> 10107889; Manufacturer (none) -> Littelfuse Inc.; Manufacturer_No (none) -> 2016L100/33
- FL1: Description (none) -> FILTER CC, 1MHZ-1GHZ, 10A, 50V; Item Number (none) -> 10022532; Manufacturer (none) -> Murata Electronics; Manufacturer_No (none) -> BNX002-01; Note (none) -> BNX002-11 is also on BOM
- J1, J2, J3, J5, J6, J7: Description (none) -> CONNECTOR 2 CONTACTS, 3.5A, HT 6.5MM; Item Number (none) -> 10021350; Manufacturer (none) -> Antelec; Manufacturer_No (none) -> ACPD25410265; Note (none) -> Need to request datasheet
- J11: footprint (none) -> Connector_Molex:Molex_Micro-Fit_3.0_43650-0215_1x02_P3.00mm_Vertical; Description (none) -> HEADER TH MOLEX MICRO-FIT 2 CIRCUITS 3MM 5A 250V; Item Number (none) -> 10107892; Manufacturer (none) -> Molex; Manufacturer_No (none) -> 0436500229
- J4, J8: Description (none) -> CONNECTOR, 1 CONTACTS, TEST PROBE; Item Number (none) -> 10023419; Manufacturer (none) -> Ingun; Manufacturer_No (none) -> GKS 913 305 230 A 15 02 S
- J9: Description (none) -> HEADER 2 PIN FRICTION LOCK MOLEX KK 156 SERIES; Item Number (none) -> 10107890; Manufacturer (none) -> Molex; Manufacturer_No (none) -> 0026614020
- R1, R10, R17, R19, R21, R30, R53, R56, R7: Description (none) -> RESISTOR,10K OHM.0.063W,+/-1%,0603; Item Number (none) -> 10022548; Manufacturer (none) -> Yageo; Manufacturer_No (none) -> RC0603FR-0710KL
- R12, R18, R2, R22, R54: Description (none) -> RESISTOR, 15K OHM, 0603, +/-1%; Item Number (none) -> 10023238; Manufacturer (none) -> Yageo; Manufacturer_No (none) -> CRCW060315K0FKEAHP; Note (none) -> BOM listed ASJ CR16153FL
- R13, R20, R23, R52, R8: Description (none) -> RESISTOR 22 KOHM 0.063W +/-1% 0603; Item Number (none) -> 10113300; Manufacturer (none) -> Yageo; Manufacturer_No (none) -> RC0603JR-0722KL
- R14, R4: Description (none) -> RESISTOR, 1K OHM, 0.063W,+/-1%, 0603; Item Number (none) -> 10022554; Manufacturer (none) -> Bourns; Manufacturer_No (none) -> CR0603-FX-1001ELF
- R15, R5: Description (none) -> RESISTOR 18 KOHM 0.063W +/-1% 0603; Item Number (none) -> 10113299; Manufacturer (none) -> Yageo; Manufacturer_No (none) -> RC0603FR-0718KL
- R16, R27, R3: Description (none) -> RES 100K OHM 1/10W 1% 0603 SMD; Item Number (none) -> 10001204; Manufacturer (none) -> Yageo; Manufacturer_No (none) -> RC0603FR-07100KL
- R24: Description (none) -> RESISTOR 0,015 OHM, 2W, +/-1%, 2512; Item Number (none) -> 10000838; Manufacturer (none) -> Welwyn; Manufacturer_No (none) -> LRF2512-R015FW
- R25: Description (none) -> RES,0OHM 1/8W 5% 1206; Item Number (none) -> 312937; Manufacturer (none) -> Panasonic; Manufacturer_No (none) -> ERJ-8GEY0R00V
- R28: Description (none) -> RESISTOR 66,5K OHM, 0,063W, +/-0,1%, 0603; Item Number (none) -> 10000836; Manufacturer (none) -> Welwyn; Manufacturer_No (none) -> PCF0603R-66K5BT1
- R29: Description (none) -> RESISTOR 40.2KOHM 0.1% 0.063W 0603; Item Number (none) -> 10021070; Manufacturer (none) -> Welwyn; Manufacturer_No (none) -> PCF0603-R-40K2BT1
- R32: Description (none) -> RESISTOR 470 OHM 1/8W 5% 1206; Item Number (none) -> 10107895; Manufacturer (none) -> Yageo; Manufacturer_No (none) -> RC1206JR-07470RL
- R50, R51: Description (none) -> RESISTOR 100 OHM 0.063W +/-1% 0603; Manufacturer (none) -> Yageo; Manufacturer_No (none) -> RC0603FR-07100RL; Note (none) -> DNP
- R55: Description (none) -> RESISTOR,47K OHM,0.063W,+/-1%,0603; Item Number (none) -> 10022734; Manufacturer (none) -> Yageo; Manufacturer_No (none) -> RC0603FR-0747KL
- R57, R58: Description (none) -> RES SMD 0 OHM JUMPER 1/10W 0603; Manufacturer (none) -> Yageo; Manufacturer_No (none) -> RC0603JR-070RL; Note (none) -> DNP
- RL1: Description (none) -> RELAY 24V 2POLES 8A RT2; Item Number (none) -> 10021053; Manufacturer (none) -> Finder; Manufacturer_No (none) -> 41.52.9.024.0010
- T1, T10, T12, T13, T15, T6, T7: Description (none) -> MOSFET N-CH 60V 115MA SOT23-3; Item Number (none) -> 10002095; Manufacturer (none) -> ON Semiconductor; Manufacturer_No (none) -> 2N7002LT1G
- T14, T2, T4, T8, T9: symbol Device:Q_NMOS_GDS -> Device:Q_PMOS_GDSD; Description (none) -> TRANSISTOR MOSFET, 60V, 50A, P CHANNEL; Item Number (none) -> 10095972; Manufacturer (none) -> Vishay Siliconix; Manufacturer_No (none) -> SUD50P06-15L-E3
- U3: Description (none) -> IC,CURRENT SHUNT MONITOR,MSOP; Item Number (none) -> 10022891; Manufacturer (none) -> Texas Instruments; Manufacturer_No (none) -> INA170EA/2K5
Connections:
- net at T2.2 (D), T4.2 (D): now also T2.4 (D), T4.4 (D)
- net at T8.2 (D), T9.2 (D): now also T8.4 (D), T9.4 (D)
- net at D9.1 (K), F1.1, R25.2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: now also T14.4 (D)

Commit message: Created Project Footprint Library
Parts:
- F1: footprint (none) -> 10106052 PowerPack:FUS4755X155N_1
- FL1: footprint (none) -> 10106052 PowerPack:BNX00201_1
- J4: footprint (none) -> 10106052 PowerPack:GKS-913-305-230-A-15-02-S_1
- J9: footprint (none) -> 10106052 PowerPack:CON2PHDR1000W777L396P_1
Changed lines of the file:
@@
 F 0 "J4" H 11300 2675 50  0000 R CNN
 F 1 "GKS 913 305 230 A 15 02 S" H 11600 2775 50  0000 R CNN
-F 2 "" H 11400 2700 50  0001 C CNN
+F 2 "10106052 PowerPack:GKS-913-305-230-A-15-02-S_1" H 11400 2700 50  0001 C CNN
 F 3 "https://worbis.shop/gks-913-306-230-a-1502-s.html" H 11400 2700 50  0001 C CNN
 F 4 "CONNECTOR, 1 CONTACTS, TEST PROBE" H 11400 2700 50  0001 C CNN "Description"
@@
 F 0 "FL1" H 9725 9448 50  0000 C CNN
 F 1 "BNX002-11" H 9725 9357 50  0000 C CNN
-F 2 "" H 9680 9120 50  0001 C CNN
+F 2 "10106052 PowerPack:BNX00201_1" H 9680 9120 50  0001 C CNN
 F 3 "https://media.digikey.com/pdf/Data%20Sheets/Murata%20PDFs/BNX00x_Series.pdf" H 9680 9120 50  0001 C CNN
 F 4 "FILTER CC, 1MHZ-1GHZ, 10A, 50V" H 9750 9075 50  0001 C CNN "Description"
@@
 F 0 "F1" V 2553 7225 50  0000 C CNN
 F 1 "Fuse" V 2644 7225 50  0000 C CNN
-F 2 "" V 2680 7225 50  0001 C CNN
+F 2 "10106052 PowerPack:FUS4755X155N_1" V 2680 7225 50  0001 C CNN
 F 3 "https://www.littelfuse.com/~/media/electronics/datasheets/resettable_ptcs/littelfuse_ptc_2016l_datasheet.pdf.pdf" H 2750 7225 50  0001 C CNN
 F 4 "PTC RESETTABLE 33V 1.1A 2016 SMD" H 2750 7225 50  0001 C CNN "Description"
@@
 F 0 "J9" H 1850 7175 50  0000 C CNN
 F 1 "26-61-4020" H 1775 7050 50  0000 C CNN
-F 2 "" H 1950 7225 50  0001 C CNN
+F 2 "10106052 PowerPack:CON2PHDR1000W777L396P_1" H 1950 7225 50  0001 C CNN
 F 3 "https://www.molex.com/pdm_docs/sd/026614020_sd.pdf" H 1950 7225 50  0001 C CNN
 F 4 "HEADER 2 PIN FRICTION LOCK MOLEX KK 156 SERIES" H 1950 7225 50  0001 C CNN "Description"

Commit message: Footprints relinked
Parts:
- C1, C10, C11, C12, C14, C4: footprint Capacitor_SMD:C_0603_1608Metric -> 10106052 PowerPack:CAPC1608X86N
- C8, C9: footprint Capacitor_THT:CP_Radial_D8.0mm_P3.50mm -> 10106052 PowerPack:CAPPRD350W60D800H1250PBA
- D1, D7, D9: footprint Diode_SMD:D_SMA -> 10106052 PowerPack:DIOM5126X203N_SWP
- D15, D2, D8: footprint Package_TO_SOT_SMD:SOT-323_SC-70 -> 10106052 PowerPack:SOT65P220X110-3N
- D3, D4, D6: footprint Diode_SMD:D_SOD-323 -> 10106052 PowerPack:SOD2512X110N_SWP
- F1: footprint 10106052 PowerPack:FUS4755X155N_1 -> 10106052 PowerPack:FUS4755X155N
- FL1: footprint 10106052 PowerPack:BNX00201_1 -> 10106052 PowerPack:BNX00201
- J1, J2, J3, J5, J6, J7: footprint Connector_PinHeader_2.54mm:PinHeader_1x02_P2.54mm_Vertical -> 10106052 PowerPack:CON254W80L508T254H600P
- J11: footprint Connector_Molex:Molex_Micro-Fit_3.0_43650-0215_1x02_P3.00mm_Vertical -> 10106052 PowerPack:CON-43650-0229
- J4: footprint 10106052 PowerPack:GKS-913-305-230-A-15-02-S_1 -> 10106052 PowerPack:GKS-913-305-230-A-15-02-S
- J8: footprint (none) -> 10106052 PowerPack:GKS-913-305-230-A-15-02-S
- J9: footprint 10106052 PowerPack:CON2PHDR1000W777L396P_1 -> 10106052 PowerPack:CON2PHDR1000W777L396P
- NT1: footprint (none) -> 10106052 PowerPack:STAR
- R1, R10, R12, R13, R14, R15, R16, R17, R18, R19, R2, R20, R21, R22, R23, R27, R28, R29, R3, R30, R4, R5, R50, R51, R52, R53, R54, R55, R56, R57, R58, R7, R8: footprint Resistor_SMD:R_0603_1608Metric -> 10106052 PowerPack:RESC1608X50AN
- R24: footprint Resistor_SMD:R_2512_6332Metric -> 10106052 PowerPack:RESC6533X80N
- R25, R32: footprint Resistor_SMD:R_1206_3216Metric -> 10106052 PowerPack:RESC3216X60N
- RL1: footprint Relay_THT:Relay_DPDT_Finder_40.52 -> 10106052 PowerPack:RLY-41-52-9-024-0010
- T1, T10, T12, T13, T15, T6, T7: footprint Package_TO_SOT_SMD:SOT-23 -> 10106052 PowerPack:SOT92P240X120-3N
- T14, T2, T4, T8, T9: footprint Package_TO_SOT_SMD:TO-252-3_TabPin2 -> 10106052 PowerPack:TO228P1003X238-3_4N
- U3: footprint Package_SO:MSOP-8_3x3mm_P0.65mm -> 10106052 PowerPack:SOP65P490X110-8N

Commit message: Added 3D Models, corrected orientation of parts on schematic, added TX/RX TP
Parts:
- D1, D7, D9: symbol Device:D_Schottky -> 10106052_PowerPack:SMA6J28A
- D3, D4, D6: symbol Device:D -> 10106052_PowerPack:PMEG4005AEA
- T14, T2, T4, T8, T9: Description TRANSISTOR MOSFET, 60V, 50A, P CHANNEL -> TRANSISTOR MOSFET, 60V, 50A, P CHANNEL, TO252
Connections:
- net +VDC_PERM: now also D3.2 (K), D4.2 (K), D6.2 (K); no longer D3.1 (K), D4.1 (K), D6.1 (K)
- net GND: now also D1.1 (A), D7.1 (A), D9.1 (A); no longer D1.2 (A), D7.2 (A), D9.2 (A)
- net GNDA: now also C4.1, R19.1; no longer C4.2, R19.2
- net VBAT2_MEAS: now also C4.2, R16.1, R19.2; no longer C4.1, R16.2, R19.1
- net V_DC_CHARGER: now also D4.1 (A); no longer D4.2 (A)
- net at J1.1 (Pin_1), J1.2 (Pin_2), R2.1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: now also D1.2 (K), D3.1 (A); no longer D1.1 (K), D3.2 (A)
- net at J5.1 (Pin_1), J5.2 (Pin_2), R18.1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: now also D6.1 (A), D7.2 (K), R16.2; no longer D6.2 (A), D7.1 (K), R16.1
- net at F1.1, R25.2, R27.1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: now also D9.2 (K); no longer D9.1 (K)
Other:
- moved on the sheet: D3, D4, D6
Changed lines of the file:
@@
 ID_BAT_READ
 $Comp
-L Device:D_Schottky D1
+L 10106052_PowerPack:SMA6J28A D1
 U 1 1 5E8958A9
 P 8700 2325
@@
 ID_BAT2
 $Comp
-L Device:D_Schottky D7
+L 10106052_PowerPack:SMA6J28A D7
 U 1 1 5E8B3A76
 P 8700 5075
@@
 F 2 "10106052 PowerPack:TO228P1003X238-3_4N" H 7975 1925 50  0001 C CNN
 F 3 "http://www.vishay.com/docs/72250/sud50p06.pdf" H 7775 1825 50  0001 C CNN
-F 4 "TRANSISTOR MOSFET, 60V, 50A, P CHANNEL" H 7775 1825 50  0001 C CNN "Description"
+F 4 "TRANSISTOR MOSFET, 60V, 50A, P CHANNEL, TO252" H 7775 1825 50  0001 C CNN "Description"
 F 5 "10095972" H 7775 1825 50  0001 C CNN "Item Number"
 F 6 "Vishay Siliconix" H 7775 1825 50  0001 C CNN "Manufacturer"
@@
 F 2 "10106052 PowerPack:TO228P1003X238-3_4N" H 7975 2800 50  0001 C CNN
 F 3 "http://www.vishay.com/docs/72250/sud50p06.pdf" H 7775 2700 50  0001 C CNN
-F 4 "TRANSISTOR MOSFET, 60V, 50A, P CHANNEL" H 7775 2700 50  0001 C CNN "Description"
+F 4 "TRANSISTOR MOSFET, 60V, 50A, P CHANNEL, TO252" H 7775 2700 50  0001 C CNN "Description"
 F 5 "10095972" H 7775 2700 50  0001 C CNN "Item Number"
 F 6 "Vishay Siliconix" H 7775 2700 50  0001 C CNN "Manufacturer"
@@
 F 2 "10106052 PowerPack:TO228P1003X238-3_4N" H 7225 4675 50  0001 C CNN
 F 3 "http://www.vishay.com/docs/72250/sud50p06.pdf" H 7025 4575 50  0001 C CNN
-F 4 "TRANSISTOR MOSFET, 60V, 50A, P CHANNEL" H 7025 4575 50  0001 C CNN "Description"
+F 4 "TRANSISTOR MOSFET, 60V, 50A, P CHANNEL, TO252" H 7025 4575 50  0001 C CNN "Description"
 F 5 "10095972" H 7025 4575 50  0001 C CNN "Item Number"
 F 6 "Vishay Siliconix" H 7025 4575 50  0001 C CNN "Manufacturer"
@@
 F 2 "10106052 PowerPack:TO228P1003X238-3_4N" H 7225 5550 50  0001 C CNN
 F 3 "http://www.vishay.com/docs/72250/sud50p06.pdf" H 7025 5450 50  0001 C CNN
-F 4 "TRANSISTOR MOSFET, 60V, 50A, P CHANNEL" H 7025 5450 50  0001 C CNN "Description"
+F 4 "TRANSISTOR MOSFET, 60V, 50A, P CHANNEL, TO252" H 7025 5450 50  0001 C CNN "Description"
 F 5 "10095972" H 7025 5450 50  0001 C CNN "Item Number"
 F 6 "Vishay Siliconix" H 7025 5450 50  0001 C CNN "Manufacturer"
@@
 Connection ~ 4550 1425
 Wire Wire Line
-	4900 975  5275 975
-Wire Wire Line
 	7875 975  7875 1425
 $Comp
@@
 F 7 "RC0603FR-07100KL" H 4150 4025 50  0001 C CNN "Manufacturer_No"
 	1    4150 4025
-	1    0    0    -1
+	1    0    0    1
 $EndComp
 $Comp
@@
 F 7 "RC0603FR-0710KL" H 4150 4500 50  0001 C CNN "Manufacturer_No"
 	1    4150 4500
-	1    0    0    -1
+	1    0    0    1
 $EndComp
 $Comp
@@
 F 7 "C0603C104K5RACTU" H 3800 4500 50  0001 C CNN "Manufacturer_No"
 	1    3800 4500
-	1    0    0    -1
+	1    0    0    1
 $EndComp
 $Comp
@@
 	7125 3825 7125 4175
 $Comp
-L Device:D D3
+L 10106052_PowerPack:PMEG4005AEA D3
 U 1 1 5E9EE36A
-P 3050 2225
-F 0 "D3" H 2925 2300 50  0000 C CNN
-F 1 "PMEG4005AEA" H 3375 2300 50  0000 C CNN
-F 2 "10106052 PowerPack:SOD2512X110N_SWP" H 3050 2225 50  0001 C CNN
-F 3 "https://assets.nexperia.com/documents/data-sheet/PMEG4005AEA.pdf" H 3050 2225 50  0001 C CNN
-F 4 "DIODE SCHOTTKY, 500MA,40V,SOD323" H 3050 2225 50  0001 C CNN "Description"
-F 5 "10022515" H 3050 2225 50  0001 C CNN "Item Number"
-F 6 "Nexperia USA Inc." H 3050 2225 50  0001 C CNN "Manufacturer"
-F 7 "PMEG4005AEA,115" H 3050 2225 50  0001 C CNN "Manufacturer_No"
-	1    3050 2225
-	1    0    0    -1
-$EndComp
-$Comp
-L Device:D D4
+P 3050 2200
+F 0 "D3" H 2925 2275 50  0000 C CNN
+F 1 "PMEG4005AEA" H 3375 2275 50  0000 C CNN
+F 2 "10106052 PowerPack:SOD2512X110N_SWP" H 3050 2200 50  0001 C CNN
+F 3 "https://assets.nexperia.com/documents/data-sheet/PMEG4005AEA.pdf" H 3050 2200 50  0001 C CNN
+F 4 "DIODE SCHOTTKY, 500MA,40V,SOD323" H 3050 2200 50  0001 C CNN "Description"
+F 5 "10022515" H 3050 2200 50  0001 C CNN "Item Number"
+F 6 "Nexperia USA Inc." H 3050 2200 50  0001 C CNN "Manufacturer"
+F 7 "PMEG4005AEA,115" H 3050 2200 50  0001 C CNN "Manufacturer_No"
+	1    3050 2200
+	1    0    0    -1
+$EndComp
+$Comp
+L 10106052_PowerPack:PMEG4005AEA D4
 U 1 1 5E9EF925
-P 3050 2475
-F 0 "D4" H 2925 2550 50  0000 C CNN
-F 1 "PMEG4005AEA" H 3375 2550 50  0000 C CNN
-F 2 "10106052 PowerPack:SOD2512X110N_SWP" H 3050 2475 50  0001 C CNN
-F 3 "https://assets.nexperia.com/documents/data-sheet/PMEG4005AEA.pdf" H 3050 2475 50  0001 C CNN
-F 4 "DIODE SCHOTTKY, 500MA,40V,SOD323" H 3050 2475 50  0001 C CNN "Description"
-F 5 "10022515" H 3050 2475 50  0001 C CNN "Item Number"
-F 6 "Nexperia USA Inc." H 3050 2475 50  0001 C CNN "Manufacturer"
-F 7 "PMEG4005AEA,115" H 3050 2475 50  0001 C CNN "Manufacturer_No"
-	1    3050 2475
-	1    0    0    -1
-$EndComp
-$Comp
-L Device:D D6
+P 3050 2450
+F 0 "D4" H 2925 2525 50  0000 C CNN
+F 1 "PMEG4005AEA" H 3375 2525 50  0000 C CNN
+F 2 "10106052 PowerPack:SOD2512X110N_SWP" H 3050 2450 50  0001 C CNN
+F 3 "https://assets.nexperia.com/documents/data-sheet/PMEG4005AEA.pdf" H 3050 2450 50  0001 C CNN
+F 4 "DIODE SCHOTTKY, 500MA,40V,SOD323" H 3050 2450 50  0001 C CNN "Description"
+F 5 "10022515" H 3050 2450 50  0001 C CNN "Item Number"
+F 6 "Nexperia USA Inc." H 3050 2450 50  0001 C CNN "Manufacturer"
+F 7 "PMEG4005AEA,115" H 3050 2450 50  0001 C CNN "Manufacturer_No"
+	1    3050 2450
+	1    0    0    -1
+$EndComp
+$Comp
+L 10106052_PowerPack:PMEG4005AEA D6
 U 1 1 5E9EFC87
-P 3050 2725
-F 0 "D6" H 2925 2800 50  0000 C CNN
-F 1 "PMEG4005AEA" H 3375 2800 50  0000 C CNN
-F 2 "10106052 PowerPack:SOD2512X110N_SWP" H 3050 2725 50  0001 C CNN
-F 3 "https://assets.nexperia.com/documents/data-sheet/PMEG4005AEA.pdf" H 3050 2725 50  0001 C CNN
-F 4 "DIODE SCHOTTKY, 500MA,40V,SOD323" H 3050 2725 50  0001 C CNN "Description"
-F 5 "10022515" H 3050 2725 50  0001 C CNN "Item Number"
-F 6 "Nexperia USA Inc." H 3050 2725 50  0001 C CNN "Manufacturer"
-F 7 "PMEG4005AEA,115" H 3050 2725 50  0001 C CNN "Manufacturer_No"
-	1    3050 2725
-	1    0    0    -1
-$EndComp
-Wire Wire Line
-	3200 2225 5275 2225
-Wire Wire Line
-	5275 2225 5275 975
-Connection ~ 5275 975
-Wire Wire Line
-	5275 975  7875 975
-Wire Wire Line
-	3200 2725 4150 2725
-Wire Wire Line
-	4150 2725 4150 3825
+P 3050 2700
+F 0 "D6" H 2925 2775 50  0000 C CNN
+F 1 "PMEG4005AEA" H 3375 2775 50  0000 C CNN
+F 2 "10106052 PowerPack:SOD2512X110N_SWP" H 3050 2700 50  0001 C CNN
+F 3 "https://assets.nexperia.com/documents/data-sheet/PMEG4005AEA.pdf" H 3050 2700 50  0001 C CNN
+F 4 "DIODE SCHOTTKY, 500MA,40V,SOD323" H 3050 2700 50  0001 C CNN "Description"
+F 5 "10022515" H 3050 2700 50  0001 C CNN "Item Number"
+F 6 "Nexperia USA Inc." H 3050 2700 50  0001 C CNN "Manufacturer"
+F 7 "PMEG4005AEA,115" H 3050 2700 50  0001 C CNN "Manufacturer_No"
+	1    3050 2700
+	1    0    0    -1
+$EndComp
+Wire Wire Line
+	3200 2700 4150 2700
 Connection ~ 4150 3825
 Wire Wire Line
-	3200 2475 3725 2475
+	3200 2450 3725 2450
 Text HLabel 4950 7725 2    50   Output ~ 0
 V_DC_CHARGER
-Wire Wire Line
-	2900 2225 2750 2225
-Wire Wire Line
-	2750 2225 2750 2475
-Wire Wire Line
-	2750 2725 2900 2725
-Wire Wire Line
-	2900 2475 2750 2475
-Connection ~ 2750 2475
-Wire Wire Line
-	2750 2475 2750 2725
-Wire Wire Line
-	2750 2475 2575 2475
 $Comp
 L 10106052_PowerPack:INA170 U3
@@
 F 2 "10106052 PowerPack:TO228P1003X238-3_4N" H 6850 7425 50  0001 C CNN
 F 3 "http://www.vishay.com/docs/72250/sud50p06.pdf" H 6650 7325 50  0001 C CNN
-F 4 "TRANSISTOR MOSFET, 60V, 50A, P CHANNEL" H 6650 7325 50  0001 C CNN "Description"
+F 4 "TRANSISTOR MOSFET, 60V, 50A, P CHANNEL, TO252" H 6650 7325 50  0001 C CNN "Description"
 F 5 "10095972" H 6650 7325 50  0001 C CNN "Item Number"
 F 6 "Vishay Siliconix" H 6650 7325 50  0001 C CNN "Manufacturer"
@@
 V_DC_CHARGER
 $Comp
-L Device:D_Schottky D9
+L 10106052_PowerPack:SMA6J28A D9
 U 1 1 5ED5C669
 P 3150 7625
@@
 L 10106052_PowerPack:+VDC_PERM #PWR0120
 U 1 1 5E8C661B
-P 2575 2475
-F 0 "#PWR0120" H 2575 2325 50  0001 C CNN
-F 1 "+VDC_PERM" V 2590 2602 50  0000 L CNN
-F 2 "" H 2575 2475 50  0001 C CNN
-F 3 "" H 2575 2475 50  0001 C CNN
-	1    2575 2475
+P 2575 2450
+F 0 "#PWR0120" H 2575 2300 50  0001 C CNN
+F 1 "+VDC_PERM" V 2590 2577 50  0000 L CNN
+F 2 "" H 2575 2450 50  0001 C CNN
+F 3 "" H 2575 2450 50  0001 C CNN
+	1    2575 2450
 	0    -1   -1   0
 $EndComp
 Text HLabel 9275 7325 0    50   Input ~ 0
 +3.0VREF
-Text Label 3725 2475 0    50   ~ 0
+Text Label 3725 2450 0    50   ~ 0
 V_DC_CHARGER
 Text Label 7175 6125 0    50   ~ 0
@@
 L power:PWR_FLAG #FLG0104
 U 1 1 5E97BAC7
-P 2750 2725
-F 0 "#FLG0104" H 2750 2800 50  0001 C CNN
-F 1 "PWR_FLAG" V 2750 2852 50  0000 L CNN
-F 2 "" H 2750 2725 50  0001 C CNN
-F 3 "~" H 2750 2725 50  0001 C CNN
-	1    2750 2725
+P 2750 2700
+F 0 "#FLG0104" H 2750 2775 50  0001 C CNN
+F 1 "PWR_FLAG" V 2750 2827 50  0000 L CNN
+F 2 "" H 2750 2700 50  0001 C CNN
+F 3 "~" H 2750 2700 50  0001 C CNN
+	1    2750 2700
 	0    -1   -1   0
 $EndComp
-Connection ~ 2750 2725
 Wire Wire Line
 	7225 5250 7225 5175
@@
 Wire Wire Line
 	6375 7225 5775 7225
+Wire Wire Line
+	2900 2200 2750 2200
+Wire Wire Line
+	4150 2700 4150 3825
+Wire Wire Line
+	2900 2450 2750 2450
+Wire Wire Line
+	2750 2200 2750 2450
+Connection ~ 2750 2700
+Wire Wire Line
+	2750 2700 2900 2700
+Connection ~ 2750 2450
+Wire Wire Line
+	2750 2450 2575 2450
+Wire Wire Line
+	2750 2450 2750 2700
+Wire Wire Line
+	4900 975  5300 975
+Wire Wire Line
+	3200 2200 5300 2200
+Wire Wire Line
+	5300 2200 5300 975
+Connection ~ 5300 975
+Wire Wire Line
+	5300 975  7875 975
 $EndSCHEMATC
