File: 10106052 PowerPack/utils.sch (KiCad schematic (older format))
At the start: 19 parts, among them J10 S2B-ZR-SM4A-TF, T11 SI2300DS-T1-GE3, T3 SI2309CDS-T1-GE3, T5 SI2300DS-T1-GE3, U1 NCV87722DT50RKG, U2 LM4120AIM5-3.0, U6 MCP9700A-E_TO

Commit message: PowerPack schematic toplevel done
Changed lines of the file:
@@
 $Descr A4 11693 8268
 encoding utf-8
-Sheet 4 4
-Title ""
-Date ""
-Rev ""
+Sheet 3 4
+Title "Utils"
+Date "2020-04-05"
+Rev "1"
 Comp ""
 Comment1 ""
@@
 P 9000 2050
 AR Path="/5E878266/5E8CB2D2" Ref="#PWR?"  Part="1"
-AR Path="/5E8CA2BD/5E8CB2D2" Ref="#PWR?"  Part="1"
-F 0 "#PWR?" H 9000 1900 50  0001 C CNN
+AR Path="/5E8CA2BD/5E8CB2D2" Ref="#PWR0121"  Part="1"
+F 0 "#PWR0121" H 9000 1900 50  0001 C CNN
 F 1 "+5V" H 9015 2223 50  0000 C CNN
 F 2 "" H 9000 2050 50  0001 C CNN
@@
 P 9000 2800
 AR Path="/5E878266/5E8CB2DA" Ref="#PWR?"  Part="1"
-AR Path="/5E8CA2BD/5E8CB2DA" Ref="#PWR?"  Part="1"
-F 0 "#PWR?" H 9000 2550 50  0001 C CNN
+AR Path="/5E8CA2BD/5E8CB2DA" Ref="#PWR0122"  Part="1"
+F 0 "#PWR0122" H 9000 2550 50  0001 C CNN
 F 1 "GNDA" H 9005 2627 50  0000 C CNN
 F 2 "" H 9000 2800 50  0001 C CNN
@@
 P 9000 5725
 AR Path="/5E87821E/5E8CDD85" Ref="#PWR?"  Part="1"
-AR Path="/5E8CA2BD/5E8CDD85" Ref="#PWR?"  Part="1"
-F 0 "#PWR?" H 9000 5475 50  0001 C CNN
+AR Path="/5E8CA2BD/5E8CDD85" Ref="#PWR0123"  Part="1"
+F 0 "#PWR0123" H 9000 5475 50  0001 C CNN
 F 1 "GND" H 9000 5575 50  0000 C CNN
 F 2 "" H 9000 5725 50  0001 C CNN
@@
 P 9000 4425
 AR Path="/5E87821E/5E8CDD8E" Ref="#PWR?"  Part="1"
-AR Path="/5E8CA2BD/5E8CDD8E" Ref="#PWR?"  Part="1"
-F 0 "#PWR?" H 9000 4275 50  0001 C CNN
+AR Path="/5E8CA2BD/5E8CDD8E" Ref="#PWR0124"  Part="1"
+F 0 "#PWR0124" H 9000 4275 50  0001 C CNN
 F 1 "+5V" H 9015 4598 50  0000 C CNN
 F 2 "" H 9000 4425 50  0001 C CNN
@@
 P 3350 6100
 AR Path="/5E8781F8/5E8CF8BF" Ref="#PWR?"  Part="1"
-AR Path="/5E8CA2BD/5E8CF8BF" Ref="#PWR?"  Part="1"
-F 0 "#PWR?" H 3350 5850 50  0001 C CNN
+AR Path="/5E8CA2BD/5E8CF8BF" Ref="#PWR0125"  Part="1"
+F 0 "#PWR0125" H 3350 5850 50  0001 C CNN
 F 1 "GNDA" H 3355 5927 50  0000 C CNN
 F 2 "" H 3350 6100 50  0001 C CNN
@@
 P 3775 5250
 AR Path="/5E8781F8/5E8CF8CB" Ref="#PWR?"  Part="1"
-AR Path="/5E8CA2BD/5E8CF8CB" Ref="#PWR?"  Part="1"
-F 0 "#PWR?" H 3775 5100 50  0001 C CNN
+AR Path="/5E8CA2BD/5E8CF8CB" Ref="#PWR0126"  Part="1"
+F 0 "#PWR0126" H 3775 5100 50  0001 C CNN
 F 1 "+5V" H 3790 5423 50  0000 C CNN
 F 2 "" H 3775 5250 50  0001 C CNN
@@
 P 4725 3000
 AR Path="/5E87819A/5E8D1CDF" Ref="#PWR?"  Part="1"
-AR Path="/5E8CA2BD/5E8D1CDF" Ref="#PWR?"  Part="1"
-F 0 "#PWR?" H 4725 2750 50  0001 C CNN
+AR Path="/5E8CA2BD/5E8D1CDF" Ref="#PWR0127"  Part="1"
+F 0 "#PWR0127" H 4725 2750 50  0001 C CNN
 F 1 "GND" H 4730 2827 50  0000 C CNN
 F 2 "" H 4725 3000 50  0001 C CNN
@@
 P 5375 2075
 AR Path="/5E87819A/5E8D1CE6" Ref="#PWR?"  Part="1"
-AR Path="/5E8CA2BD/5E8D1CE6" Ref="#PWR?"  Part="1"
-F 0 "#PWR?" H 5375 1925 50  0001 C CNN
+AR Path="/5E8CA2BD/5E8D1CE6" Ref="#PWR0128"  Part="1"
+F 0 "#PWR0128" H 5375 1925 50  0001 C CNN
 F 1 "+5V" H 5390 2248 50  0000 C CNN
 F 2 "" H 5375 2075 50  0001 C CNN
@@
 P 4150 3025
 AR Path="/5E87819A/5E8D1D2F" Ref="#PWR?"  Part="1"
-AR Path="/5E8CA2BD/5E8D1D2F" Ref="#PWR?"  Part="1"
-F 0 "#PWR?" H 4150 2775 50  0001 C CNN
+AR Path="/5E8CA2BD/5E8D1D2F" Ref="#PWR0129"  Part="1"
+F 0 "#PWR0129" H 4150 2775 50  0001 C CNN
 F 1 "GND" H 4155 2852 50  0000 C CNN
 F 2 "" H 4150 3025 50  0001 C CNN
@@
 P 3675 1600
 AR Path="/5E87819A/5E8D1D50" Ref="#PWR?"  Part="1"
-AR Path="/5E8CA2BD/5E8D1D50" Ref="#PWR?"  Part="1"
-F 0 "#PWR?" H 3675 1450 50  0001 C CNN
+AR Path="/5E8CA2BD/5E8D1D50" Ref="#PWR0130"  Part="1"
+F 0 "#PWR0130" H 3675 1450 50  0001 C CNN
 F 1 "+VDC_PERM" H 3690 1773 50  0000 C CNN
 F 2 "" H 3675 1600 50  0001 C CNN
@@
 $EndComp
 $Comp
-L power:GNDA #PWR?
+L power:GNDA #PWR0131
 U 1 1 5E905EEE
 P 4875 5650
-F 0 "#PWR?" H 4875 5400 50  0001 C CNN
+F 0 "#PWR0131" H 4875 5400 50  0001 C CNN
 F 1 "GNDA" H 4880 5477 50  0000 C CNN
 F 2 "" H 4875 5650 50  0001 C CNN
@@
 Text Notes 2500 750  0    100  ~ 0
 +5V Power Supply
+$Comp
+L power:PWR_FLAG #FLG0101
+U 1 1 5E972989
+P 2950 6100
+F 0 "#FLG0101" H 2950 6175 50  0001 C CNN
+F 1 "PWR_FLAG" H 2950 6273 50  0000 C CNN
+F 2 "" H 2950 6100 50  0001 C CNN
+F 3 "~" H 2950 6100 50  0001 C CNN
+	1    2950 6100
+	-1   0    0    1
+$EndComp
+Connection ~ 2950 6100
+$Comp
+L power:PWR_FLAG #FLG0102
+U 1 1 5E9753B6
+P 5375 3000
+F 0 "#FLG0102" H 5375 3075 50  0001 C CNN
+F 1 "PWR_FLAG" H 5375 3173 50  0000 C CNN
+F 2 "" H 5375 3000 50  0001 C CNN
+F 3 "~" H 5375 3000 50  0001 C CNN
+	1    5375 3000
+	-1   0    0    1
+$EndComp
+Connection ~ 5375 3000
 $EndSCHEMATC

Commit message: Added ICSP Prog label
Parts:
- U6: symbol dk_Temperature-Sensors-Analog-and-Digital-Output:MCP9700A-E_TO -> 10106052-PowerPack-rescue:MCP9700A-E_TO-dk_Temperature-Sensors-Analog-and-Digital-Output
Changed lines of the file:
@@
 $EndDescr
 $Comp
-L dk_Temperature-Sensors-Analog-and-Digital-Output:MCP9700A-E_TO U?
+L 10106052-PowerPack-rescue:MCP9700A-E_TO-dk_Temperature-Sensors-Analog-and-Digital-Output U?
 U 1 1 5E8CB2CC
 P 9000 2425

Commit message: PCB Added and Schematic Footprints Added
Parts:
- C2, C30, C5, C6, C7: footprint (none) -> Capacitor_SMD:C_0603_1608Metric
- C3: footprint (none) -> Capacitor_SMD:C_1210_3225Metric
- D5: footprint digikey-footprints:SOT-23-3 -> Package_TO_SOT_SMD:SOT-23
- R11, R31, R6, R9: footprint (none) -> Resistor_SMD:R_0603_1608Metric
- R26: footprint (none) -> Resistor_SMD:R_1206_3216Metric
- T11, T3, T5: footprint (none) -> Package_TO_SOT_SMD:SOT-23
- U1: footprint (none) -> Package_TO_SOT_SMD:TO-263-7_TabPin4
- U2: footprint Package_TO_SOT_SMD:SOT-23-5_HandSoldering -> Package_TO_SOT_SMD:SOT-23-5
Changed lines of the file:
@@
 F 0 "C30" H 8300 2575 50  0000 L CNN
 F 1 "100n" H 8300 2400 50  0000 L CNN
-F 2 "" H 8638 2325 50  0001 C CNN
+F 2 "Capacitor_SMD:C_0603_1608Metric" H 8638 2325 50  0001 C CNN
 F 3 "~" H 8600 2475 50  0001 C CNN
 	1    8600 2475
@@
 F 0 "T11" H 9106 5296 50  0000 L CNN
 F 1 "SI2300DS-T1-GE3" H 9106 5205 50  0000 L CNN
-F 2 "" H 9100 5350 50  0001 C CNN
+F 2 "Package_TO_SOT_SMD:SOT-23" H 9100 5350 50  0001 C CNN
 F 3 "~" H 8900 5250 50  0001 C CNN
 	1    8900 5250
@@
 F 0 "R31" H 8695 5521 50  0000 L CNN
 F 1 "22k" H 8695 5430 50  0000 L CNN
-F 2 "" V 8555 5475 50  0001 C CNN
+F 2 "Resistor_SMD:R_0603_1608Metric" V 8555 5475 50  0001 C CNN
 F 3 "~" H 8625 5475 50  0001 C CNN
 	1    8625 5475
@@
 F 0 "R26" H 9070 4696 50  0000 L CNN
 F 1 "68" H 9070 4605 50  0000 L CNN
-F 2 "" V 8930 4650 50  0001 C CNN
+F 2 "Resistor_SMD:R_1206_3216Metric" V 8930 4650 50  0001 C CNN
 F 3 "~" H 9000 4650 50  0001 C CNN
 	1    9000 4650
@@
 F 0 "U2" H 4400 5965 50  0000 C CNN
 F 1 "LM4120AIM5-3.0" H 4400 5874 50  0000 C CNN
-F 2 "Package_TO_SOT_SMD:SOT-23-5_HandSoldering" H 4400 5600 50  0001 C CNN
+F 2 "Package_TO_SOT_SMD:SOT-23-5" H 4400 5600 50  0001 C CNN
 F 3 "" H 4400 5600 50  0001 C CNN
 	1    4400 5600
@@
 F 0 "C7" H 3890 5946 50  0000 L CNN
 F 1 "100n" H 3890 5855 50  0000 L CNN
-F 2 "" H 3813 5750 50  0001 C CNN
+F 2 "Capacitor_SMD:C_0603_1608Metric" H 3813 5750 50  0001 C CNN
 F 3 "~" H 3775 5900 50  0001 C CNN
 	1    3775 5900
@@
 F 0 "C6" H 3465 5946 50  0000 L CNN
 F 1 "1u" H 3465 5855 50  0000 L CNN
-F 2 "" H 3388 5750 50  0001 C CNN
+F 2 "Capacitor_SMD:C_0603_1608Metric" H 3388 5750 50  0001 C CNN
 F 3 "~" H 3350 5900 50  0001 C CNN
 	1    3350 5900
@@
 F 0 "C5" H 3065 5946 50  0000 L CNN
 F 1 "100n" H 3065 5855 50  0000 L CNN
-F 2 "" H 2988 5750 50  0001 C CNN
+F 2 "Capacitor_SMD:C_0603_1608Metric" H 2988 5750 50  0001 C CNN
 F 3 "~" H 2950 5900 50  0001 C CNN
 	1    2950 5900
@@
 F 0 "U1" H 4725 2765 50  0000 C CNN
 F 1 "NCV87722DT50RKG" H 4725 2674 50  0000 C CNN
-F 2 "" H 4725 2200 50  0001 C CNN
+F 2 "Package_TO_SOT_SMD:TO-263-7_TabPin4" H 4725 2200 50  0001 C CNN
 F 3 "" H 4725 2200 50  0001 C CNN
 	1    4725 2350
@@
 F 0 "C2" H 5490 2596 50  0000 L CNN
 F 1 "10u" H 5490 2505 50  0000 L CNN
-F 2 "" H 5413 2400 50  0001 C CNN
+F 2 "Capacitor_SMD:C_0603_1608Metric" H 5413 2400 50  0001 C CNN
 F 3 "~" H 5375 2550 50  0001 C CNN
 	1    5375 2550
@@
 F 0 "T3" H 3281 2146 50  0000 L CNN
 F 1 "SI2309CDS-T1-GE3" H 3281 2055 50  0000 L CNN
-F 2 "" H 3275 2200 50  0001 C CNN
+F 2 "Package_TO_SOT_SMD:SOT-23" H 3275 2200 50  0001 C CNN
 F 3 "~" H 3075 2100 50  0001 C CNN
 	1    3075 2100
@@
 F 0 "T5" H 2606 2746 50  0000 L CNN
 F 1 "SI2300DS-T1-GE3" H 2606 2655 50  0000 L CNN
-F 2 "" H 2600 2800 50  0001 C CNN
+F 2 "Package_TO_SOT_SMD:SOT-23" H 2600 2800 50  0001 C CNN
 F 3 "~" H 2400 2700 50  0001 C CNN
 	1    2400 2700
@@
 F 0 "R9" H 2570 2346 50  0000 L CNN
 F 1 "10k" H 2570 2255 50  0000 L CNN
-F 2 "" V 2430 2300 50  0001 C CNN
+F 2 "Resistor_SMD:R_0603_1608Metric" V 2430 2300 50  0001 C CNN
 F 3 "~" H 2500 2300 50  0001 C CNN
 	1    2500 2300
@@
 F 0 "R6" V 2593 1725 50  0000 C CNN
 F 1 "10k" V 2684 1725 50  0000 C CNN
-F 2 "" V 2730 1725 50  0001 C CNN
+F 2 "Resistor_SMD:R_0603_1608Metric" V 2730 1725 50  0001 C CNN
 F 3 "~" H 2800 1725 50  0001 C CNN
 	1    2800 1725
@@
 F 0 "R11" V 2100 2975 50  0000 C CNN
 F 1 "10k" V 2000 3000 50  0000 C CNN
-F 2 "" V 2130 3000 50  0001 C CNN
+F 2 "Resistor_SMD:R_0603_1608Metric" V 2130 3000 50  0001 C CNN
 F 3 "~" H 2200 3000 50  0001 C CNN
 	1    2200 3000
@@
 F 0 "C3" H 4265 2771 50  0000 L CNN
 F 1 "1u" H 4265 2680 50  0000 L CNN
-F 2 "" H 4188 2575 50  0001 C CNN
+F 2 "Capacitor_SMD:C_1210_3225Metric" H 4188 2575 50  0001 C CNN
 F 3 "~" H 4150 2725 50  0001 C CNN
 	1    4150 2725
@@
 F 0 "D5" V 2475 3900 60  0000 C CNN
 F 1 "BAS70-05" V 2350 4075 60  0000 C CNN
-F 2 "digikey-footprints:SOT-23-3" H 2700 3950 60  0001 L CNN
+F 2 "Package_TO_SOT_SMD:SOT-23" H 2700 3950 60  0001 L CNN
 F 3 "https://www.diodes.com/assets/Datasheets/ds11005.pdf" H 2700 4050 60  0001 L CNN
 F 4 "BAT54C-FDICT-ND" H 2700 4150 60  0001 L CNN "Digi-Key_PN"

Commit message: Added parameters to components
Parts:
- C2: Description (none) -> CAPACITOR CERAMIC 10UF 6.3V 20% X5R 0603; Item Number (none) -> 10021370; Manufacturer (none) -> Kemet; Manufacturer_No (none) -> C0603C106M9PACTM; Note (none) -> BOM lists C0603C106M9PACTM but only TU was found
- C3: Description (none) -> CAPACITOR CERAMIC 1UF 50V X5R 10% 1210; Item Number (none) -> 10107885; Manufacturer (none) -> Kemet; Manufacturer_No (none) -> C1210C105K5PACTU
- C30, C5, C7: Description (none) -> CAPACITOR CERAMIC 100NF 50V 10% X7R 0603; Item Number (none) -> 10021386; Manufacturer (none) -> Kemet; Manufacturer_No (none) -> C0603C104K5RACTU
- C6: Description (none) -> CAPACITOR CERAMIC 1UF 10V 10% X5R 0402; Item Number (none) -> 10021369; Manufacturer (none) -> Kemet; Manufacturer_No (none) -> C0402C105K8PACTU
- D5: Description DIODE ARRAY SCHOTTKY 30V SOT23-3 -> DIODE SCHOTTKY DUAL 70V 100MA SOT-23; Digi-Key_PN BAT54C-FDICT-ND -> (none); Item Number (none) -> 10107888; MPN BAT54C-7-F -> (none); Manufacturer Diodes Incorporated -> Vishay; Manufacturer_No (none) -> BAS70-05-E3-08
- J10: Description (none) -> CONNECTOR, ZH, 2 CIRCUITS, 1.5 MM; Item Number (none) -> 10107891; Manufacturer (none) -> JST; Manufacturer_No (none) -> S2B-ZR-SM4A-TF(LF)(SN)
- R11, R6, R9: Description (none) -> RESISTOR,10K OHM.0.063W,+/-1%,0603; Item Number (none) -> 10022548; Manufacturer (none) -> Yageo; Manufacturer_No (none) -> RC0603FR-0710KL
- R26: Description (none) -> RESISTOR 68 OHM 1/4W 5% 1206; Item Number (none) -> 10126895; Manufacturer (none) -> Yageo; Manufacturer_No (none) -> RC1206JR-0768RL; Note (none) -> BOM has CRCW120668RJKEA
- R31: Description (none) -> RESISTOR 22 KOHM 0.063W +/-1% 0603; Item Number (none) -> 10113300; Manufacturer (none) -> Yageo; Manufacturer_No (none) -> RC0603JR-0722KL
- T11, T5: Description (none) -> MOSFET N-CH 30V SOT-23; Item Number (none) -> GR102887; Manufacturer (none) -> Vishay Siliconix; Manufacturer_No (none) -> SI2300DS-T1-GE3
- T3: Description (none) -> TRANSISTOR MOS P CHANNEL, 60V, 1.6A, SOT23; Item Number (none) -> 10060356; Manufacturer (none) -> Vishay Siliconix; Manufacturer_No (none) -> SI2309CDS-T1-GE3
- U1: Description (none) -> IC REG LINEAR 5V/3.3V 350MA D2PAK-7; Item Number (none) -> 10113304; Manufacturer (none) -> ON Semiconductor; Manufacturer_No (none) -> NCV87725D7S50R4G
- U2: Description (none) -> IC,VOLTAGE REFERENCE,5MA,3V +/-2%,SOT23; Item Number (none) -> 10022896; Manufacturer (none) -> Texas Instruments; Manufacturer_No (none) -> LM4120AIM5-3.0/NOPB
- U6: footprint digikey-footprints:TO-92-3 -> Package_TO_SOT_THT:TO-92; Description SENSOR ANALOG -40C-125C TO92-3 -> IC LINEAR ACTIVE THERMISTOR MCP9700 TO-92; Item Number (none) -> 10107900; MPN MCP9700A-E/TO -> (none); Manufacturer_No (none) -> MCP9700A-E/TO; Note (none) -> AT part not available

Commit message: Created Project Footprint Library
Parts:
- J10: footprint (none) -> 10106052 PowerPack:CON-S2B-ZR-SM4A-TF_1
Changed lines of the file:
@@
 F 0 "J10" H 9422 4849 50  0000 R CNN
 F 1 "S2B-ZR-SM4A-TF" H 9422 4758 50  0000 R CNN
-F 2 "" H 9450 4875 50  0001 C CNN
+F 2 "10106052 PowerPack:CON-S2B-ZR-SM4A-TF_1" H 9450 4875 50  0001 C CNN
 F 3 "http://www.jst-mfg.com/product/pdf/eng/eZH.pdf" H 9450 4875 50  0001 C CNN
 F 4 "CONNECTOR, ZH, 2 CIRCUITS, 1.5 MM" H 9450 4875 50  0001 C CNN "Description"

Commit message: Footprints relinked
Parts:
- C2, C30, C5, C6, C7: footprint Capacitor_SMD:C_0603_1608Metric -> 10106052 PowerPack:CAPC1608X86N
- C3: footprint Capacitor_SMD:C_1210_3225Metric -> 10106052 PowerPack:CAPC3225X155N
- D5, T11, T3, T5: footprint Package_TO_SOT_SMD:SOT-23 -> 10106052 PowerPack:SOT92P240X120-3N
- J10: footprint 10106052 PowerPack:CON-S2B-ZR-SM4A-TF_1 -> 10106052 PowerPack:CON-S2B-ZR-SM4A-TF
- R11, R31, R6, R9: footprint Resistor_SMD:R_0603_1608Metric -> 10106052 PowerPack:RESC1608X50AN
- R26: footprint Resistor_SMD:R_1206_3216Metric -> 10106052 PowerPack:RESC3216X60N
- U1: footprint Package_TO_SOT_SMD:TO-263-7_TabPin4 -> 10106052 PowerPack:TO170P1420X457-8NA
- U2: footprint Package_TO_SOT_SMD:SOT-23-5 -> 10106052 PowerPack:SOT95P279X142-5N
- U6: footprint Package_TO_SOT_THT:TO-92 -> 10106052 PowerPack:TO-92
Changed lines of the file:
@@
 F 0 "U6" H 9175 2675 60  0000 R CNN
 F 1 "MCP9700A-E_TO" H 9825 2175 60  0000 R CNN
-F 2 "Package_TO_SOT_THT:TO-92" H 9200 2625 60  0001 L CNN
+F 2 "10106052 PowerPack:TO-92" H 9200 2625 60  0001 L CNN
 F 3 "http://ww1.microchip.com/downloads/en/DeviceDoc/20001942G.pdf" H 9200 2725 60  0001 L CNN
 F 4 "MCP9700A-E/TO-ND" H 9200 2825 60  0001 L CNN "Digi-Key_PN"
@@
 F 0 "C30" H 8300 2575 50  0000 L CNN
 F 1 "100n" H 8300 2400 50  0000 L CNN
-F 2 "Capacitor_SMD:C_0603_1608Metric" H 8638 2325 50  0001 C CNN
+F 2 "10106052 PowerPack:CAPC1608X86N" H 8638 2325 50  0001 C CNN
 F 3 "https://api.kemet.com/component-edge/download/datasheet/C0603C104K5RACTU.pdf" H 8600 2475 50  0001 C CNN
 F 4 "CAPACITOR CERAMIC 100NF 50V 10% X7R 0603" H 8600 2475 50  0001 C CNN "Description"
@@
 F 0 "J10" H 9422 4849 50  0000 R CNN
 F 1 "S2B-ZR-SM4A-TF" H 9422 4758 50  0000 R CNN
-F 2 "10106052 PowerPack:CON-S2B-ZR-SM4A-TF_1" H 9450 4875 50  0001 C CNN
+F 2 "10106052 PowerPack:CON-S2B-ZR-SM4A-TF" H 9450 4875 50  0001 C CNN
 F 3 "http://www.jst-mfg.com/product/pdf/eng/eZH.pdf" H 9450 4875 50  0001 C CNN
 F 4 "CONNECTOR, ZH, 2 CIRCUITS, 1.5 MM" H 9450 4875 50  0001 C CNN "Description"
@@
 F 0 "T11" H 9106 5296 50  0000 L CNN
 F 1 "SI2300DS-T1-GE3" H 9106 5205 50  0000 L CNN
-F 2 "Package_TO_SOT_SMD:SOT-23" H 9100 5350 50  0001 C CNN
+F 2 "10106052 PowerPack:SOT92P240X120-3N" H 9100 5350 50  0001 C CNN
 F 3 "http://www.vishay.com/docs/65701/si2300ds.pdf" H 8900 5250 50  0001 C CNN
 F 4 "MOSFET N-CH 30V SOT-23" H 8900 5250 50  0001 C CNN "Description"
@@
 F 0 "R31" H 8695 5521 50  0000 L CNN
 F 1 "22k" H 8695 5430 50  0000 L CNN
-F 2 "Resistor_SMD:R_0603_1608Metric" V 8555 5475 50  0001 C CNN
+F 2 "10106052 PowerPack:RESC1608X50AN" V 8555 5475 50  0001 C CNN
 F 3 "https://www.yageo.com/upload/media/product/productsearch/datasheet/rchip/PYu-RC_Group_51_RoHS_L_10.pdf" H 8625 5475 50  0001 C CNN
 F 4 "RESISTOR 22 KOHM 0.063W +/-1% 0603" H 8625 5475 50  0001 C CNN "Description"
@@
 F 0 "R26" H 9070 4696 50  0000 L CNN
 F 1 "68" H 9070 4605 50  0000 L CNN
-F 2 "Resistor_SMD:R_1206_3216Metric" V 8930 4650 50  0001 C CNN
+F 2 "10106052 PowerPack:RESC3216X60N" V 8930 4650 50  0001 C CNN
 F 3 "https://www.yageo.com/upload/media/product/productsearch/datasheet/rchip/PYu-RC_Group_51_RoHS_L_10.pdf" H 9000 4650 50  0001 C CNN
 F 4 "RESISTOR 68 OHM 1/4W 5% 1206" H 9000 4650 50  0001 C CNN "Description"
@@
 F 0 "U2" H 4400 5965 50  0000 C CNN
 F 1 "LM4120AIM5-3.0" H 4400 5874 50  0000 C CNN
-F 2 "Package_TO_SOT_SMD:SOT-23-5" H 4400 5600 50  0001 C CNN
+F 2 "10106052 PowerPack:SOT95P279X142-5N" H 4400 5600 50  0001 C CNN
 F 3 "http://www.ti.com/general/docs/suppproductinfo.tsp?distId=10&gotoUrl=http%3A%2F%2Fwww.ti.com%2Flit%2Fgpn%2Flm4120" H 4400 5600 50  0001 C CNN
 F 4 "IC,VOLTAGE REFERENCE,5MA,3V +/-2%,SOT23" H 4400 5600 50  0001 C CNN "Description"
@@
 F 0 "C7" H 3890 5946 50  0000 L CNN
 F 1 "100n" H 3890 5855 50  0000 L CNN
-F 2 "Capacitor_SMD:C_0603_1608Metric" H 3813 5750 50  0001 C CNN
+F 2 "10106052 PowerPack:CAPC1608X86N" H 3813 5750 50  0001 C CNN
 F 3 "https://api.kemet.com/component-edge/download/datasheet/C0603C104K5RACTU.pdf" H 3775 5900 50  0001 C CNN
 F 4 "CAPACITOR CERAMIC 100NF 50V 10% X7R 0603" H 3775 5900 50  0001 C CNN "Description"
@@
 F 0 "C6" H 3465 5946 50  0000 L CNN
 F 1 "1u" H 3465 5855 50  0000 L CNN
-F 2 "Capacitor_SMD:C_0603_1608Metric" H 3388 5750 50  0001 C CNN
+F 2 "10106052 PowerPack:CAPC1608X86N" H 3388 5750 50  0001 C CNN
 F 3 "https://api.kemet.com/component-edge/download/datasheet/C0402C105K8PACTU.pdf" H 3350 5900 50  0001 C CNN
 F 4 "CAPACITOR CERAMIC 1UF 10V 10% X5R 0402" H 3350 5900 50  0001 C CNN "Description"
@@
 F 0 "C5" H 3065 5946 50  0000 L CNN
 F 1 "100n" H 3065 5855 50  0000 L CNN
-F 2 "Capacitor_SMD:C_0603_1608Metric" H 2988 5750 50  0001 C CNN
+F 2 "10106052 PowerPack:CAPC1608X86N" H 2988 5750 50  0001 C CNN
 F 3 "https://api.kemet.com/component-edge/download/datasheet/C0603C104K5RACTU.pdf" H 2950 5900 50  0001 C CNN
 F 4 "CAPACITOR CERAMIC 100NF 50V 10% X7R 0603" H 2950 5900 50  0001 C CNN "Description"
@@
 F 0 "U1" H 4725 2765 50  0000 C CNN
 F 1 "NCV87722DT50RKG" H 4725 2674 50  0000 C CNN
-F 2 "Package_TO_SOT_SMD:TO-263-7_TabPin4" H 4725 2200 50  0001 C CNN
+F 2 "10106052 PowerPack:TO170P1420X457-8NA" H 4725 2200 50  0001 C CNN
 F 3 "http://www.onsemi.com/pub/Collateral/NCV8772-D.PDF" H 4725 2200 50  0001 C CNN
 F 4 "IC REG LINEAR 5V/3.3V 350MA D2PAK-7" H 4725 2350 50  0001 C CNN "Description"
@@
 F 0 "C2" H 5490 2596 50  0000 L CNN
 F 1 "10u" H 5490 2505 50  0000 L CNN
-F 2 "Capacitor_SMD:C_0603_1608Metric" H 5413 2400 50  0001 C CNN
+F 2 "10106052 PowerPack:CAPC1608X86N" H 5413 2400 50  0001 C CNN
 F 3 "https://api.kemet.com/component-edge/download/datasheet/C0603C106M9PACTU.pdf" H 5375 2550 50  0001 C CNN
 F 4 "CAPACITOR CERAMIC 10UF 6.3V 20% X5R 0603" H 5375 2550 50  0001 C CNN "Description"
@@
 F 0 "T3" H 3281 2146 50  0000 L CNN
 F 1 "SI2309CDS-T1-GE3" H 3281 2055 50  0000 L CNN
-F 2 "Package_TO_SOT_SMD:SOT-23" H 3275 2200 50  0001 C CNN
+F 2 "10106052 PowerPack:SOT92P240X120-3N" H 3275 2200 50  0001 C CNN
 F 3 "http://www.vishay.com/docs/68980/si2309cd.pdf" H 3075 2100 50  0001 C CNN
 F 4 "TRANSISTOR MOS P CHANNEL, 60V, 1.6A, SOT23" H 3075 2100 50  0001 C CNN "Description"
@@
 F 0 "T5" H 2606 2746 50  0000 L CNN
 F 1 "SI2300DS-T1-GE3" H 2606 2655 50  0000 L CNN
-F 2 "Package_TO_SOT_SMD:SOT-23" H 2600 2800 50  0001 C CNN
+F 2 "10106052 PowerPack:SOT92P240X120-3N" H 2600 2800 50  0001 C CNN
 F 3 "http://www.vishay.com/docs/65701/si2300ds.pdf" H 2400 2700 50  0001 C CNN
 F 4 "MOSFET N-CH 30V SOT-23" H 2400 2700 50  0001 C CNN "Description"
@@
 F 0 "R9" H 2570 2346 50  0000 L CNN
 F 1 "10k" H 2570 2255 50  0000 L CNN
-F 2 "Resistor_SMD:R_0603_1608Metric" V 2430 2300 50  0001 C CNN
+F 2 "10106052 PowerPack:RESC1608X50AN" V 2430 2300 50  0001 C CNN
 F 3 "https://www.yageo.com/upload/media/product/productsearch/datasheet/rchip/PYu-RC_Group_51_RoHS_L_10.pdf" H 2500 2300 50  0001 C CNN
 F 4 "RESISTOR,10K OHM.0.063W,+/-1%,0603" H 2500 2300 50  0001 C CNN "Description"
@@
 F 0 "R6" V 2593 1725 50  0000 C CNN
 F 1 "10k" V 2684 1725 50  0000 C CNN
-F 2 "Resistor_SMD:R_0603_1608Metric" V 2730 1725 50  0001 C CNN
+F 2 "10106052 PowerPack:RESC1608X50AN" V 2730 1725 50  0001 C CNN
 F 3 "https://www.yageo.com/upload/media/product/productsearch/datasheet/rchip/PYu-RC_Group_51_RoHS_L_10.pdf" H 2800 1725 50  0001 C CNN
 F 4 "RESISTOR,10K OHM.0.063W,+/-1%,0603" H 2800 1725 50  0001 C CNN "Description"
@@
 F 0 "R11" V 2100 2975 50  0000 C CNN
 F 1 "10k" V 2000 3000 50  0000 C CNN
-F 2 "Resistor_SMD:R_0603_1608Metric" V 2130 3000 50  0001 C CNN
+F 2 "10106052 PowerPack:RESC1608X50AN" V 2130 3000 50  0001 C CNN
 F 3 "https://www.yageo.com/upload/media/product/productsearch/datasheet/rchip/PYu-RC_Group_51_RoHS_L_10.pdf" H 2200 3000 50  0001 C CNN
 F 4 "RESISTOR,10K OHM.0.063W,+/-1%,0603" H 2200 3000 50  0001 C CNN "Description"
@@
 F 0 "C3" H 4265 2771 50  0000 L CNN
 F 1 "1u" H 4265 2680 50  0000 L CNN
-F 2 "Capacitor_SMD:C_1210_3225Metric" H 4188 2575 50  0001 C CNN
+F 2 "10106052 PowerPack:CAPC3225X155N" H 4188 2575 50  0001 C CNN
 F 3 "https://api.kemet.com/component-edge/download/datasheet/C1210C105K5PACTU.pdf" H 4150 2725 50  0001 C CNN
 F 4 "CAPACITOR CERAMIC 1UF 50V X5R 10% 1210" H 4150 2725 50  0001 C CNN "Description"
@@
 F 0 "D5" V 2475 3900 60  0000 C CNN
 F 1 "BAS70-05" V 2350 4075 60  0000 C CNN
-F 2 "Package_TO_SOT_SMD:SOT-23" H 2700 3950 60  0001 L CNN
+F 2 "10106052 PowerPack:SOT92P240X120-3N" H 2700 3950 60  0001 L CNN
 F 3 "http://www.vishay.com/docs/85702/bas70.pdf" H 2700 4050 60  0001 L CNN
 F 4 "" H 2700 4150 60  0001 L CNN "Digi-Key_PN"
