File: 10106052 PowerPack/utils.sch (KiCad schematic (older format))
At the start: 19 parts, among them J10 S2B-ZR-SM4A-TF, T11 SI2300DS-T1-GE3, T3 SI2309CDS-T1-GE3, T5 SI2300DS-T1-GE3, U1 NCV87722DT50RKG, U2 LM4120AIM5-3.0, U6 MCP9700A-E_TO

Commit message: Added 3D Models, corrected orientation of parts on schematic, added TX/RX TP
Parts:
- T3: symbol Device:Q_NMOS_GSD -> Device:Q_PMOS_GSD
Connections:
- net +3.0VREF: now also C5.2, C6.2; no longer C5.1, C6.1
- net +5V: now also C30.2; no longer C30.1
- net +VDC_PERM: now also C3.2, T3.2 (S); no longer C3.1, T3.3 (D)
- net GND: now also C3.1; no longer C3.2
- net GNDA: now also C30.1, C5.1, C6.1; no longer C30.2, C5.2, C6.2
- net at D5.3 (K), U1.4 (EN): now also T3.3 (D); no longer T3.2 (S)
Other:
- moved on the sheet: C2
Changed lines of the file:
@@
 F 7 "C0603C104K5RACTU" H 8600 2475 50  0001 C CNN "Manufacturer_No"
 	1    8600 2475
-	1    0    0    -1
+	1    0    0    1
 $EndComp
 Wire Wire Line
@@
 F 7 "C0402C105K8PACTU" H 3350 5900 50  0001 C CNN "Manufacturer_No"
 	1    3350 5900
-	1    0    0    -1
+	1    0    0    1
 $EndComp
 $Comp
@@
 F 7 "C0603C104K5RACTU" H 2950 5900 50  0001 C CNN "Manufacturer_No"
 	1    2950 5900
-	1    0    0    -1
+	1    0    0    1
 $EndComp
 Wire Wire Line
@@
 L Device:C C?
 U 1 1 5E8D1CD4
-P 5375 2550
+P 5400 2550
 AR Path="/5E87819A/5E8D1CD4" Ref="C?"  Part="1"
 AR Path="/5E8CA2BD/5E8D1CD4" Ref="C2"  Part="1"
-F 0 "C2" H 5490 2596 50  0000 L CNN
-F 1 "10u" H 5490 2505 50  0000 L CNN
-F 2 "10106052 PowerPack:CAPC1608X86N" H 5413 2400 50  0001 C CNN
-F 3 "https://api.kemet.com/component-edge/download/datasheet/C0603C106M9PACTU.pdf" H 5375 2550 50  0001 C CNN
-F 4 "CAPACITOR CERAMIC 10UF 6.3V 20% X5R 0603" H 5375 2550 50  0001 C CNN "Description"
-F 5 "10021370" H 5375 2550 50  0001 C CNN "Item Number"
-F 6 "C0603C106M9PACTM" H 5375 2550 50  0001 C CNN "Manufacturer_No"
-F 7 "BOM lists C0603C106M9PACTM but only TU was found" H 5375 2550 50  0001 C CNN "Note"
-F 8 "Kemet" H 5375 2550 50  0001 C CNN "Manufacturer"
-	1    5375 2550
-	1    0    0    -1
-$EndComp
-Wire Wire Line
-	5375 2400 5375 2250
-Wire Wire Line
-	5375 2250 5125 2250
-Wire Wire Line
-	5375 2700 5375 3000
-Wire Wire Line
-	5375 3000 4725 3000
+F 0 "C2" H 5515 2596 50  0000 L CNN
+F 1 "10u" H 5515 2505 50  0000 L CNN
+F 2 "10106052 PowerPack:CAPC1608X86N" H 5438 2400 50  0001 C CNN
+F 3 "https://api.kemet.com/component-edge/download/datasheet/C0603C106M9PACTU.pdf" H 5400 2550 50  0001 C CNN
+F 4 "CAPACITOR CERAMIC 10UF 6.3V 20% X5R 0603" H 5400 2550 50  0001 C CNN "Description"
+F 5 "10021370" H 5400 2550 50  0001 C CNN "Item Number"
+F 6 "C0603C106M9PACTM" H 5400 2550 50  0001 C CNN "Manufacturer_No"
+F 7 "BOM lists C0603C106M9PACTM but only TU was found" H 5400 2550 50  0001 C CNN "Note"
+F 8 "Kemet" H 5400 2550 50  0001 C CNN "Manufacturer"
+	1    5400 2550
+	1    0    0    -1
+$EndComp
+Wire Wire Line
+	5400 2400 5400 2250
+Wire Wire Line
+	5400 2700 5400 3000
 Wire Wire Line
 	4725 3000 4725 2700
@@
 	1    0    0    -1
 $EndComp
-Connection ~ 4725 3000
 $Comp
 L power:+5V #PWR?
 U 1 1 5E8D1CE6
-P 5375 2075
+P 5400 2075
 AR Path="/5E87819A/5E8D1CE6" Ref="#PWR?"  Part="1"
 AR Path="/5E8CA2BD/5E8D1CE6" Ref="#PWR0128"  Part="1"
-F 0 "#PWR0128" H 5375 1925 50  0001 C CNN
-F 1 "+5V" H 5390 2248 50  0000 C CNN
-F 2 "" H 5375 2075 50  0001 C CNN
-F 3 "" H 5375 2075 50  0001 C CNN
-	1    5375 2075
-	1    0    0    -1
-$EndComp
-Wire Wire Line
-	5375 2075 5375 2250
-Connection ~ 5375 2250
+F 0 "#PWR0128" H 5400 1925 50  0001 C CNN
+F 1 "+5V" H 5415 2248 50  0000 C CNN
+F 2 "" H 5400 2075 50  0001 C CNN
+F 3 "" H 5400 2075 50  0001 C CNN
+	1    5400 2075
+	1    0    0    -1
+$EndComp
+Wire Wire Line
+	5400 2075 5400 2250
+Connection ~ 5400 2250
 NoConn ~ 5125 2450
 $Comp
-L Device:Q_NMOS_GSD T?
+L Device:Q_PMOS_GSD T?
 U 1 1 5E8D1CEF
 P 3075 2100
@@
 F 7 "SI2309CDS-T1-GE3" H 3075 2100 50  0001 C CNN "Manufacturer_No"
 	1    3075 2100
-	1    0    0    -1
+	1    0    0    1
 $EndComp
 $Comp
@@
 F 7 "C1210C105K5PACTU" H 4150 2725 50  0001 C CNN "Manufacturer_No"
 	1    4150 2725
-	1    0    0    -1
+	1    0    0    1
 $EndComp
 Wire Wire Line
@@
 L power:PWR_FLAG #FLG0102
 U 1 1 5E9753B6
-P 5375 3000
-F 0 "#FLG0102" H 5375 3075 50  0001 C CNN
-F 1 "PWR_FLAG" H 5375 3173 50  0000 C CNN
-F 2 "" H 5375 3000 50  0001 C CNN
-F 3 "~" H 5375 3000 50  0001 C CNN
-	1    5375 3000
+P 5400 3000
+F 0 "#FLG0102" H 5400 3075 50  0001 C CNN
+F 1 "PWR_FLAG" H 5400 3173 50  0000 C CNN
+F 2 "" H 5400 3000 50  0001 C CNN
+F 3 "~" H 5400 3000 50  0001 C CNN
+	1    5400 3000
 	-1   0    0    1
 $EndComp
-Connection ~ 5375 3000
+Connection ~ 5400 3000
+Wire Wire Line
+	5125 2250 5400 2250
+Wire Wire Line
+	4725 3000 5400 3000
+Connection ~ 4725 3000
 $EndSCHEMATC

Commit message: powerpack-dev
Parts:
- U6: symbol 10106052-PowerPack-rescue:MCP9700A-E_TO-dk_Temperature-Sensors-Analog-and-Digital-Output -> 10106052_PowerPack:MCP9700A-E_TO
Connections:
- net +5V: now also C2.2, C7.2, R26.2; no longer C2.1, C7.1, R26.1
- net GND: now also C2.1; no longer C2.2
- net GNDA: now also C7.1; no longer C7.2
- net at J10.1 (Pin_1): now also R26.1; no longer R26.2
Changed lines of the file:
@@
 $EndDescr
 $Comp
-L 10106052-PowerPack-rescue:MCP9700A-E_TO-dk_Temperature-Sensors-Analog-and-Digital-Output U?
+L 10106052_PowerPack:MCP9700A-E_TO U?
 U 1 1 5E8CB2CC
 P 9000 2425
@@
 AR Path="/5E87821E/5E8CDD76" Ref="R?"  Part="1"
 AR Path="/5E8CA2BD/5E8CDD76" Ref="R26"  Part="1"
-F 0 "R26" H 9070 4696 50  0000 L CNN
-F 1 "68" H 9070 4605 50  0000 L CNN
+F 0 "R26" H 8930 4604 50  0000 R CNN
+F 1 "68" H 8930 4695 50  0000 R CNN
 F 2 "10106052 PowerPack:RESC3216X60N" V 8930 4650 50  0001 C CNN
 F 3 "https://www.yageo.com/upload/media/product/productsearch/datasheet/rchip/PYu-RC_Group_51_RoHS_L_10.pdf" H 9000 4650 50  0001 C CNN
@@
 F 8 "BOM has CRCW120668RJKEA" H 9000 4650 50  0001 C CNN "Note"
 	1    9000 4650
-	1    0    0    -1
+	-1   0    0    1
 $EndComp
 Wire Wire Line
@@
 AR Path="/5E8781F8/5E8CF89F" Ref="C?"  Part="1"
 AR Path="/5E8CA2BD/5E8CF89F" Ref="C7"  Part="1"
-F 0 "C7" H 3890 5946 50  0000 L CNN
-F 1 "100n" H 3890 5855 50  0000 L CNN
+F 0 "C7" H 3660 5854 50  0000 R CNN
+F 1 "100n" H 3660 5945 50  0000 R CNN
 F 2 "10106052 PowerPack:CAPC1608X86N" H 3813 5750 50  0001 C CNN
 F 3 "https://api.kemet.com/component-edge/download/datasheet/C0603C104K5RACTU.pdf" H 3775 5900 50  0001 C CNN
@@
 F 7 "C0603C104K5RACTU" H 3775 5900 50  0001 C CNN "Manufacturer_No"
 	1    3775 5900
-	1    0    0    -1
+	-1   0    0    1
 $EndComp
 $Comp
@@
 AR Path="/5E87819A/5E8D1CD4" Ref="C?"  Part="1"
 AR Path="/5E8CA2BD/5E8D1CD4" Ref="C2"  Part="1"
-F 0 "C2" H 5515 2596 50  0000 L CNN
-F 1 "10u" H 5515 2505 50  0000 L CNN
+F 0 "C2" H 5285 2504 50  0000 R CNN
+F 1 "10u" H 5285 2595 50  0000 R CNN
 F 2 "10106052 PowerPack:CAPC1608X86N" H 5438 2400 50  0001 C CNN
 F 3 "https://api.kemet.com/component-edge/download/datasheet/C0603C106M9PACTU.pdf" H 5400 2550 50  0001 C CNN
@@
 F 8 "Kemet" H 5400 2550 50  0001 C CNN "Manufacturer"
 	1    5400 2550
-	1    0    0    -1
-$EndComp
-Wire Wire Line
+	-1   0    0    1
+$EndComp
+Wire Wire Line
