File: 10106052 PowerPack/10106052 PowerPack.kicad_pcb (KiCad board)
At the start: 4 copper layers, 0 parts

Commit message: Import drawing as Cmts.User layer
Parts:
- added H1: MountingHole, MountingHole:MountingHole_3.2mm_M3_ISO7380, F.Cu at (-264.4, -174.4)
Other:
- board outline added: 210 x 34 mm

Commit message: PCB Added and Schematic Footprints Added
Parts:
- removed H1: MountingHole, MountingHole:MountingHole_3.2mm_M3_ISO7380
- added C1: CAPC1608X86N, CAPC1608X86N_15, B.Cu at (382.6, 29.3)
- added C10: CAPC1608X86N, CAPC1608X86N_14, B.Cu at (414.8, 52.4)
- added C11: CAPC1608X86N, CAPC1608X86N_13, B.Cu at (404.3, 46.8)
- added C12: CAPC1608X86N, CAPC1608X86N_12, B.Cu at (404.3, 49.5)
- added C14: CAPC1608X86N, CAPC1608X86N_11, B.Cu at (458.5, 50.0)
- added C2: CAPC1608X86N, CAPC1608X86N_10, B.Cu at (430.8, 32.8)
- added C22: CAPC1608X86N, CAPC1608X86N_6, B.Cu at (320.8, 39.3)
- added C23: CAPC1608X86N, CAPC1608X86N_9, B.Cu at (320.8, 37.0)
- added C24: CAPC1608X86N, CAPC1608X86N_8, B.Cu at (319.8, 55.5)
- added C25: CAPC1608X86N, CAPC1608X86N_7, B.Cu at (296.4, 40.1)
- added C3: CAPC3225X155N, CAPC3225X155N_1, B.Cu at (418.1, 38.0)
- added C30: CAPC1608X86N, CAPC1608X86N_6, B.Cu at (472.7, 50.7)
- added C4: CAPC1608X86N, CAPC1608X86N_5, B.Cu at (351.1, 52.3)
- added C5: CAPC1608X86N, CAPC1608X86N_4, B.Cu at (333.1, 50.4)
- added C6: CAPC1005X60N, CAPC1005X60N_1, B.Cu at (334.8, 50.5)
- added C7: CAPC1608X86N, CAPC1608X86N_3, B.Cu at (341.3, 52.0)
- added C8: CAPPRD350W60D800H1250PBA, CAPPRD350W60D800H1250PBA_1, F.Cu at (452.1, 51.3)
- added C9: CAPPRD350W60D800H1250PAAAAA, CAPPRD350W60D800H1250PAAAAA_1, F.Cu at (452.1, 41.8)
- added D1: DIOM5126X203N_SWP, DIOM5126X203N_SWP_4, B.Cu at (391.8, 48.8)
- added D10: SOT95P275X110-6N, SOT95P275X110-6N_4, B.Cu at (297.8, 54.5)
- added D11: SOT95P275X110-6N, SOT95P275X110-6N_3, B.Cu at (300.8, 47.9)
- added D12: SOT95P275X110-6N, SOT95P275X110-6N_2, B.Cu at (300.8, 40.3)
- added D13: SOT95P275X110-6N, SOT95P275X110-6N_1, B.Cu at (297.8, 33.7)
- added D14: DIOM5126X203N_SWP, DIOM5126X203N_SWP_3, B.Cu at (294.7, 44.3)
- added D15: SOT65P220X110-3N, SOT65P220X110-3N_3, B.Cu at (376.1, 39.0)
- added D2: SOT65P220X110-3N, SOT65P220X110-3N_2, B.Cu at (379.8, 39.0)
- added D3: SOD2512X110N_SWP, SOD2512X110N_SWP_3, B.Cu at (389.1, 28.8)
- added D4: SOD2512X110N_SWP, SOD2512X110N_SWP_2, B.Cu at (430.1, 28.8)
- added D5: SOT92P240X120-3N, SOT92P240X120-3N_1, B.Cu at (426.8, 29.8)
- added D6: SOD2512X110N_SWP, SOD2512X110N_SWP_1, B.Cu at (355.3, 28.8)
- added D7: DIOM5126X203N_SWP, DIOM5126X203N_SWP_2, B.Cu at (352.1, 36.8)
- added D8: SOT65P220X110-3N, SOT65P220X110-3N_1, B.Cu at (339.3, 39.3)
- added D9: DIOM5126X203N_SWP, DIOM5126X203N_SWP_1, B.Cu at (452.8, 36.8)
- added F1: FUS4755X155N, FUS4755X155N_1, B.Cu at (448.3, 37.3)
- added FID1: FIDUCIAL, FIDUCIAL_1, F.Cu at (277.3, 27.5)
- added FID2: FIDUCIAL, FIDUCIAL_1, F.Cu at (482.8, 53.0)
- added FL1: BNX00201, BNX00201_1, F.Cu at (477.2, 44.3)
- added J1: CON254W80L508T254H600P, CON254W80L508T254H600P_6, F.Cu at (386.5, 46.8)
- added J10: CON-S2B-ZR-SM4A-TF, CON-S2B-ZR-SM4A-TF_1, B.Cu at (471.6, 31.5)
- added J11: CON-43650-0229, CON-43650-0229_1, F.Cu at (480.1, 31.8)
- added J12: CON-52207-1960, CON-52207-1960_1, B.Cu at (288.9, 42.3)
- added J13: CON-S5B-ZR-SM4A-TF, CON-S5B-ZR-SM4A-TF_1, B.Cu at (333.8, 31.5)
- added J2: CON254W80L508T254H600P, CON254W80L508T254H600P_5, F.Cu at (386.5, 42.8)
- added J3: CON254W80L508T254H600P, CON254W80L508T254H600P_4, F.Cu at (386.5, 38.8)
- added J4: GKS-913-305-230-A-15-02-S, GKS-913-305-230-A-15-02-S_1, F.Cu at (386.5, 34.8)
- added J5: CON254W80L508T254H600P, CON254W80L508T254H600P_3, F.Cu at (346.9, 34.8)
- added J6: CON254W80L508T254H600P, CON254W80L508T254H600P_2, F.Cu at (346.9, 38.8)
- added J7: CON254W80L508T254H600P, CON254W80L508T254H600P_1, F.Cu at (346.9, 42.8)
- added J8: GKS-913-305-230-A-15-02-S, GKS-913-305-230-A-15-02-S_1, F.Cu at (346.9, 46.8)
- added J9: CON2PHDR1000W777L396P, CON2PHDR1000W777L396P_1, F.Cu at (450.6, 30.3)
- added MT1: MTHOLE1, MTHOLE1_1, F.Cu at (367.1, 31.3)
- added R1: RESC1608X50AN, RESC1608X50AN_49, B.Cu at (396.3, 43.0)
- added R10: RESC1608X50AN, RESC1608X50AN_48, B.Cu at (409.8, 41.3)
- added R11: RESC1608X50AN, RESC1608X50AN_47, B.Cu at (422.8, 32.8)
- added R12: RESC1608X50AN, RESC1608X50AN_46, B.Cu at (405.1, 41.3)
- added R13: RESC1608X50AN, RESC1608X50AN_45, B.Cu at (400.8, 50.3)
- added R14: RESC1608X50AN, RESC1608X50AN_44, B.Cu at (342.8, 33.0)
- added R15: RESC1608X50AN, RESC1608X50AN_43, B.Cu at (342.8, 42.8)
- added R16: RESC1608X50AN, RESC1608X50AN_42, B.Cu at (356.8, 51.5)
- added R17: RESC1608X50AN, RESC1608X50AN_41, B.Cu at (359.6, 49.8)
- added R18: RESC1608X50AN, RESC1608X50AN_40, B.Cu at (359.6, 48.0)
- added R19: RESC1608X50AN, RESC1608X50AN_39, B.Cu at (353.1, 52.3)
- added R2: RESC1608X50AN, RESC1608X50AN_38, B.Cu at (396.3, 41.3)
- added R20: RESC1608X50AN, RESC1608X50AN_37, B.Cu at (362.7, 55.3)
- added R21: RESC1608X50AN, RESC1608X50AN_36, B.Cu at (368.3, 49.7)
- added R22: RESC1608X50AN, RESC1608X50AN_35, B.Cu at (368.3, 48.0)
- added R23: RESC1608X50AN, RESC1608X50AN_34, B.Cu at (367.6, 55.3)
- added R24: RESC6533X80N, RESC6533X80N_1, B.Cu at (410.1, 46.8)
- added R25: RESC3216X60N, RESC3216X60N_4, B.Cu at (462.1, 46.3)
- added R26: RESC3216X60N, RESC3216X60N_3, B.Cu at (470.1, 37.0)
- added R27: RESC1608X50AN, RESC1608X50AN_33, B.Cu at (456.8, 45.5)
- added R28: RESC1608X50AN, RESC1608X50AN_32, B.Cu at (404.3, 53.0)
- added R29: RESC1608X50AN, RESC1608X50AN_31, B.Cu at (404.3, 51.3)
- added R3: RESC1608X50AN, RESC1608X50AN_30, B.Cu at (386.6, 29.3)
- added R30: RESC1608X50AN, RESC1608X50AN_29, B.Cu at (456.8, 50.0)
- added R31: RESC1608X50AN, RESC1608X50AN_28, B.Cu at (473.1, 38.5)
- added R32: RESC3216X60N, RESC3216X60N_2, B.Cu at (462.1, 51.3)
- added R33: RESC1608X50AN, RESC1608X50AN_27, B.Cu at (306.3, 35.3)
- added R34: RESC1608X50AN, RESC1608X50AN_26, B.Cu at (306.3, 37.3)
- added R35: RESC1608X50AN, RESC1608X50AN_25, B.Cu at (306.3, 39.0)
- added R36: RESC1608X50AN, RESC1608X50AN_24, B.Cu at (306.3, 40.8)
- added R37: RESC1608X50AN, RESC1608X50AN_23, B.Cu at (306.3, 44.5)
- added R38: RESC1608X50AN, RESC1608X50AN_22, B.Cu at (306.3, 46.3)
- added R39: RESC1608X50AN, RESC1608X50AN_21, B.Cu at (306.3, 42.5)
- added R4: RESC1608X50AN, RESC1608X50AN_20, B.Cu at (382.1, 46.8)
- added R40: RESC1608X50AN, RESC1608X50AN_11, B.Cu at (306.3, 48.0)
- added R41: RESC1608X50AN, RESC1608X50AN_19, B.Cu at (331.2, 40.8)
- added R42: RESC1608X50AN, RESC1608X50AN_18, B.Cu at (306.3, 49.8)
- added R43: RESC1608X50AN, RESC1608X50AN_17, B.Cu at (306.3, 51.5)
- added R44: RESC3216X60N, RESC3216X60N_1, B.Cu at (294.4, 47.1)
- added R45: RESC1608X50AN, RESC1608X50AN_6, B.Cu at (306.3, 53.3)
- added R46: RESC1608X50AN, RESC1608X50AN_16, B.Cu at (306.3, 55.0)
- added R47: RESC1608X50AN, RESC1608X50AN_15, B.Cu at (306.3, 56.8)
- added R48: RESC1608X50AN, RESC1608X50AN_14, B.Cu at (293.2, 41.8)
- added R49: RESC1608X50AN, RESC1608X50AN_13, B.Cu at (296.4, 41.8)
- added R5: RESC1608X50AN, RESC1608X50AN_12, B.Cu at (382.1, 38.8)
- added R50: CAPC1608X86N, CAPC1608X86N_2, B.Cu at (382.1, 42.8)
- added R51: CAPC1608X86N, CAPC1608X86N_1, B.Cu at (342.8, 36.8)
- added R52: RESC1608X50AN, RESC1608X50AN_11, B.Cu at (440.3, 52.5)
- added R53: RESC1608X50AN, RESC1608X50AN_10, B.Cu at (443.1, 48.0)
- added R54: RESC1608X50AN, RESC1608X50AN_9, B.Cu at (437.1, 48.0)
- added R55: RESC1608X50AN, RESC1608X50AN_8, B.Cu at (445.3, 48.0)
- added R56: RESC1608X50AN, RESC1608X50AN_7, B.Cu at (440.3, 54.0)
- added R57: RESC1608X50AN, RESC1608X50AN_6, B.Cu at (379.5, 42.0)
- added R58: RESC1608X50AN, RESC1608X50AN_5, B.Cu at (342.8, 39.8)
- added R6: RESC1608X50AN, RESC1608X50AN_4, B.Cu at (416.8, 32.8)
- added R7: RESC1608X50AN, RESC1608X50AN_3, B.Cu at (384.6, 29.3)
- added R8: RESC1608X50AN, RESC1608X50AN_2, B.Cu at (396.3, 50.3)
- added R9: RESC1608X50AN, RESC1608X50AN_1, B.Cu at (419.8, 29.8)
- added RL1: RLY-41-52-9-024-0010, RLY-41-52-9-024-0010_1, F.Cu at (466.6, 54.5)
- added RX: TP-40R-NSA, TP-40R-NSA_1, F.Cu at (318.2, 36.8)
- added STAR1: STAR, STAR_1, B.Cu at (387.2, 55.9)
- added T1: SOT95P237X112-3N, SOT95P237X112-3N_10, B.Cu at (396.3, 47.3)
- added T10: SOT95P237X112-3N, SOT95P237X112-3N_9, B.Cu at (367.6, 52.3)
- added T11: SOT95P237X112-3N, SOT95P237X112-3N_8, B.Cu at (473.1, 35.5)
- added T12: SOT95P237X112-3N, SOT95P237X112-3N_7, B.Cu at (378.6, 46.5)
- added T13: SOT95P237X112-3N, SOT95P237X112-3N_6, B.Cu at (335.6, 39.5)
- added T14: TO228P1003X238-3_4N, TO228P1003X238-3_4N_5, B.Cu at (440.3, 39.8)
- added T15: SOT95P237X112-3N, SOT95P237X112-3N_5, B.Cu at (440.3, 49.8)
- added T2: TO228P1003X238-3_4N, TO228P1003X238-3_4N_4, B.Cu at (396.3, 34.3)
- added T3: SOT95P237X112-3N, SOT95P237X112-3N_4, B.Cu at (416.8, 29.8)
- added T4: TO228P1003X238-3_4N, TO228P1003X238-3_4N_3, B.Cu at (405.1, 34.3)
- added T5: SOT95P237X112-3N, SOT95P237X112-3N_3, B.Cu at (422.8, 29.8)
- added T6: SOT95P237X112-3N, SOT95P237X112-3N_2, B.Cu at (400.8, 47.3)
- added T7: SOT95P237X112-3N, SOT95P237X112-3N_1, B.Cu at (362.7, 52.3)
- added T8: TO228P1003X238-3_4N, TO228P1003X238-3_4N_2, B.Cu at (359.6, 41.0)
- added T9: TO228P1003X238-3_4N, TO228P1003X238-3_4N_1, B.Cu at (368.3, 41.0)
- added TX: TP-40R-NSA, TP-40R-NSA_1, F.Cu at (318.2, 38.6)
- added U1: TO170P1420X457-8NA, TO170P1420X457-8NA_1, B.Cu at (426.5, 41.0)
- added U2: SOT95P279X142-5N, SOT95P279X142-5N_1, B.Cu at (338.6, 50.5)
- added U3: SOP65P490X110-8N, SOP65P490X110-8N_1, B.Cu at (410.1, 51.3)
- added U4: QFP80P1200X1200X120-44N, QFP80P1200X1200X120-44N_1, B.Cu at (320.3, 47.3)
- added U6: TO-92, TO-92_1, F.Cu at (473.9, 52.9)
Routing:
- net GND: track 0.00 -> 475.6 mm, vias 0 -> 29
- net +5V: track 0.00 -> 416.2 mm, vias 0 -> 17
- net AGND: track 0.00 -> 292.8 mm, vias 0 -> 4
- net V_DC_CHARGER: track 0.00 -> 201.4 mm, vias 0 -> 5
- net TEMP_MEAS: track 0.00 -> 180.4 mm, vias 0 -> 3
- net +VDC_PERM: track 0.00 -> 178.2 mm, vias 0 -> 3
- net V_CH: track 0.00 -> 163.2 mm, vias 0 -> 5
- net FAN_EN: track 0.00 -> 162.7 mm, vias 0 -> 2
- net BP: track 0.00 -> 152.0 mm, vias 0 -> 2
- net V_EN: track 0.00 -> 124.9 mm, vias 0 -> 5
- net +3.0VREF: track 0.00 -> 101.2 mm, vias 0 -> 2
- net CHARG_BAT1: track 0.00 -> 95.4 mm, vias 0 -> 2
- net DISCH_BAT1: track 0.00 -> 91.1 mm, vias 0 -> 4
- net IBAT_MEAS: track 0.00 -> 88.9 mm, vias 0 -> 3
- net N16104935: track 0.00 -> 88.7 mm, vias 0 -> 1
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- added copper zone on B.Cu, net GND
- added copper zone on F.Cu, net GND
Other:
- copper layers 4 -> 2
- net class Default: clearance 0.1524 -> 0.2; trace_width 0.254 -> 0.25; via_dia 0.6858 -> 0.8; via_drill 0.3302 -> 0.4
- rule pad_to_mask_clearance: 0 -> 0.051
- rule solder_mask_min_width: 0.1016 -> 0.25
- rule trace_clearance: 0.1524 -> 0.2
- rule trace_min: 0.127 -> 0.2
- rule via_min_drill: 0.254 -> 0.3
- rule via_min_size: 0.4572 -> 0.4
- board text added: "+3.0REF"
- board text added: "+5V"
- board text added: "+VDC_PERM"
- board text added: "11.0"
- board text added: "12.40"
- board text added: "126.0"
- board text added: "17.00"
- board text added: "20.0"
- board text added: "210"
- board text added: "28.0"
- board text added: "53.5"
- board text added: "6"
- board text added: "6.0"
- board text added: "AGND"
- board text added: "BOTTOM SIDE"
- board text added: "BP"
- board text added: "BP_INFO"
- board text added: "CHG_BAT1"
- board text added: "CHG_BAT2"
- board text added: "COVIDIEN"
- board text added: "DISCHG_BAT1"
- board text added: "DISCHG_BAT2"
- board text added: "FAN_EN"
- board text added: "GND"
- board text added: "HEIGHT RESTRICTION OF 7MM"
- board text added: "IBAT_MEAS"
- board text added: "ID_BAT1"
- board text added: "ID_BAT2"
- board text added: "ID_BAT_READ"
- board text added: "J12"
- board text added: "L1"
- board text added: "L2"
- board text added: "LAYER 1 - PRIMARY SIDE"
- board text added: "LAYER 2 - SECONDARY SIDE"
- board text added: "LAYER 4 - BOTTOM"
- board text added: "MCLR"
- board text added: "ON THIS SIDE OF THE BOARD"
- board text added: "PASTE BOTTOM"
- board text added: "PASTE TOP"
- board text added: "PGC"
- board text added: "PGD"
- board text added: "Powerpack2 Board, 10106054 Rev A"
- board text added: "RESIST BOTTOM"
- board text added: "RESIST TOP"
- board text added: "SILKSCREEN BOTTOM"
- board text added: "SILKSCREEN TOP"
- board text added: "TEMP_BAT1"
- board text added: "TEMP_BAT2"
- board text added: "TEMP_MEAS"
- board text added: "VBAT1_MEAS"
- board text added: "VBAT2_MEAS"
- board text added: "V_CH"
- board text added: "V_DC_CHARGER"
- board text added: "V_EN"
- board text added: "\U+2205"

Commit message: powerpack-dev
Parts:
- removed RX, TX: TP-40R-NSA, TP-40R-NSA_1
- added RX1: TP-40R-NSA, TP-40R-NSA_1, F.Cu at (318.2, 36.8)
- added TX1: TP-40R-NSA, TP-40R-NSA_1, F.Cu at (318.2, 38.6)
Changed lines of the file:
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@@
-(kicad_pcb (version 20171130) (host pcbnew 5.1.5+dfsg1-2~bpo10+1)
+(kicad_pcb (version 20171130) (host pcbnew 5.1.5-52549c5~86~ubuntu18.04.1)
   (general
     (thickness 1.6)
@@
     (add_net +5V)
     (add_net +VDC_PERM)
-    (add_net "/Microcontroller block/RX")
-    (add_net "/Microcontroller block/TX")
     (add_net AGND)
     (add_net BP)
@@
     (add_net N16383725)
     (add_net N16384319)
-    (add_net "Net-(FL1-Pad1)")
-    (add_net "Net-(FL1-Pad2)")
-    (add_net "Net-(FL1-Pad3)")
-    (add_net "Net-(FL1-Pad4)")
-    (add_net "Net-(RL1-Pad14)")
-    (add_net "Net-(RL1-Pad24)")
-    (add_net "Net-(U1-Pad2)")
-    (add_net "Net-(U2-Pad1)")
-    (add_net "Net-(U3-Pad7)")
-    (add_net "Net-(U4-Pad12)")
-    (add_net "Net-(U4-Pad13)")
-    (add_net "Net-(U4-Pad33)")
-    (add_net "Net-(U4-Pad34)")
     (add_net PGC)
     (add_net PGD)
@@
     (at 318.2034 38.6434)
     (attr smd)
-    (fp_text reference TX (at -2.0193 0.2159 unlocked) (layer F.SilkS)
+    (fp_text reference TX1 (at -2.0193 0.2159 unlocked) (layer F.SilkS)
       (effects (font (size 0.216611 0.227838) (thickness 0.0254)))
     )
@@
     (at 318.2034 36.7892)
     (attr smd)
-    (fp_text reference RX (at -2.0447 0.2159 unlocked) (layer F.SilkS)
+    (fp_text reference RX1 (at -2.0447 0.2159 unlocked) (layer F.SilkS)
       (effects (font (size 0.216611 0.227838) (thickness 0.0254)))
     )

Commit message: Schematic Synched to PCB
Parts:
- C1, C14, C23, C24, C25, C30, C4, C5, C7: value CAPC1608X86N -> 100n
- C10, C11, C12: value CAPC1608X86N -> 10n
- C2, C22: value CAPC1608X86N -> 10u
- C3: value CAPC3225X155N -> 1u
- C6: value CAPC1005X60N -> 1u
- C8: value CAPPRD350W60D800H1250PBA -> 100u
- C9: value CAPPRD350W60D800H1250PAAAAA -> 100u
- D1, D14, D7, D9: value DIOM5126X203N_SWP -> SMA6J28A
- D10, D11, D12, D13: value SOT95P275X110-6N -> PESD5V0S4UD
- D15: value SOT65P220X110-3N -> BAT54CWT1G
- D2, D8: value SOT65P220X110-3N -> SP0502BAHTG
- D3, D4, D6: value SOD2512X110N_SWP -> PMEG4005AEA
- D5: value SOT92P240X120-3N -> BAS70-05
- F1: value FUS4755X155N -> Fuse
- FL1: value BNX00201 -> BNX002-11
- J1, J2, J3, J5, J6, J7: value CON254W80L508T254H600P -> 811-S1-002-10-015101
- J10: value CON-S2B-ZR-SM4A-TF -> S2B-ZR-SM4A-TF
- J11: value CON-43650-0229 -> 43650-0229
- J12: value CON-52207-1960 -> Molex_52207-1933_1x19-1MP_P1.00mm_Horizontal
- J13: value CON-S5B-ZR-SM4A-TF -> S5B-ZR-SM4A-TF
- J4, J8: value GKS-913-305-230-A-15-02-S -> GKS 913 305 230 A 15 02 S
- J9: value CON2PHDR1000W777L396P -> 26-61-4020
- R1, R10, R11, R17, R19, R21, R30, R49, R53, R56, R6, R7, R9: value RESC1608X50AN -> 10k
- R12, R18, R2, R22, R54: value RESC1608X50AN -> 15k
- R13, R20, R23, R31, R52, R8: value RESC1608X50AN -> 22k
- R14, R33, R34, R35, R36, R37, R38, R39, R4, R40, R42, R43, R45, R46, R47: value RESC1608X50AN -> 1k
- R15, R5: value RESC1608X50AN -> 18k
- R16, R27, R3: value RESC1608X50AN -> 100k
- R24: value RESC6533X80N -> 0.015
- R25: value RESC3216X60N -> 0
- R26: value RESC3216X60N -> 68
- R28: value RESC1608X50AN -> 66.5k
- R29: value RESC1608X50AN -> 40.2k
- R32: value RESC3216X60N -> 470
- R41: value RESC1608X50AN -> 4.7k
- R44: value RESC3216X60N -> 4.7k
- R48: value RESC1608X50AN -> 62k
- R50, R51: value CAPC1608X86N -> 100
- R55: value RESC1608X50AN -> 47k
- R57, R58: value RESC1608X50AN -> 0
- RL1: value RLY-41-52-9-024-0010 -> 41.52.9.024.0010
- RX1, TX1: value TP-40R-NSA -> TestPoint
- STAR1: value STAR -> Net-Tie_2
- T1, T10, T12, T13, T15, T6, T7: value SOT95P237X112-3N -> 2N7002TA
- T11, T5: value SOT95P237X112-3N -> SI2300DS-T1-GE3
- T14, T2, T4, T8, T9: value TO228P1003X238-3_4N -> SUD50P06-15
- T3: value SOT95P237X112-3N -> SI2309CDS-T1-GE3
- U1: value TO170P1420X457-8NA -> NCV87722DT50RKG
- U2: value SOT95P279X142-5N -> LM4120AIM5-3.0
- U3: value SOP65P490X110-8N -> INA170
- U4: value QFP80P1200X1200X120-44N -> PIC18F43K22T-IPT
- U6: value TO-92 -> MCP9700A-E_TO
Connections:
- net AGND renamed GNDA
- net BP renamed /BP
- net BP_INFO renamed /Microcontroller block/BP_INFO
- net CHARG_BAT1 renamed /CHARG_BAT1
- net CHARG_BAT2 renamed /CHARG_BAT2
- net DISCH_BAT1 renamed /DISCH_BAT1
- net DISCH_BAT2 renamed /DISCH_BAT2
- net FAN_EN renamed /FAN_EN
- net IBAT_MEAS renamed /IBAT_MEAS
- net ID_BAT1 renamed /ID_BAT1
- net ID_BAT2 renamed /ID_BAT2
- net ID_BAT_READ renamed /ID_BAT_READ
- net MCLR renamed /Microcontroller block/MCLR
- net N16098669 renamed Net-(D9-Pad2)
- net N16099163 renamed Net-(R1-Pad2)
- net N16099172 renamed Net-(R1-Pad1)
- net N16099189 renamed Net-(D1-Pad2)
- net N16099430 renamed Net-(R10-Pad2)
- net N16099438 renamed Net-(R10-Pad1)
- net N16099574 renamed Net-(T2-Pad4)
- net N16102944 renamed Net-(R17-Pad2)
- net N16102952 renamed Net-(R17-Pad1)
- net N16102968 renamed Net-(D6-Pad1)
- net N16103028 renamed Net-(R21-Pad2)
- net N16103036 renamed Net-(R21-Pad1)
- net N16103052 renamed Net-(T8-Pad4)
- net N16104931 renamed /Switching block/+BATT_BUS
- net N16104935 renamed Net-(C8-Pad1)
- net N16108884 renamed Net-(J2-Pad1)
- net N16114574 renamed Net-(R33-Pad2)
- net N16114708 renamed Net-(R34-Pad2)
- net N16114712 renamed Net-(R35-Pad2)
- net N16114784 renamed Net-(R36-Pad2)
- net N16114788 renamed Net-(R39-Pad2)
- net N16114860 renamed Net-(R37-Pad2)
- net N16114864 renamed Net-(R38-Pad2)
- net N16120987 renamed Net-(D15-Pad2)
- net N16121186 renamed Net-(D15-Pad1)
- net N16123242 renamed Net-(R40-Pad2)
- net N16123728 renamed Net-(R42-Pad2)
- net N16123740 renamed Net-(R43-Pad2)
- net N16123752 renamed Net-(R45-Pad2)
- net N16124630 renamed Net-(D13-Pad3)
- net N16124642 renamed Net-(D13-Pad4)
- net N16124654 renamed Net-(D13-Pad6)
- net N16124670 renamed Net-(D12-Pad1)
- net N16124678 renamed Net-(D12-Pad3)
- net N16124694 renamed Net-(D12-Pad4)
- net N16124795 renamed Net-(D12-Pad6)
- net N16125012 renamed Net-(D11-Pad1)
- net N16125020 renamed Net-(D11-Pad3)
- net N16125036 renamed Net-(D11-Pad4)
- net N16125044 renamed Net-(D11-Pad6)
- net N16125060 renamed Net-(D10-Pad1)
- net N16125068 renamed Net-(D10-Pad3)
- net N16128468 renamed Net-(R28-Pad2)
- net N16140479 renamed Net-(J10-Pad2)
- net N16140749 renamed Net-(J10-Pad1)
- net N16147060 renamed Net-(D2-Pad2)
- net N16148240 renamed Net-(D8-Pad2)
- net N16163380 renamed Net-(R47-Pad2)
- net N16171508 renamed Net-(J12-Pad7)
- net N16173153 renamed Net-(R46-Pad2)
- net N16188495 renamed Net-(R6-Pad2)
- net N16188649 renamed Net-(R9-Pad2)
- net N16216077 renamed Net-(J6-Pad1)
- net N16275854 renamed Net-(FL1-PadB)
- net N16275858 renamed Net-(FL1-PadPSG)
- net N16285730 renamed Net-(R32-Pad1)
- net N16293601 renamed Net-(F1-Pad1)
- net N16382223 renamed Net-(R52-Pad2)
- net N16383725 renamed Net-(R53-Pad1)
- net N16384319 renamed Net-(R53-Pad2)
- net PGC renamed /Microcontroller block/PGC
- net PGD renamed /Microcontroller block/PGD
- net RX renamed Net-(RX1-Pad1)
- net TEMP_BAT1 renamed /TEMP_BAT1
- net TEMP_BAT2 renamed /TEMP_BAT2
- net TEMP_MEAS renamed /TEMP_MEAS
- net TX renamed Net-(TX1-Pad1)
- net VBAT1_MEAS renamed /VBAT1_MEAS
- net VBAT2_MEAS renamed /VBAT2_MEAS
- net V_CH renamed /V_CH
- net V_DC_CHARGER renamed /V_DC_CHARGER
- net V_EN renamed /V_EN
- net X00088 renamed Net-(FL1-PadCB)
- net X00089 renamed Net-(FL1-PadCG1)
- D5 pad 3: N16136951 -> Net-(D5-Pad3)
- RL1 pad 14: (no net) -> Net-(RL1-Pad14)
- RL1 pad 24: (no net) -> Net-(RL1-Pad24)
- T3 pad 3: N16136951 -> Net-(D5-Pad3)
- U1 pad 2: (no net) -> Net-(U1-Pad2)
- U1 pad 3: (no net) -> GND
- U1 pad 4: GND -> Net-(D5-Pad3)
- U1 pad 5: N16136951 -> +5V
- U1 pad 6: GND -> (no net)
- U1 pad 7: +5V -> (no net)
- U1 pad 8: GND -> (no net)
- U2 pad 1: (no net) -> Net-(U2-Pad1)
- U3 pad 7: (no net) -> Net-(U3-Pad7)
- U4 pad 12: (no net) -> Net-(U4-Pad12)
- U4 pad 13: (no net) -> Net-(U4-Pad13)
- U4 pad 33: (no net) -> Net-(U4-Pad33)
- U4 pad 34: (no net) -> Net-(U4-Pad34)

Commit message: Added some design rules
Other:
- net class 0.6mm added: clearance 0.5, trace_width 0.25, via_dia 1, via_drill 0.4
- net class ClearanceClass_3(RuleSet) added: clearance 0.25, trace_width 0.25, via_dia 1, via_drill 0.4
- net class Default: clearance 0.2 -> 0.25; via_dia 0.8 -> 1
- rule trace_clearance: 0.2 -> 0.25

Commit message: correctly associate pcb footprints to library
Parts:
- C1: footprint CAPC1608X86N_15 -> 10106052 PowerPack:CAPC1608X86N
- C10: footprint CAPC1608X86N_14 -> 10106052 PowerPack:CAPC1608X86N
- C11: footprint CAPC1608X86N_13 -> 10106052 PowerPack:CAPC1608X86N
- C12: footprint CAPC1608X86N_12 -> 10106052 PowerPack:CAPC1608X86N
- C14: footprint CAPC1608X86N_11 -> 10106052 PowerPack:CAPC1608X86N
- C2: footprint CAPC1608X86N_10 -> 10106052 PowerPack:CAPC1608X86N
- C22, C30: footprint CAPC1608X86N_6 -> 10106052 PowerPack:CAPC1608X86N
- C23: footprint CAPC1608X86N_9 -> 10106052 PowerPack:CAPC1608X86N
- C24: footprint CAPC1608X86N_8 -> 10106052 PowerPack:CAPC1608X86N
- C25: footprint CAPC1608X86N_7 -> 10106052 PowerPack:CAPC1608X86N
- C3: footprint CAPC3225X155N_1 -> 10106052 PowerPack:CAPC3225X155N
- C4: footprint CAPC1608X86N_5 -> 10106052 PowerPack:CAPC1608X86N
- C5: footprint CAPC1608X86N_4 -> 10106052 PowerPack:CAPC1608X86N
- C6: footprint CAPC1005X60N_1 -> 10106052 PowerPack:CAPC1005X60N
- C7: footprint CAPC1608X86N_3 -> 10106052 PowerPack:CAPC1608X86N
- C8: footprint CAPPRD350W60D800H1250PBA_1 -> 10106052 PowerPack:CAPPRD350W60D800H1250PBA
- C9: footprint CAPPRD350W60D800H1250PAAAAA_1 -> 10106052 PowerPack:CAPPRD350W60D800H1250PAAAAA
- D1: footprint DIOM5126X203N_SWP_4 -> 10106052 PowerPack:DIOM5126X203N_SWP
- D10: footprint SOT95P275X110-6N_4 -> 10106052 PowerPack:SOT95P275X110-6N
- D11: footprint SOT95P275X110-6N_3 -> 10106052 PowerPack:SOT95P275X110-6N
- D12: footprint SOT95P275X110-6N_2 -> 10106052 PowerPack:SOT95P275X110-6N
- D13: footprint SOT95P275X110-6N_1 -> 10106052 PowerPack:SOT95P275X110-6N
- D14: footprint DIOM5126X203N_SWP_3 -> 10106052 PowerPack:DIOM5126X203N_SWP
- D15: footprint SOT65P220X110-3N_3 -> 10106052 PowerPack:SOT65P220X110-3N
- D2: footprint SOT65P220X110-3N_2 -> 10106052 PowerPack:SOT65P220X110-3N
- D3: footprint SOD2512X110N_SWP_3 -> 10106052 PowerPack:SOD2512X110N_SWP
- D4: footprint SOD2512X110N_SWP_2 -> 10106052 PowerPack:SOD2512X110N_SWP
- D5: footprint SOT92P240X120-3N_1 -> 10106052 PowerPack:SOT92P240X120-3N
- D6: footprint SOD2512X110N_SWP_1 -> 10106052 PowerPack:SOD2512X110N_SWP
- D7: footprint DIOM5126X203N_SWP_2 -> 10106052 PowerPack:DIOM5126X203N_SWP
- D8: footprint SOT65P220X110-3N_1 -> 10106052 PowerPack:SOT65P220X110-3N
- D9: footprint DIOM5126X203N_SWP_1 -> 10106052 PowerPack:DIOM5126X203N_SWP
- F1: footprint FUS4755X155N_1 -> 10106052 PowerPack:FUS4755X155N
- FID1, FID2: footprint FIDUCIAL_1 -> 10106052 PowerPack:FIDUCIAL
- FL1: footprint BNX00201_1 -> 10106052 PowerPack:BNX00201
- J1: footprint CON254W80L508T254H600P_6 -> 10106052 PowerPack:CON254W80L508T254H600P
- J10: footprint CON-S2B-ZR-SM4A-TF_1 -> 10106052 PowerPack:CON-S2B-ZR-SM4A-TF
- J11: footprint CON-43650-0229_1 -> 10106052 PowerPack:CON-43650-0229
- J12: footprint CON-52207-1960_1 -> 10106052 PowerPack:CON-52207-1960
- J13: footprint CON-S5B-ZR-SM4A-TF_1 -> 10106052 PowerPack:CON-S5B-ZR-SM4A-TF
- J2: footprint CON254W80L508T254H600P_5 -> 10106052 PowerPack:CON254W80L508T254H600P
- J3: footprint CON254W80L508T254H600P_4 -> 10106052 PowerPack:CON254W80L508T254H600P
- J4, J8: footprint GKS-913-305-230-A-15-02-S_1 -> 10106052 PowerPack:GKS-913-305-230-A-15-02-S
- J5: footprint CON254W80L508T254H600P_3 -> 10106052 PowerPack:CON254W80L508T254H600P
- J6: footprint CON254W80L508T254H600P_2 -> 10106052 PowerPack:CON254W80L508T254H600P
- J7: footprint CON254W80L508T254H600P_1 -> 10106052 PowerPack:CON254W80L508T254H600P
- J9: footprint CON2PHDR1000W777L396P_1 -> 10106052 PowerPack:CON2PHDR1000W777L396P
- MT1: footprint MTHOLE1_1 -> 10106052 PowerPack:MTHOLE1
- R1: footprint RESC1608X50AN_49 -> 10106052 PowerPack:RESC1608X50AN
- R10: footprint RESC1608X50AN_48 -> 10106052 PowerPack:RESC1608X50AN
- R11: footprint RESC1608X50AN_47 -> 10106052 PowerPack:RESC1608X50AN
- R12: footprint RESC1608X50AN_46 -> 10106052 PowerPack:RESC1608X50AN
- R13: footprint RESC1608X50AN_45 -> 10106052 PowerPack:RESC1608X50AN
- R14: footprint RESC1608X50AN_44 -> 10106052 PowerPack:RESC1608X50AN
- R15: footprint RESC1608X50AN_43 -> 10106052 PowerPack:RESC1608X50AN
- R16: footprint RESC1608X50AN_42 -> 10106052 PowerPack:RESC1608X50AN
- R17: footprint RESC1608X50AN_41 -> 10106052 PowerPack:RESC1608X50AN
- R18: footprint RESC1608X50AN_40 -> 10106052 PowerPack:RESC1608X50AN
- R19: footprint RESC1608X50AN_39 -> 10106052 PowerPack:RESC1608X50AN
- R2: footprint RESC1608X50AN_38 -> 10106052 PowerPack:RESC1608X50AN
- R20: footprint RESC1608X50AN_37 -> 10106052 PowerPack:RESC1608X50AN
- R21: footprint RESC1608X50AN_36 -> 10106052 PowerPack:RESC1608X50AN
- R22: footprint RESC1608X50AN_35 -> 10106052 PowerPack:RESC1608X50AN
- R23: footprint RESC1608X50AN_34 -> 10106052 PowerPack:RESC1608X50AN
- R24: footprint RESC6533X80N_1 -> 10106052 PowerPack:RESC6533X80N
- R25: footprint RESC3216X60N_4 -> 10106052 PowerPack:RESC3216X60N
- R26: footprint RESC3216X60N_3 -> 10106052 PowerPack:RESC3216X60N
- R27: footprint RESC1608X50AN_33 -> 10106052 PowerPack:RESC1608X50AN
- R28: footprint RESC1608X50AN_32 -> 10106052 PowerPack:RESC1608X50AN
- R29: footprint RESC1608X50AN_31 -> 10106052 PowerPack:RESC1608X50AN
- R3: footprint RESC1608X50AN_30 -> 10106052 PowerPack:RESC1608X50AN
- R30: footprint RESC1608X50AN_29 -> 10106052 PowerPack:RESC1608X50AN
- R31: footprint RESC1608X50AN_28 -> 10106052 PowerPack:RESC1608X50AN
- R32: footprint RESC3216X60N_2 -> 10106052 PowerPack:RESC3216X60N
- R33: footprint RESC1608X50AN_27 -> 10106052 PowerPack:RESC1608X50AN
- R34: footprint RESC1608X50AN_26 -> 10106052 PowerPack:RESC1608X50AN
- R35: footprint RESC1608X50AN_25 -> 10106052 PowerPack:RESC1608X50AN
- R36: footprint RESC1608X50AN_24 -> 10106052 PowerPack:RESC1608X50AN
- R37: footprint RESC1608X50AN_23 -> 10106052 PowerPack:RESC1608X50AN
- R38: footprint RESC1608X50AN_22 -> 10106052 PowerPack:RESC1608X50AN
- R39: footprint RESC1608X50AN_21 -> 10106052 PowerPack:RESC1608X50AN
- R4: footprint RESC1608X50AN_20 -> 10106052 PowerPack:RESC1608X50AN
- R40, R52: footprint RESC1608X50AN_11 -> 10106052 PowerPack:RESC1608X50AN
- R41: footprint RESC1608X50AN_19 -> 10106052 PowerPack:RESC1608X50AN
- R42: footprint RESC1608X50AN_18 -> 10106052 PowerPack:RESC1608X50AN
- R43: footprint RESC1608X50AN_17 -> 10106052 PowerPack:RESC1608X50AN
- R44: footprint RESC3216X60N_1 -> 10106052 PowerPack:RESC3216X60N
- R45, R57: footprint RESC1608X50AN_6 -> 10106052 PowerPack:RESC1608X50AN
- R46: footprint RESC1608X50AN_16 -> 10106052 PowerPack:RESC1608X50AN
- R47: footprint RESC1608X50AN_15 -> 10106052 PowerPack:RESC1608X50AN
- R48: footprint RESC1608X50AN_14 -> 10106052 PowerPack:RESC1608X50AN
- R49: footprint RESC1608X50AN_13 -> 10106052 PowerPack:RESC1608X50AN
- R5: footprint RESC1608X50AN_12 -> 10106052 PowerPack:RESC1608X50AN
- R50: footprint CAPC1608X86N_2 -> 10106052 PowerPack:CAPC1608X86N
- R51: footprint CAPC1608X86N_1 -> 10106052 PowerPack:CAPC1608X86N
- R53: footprint RESC1608X50AN_10 -> 10106052 PowerPack:RESC1608X50AN
- R54: footprint RESC1608X50AN_9 -> 10106052 PowerPack:RESC1608X50AN
- R55: footprint RESC1608X50AN_8 -> 10106052 PowerPack:RESC1608X50AN
- R56: footprint RESC1608X50AN_7 -> 10106052 PowerPack:RESC1608X50AN
- R58: footprint RESC1608X50AN_5 -> 10106052 PowerPack:RESC1608X50AN
- R6: footprint RESC1608X50AN_4 -> 10106052 PowerPack:RESC1608X50AN
- R7: footprint RESC1608X50AN_3 -> 10106052 PowerPack:RESC1608X50AN
- R8: footprint RESC1608X50AN_2 -> 10106052 PowerPack:RESC1608X50AN
- R9: footprint RESC1608X50AN_1 -> 10106052 PowerPack:RESC1608X50AN
- RL1: footprint RLY-41-52-9-024-0010_1 -> 10106052 PowerPack:RLY-41-52-9-024-0010
- RX1, TX1: footprint TP-40R-NSA_1 -> 10106052 PowerPack:TP-40R-NSA
- STAR1: footprint STAR_1 -> 10106052 PowerPack:STAR
- T1: footprint SOT95P237X112-3N_10 -> 10106052 PowerPack:SOT95P237X112-3N
- T10: footprint SOT95P237X112-3N_9 -> 10106052 PowerPack:SOT95P237X112-3N
- T11: footprint SOT95P237X112-3N_8 -> 10106052 PowerPack:SOT95P237X112-3N
- T12: footprint SOT95P237X112-3N_7 -> 10106052 PowerPack:SOT95P237X112-3N
- T13: footprint SOT95P237X112-3N_6 -> 10106052 PowerPack:SOT95P237X112-3N
- T14: footprint TO228P1003X238-3_4N_5 -> 10106052 PowerPack:TO228P1003X238-3_4N
- T15: footprint SOT95P237X112-3N_5 -> 10106052 PowerPack:SOT95P237X112-3N
- T2: footprint TO228P1003X238-3_4N_4 -> 10106052 PowerPack:TO228P1003X238-3_4N
- T3: footprint SOT95P237X112-3N_4 -> 10106052 PowerPack:SOT95P237X112-3N
- T4: footprint TO228P1003X238-3_4N_3 -> 10106052 PowerPack:TO228P1003X238-3_4N
- T5: footprint SOT95P237X112-3N_3 -> 10106052 PowerPack:SOT95P237X112-3N
- T6: footprint SOT95P237X112-3N_2 -> 10106052 PowerPack:SOT95P237X112-3N
- T7: footprint SOT95P237X112-3N_1 -> 10106052 PowerPack:SOT95P237X112-3N
- T8: footprint TO228P1003X238-3_4N_2 -> 10106052 PowerPack:TO228P1003X238-3_4N
- T9: footprint TO228P1003X238-3_4N_1 -> 10106052 PowerPack:TO228P1003X238-3_4N
- U1: footprint TO170P1420X457-8NA_1 -> 10106052 PowerPack:TO170P1420X457-8NA
- U2: footprint SOT95P279X142-5N_1 -> 10106052 PowerPack:SOT95P279X142-5N
- U3: footprint SOP65P490X110-8N_1 -> 10106052 PowerPack:SOP65P490X110-8N
- U4: footprint QFP80P1200X1200X120-44N_1 -> 10106052 PowerPack:QFP80P1200X1200X120-44N
- U6: footprint TO-92_1 -> 10106052 PowerPack:TO-92
