File: CPU_RB0505/cpu.sch (KiCad schematic (older format))
At the start: 10 parts

Commit message: Update CPU sheet
Parts:
- added RN?: R_Network04, Resistor_THT:R_Array_SIP5, symbol Device:R_Network04
Connections:
- net SPEED_MEASURE: now reaches U?.47 (P2.0-CC0IO)
- net BRAKE: now reaches U?.48 (P2.1-CC1IO)
- net DEF-TURB: now reaches U?.49 (P2.2-CC2IO)
- net ENABLE-TURB: now reaches U?.50 (P2.3-CC3IO)
- net WDOG: now reaches U?.51 (P2.4-CC4IO)
- net +3.3V-FAILURE: now reaches U?.52 (P2.5-CC5IO)
- net +5VREF-FAILURE: now reaches U?.53 (P2.6-CC6IO)
- net +10VREF-FAILURE: now reaches U?.54 (P2.7-CC7IO)
- net BUSY-ME1: now reaches U?.57 (P2.8-CC8IO-EX0IN)
- net BUSY-ME1: now also RN?.5 (R4)
- net BUSY-ME2: now reaches U?.58 (P2.9-CC9IO-EX1IN)
- net BUSY-ME2: now also RN?.4 (R3)
- net USB_BUSY_E: now reaches U?.59 (P2.10-CC10IOIO-EX2IN)
- net BUSY-AFF: now reaches U?.60 (P2.11-CC11IOIO-EX3IN)
- net TEST-RAP-ALARM: now reaches U?.61 (P2.12-CC12IOIO-EX4IN)
- net TEST-RAP-ALARM: now also RN?.3 (R2)
- net INV-STOP: now reaches U?.62 (P2.13-CC13IOIO-EX5IN)
- net RAP-ALARM: now reaches U?.63 (P2.14-CC14IOIO-EX6IN)
- net CMD_ME1: now reaches U?.64 (P2.15-CC15IOIO-EX7IN-T7IN)
- new net +5V: RN?.1 (common)
- no-connect marks 0 -> 1
Other:
- moved on the sheet: U?C, U?D, U?F

Commit message: Updating CPU sheet
Parts:
- removed RN?: R_Network04, Resistor_THT:R_Array_SIP5, symbol Device:R_Network04
- added CN?: C_Pack04, symbol CPU_RB0505:C_Pack04
- added RN? (x2): R_Pack04, symbol Device:R_Pack04
Connections:
- net labels added: GND
- wire segments 71 -> 107
Other:
- moved on the sheet: U?D, U?F, U?H, U?I
Changed lines of the file:
@@
 Connection ~ 6350 1850
 Connection ~ 6450 1750
+Connection ~ 6150 1200
+Connection ~ 6250 1200
+Connection ~ 6350 1200
+Connection ~ 6150 2500
+Connection ~ 5850 3500
+Connection ~ 5950 3400
+Connection ~ 6050 3300
+Connection ~ 6150 3200
 NoConn ~ 6150 1650
 Entry Wire Line
@@
 	5000 2450 5250 2450
 Wire Wire Line
+	5000 2900 5250 2900
+Wire Wire Line
+	5000 3000 5250 3000
+Wire Wire Line
+	5000 3100 5250 3100
+Wire Wire Line
+	5000 3200 6150 3200
+Wire Wire Line
+	5000 3300 6050 3300
+Wire Wire Line
+	5000 3400 5950 3400
+Wire Wire Line
+	5000 3500 5850 3500
+Wire Wire Line
+	5000 3600 5250 3600
+Wire Wire Line
+	5000 3700 5250 3700
+Wire Wire Line
+	5000 3800 5250 3800
+Wire Wire Line
+	5000 3900 5250 3900
+Wire Wire Line
+	5000 4000 5250 4000
+Wire Wire Line
+	5000 4100 5250 4100
+Wire Wire Line
+	5000 4200 5250 4200
+Wire Wire Line
+	5000 4400 5250 4400
+Wire Wire Line
+	5850 2500 5850 2550
+Wire Wire Line
+	5850 2950 5850 3500
+Wire Wire Line
+	5850 3500 6200 3500
+Wire Wire Line
+	5950 2250 5950 2550
+Wire Wire Line
+	5950 2950 5950 3400
+Wire Wire Line
+	5950 3400 6200 3400
+Wire Wire Line
+	6050 2500 6150 2500
+Wire Wire Line
+	6050 2550 6050 2500
+Wire Wire Line
+	6050 2950 6050 3300
+Wire Wire Line
+	6050 3300 6200 3300
+Wire Wire Line
 	6150 1200 6150 1250
 Wire Wire Line
+	6150 1200 6250 1200
+Wire Wire Line
+	6150 2500 6150 2550
+Wire Wire Line
+	6150 2950 6150 3200
+Wire Wire Line
+	6150 3200 6200 3200
+Wire Wire Line
+	6250 1200 6250 1250
+Wire Wire Line
+	6250 1200 6350 1200
+Wire Wire Line
 	6250 1650 6250 2150
 Wire Wire Line
 	6250 2150 6750 2150
 Wire Wire Line
+	6350 1200 6350 1250
+Wire Wire Line
+	6350 1200 6450 1200
+Wire Wire Line
 	6350 1650 6350 1850
 Wire Wire Line
 	6350 1850 6750 1850
 Wire Wire Line
+	6450 1250 6450 1200
+Wire Wire Line
 	6450 1650 6450 1750
 Wire Wire Line
 	6450 1750 6750 1750
+Wire Wire Line
+	6450 2250 5950 2250
+Wire Wire Line
+	6450 2350 6450 2250
 Wire Bus Line
 	2500 1050 2500 1250
 Wire Bus Line
-	2500 1250 2500 1350
-Wire Bus Line
-	2500 1350 2500 1550
-Wire Bus Line
-	2500 1550 2500 1650
-Wire Bus Line
-	2500 1650 2500 1850
-Wire Bus Line
-	2500 1850 2500 1950
+	2500 1250 2500 1450
+Wire Bus Line
+	2500 1450 2500 1650
+Wire Bus Line
+	2500 1650 2500 1750
+Wire Bus Line
+	2500 1750 2500 1950
 Wire Bus Line
 	2500 1950 2500 2150
@@
 	2500 3850 2500 4050
 Wire Bus Line
-	2500 4050 2500 4250
-Wire Bus Line
-	2500 4250 2500 4450
-Wire Bus Line
-	2500 4450 2500 5150
-Wire Bus Line
-	2500 5150 2500 5250
+	2500 4050 2500 4150
+Wire Bus Line
+	2500 4150 2500 4350
+Wire Bus Line
+	2500 4350 2500 4550
+Wire Bus Line
+	2500 4550 2500 5250
 Wire Bus Line
 	2500 5250 2500 5450
@@
 $Comp
 L power:+5V #PWR?
+U 1 1 5E9112EF
+P 5850 2500
+F 0 "#PWR?" H 5850 2350 50  0001 C CNN
+F 1 "+5V" H 5865 2673 50  0000 C CNN
+F 2 "" H 5850 2500 50  0001 C CNN
+F 3 "" H 5850 2500 50  0001 C CNN
+	1    5850 2500
+	1    0    0    -1
+$EndComp
+$Comp
+L power:+5V #PWR?
 U 1 1 5E900EF9
 P 6150 1200
@@
 $EndComp
 $Comp
-L Device:R_Network04 RN?
-U 1 1 5E8FF62E
+L power:+5V #PWR?
+U 1 1 5E9100BA
+P 6150 2500
+F 0 "#PWR?" H 6150 2350 50  0001 C CNN
+F 1 "+5V" H 6165 2673 50  0000 C CNN
+F 2 "" H 6150 2500 50  0001 C CNN
+F 3 "" H 6150 2500 50  0001 C CNN
+	1    6150 2500
+	1    0    0    -1
+$EndComp
+$Comp
+L power:GND #PWR?
+U 1 1 5E911FD4
+P 6450 2350
+F 0 "#PWR?" H 6450 2100 50  0001 C CNN
+F 1 "GND" H 6455 2177 50  0000 C CNN
+F 2 "" H 6450 2350 50  0001 C CNN
+F 3 "" H 6450 2350 50  0001 C CNN
+	1    6450 2350
+	1    0    0    -1
+$EndComp
+$Comp
+L Device:R_Pack04 RN?
+U 1 1 5E90F641
+P 6050 2750
+F 0 "RN?" H 6237 2795 50  0000 L CNN
+F 1 "R_Pack04" H 6237 2705 50  0000 L CNN
+F 2 "" V 6325 2750 50  0001 C CNN
+F 3 "~" H 6050 2750 50  0001 C CNN
+	1    6050 2750
+	1    0    0    -1
+$EndComp
+$Comp
+L Device:R_Pack04 RN?
+U 1 1 5E90CE51
 P 6350 1450
 F 0 "RN?" H 6537 1495 50  0000 L CNN
-F 1 "R_Network04" H 6537 1405 50  0000 L CNN
-F 2 "Resistor_THT:R_Array_SIP5" V 6625 1450 50  0001 C CNN
-F 3 "http://www.vishay.com/docs/31509/csc.pdf" H 6350 1450 50  0001 C CNN
+F 1 "R_Pack04" H 6537 1405 50  0000 L CNN
+F 2 "" V 6625 1450 50  0001 C CNN
+F 3 "~" H 6350 1450 50  0001 C CNN
 	1    6350 1450
 	1    0    0    -1
 $EndComp
 $Comp
+L CPU_RB0505:C_Pack04 CN?
+U 1 1 5E918C34
+P 6900 2750
+F 0 "CN?" H 7087 2795 50  0000 L CNN
+F 1 "C_Pack04" H 7087 2705 50  0000 L CNN
+F 2 "" V 7175 2750 50  0001 C CNN
+F 3 "" H 6900 2750 50  0001 C CNN
+	1    6900 2750
+	1    0    0    -1
+$EndComp
+$Comp
 L CPU_RB0505:ST10F276Z5 U?
 U 8 1 5E9C336E
-P 6750 3000
-F 0 "U?" H 6758 3664 50  0000 C CNN
-F 1 "ST10F276Z5" H 6758 3573 50  0000 C CNN
-F 2 "Package_QFP:LQFP-144_20x20mm_P0.5mm" H 6800 3350 50  0001 C CNN
-F 3 "https://www.st.com/content/ccc/resource/technical/document/datasheet/92/18/5e/9c/68/61/42/f6/CD00115722.pdf/files/CD00115722.pdf/jcr:content/translations/en.CD00115722.pdf" H 5250 3350 50  0001 C CNN
-	8    6750 3000
+P 8800 1700
+F 0 "U?" H 8808 2364 50  0000 C CNN
+F 1 "ST10F276Z5" H 8808 2273 50  0000 C CNN
+F 2 "Package_QFP:LQFP-144_20x20mm_P0.5mm" H 8850 2050 50  0001 C CNN
+F 3 "https://www.st.com/content/ccc/resource/technical/document/datasheet/92/18/5e/9c/68/61/42/f6/CD00115722.pdf/files/CD00115722.pdf/jcr:content/translations/en.CD00115722.pdf" H 7300 2050 50  0001 C CNN
+	8    8800 1700
 	1    0    0    -1
 $EndComp
@@
 L CPU_RB0505:ST10F276Z5 U?
 U 9 1 5E9C4E56
-P 6650 4500
-F 0 "U?" H 6550 3927 50  0000 C CNN
-F 1 "ST10F276Z5" H 6550 3836 50  0000 C CNN
-F 2 "Package_QFP:LQFP-144_20x20mm_P0.5mm" H 6700 4850 50  0001 C CNN
-F 3 "https://www.st.com/content/ccc/resource/technical/document/datasheet/92/18/5e/9c/68/61/42/f6/CD00115722.pdf/files/CD00115722.pdf/jcr:content/translations/en.CD00115722.pdf" H 5150 4850 50  0001 C CNN
-	9    6650 4500
+P 7500 5250
+F 0 "U?" H 7400 4677 50  0000 C CNN
+F 1 "ST10F276Z5" H 7400 4586 50  0000 C CNN
+F 2 "Package_QFP:LQFP-144_20x20mm_P0.5mm" H 7550 5600 50  0001 C CNN
+F 3 "https://www.st.com/content/ccc/resource/technical/document/datasheet/92/18/5e/9c/68/61/42/f6/CD00115722.pdf/files/CD00115722.pdf/jcr:content/translations/en.CD00115722.pdf" H 6000 5600 50  0001 C CNN
+	9    7500 5250
 	1    0    0    -1
 $EndComp
@@
 L CPU_RB0505:ST10F276Z5 U?
 U 4 1 5E9B3194
-P 5250 4000
-F 0 "U?" H 5333 5114 50  0000 C CNN
-F 1 "ST10F276Z5" H 5333 5023 50  0000 C CNN
-F 2 "Package_QFP:LQFP-144_20x20mm_P0.5mm" H 5300 4350 50  0001 C CNN
-F 3 "https://www.st.com/content/ccc/resource/technical/document/datasheet/92/18/5e/9c/68/61/42/f6/CD00115722.pdf/files/CD00115722.pdf/jcr:content/translations/en.CD00115722.pdf" H 3750 4350 50  0001 C CNN
-	4    5250 4000
+P 4400 3700
+F 0 "U?" H 4483 4814 50  0000 C CNN
+F 1 "ST10F276Z5" H 4483 4723 50  0000 C CNN
+F 2 "Package_QFP:LQFP-144_20x20mm_P0.5mm" H 4450 4050 50  0001 C CNN
+F 3 "https://www.st.com/content/ccc/resource/technical/document/datasheet/92/18/5e/9c/68/61/42/f6/CD00115722.pdf/files/CD00115722.pdf/jcr:content/translations/en.CD00115722.pdf" H 2900 4050 50  0001 C CNN
+	4    4400 3700
 	1    0    0    -1
 $EndComp
@@
 L CPU_RB0505:ST10F276Z5 U?
 U 6 1 5E9B9492
-P 4300 3750
-F 0 "U?" H 4358 4614 50  0000 C CNN
-F 1 "ST10F276Z5" H 4358 4523 50  0000 C CNN
-F 2 "Package_QFP:LQFP-144_20x20mm_P0.5mm" H 4350 4100 50  0001 C CNN
-F 3 "https://www.st.com/content/ccc/resource/technical/document/datasheet/92/18/5e/9c/68/61/42/f6/CD00115722.pdf/files/CD00115722.pdf/jcr:content/translations/en.CD00115722.pdf" H 2800 4100 50  0001 C CNN
-	6    4300 3750
-	1    0    0    -1
-$EndComp
+P 4250 5650
+F 0 "U?" H 4308 6514 50  0000 C CNN
+F 1 "ST10F276Z5" H 4308 6423 50  0000 C CNN
+F 2 "Package_QFP:LQFP-144_20x20mm_P0.5mm" H 4300 6000 50  0001 C CNN
+F 3 "https://www.st.com/content/ccc/resource/technical/document/datasheet/92/18/5e/9c/68/61/42/f6/CD00115722.pdf/files/CD00115722.pdf/jcr:content/translations/en.CD00115722.pdf" H 2750 6000 50  0001 C CNN
+	6    4250 5650
+	1    0    0    -1
+$EndComp

Commit message: Continuing CPU work
Parts:
- added R10: 1k5, symbol Device:R_Small
Connections:
- net labels added: ALARM-INHIB, BHE, CD-O2, CD-VALVE, CMD_ALE1, COM1, COM2, COM3, CONS-VIT, KEY-1, KEY-2, LED-AL-O, LED-AL-R, MRST-SPI-0_E, MTSR-SPI-0, PWM-BUZ, RESET_USB, RF, RX_UART_ST_E, SCLK-SPI-0, SEC-BUZ, TX_UART_ST_E
- wire segments 107 -> 132
- no-connect marks 1 -> 2
Other:
- note added: "To USB/UART\nPower Supply Board"
- note added: "}"
- moved on the sheet: U?F, U?H, U?I
Changed lines of the file:
@@
 Connection ~ 6050 3300
 Connection ~ 6150 3200
+Connection ~ 6700 3200
+Connection ~ 6800 3300
+Connection ~ 7000 3500
+Connection ~ 6450 2250
+Connection ~ 6700 2250
+Connection ~ 6800 2250
+Connection ~ 6900 2250
+Connection ~ 5750 6100
 NoConn ~ 6150 1650
+NoConn ~ 6900 2950
 Entry Wire Line
 	2400 1150 2500 1050
@@
 	5000 4400 5250 4400
 Wire Wire Line
+	5000 5800 5900 5800
+Wire Wire Line
+	5000 5900 5900 5900
+Wire Wire Line
+	5000 6000 5900 6000
+Wire Wire Line
+	5000 6100 5750 6100
+Wire Wire Line
+	5000 6200 5500 6200
+Wire Wire Line
+	5000 6300 5050 6300
+Wire Wire Line
+	5000 6400 5050 6400
+Wire Wire Line
+	5000 6500 5050 6500
+Wire Wire Line
+	5700 6200 5750 6200
+Wire Wire Line
+	5750 6100 5900 6100
+Wire Wire Line
+	5750 6200 5750 6100
+Wire Wire Line
 	5850 2500 5850 2550
 Wire Wire Line
 	5850 2950 5850 3500
 Wire Wire Line
-	5850 3500 6200 3500
+	5850 3500 7000 3500
 Wire Wire Line
 	5950 2250 5950 2550
@@
 	5950 2950 5950 3400
 Wire Wire Line
-	5950 3400 6200 3400
+	5950 3400 7150 3400
 Wire Wire Line
 	6050 2500 6150 2500
@@
 	6050 2950 6050 3300
 Wire Wire Line
-	6050 3300 6200 3300
+	6050 3300 6800 3300
 Wire Wire Line
 	6150 1200 6150 1250
@@
 	6150 2950 6150 3200
 Wire Wire Line
-	6150 3200 6200 3200
+	6150 3200 6700 3200
 Wire Wire Line
 	6250 1200 6250 1250
@@
 	6450 2250 5950 2250
 Wire Wire Line
+	6450 2250 6700 2250
+Wire Wire Line
 	6450 2350 6450 2250
+Wire Wire Line
+	6700 2250 6700 2550
+Wire Wire Line
+	6700 2250 6800 2250
+Wire Wire Line
+	6700 2950 6700 3200
+Wire Wire Line
+	6700 3200 7150 3200
+Wire Wire Line
+	6800 2250 6800 2550
+Wire Wire Line
+	6800 2250 6900 2250
+Wire Wire Line
+	6800 2950 6800 3300
+Wire Wire Line
+	6800 3300 7150 3300
+Wire Wire Line
+	6900 2250 6900 2550
+Wire Wire Line
+	6900 2250 7000 2250
+Wire Wire Line
+	7000 2250 7000 2550
+Wire Wire Line
+	7000 2950 7000 3500
+Wire Wire Line
+	7000 3500 7150 3500
 Wire Bus Line
 	2500 1050 2500 1250
 Wire Bus Line
-	2500 1250 2500 1450
-Wire Bus Line
-	2500 1450 2500 1650
-Wire Bus Line
-	2500 1650 2500 1750
+	2500 1250 2500 1350
+Wire Bus Line
+	2500 1350 2500 1550
+Wire Bus Line
+	2500 1550 2500 1750
 Wire Bus Line
 	2500 1750 2500 1950
@@
 	2500 3150 2500 3350
 Wire Bus Line
-	2500 3350 2500 3550
-Wire Bus Line
-	2500 3550 2500 3750
-Wire Bus Line
-	2500 3750 2500 3850
-Wire Bus Line
-	2500 3850 2500 4050
-Wire Bus Line
-	2500 4050 2500 4150
+	2500 3350 2500 3450
+Wire Bus Line
+	2500 3450 2500 3650
+Wire Bus Line
+	2500 3650 2500 3850
+Wire Bus Line
+	2500 3850 2500 3950
+Wire Bus Line
+	2500 3950 2500 4150
 Wire Bus Line
 	2500 4150 2500 4350
@@
 	2500 4350 2500 4550
 Wire Bus Line
-	2500 4550 2500 5250
-Wire Bus Line
-	2500 5250 2500 5450
+	2500 4550 2500 5150
+Wire Bus Line
+	2500 5150 2500 5350
+Wire Bus Line
+	2500 5350 2500 5450
 Wire Bus Line
 	2600 1050 2500 1050
+Text Notes 5950 4000 0    50   ~ 0
+To USB/UART\nPower Supply Board
+Text Notes 5950 4000 2    118  ~ 0
+}
 Text Label 2250 1150 0    50   ~ 0
 D0
@@
 Text HLabel 2600 3050 2    50   Output ~ 0
 A[0..19]
+Text HLabel 5050 6300 2    50   Output ~ 0
+SEC-BUZ
+Text HLabel 5050 6400 2    50   Output ~ 0
+LED-AL-O
+Text HLabel 5050 6500 2    50   Output ~ 0
+LED-AL-R
 Text HLabel 5250 950  2    50   Input ~ 0
 SPEED_MEASURE
@@
 Text HLabel 5250 2450 2    50   Output ~ 0
 CMD_ME1
+Text HLabel 5250 2900 2    50   Output ~ 0
+COM1
+Text HLabel 5250 3000 2    50   Output ~ 0
+COM2
+Text HLabel 5250 3100 2    50   Output ~ 0
+COM3
+Text HLabel 5250 3600 2    50   Output ~ 0
+RF
+Text HLabel 5250 3700 2    50   Input ~ 0
+MRST-SPI-0_E
+Text HLabel 5250 3800 2    50   Output ~ 0
+MTSR-SPI-0
+Text HLabel 5250 3900 2    50   Output ~ 0
+TX_UART_ST_E
+Text HLabel 5250 4000 2    50   Input ~ 0
+RX_UART_ST_E
+Text HLabel 5250 4100 2    50   Output ~ 0
+BHE
+Text HLabel 5250 4200 2    50   Output ~ 0
+SCLK-SPI-0
+Text HLabel 5250 4400 2    50   Output ~ 0
+CMD_ALE1
+Text HLabel 5900 5800 2    50   Output ~ 0
+CONS-VIT
+Text HLabel 5900 5900 2    50   Output ~ 0
+CD-VALVE
+Text HLabel 5900 6000 2    50   Output ~ 0
+CD-O2
+Text HLabel 5900 6100 2    50   Output ~ 0
+PWM-BUZ
 Text HLabel 6750 1750 2    50   Input ~ 0
 BUSY-ME1
@@
 Text HLabel 6750 2150 2    50   Input ~ 0
 TEST-RAP-ALARM
+Text HLabel 7150 3200 2    50   Input ~ 0
+KEY-1
+Text HLabel 7150 3300 2    50   Input ~ 0
+KEY-2
+Text HLabel 7150 3400 2    50   Output ~ 0
+RESET_USB
+Text HLabel 7150 3500 2    50   Input ~ 0
+ALARM-INHIB
 $Comp
 L power:+5V #PWR?
@@
 $EndComp
 $Comp
+L Device:R_Small R10
+U 1 1 5E9342A9
+P 5600 6200
+F 0 "R10" V 5795 6200 50  0000 C CNN
+F 1 "1k5" V 5704 6200 50  0000 C CNN
+F 2 "" H 5600 6200 50  0001 C CNN
+F 3 "~" H 5600 6200 50  0001 C CNN
+	1    5600 6200
+	0    -1   1    0
+$EndComp
+$Comp
 L Device:R_Pack04 RN?
 U 1 1 5E90F641
@@
 L CPU_RB0505:ST10F276Z5 U?
 U 8 1 5E9C336E
-P 8800 1700
-F 0 "U?" H 8808 2364 50  0000 C CNN
-F 1 "ST10F276Z5" H 8808 2273 50  0000 C CNN
-F 2 "Package_QFP:LQFP-144_20x20mm_P0.5mm" H 8850 2050 50  0001 C CNN
-F 3 "https://www.st.com/content/ccc/resource/technical/document/datasheet/92/18/5e/9c/68/61/42/f6/CD00115722.pdf/files/CD00115722.pdf/jcr:content/translations/en.CD00115722.pdf" H 7300 2050 50  0001 C CNN
-	8    8800 1700
+P 4350 6150
+F 0 "U?" H 4358 5564 50  0000 C CNN
+F 1 "ST10F276Z5" H 4358 5473 50  0000 C CNN
+F 2 "Package_QFP:LQFP-144_20x20mm_P0.5mm" H 4400 6500 50  0001 C CNN
+F 3 "https://www.st.com/content/ccc/resource/technical/document/datasheet/92/18/5e/9c/68/61/42/f6/CD00115722.pdf/files/CD00115722.pdf/jcr:content/translations/en.CD00115722.pdf" H 2850 6500 50  0001 C CNN
+	8    4350 6150
 	1    0    0    -1
 $EndComp
@@
 L CPU_RB0505:ST10F276Z5 U?
 U 9 1 5E9C4E56
-P 7500 5250
-F 0 "U?" H 7400 4677 50  0000 C CNN
-F 1 "ST10F276Z5" H 7400 4586 50  0000 C CNN
-F 2 "Package_QFP:LQFP-144_20x20mm_P0.5mm" H 7550 5600 50  0001 C CNN
-F 3 "https://www.st.com/content/ccc/resource/technical/document/datasheet/92/18/5e/9c/68/61/42/f6/CD00115722.pdf/files/CD00115722.pdf/jcr:content/translations/en.CD00115722.pdf" H 6000 5600 50  0001 C CNN
-	9    7500 5250
+P 4250 5100
+F 0 "U?" H 4150 4527 50  0000 C CNN
+F 1 "ST10F276Z5" H 4150 4436 50  0000 C CNN
+F 2 "Package_QFP:LQFP-144_20x20mm_P0.5mm" H 4300 5450 50  0001 C CNN
+F 3 "https://www.st.com/content/ccc/resource/technical/document/datasheet/92/18/5e/9c/68/61/42/f6/CD00115722.pdf/files/CD00115722.pdf/jcr:content/translations/en.CD00115722.pdf" H 2750 5450 50  0001 C CNN
+	9    4250 5100
 	1    0    0    -1
 $EndComp
@@
 L CPU_RB0505:ST10F276Z5 U?
 U 6 1 5E9B9492
-P 4250 5650
-F 0 "U?" H 4308 6514 50  0000 C CNN
-F 1 "ST10F276Z5" H 4308 6423 50  0000 C CNN
-F 2 "Package_QFP:LQFP-144_20x20mm_P0.5mm" H 4300 6000 50  0001 C CNN
-F 3 "https://www.st.com/content/ccc/resource/technical/document/datasheet/92/18/5e/9c/68/61/42/f6/CD00115722.pdf/files/CD00115722.pdf/jcr:content/translations/en.CD00115722.pdf" H 2750 6000 50  0001 C CNN
-	6    4250 5650
-	1    0    0    -1
-$EndComp
+P 10900 2300
+F 0 "U?" H 10958 3164 50  0000 C CNN
+F 1 "ST10F276Z5" H 10958 3073 50  0000 C CNN
+F 2 "Package_QFP:LQFP-144_20x20mm_P0.5mm" H 10950 2650 50  0001 C CNN
+F 3 "https://www.st.com/content/ccc/resource/technical/document/datasheet/92/18/5e/9c/68/61/42/f6/CD00115722.pdf/files/CD00115722.pdf/jcr:content/translations/en.CD00115722.pdf" H 9400 2650 50  0001 C CNN
+	6    10900 2300
+	1    0    0    -1
+$EndComp
