File: CPU_RB0505/10125623A00_5.sch (KiCad schematic (older format))
At the start: 46 parts, among them IC21 LT1236ACS8-5, IC23 LT1236ACS8-10, IC24 STM809LWX, IC25 STM809LWX, IC26 LF33CDT, IC29 TPS5430, IC36 STM809TWX, T10 FZT953, T11 FZT953, T12 FZT953

Commit message: Schematics updated from symbols
Parts:
- C105, C107, C46, C47, C74, C79, C80, C82, C83, C90, C91, C97: Description (none) -> CAPACITOR CERAMIC, 100NF, +/-10%, 50V, X7R,0805; Item Number (none) -> 10022135; Manufacturer (none) -> YAGEO_RMS1; Manufacturer2 (none) -> MURATA MANUFACTURING CO., LTD.; Manufacturer3 (none) -> YAGEO_RMS1; Manufacturer4 (none) -> SAMSUNG_RMS1; Manufacturer5 (none) -> YAGEO_RMS1; Manufacturer6 (none) -> AVX_RMS1; Manufacturer_Desc (none) -> CAPACITOR, CERAMIC, MULTILAYER, 50 V, X7R, 0.1 UF, SURFACE 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; Manufacturer_Desc2 (none) -> MONOLITHIC CERAMIC CAPACITOR; Manufacturer_Desc3 (none) -> CAPACITOR, CERAMIC, MULTILAYER, 50 V, X7R, 0.1 UF, SURFACE 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; Manufacturer_Desc4 (none) -> MULTILAYER CERAMIC CAPACITOR; Manufacturer_Desc5 (none) -> CAP CER .1UF 50V 10% X7R 0805; Manufacturer_Desc6 (none) -> CAPACITOR CERAMIC, 100NF, +/-10%, 50V, X7R,0805, X7R DIELEC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; Manufacturer_No (none) -> 223858055649; Manufacturer_No2 (none) -> GRM21BR71H104KA01L; Manufacturer_No3 (none) -> 223858015649; Manufacturer_No4 (none) -> CL21B104KBCNNNC; Manufacturer_No5 (none) -> CC0805KRX7R9BB104; Manufacturer_No6 (none) -> 08055C104KAT2A
- C106: Description (none) -> CAPACITOR ELECTROLYTIC, 220UF,16V+/-20%; Item Number (none) -> 10022622; Manufacturer (none) -> PANASONIC_RMS1; Manufacturer2 (none) -> ELNA AMERICA, INC.; Manufacturer3 (none) -> ELNA AMERICA, INC.; Manufacturer_Desc (none) -> ALUMINUM ELETROLYTIC CAPACITORS/FK; Manufacturer_Desc3 (none) -> CHIP TYPE, LOW IMPEDANCE CAP.; Manufacturer_No (none) -> EEEFK1C221P; Manufacturer_No2 (none) -> RVD-16V221MG68U-R; Manufacturer_No3 (none) -> RVZ-16V221MG68U
- C108, C117, C92: Description (none) -> CAPACITOR TANTALUM, 1UF,35V, +/-10%; Item Number (none) -> 10022959; Manufacturer (none) -> KEMET; Manufacturer2 (none) -> KEMET; Manufacturer_Desc (none) -> Cap, Tantalum, Polarized, 35V, 20% +/-Tol, 1uF, Surface Mou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; Manufacturer_Desc2 (none) -> Cap, Tantalum, Polarized, 35V, 10% +/-Tol, 1uF, Surface Mou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; Manufacturer_No (none) -> T491A105M035AT; Manufacturer_No2 (none) -> T495A105K035ATE3K0
- C21, C88: Description (none) -> CAPACITOR ELECTROLYTIC, 100UF, 35V +/-20%; Item Number (none) -> 10022963; Manufacturer (none) -> MULTICOMP (920630); Manufacturer2 (none) -> LELON; Manufacturer_Desc (none) -> ELECTROLYTIC CAPACITOR; Manufacturer_Desc2 (none) -> ALUMINIUM ELECTROLYTIC CAPACITOR; Manufacturer_No (none) -> MCRH35V107M8X11; Manufacturer_No2 (none) -> RXW101M1V-SA-0811
- C81, C85: Description (none) -> CAPACITOR TANTALUM, 10UF, 25V, +/-10%; Item Number (none) -> 10022608; Manufacturer (none) -> KEMET; Manufacturer2 (none) -> KEMET; Manufacturer_Desc (none) -> Cap, Tantalum, Polarized, 25V, 10% +/-Tol, 10uF, Surface Mo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; Manufacturer_Desc2 (none) -> Cap, Tantalum, Polarized, 25V, 10% +/-Tol, 10uF, Surface Mo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; Manufacturer_No (none) -> T491C106K025AT; Manufacturer_No2 (none) -> T495C106K025ATE275
- D11: Description (none) -> DIODE SCHOTTKY, 30V, 200MA; Item Number (none) -> 10022652; Manufacturer (none) -> NXP SEMICONDUCTORS_RMS1; Manufacturer2 (none) -> NXP SEMICONDUCTORS_RMS1; Manufacturer_Desc2 (none) -> SCHOTTKY BARRIER DOUBLE DIODE; Manufacturer_No (none) -> BAT54,215; Manufacturer_No2 (none) -> BAT54
- D4: Description (none) -> DIODE TRANSIENT 600W,36V; Item Number (none) -> 10022654; Manufacturer (none) -> LITTLEFUSE; Manufacturer2 (none) -> ON SEMICONDUCTOR_RMS1; Manufacturer3 (none) -> LITTLEFUSE; Manufacturer_Desc (none) -> ZENER TRANSIENT VOLTAGE SUPPRESSORS; Manufacturer_Desc2 (none) -> ZENER TRANSIENT VOLTAGE SUPPRESSORS; Manufacturer_Desc3 (none) -> ZENER TRANSIENT VOLTAGE SUPPRESSORS; Manufacturer_No (none) -> 1SMB36AT3G; Manufacturer_No2 (none) -> 1SMB36AT3G; Manufacturer_No3 (none) -> SZ1SMB36AT3G
- D7: Description (none) -> DIODE SCHOTTKY, 40V, 1A; Item Number (none) -> 10097253; Manufacturer (none) -> DIODES INC_RMS1; Manufacturer_Desc (none) -> SURFACE MOUNT SCHOTTKY BARRIER RECTIFIER; Manufacturer_No (none) -> 1N5819HW-7-F
- FU2: Description (none) -> FUSE, 500MA; Item Number (none) -> 10022703; Manufacturer (none) -> LITTELFUSE_RMS1; Manufacturer_Desc (none) -> VERY FAST ACTING FUSE; Manufacturer_No (none) -> 0154.500DRT
- IC21, IC23: Description (none) -> IC,REFERENCE VOLTAGE 5V FIXED - 10 MA,SO8; Item Number (none) -> 10023039; Manufacturer (none) -> LINEAR TECHNOLOGY_RMS1; Manufacturer_Desc (none) -> PRECISION REFERENCE; Manufacturer_No (none) -> LT1236CCS8-5#TRPBF
- IC24, IC25, IC36: Description (none) -> RESET CIRCUIT, SUPERVISOR VOLTAGE 5V,SOT23; Item Number (none) -> 10022974; Manufacturer (none) -> STMICROELECTRONICS; Manufacturer_Desc (none) -> RESET CIRCUIT; Manufacturer_No (none) -> STM809LWX6F
- IC26: Description (none) -> REGULATOR 3.3 V 2% 500MA LOW DROPOUT,DPACK; Item Number (none) -> 10022892; Manufacturer (none) -> ST MICROELECTRONIC; Manufacturer2 (none) -> STMICROELECTRONICS; Manufacturer_Desc (none) -> VERY LOW DROP VOLTAGE REGULATOR; Manufacturer_Desc2 (none) -> VERY LOW DROP VOLTAGE REGULATOR; Manufacturer_No (none) -> LF33CDT; Manufacturer_No2 (none) -> LF33CDT-TR
- IC29: Description (none) -> REGULATOR, 5.5V TO 36V,3A; Item Number (none) -> 10022895; Manufacturer (none) -> TEXAS INSTRUMENTS_RMS1; Manufacturer2 (none) -> TEXAS INSTRUMENTS_RMS1; Manufacturer_Desc (none) -> 3A, WIDE INPUT RANGE, CONVERTER; Manufacturer_No (none) -> TPS 5430 DDA; Manufacturer_No2 (none) -> TPS5430DDAR
- JP9: Description (none) -> RESISTANCE, 0 OHM,0603; Item Number (none) -> 10023185; Manufacturer (none) -> YAGEO_RMS1; Manufacturer2 (none) -> YAGEO_RMS1; Manufacturer3 (none) -> YAGEO_RMS1; Manufacturer4 (none) -> ASJ; Manufacturer5 (none) -> KAMAYA (049580); Manufacturer_Desc (none) -> RES 0.0 OHM 1/10W 0603 SMD; Manufacturer_Desc2 (none) -> JUMPER, METAL GLAZE/THICK FILM, 0.1 W, 0 OHM, SURFACE MOUNT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; Manufacturer_Desc3 (none) -> JUMPER, METAL GLAZE/THICK FILM, 0.1 W, 0 OHM, SURFACE MOUNT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; Manufacturer_Desc4 (none) -> THICK FILM CHIP RESISTOR; Manufacturer_Desc5 (none) -> JUMPER; Manufacturer_No (none) -> RC0603JR-070RL; Manufacturer_No2 (none) -> 232270296001; Manufacturer_No3 (none) -> 232270296001L; Manufacturer_No4 (none) -> CR16000ZL; Manufacturer_No5 (none) -> RMC1/16JPTP
- L30: Description (none) -> FERRITE, 2.5, 3A; Item Number (none) -> 10023186; Manufacturer (none) -> WURTH ELEKTRONIK GMBH; Manufacturer2 (none) -> WURTH ELEKTRONIK GMBH; Manufacturer_Desc (none) -> 5 HOLE SMD FERRITE BEAD; Manufacturer_Desc2 (none) -> 6 HOLE FERRITE BEAD; Manufacturer_No (none) -> 7427512; Manufacturer_No2 (none) -> 7427504
- R35, R36, R40, R44, R66, R67, R71, R73: Description (none) -> RESISTOR, 4.7 K OHM, 0.063W +/-5%; Item Number (none) -> 10022617; Manufacturer (none) -> ASJ; Manufacturer2 (none) -> YAGEO_RMS1; Manufacturer3 (none) -> YAGEO_RMS1; Manufacturer4 (none) -> YAGEO_RMS1; Manufacturer_Desc (none) -> THICK FILM CHIP RESISTOR; Manufacturer_Desc2 (none) -> RESISTOR, METAL GLAZE/THICK FILM, 0.1 W, 5 %, 100 PPM, 4700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; Manufacturer_Desc3 (none) -> RESISTOR, METAL GLAZE/THICK FILM, 0.1 W, 5 %, 100 PPM, 4700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; Manufacturer_Desc4 (none) -> RESISTOR, METAL GLAZE/THICK FILM, 0.1 W, 5 %, 100 PPM, 4700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; Manufacturer_No (none) -> CR16-472JL; Manufacturer_No2 (none) -> 232270260472L; Manufacturer_No3 (none) -> RC0603JR-074K7L; Manufacturer_No4 (none) -> 232270260472
- R41: Description (none) -> RESISTOR, 150 OHM, 0805, +/-5%; Item Number (none) -> 10023237; Manufacturer (none) -> YAGEO_RMS1; Manufacturer2 (none) -> YAGEO_RMS1; Manufacturer3 (none) -> ASJ; Manufacturer4 (none) -> YAGEO_RMS1; Manufacturer_Desc (none) -> RESISTOR, METAL GLAZE/THICK FILM, 0.125 W, 5 %, 100 PPM, 15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; Manufacturer_Desc2 (none) -> RESISTOR, METAL GLAZE/THICK FILM, 0.125 W, 5 %, 100 PPM, 15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; Manufacturer_Desc3 (none) -> THICK FILM CHIP RESISTOR; Manufacturer_Desc4 (none) -> RESISTOR, METAL GLAZE/THICK FILM, 0.125 W, 5 %, 100 PPM, 15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; Manufacturer_No (none) -> 232273061151; Manufacturer_No2 (none) -> 232273061151L; Manufacturer_No3 (none) -> CR21-151JL; Manufacturer_No4 (none) -> RC0805JR-07150RL
- T10, T11, T12: Description (none) -> RSP TRANSISTOR, BIPOLAR, PNP, 100V, 5A, SOT223; Item Number (none) -> 10023243; Manufacturer (none) -> ZETEX; Manufacturer2 (none) -> ZETEX; Manufacturer_Desc (none) -> 60 TO 100V PNP TRANSISTOR; Manufacturer_Desc2 (none) -> TRANSISTOR; Manufacturer_No (none) -> FZT953; Manufacturer_No2 (none) -> FZT953TA
