File: CPU_RB0505/10125623A00_6.sch (KiCad schematic (older format))
At the start: 69 parts, among them IC37 ARF34, J11 B3B_ZR, J18 B7B_ZR_SM3_TF, J19 B2B_ZR, J2 B8B_ZR, J20 B4B_ZR, J21 2BR254C, J4 10BRMF, J5 B2B_ZR, T17 IRLML5103, T19 BSS84

Commit message: Schematic symbols updated with BOM fields
Parts:
- C100, C38, C56: Description (none) -> CAPACITOR ARRAY, 47PF, 50V, +/-10%,NPO,0612; Item Number (none) -> 10095973; Manufacturer (none) -> YAGEO_RMS1; Manufacturer_Desc (none) -> ISOLATED C NETWORK, 50V, C0G, 0.000047UF, SURFACE MOUNT, CH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; Manufacturer_No (none) -> 225514611532
- C101: Description (none) -> CAPACITOR CERAMIC,4.7NF,25V,+/-10%,0402; Item Number (none) -> 10022976; Manufacturer (none) -> KYOCERA_RMS1; Manufacturer2 (none) -> KEMET_RMS1; Manufacturer3 (none) -> AVX_RMS1; Manufacturer_Desc (none) -> MULTILAYER CERAMIC CAPACITOR; Manufacturer_Desc2 (none) -> CERAMIC CHIP CAPACITOR; Manufacturer_Desc3 (none) -> CERAMIC CAPACITOR X7R; Manufacturer_No (none) -> CM05X7R472K25AT; Manufacturer_No2 (none) -> C0402C472K3RACTU; Manufacturer_No3 (none) -> 04023C472KAT2A
- C11, C76: Description (none) -> CAPACITOR,100NF,16V,+/-10%,X7R,0402; Item Number (none) -> 10022607; Manufacturer (none) -> MURATA; Manufacturer2 (none) -> YAGEO_RMS1; Manufacturer3 (none) -> YAGEO_RMS1; Manufacturer4 (none) -> MURATA MANUFACTURING CO., LTD.; Manufacturer_Desc (none) -> CAPACITOR, CERAMIC, MULTILAYER, 16V, X7R, 0.1UF, 0402; Manufacturer_Desc2 (none) -> CAP CER 0.1uF 16V X7R 10% 0402; Manufacturer_Desc3 (none) -> CAPACITOR, CERAMIC, MULTILAYER, 16 V, X7R, 0.1 UF, SURFACE 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; Manufacturer_Desc4 (none) -> MONOLITHIC CERAMIC CAPACITOR; Manufacturer_No (none) -> GRM155R71C104JA88J; Manufacturer_No2 (none) -> CC0402KRX7R7BB104; Manufacturer_No3 (none) -> 223878715649; Manufacturer_No4 (none) -> GRM155R71C104KA88D
- C115, C121, C122, C123, C124, C99: Description (none) -> CAPACITOR CERAMIC, 150PF,50V,+/-5,NPO, 0402; Item Number (none) -> 10022975; Manufacturer (none) -> YAGEO_RMS1; Manufacturer2 (none) -> KEMET_RMS1; Manufacturer3 (none) -> YAGEO_RMS1; Manufacturer_Desc (none) -> CAP CER 150PF 50V C0G/NPO 0402; Manufacturer_Desc2 (none) -> CERAMIC CHIP CAPACITOR; Manufacturer_Desc3 (none) -> CAPACITOR, CERAMIC, MULTILAYER, 50 V, C0G, 0.00015 UF, SURF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; Manufacturer_No (none) -> CC0402JRNPO9BN151; Manufacturer_No2 (none) -> C0402C151J5GACTU; Manufacturer_No3 (none) -> 223886915151
- C12, C13, C86: Description (none) -> CAPACITOR,47 PF,+/-5%,50V,0402; Item Number (none) -> 10022623; Manufacturer (none) -> SAMSUNG_RMS1; Manufacturer2 (none) -> KEMET_RMS1; Manufacturer3 (none) -> MURATA MANUFACTURING CO., LTD.; Manufacturer4 (none) -> KEMET_RMS1; Manufacturer5 (none) -> MURATA MANUFACTURING CO., LTD.; Manufacturer_Desc (none) -> CAP CER 47PF 50V 5% NP0 0402; Manufacturer_Desc2 (none) -> CAP,CER,SMT,0402,5%,50V,47PF; Manufacturer_Desc3 (none) -> MONOLITHIC CERAMIC CAPACITOR; Manufacturer_Desc4 (none) -> CAP,CER,SMT,0402,5%,50V,47PF; Manufacturer_Desc5 (none) -> CAP CER 47PF 50V 5% NP0 0402; Manufacturer_No (none) -> CL05C470JB5NNNC; Manufacturer_No2 (none) -> C0402C470J5GACTU; Manufacturer_No3 (none) -> GRM1555C1H470JZ01D; Manufacturer_No4 (none) -> C0402C470J5GAC; Manufacturer_No5 (none) -> GRM1555C1H470JA01D
- C75: Description (none) -> CAPACITOR TANALUM, 47UF, 10V +/-10%; Item Number (none) -> 10022962; Manufacturer (none) -> KEMET; Manufacturer_Desc (none) -> Cap, Tantalum, Polarized, 10V, 10% +/-Tol, 47uF, Surface Mo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; Manufacturer_No (none) -> T495B476K010ATE500
- C89: Description (none) -> CAPACITOR TANTALUM, 22UF, 10V,+/-10%; Item Number (none) -> 10022973; Manufacturer (none) -> KEMET; Manufacturer_Desc (none) -> Cap, Tantalum, Polarized, 10V, 10% +/-Tol, 22uF, Surface Mo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; Manufacturer_No (none) -> T495A226K010ATE1K2
- D13: Description (none) -> DIODE SCHOTTKY, 30V, 200MA; Item Number (none) -> 10022652; Manufacturer (none) -> NXP SEMICONDUCTORS_RMS1; Manufacturer2 (none) -> NXP SEMICONDUCTORS_RMS1; Manufacturer_Desc2 (none) -> SCHOTTKY BARRIER DOUBLE DIODE; Manufacturer_No (none) -> BAT54,215; Manufacturer_No2 (none) -> BAT54
- D6: Description (none) -> DIODE SCHOTTKY, 40V, 1A; Item Number (none) -> 10097253; Manufacturer (none) -> DIODES INC_RMS1; Manufacturer_Desc (none) -> SURFACE MOUNT SCHOTTKY BARRIER RECTIFIER; Manufacturer_No (none) -> 1N5819HW-7-F
- J11: Description (none) -> CONNECTOR,FIO2, 3 CONTACTS; Item Number (none) -> 10097262; Manufacturer (none) -> J.S.T. CORPORATION; Manufacturer_Desc (none) -> ZH CONNECTOR; Manufacturer_No (none) -> B3B-ZR-SM4-TF (LF)(SN)
- J18: Description (none) -> CONNECTOR, BUZZER CARD, 7 CONTACTS; Item Number (none) -> 10097265; Manufacturer (none) -> J.S.T. CORPORATION; Manufacturer_Desc (none) -> ZH CONNECTOR; Manufacturer_No (none) -> B7B-ZR-SM4-TF (LF)(SN)
- J19, J5: Description (none) -> CONNECTOR, TEMPERATURE MEASURE, 2 CONTACTS; Item Number (none) -> 10097260; Manufacturer (none) -> J.S.T. CORPORATION; Manufacturer_Desc (none) -> CONNECTOR; Manufacturer_No (none) -> B2B-ZR-SM4-TF (LF)(SN)
- J2: Description (none) -> CONNECTOR, 8 CONTACTS; Item Number (none) -> 10097257; Manufacturer (none) -> J.S.T. CORPORATION; Manufacturer_Desc (none) -> CONNECTOR; Manufacturer_No (none) -> B8B-ZR-SM4-TF (LF)(SN)
- J21: Description (none) -> CONNECTOR, O2 VALVE, 2 CONTACTS; Item Number (none) -> 10022542; Manufacturer (none) -> MOLEX_RMS1; Manufacturer_No (none) -> 22057028
- J4: Description (none) -> HEADER CONNECTOR, RIGHT ANGLE, 10 PINS; Item Number (none) -> 10052329; Manufacturer (none) -> FCI/BERG; Manufacturer2 (none) -> FCI/BERG; Manufacturer_No (none) -> 75867-101LF; Manufacturer_No2 (none) -> 88874-010LF
- L10, L12, L14, L15, L17, L21, L23, L24, L25, L26, L29, L31, L32, L33, L34, L37, L9: Description (none) -> SMD FERRITE 200MA; Item Number (none) -> 10022907; Manufacturer (none) -> WURTH ELEKTRONIK GMBH; Manufacturer_Desc (none) -> MULTILAYER-SMD-FERRITE; Manufacturer_No (none) -> 74279266
- L11, L19, L20, L22, L7: Description (none) -> SMD FERRITE, 1A,1206; Item Number (none) -> 10022911; Manufacturer (none) -> WURTH ELEKTRONIK GMBH; Manufacturer_Desc (none) -> MULTILAYER-SMD-FERRITE; Manufacturer_No (none) -> 74279218
- R11: Description (none) -> RESISTOR,3.3K OHM,0.063W,+/-1%,0603; Item Number (none) -> 10022731; Manufacturer (none) -> YAGEO_RMS1; Manufacturer2 (none) -> YAGEO_RMS1; Manufacturer3 (none) -> BOURNS_RMS1; Manufacturer4 (none) -> YAGEO_RMS1; Manufacturer_Desc (none) -> RESISTOR, METAL GLAZE/THICK FILM, 0.1 W, 1 %, 100 PPM, 3300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; Manufacturer_Desc2 (none) -> RESISTOR, METAL GLAZE/THICK FILM, 0.1 W, 1 %, 100 PPM, 3300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; Manufacturer_Desc3 (none) -> CHIP RESISTOR; Manufacturer_Desc4 (none) -> RESISTOR, METAL GLAZE/THICK FILM, 0.1 W, 1 %, 100 PPM, 3300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; Manufacturer_No (none) -> RC0603FR-073K3L; Manufacturer_No2 (none) -> 232270463302; Manufacturer_No3 (none) -> CR0603-FX-3301ELF; Manufacturer_No4 (none) -> 232270463302L
- R43, R70: Description (none) -> RESISTOR,10K OHM, 0.063W,+/-5%,0603; Item Number (none) -> 10097266; Manufacturer (none) -> YAGEO_RMS1; Manufacturer2 (none) -> YAGEO_RMS1; Manufacturer3 (none) -> VISHAY_RMS1; Manufacturer4 (none) -> ASJ; Manufacturer5 (none) -> YAGEO_RMS1; Manufacturer_Desc (none) -> RESISTOR, METAL GLAZE/THICK FILM, 0.1 W, 5 %, 100 PPM, 1000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; Manufacturer_Desc2 (none) -> RESISTOR, METAL GLAZE/THICK FILM, 0.1 W, 5 %, 100 PPM, 1000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; Manufacturer_Desc3 (none) -> THICK FILM RECTANGULAR CHIP RESISTOR; Manufacturer_Desc4 (none) -> THICK FILM CHIP RESISTOR; Manufacturer_Desc5 (none) -> RESISTOR, METAL GLAZE/THICK FILM, 0.1 W, 5 %, 100 PPM, 1000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; Manufacturer_No (none) -> 232270260103L; Manufacturer_No2 (none) -> 232270260103; Manufacturer_No3 (none) -> CRCW060310K0JNEA; Manufacturer_No4 (none) -> CR16-103JL; Manufacturer_No5 (none) -> RC0603JR-0710KL
- R48, R68: Description (none) -> RESISTOR,100 K OHM, 0.063W +/-5%; Item Number (none) -> 10022732; Manufacturer (none) -> YAGEO_RMS1; Manufacturer2 (none) -> YAGEO_RMS1; Manufacturer3 (none) -> YAGEO_RMS1; Manufacturer4 (none) -> PANASONIC_RMS1; Manufacturer_Desc (none) -> RESISTOR, METAL GLAZE/THICK FILM, 0.1 W, 5 %, 100 PPM, 1000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; Manufacturer_Desc2 (none) -> RESISTOR, METAL GLAZE/THICK FILM, 0.1 W, 5 %, 100 PPM, 1000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; Manufacturer_Desc3 (none) -> RESISTOR, METAL GLAZE/THICK FILM, 0.1 W, 5 %, 100 PPM, 1000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; Manufacturer_Desc4 (none) -> THICK FILM CHIP RESISTOR; Manufacturer_No (none) -> 232270260104L; Manufacturer_No2 (none) -> 232270260104; Manufacturer_No3 (none) -> RC0603JR-07100KL; Manufacturer_No4 (none) -> ERJ3GEYJ104V
- R69: Description (none) -> RESISTANCE, 0 OHM,0603; Item Number (none) -> 10023185; Manufacturer (none) -> YAGEO_RMS1; Manufacturer2 (none) -> YAGEO_RMS1; Manufacturer3 (none) -> YAGEO_RMS1; Manufacturer4 (none) -> ASJ; Manufacturer5 (none) -> KAMAYA (049580); Manufacturer_Desc (none) -> RES 0.0 OHM 1/10W 0603 SMD; Manufacturer_Desc2 (none) -> JUMPER, METAL GLAZE/THICK FILM, 0.1 W, 0 OHM, SURFACE MOUNT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; Manufacturer_Desc3 (none) -> JUMPER, METAL GLAZE/THICK FILM, 0.1 W, 0 OHM, SURFACE MOUNT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; Manufacturer_Desc4 (none) -> THICK FILM CHIP RESISTOR; Manufacturer_Desc5 (none) -> JUMPER; Manufacturer_No (none) -> RC0603JR-070RL; Manufacturer_No2 (none) -> 232270296001; Manufacturer_No3 (none) -> 232270296001L; Manufacturer_No4 (none) -> CR16000ZL; Manufacturer_No5 (none) -> RMC1/16JPTP
- RL1: Description (none) -> RELAY,LOW VOLTAGE 1A COIL 5VDC; Item Number (none) -> 10023252; Manufacturer (none) -> OMRON ELECTRONICS INC; Manufacturer2 (none) -> OMRON ELECTRONICS INC; Manufacturer_No (none) -> G6K-2G-TR 5 VDC; Manufacturer_No2 (none) -> G6K-2G 5 VDC
- T17: Description (none) -> RSPTRANSISTOR MOSFET, P CHANNEL, 30V,0.6A; Item Number (none) -> 10022933; Manufacturer (none) -> INTERNATIONAL RECTIFIER_RMS1; Manufacturer_Desc (none) -> POWER MOSFET; Manufacturer_No (none) -> IRLML5103TRPBF
- T19: Description (none) -> TRANSISTOR, P CHANNEL, 50V, 0.13A, 5 OHM, SOT23; Item Number (none) -> 10022157; Manufacturer (none) -> NXP SEMICONDUCTORS_RMS1; Manufacturer2 (none) -> ON SEMICONDUCTOR_RMS1; Manufacturer3 (none) -> NXP SEMICONDUCTORS_RMS1; Manufacturer_Desc (none) -> MOSFET P CHANNEL; Manufacturer_Desc2 (none) -> POWER MOSFET; Manufacturer_No (none) -> BSS84; Manufacturer_No2 (none) -> BSS84LT1G; Manufacturer_No3 (none) -> BSS84,215

Commit message: Updated J18.2 and corrected sheet numbers.
Connections:
- net labels removed: +5VSUPPLY-BOARD
Changed lines of the file:
@@
 $Descr User 17335 11946
 encoding utf-8
-Sheet 5 8
+Sheet 7 8
 Title "RB0505 CPU Board"
-Date ""
+Date "2020-04-15"
 Rev ""
 Comp ""
@@
 SUPPLY-AL-RP
 Text HLabel 3075 6650 2    70   BiDi ~ 0
-+5VSUPPLY-BOARD
++5V
 $Comp
 L cpu-board:GND #U$43
@@
 L cpu-board:C0805 C101
 U 1 1 D5229C91
-P 10275 7763
-F 0 "C101" H 10400 7826 64  0000 L CNN
-F 1 "4.7nF" H 10400 7726 42  0000 L CNN
-F 2 "10125623A00:C0805" H 10275 7763 50  0001 C CNN
-F 3 "" H 10275 7763 50  0001 C CNN
-F 4 "CAPACITOR CERAMIC,4.7NF,25V,+/-10%,0402" H 10275 7763 50  0001 C CNN "Description"
-F 5 "10022976" H 10275 7763 50  0001 C CNN "Item Number"
-F 6 "KYOCERA_RMS1" H 10275 7763 50  0001 C CNN "Manufacturer"
-F 7 "CM05X7R472K25AT" H 10275 7763 50  0001 C CNN "Manufacturer_No"
-F 8 "MULTILAYER CERAMIC CAPACITOR" H 10275 7763 50  0001 C CNN "Manufacturer_Desc"
-F 9 "KEMET_RMS1" H 10275 7763 50  0001 C CNN "Manufacturer2"
-F 10 "C0402C472K3RACTU" H 10275 7763 50  0001 C CNN "Manufacturer_No2"
-F 11 "CERAMIC CHIP CAPACITOR" H 10275 7763 50  0001 C CNN "Manufacturer_Desc2"
-F 12 "AVX_RMS1" H 10275 7763 50  0001 C CNN "Manufacturer3"
-F 13 "04023C472KAT2A" H 10275 7763 50  0001 C CNN "Manufacturer_No3"
-F 14 "CERAMIC CAPACITOR X7R" H 10275 7763 50  0001 C CNN "Manufacturer_Desc3"
-	1    10275 7763
-	1    0    0    -1
-$EndComp
+P 10275 7750
+F 0 "C101" H 10400 7813 64  0000 L CNN
+F 1 "4.7nF" H 10400 7713 42  0000 L CNN
+F 2 "10125623A00:C0805" H 10275 7750 50  0001 C CNN
+F 3 "" H 10275 7750 50  0001 C CNN
+F 4 "CAPACITOR CERAMIC,4.7NF,25V,+/-10%,0402" H 10275 7750 50  0001 C CNN "Description"
+F 5 "10022976" H 10275 7750 50  0001 C CNN "Item Number"
+F 6 "KYOCERA_RMS1" H 10275 7750 50  0001 C CNN "Manufacturer"
+F 7 "CM05X7R472K25AT" H 10275 7750 50  0001 C CNN "Manufacturer_No"
+F 8 "MULTILAYER CERAMIC CAPACITOR" H 10275 7750 50  0001 C CNN "Manufacturer_Desc"
+F 9 "KEMET_RMS1" H 10275 7750 50  0001 C CNN "Manufacturer2"
+F 10 "C0402C472K3RACTU" H 10275 7750 50  0001 C CNN "Manufacturer_No2"
+F 11 "CERAMIC CHIP CAPACITOR" H 10275 7750 50  0001 C CNN "Manufacturer_Desc2"
+F 12 "AVX_RMS1" H 10275 7750 50  0001 C CNN "Manufacturer3"
+F 13 "04023C472KAT2A" H 10275 7750 50  0001 C CNN "Manufacturer_No3"
+F 14 "CERAMIC CAPACITOR X7R" H 10275 7750 50  0001 C CNN "Manufacturer_Desc3"
+	1    10275 7750
+	1    0    0    -1
+$EndComp

Commit message: Removed 5V global label and added 5V symbol on sheet 6
Connections:
- wire segments 251 -> 252
Changed lines of the file:
@@
 Text HLabel 10050 1500 0    56   Input ~ 0
 SUPPLY-AL-RP
-Text HLabel 3075 6650 2    70   BiDi ~ 0
-+5V
 $Comp
 L cpu-board:GND #U$043
@@
 Text Notes 1900 8025 0    50   ~ 0
 *Note: in earlier version, L22 connects to +5V instead of +5VSUPPLYBOARD
+$Comp
+L cpu-board:+5V #0101
+U 1 1 5E99C70E
+P 3075 6500
+F 0 "#0101" H 3125 6550 50  0001 C CNN
+F 1 "+5V" H 3025 6550 59  0000 R CNN
+F 2 "" H 3075 6500 50  0001 C CNN
+F 3 "" H 3075 6500 50  0001 C CNN
+	1    3075 6500
+	-1   0    0    1
+$EndComp
+Wire Wire Line
+	3075 6600 3075 6650
 $EndSCHEMATC

Commit message: back anotate from cmp file
Parts:
- ANT1: footprint 10125623A00:ANTENNE -> AllModules:PT-1.0MM_TEST_1
- C100, C38, C56: footprint 10125623A00:RESEAU_1 -> AllModules:C0612-4_1
- C101, C11, C130, C86, C93, C98: footprint 10125623A00:C0805 -> AllModules:C0402_1
- C115, C12, C121, C122, C123, C124, C126, C127, C13, C76, C99: footprint 10125623A00:C0603 -> AllModules:C0402_1
- C75: footprint 10125623A00:TANTALB -> AllModules:C3528_1
- C89: footprint 10125623A00:TANTALB -> AllModules:C3216_1
- D13: footprint 10125623A00:SOT23DIO -> AllModules:SOT23-1G_1
- D6: footprint 10125623A00:SOD87 -> AllModules:SOD87_1
- IC37: footprint 10125623A00:ARF34 -> AllModules:ARF7151A_1
- J11: footprint 10125623A00:3BR -> AllModules:B3BZR-SM3TF_1
- J18: footprint 10125623A00:7B_ZR_SM3_TF -> AllModules:B7BZR-SM3TF_1
- J19, J5: footprint 10125623A00:2BR -> AllModules:B2BZR-SM3TF_1
- J2: footprint 10125623A00:8BR -> AllModules:B8BZR-SM3TF_1
- J20: footprint 10125623A00:4BR -> AllModules:B4BZR-SM3TF_1
- J21: footprint 10125623A00:2BR254C -> AllModules:MOL7395-2_1
- J4: footprint 10125623A00:MF10BR -> AllModules:BP2X5C_1
- L10, L12, L13, L14, L15, L17, L21, L23, L24, L25, L26, L27, L28, L29, L31, L32, L33, L34, L37, L9: footprint 10125623A00:0603 -> AllModules:C0603_1
- L11, L19, L20, L22, L7: footprint 10125623A00:0603 -> AllModules:RC1206_1
- R11, R43, R48, R49, R68, R69, R70: footprint 10125623A00:R0805 -> AllModules:R0603_1
- RL1: footprint 10125623A00:G6K2G -> AllModules:G6K2G_1
- T17, T19: footprint 10125623A00:SOT23MOS -> AllModules:SOT23-GSD_1

Commit message: CPU schematic updated to Kicad resistor and cap symbols
Parts:
- C101, C11, C130, C86, C93, C98: symbol cpu-board:C0805 -> Flipped_Devices:C_Small
- C115, C12, C121, C122, C123, C124, C126, C127, C13, C76, C99: symbol cpu-board:C0603 -> Flipped_Devices:C_Small
- C75, C89: symbol cpu-board:TANTALB -> Flipped_Devices:CP_Small
- R11, R43, R48, R49, R68, R69, R70: symbol cpu-board:R0805 -> Flipped_Devices:R
Connections:
- wire segments 252 -> 250
Other:
- moved on the sheet: C100, C38, C56, D13, D6, J11, J18, J19, J20, J4, J5, L12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
