File: CPU_RB0505/10125623A00_4.sch (KiCad schematic (older format))
At the start: 52 parts, among them IC15 AWM3300V, IC16 ASDX001D44R-SQ04689, IC17 AWM3300V, IC18 ASDX001D44R-SQ04689, IC19 ASDX100D44R, IC22 ASDX001D44R-SQ04689, IC27 SQ276, IC28 SQ276, IC30 SQ276, IC33 BSDX0811BARO-X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

Commit message: Schematic symbols updated with BOM fields
Parts:
- BL1, BL3: Description (none) -> EMC,FLOW SENSOR HOUSING,IC15 & IC17; Item Number (none) -> 4096600.M00.023; Manufacturer (none) -> SUZHOU ACE SHEET MATEL MANUFACTURING CO., LTD; Manufacturer_Desc (none) -> EMC,FLOW SENSOR HOUSING,IC15 & IC17 (CUSTOM PART); Manufacturer_No (none) -> 4096600.M00.023
- BL2: Description (none) -> EMC CASING - CASE 2 PRESSURE SENSORS; Item Number (none) -> 4096600.M00.002; Manufacturer (none) -> SUZHOU ACE SHEET MATEL MANUFACTURING CO., LTD; Manufacturer_Desc (none) -> EMC CASING - CASE 2 PRESSURE SENSORS (CUSTOM PART); Manufacturer_No (none) -> 4096600.M00.002
- BL4: Description (none) -> EMC CASING - CASE 3 PRESSURE SENSORS; Item Number (none) -> 4096600.M00.003; Manufacturer (none) -> SUZHOU ACE SHEET MATEL MANUFACTURING CO., LTD; Manufacturer_Desc (none) -> EMC CASING - CASE 3 PRESSURE SENSORS (CUSTOM PART); Manufacturer_No (none) -> 4096600.M00.003
- C102, C59, C65, C94: Description (none) -> CAP CERAMIC,220NF,25V,X7R,+/-10%,0805; Item Number (none) -> 10022968; Manufacturer (none) -> AVX_RMS1; Manufacturer2 (none) -> KEMET_RMS1; Manufacturer3 (none) -> AVX_RMS1; Manufacturer4 (none) -> KEMET_RMS1; Manufacturer_Desc (none) -> SMT MULTILAYER CAPACITOR; Manufacturer_Desc2 (none) -> CERAMIC CHIP CAPACITOR; Manufacturer_Desc3 (none) -> X7R DIELECTRIC; Manufacturer_Desc4 (none) -> CERAMIC CHIP CAPACITOR; Manufacturer_No (none) -> 08053C224KAZ2A; Manufacturer_No2 (none) -> C0805C224K3RAC; Manufacturer_No3 (none) -> 08053C224KAT2A; Manufacturer_No4 (none) -> C0805C224K3RACTU
- C104, C61, C64, C68, C71, C96: Description (none) -> CAPACITOR CERAMIC,4.7NF,+/-10%,50V,0603; Item Number (none) -> 10022613; Manufacturer (none) -> KEMET_RMS1; Manufacturer2 (none) -> YAGEO_RMS1; Manufacturer_Desc (none) -> CAP 4700PF 50V CERAMIC X7R 0603; Manufacturer_No (none) -> C0603C472K5RACTU; Manufacturer_No2 (none) -> CC0603KRX7R9BB472
- C60, C63, C66, C70: Description (none) -> CAPACITOR,100NF,16V,+/-10%,X7R,0402; Item Number (none) -> 10022607; Manufacturer (none) -> MURATA; Manufacturer2 (none) -> YAGEO_RMS1; Manufacturer3 (none) -> YAGEO_RMS1; Manufacturer4 (none) -> MURATA MANUFACTURING CO., LTD.; Manufacturer_Desc (none) -> CAPACITOR, CERAMIC, MULTILAYER, 16V, X7R, 0.1UF, 0402; Manufacturer_Desc2 (none) -> CAP CER 0.1uF 16V X7R 10% 0402; Manufacturer_Desc3 (none) -> CAPACITOR, CERAMIC, MULTILAYER, 16 V, X7R, 0.1 UF, SURFACE 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; Manufacturer_Desc4 (none) -> MONOLITHIC CERAMIC CAPACITOR; Manufacturer_No (none) -> GRM155R71C104JA88J; Manufacturer_No2 (none) -> CC0402KRX7R7BB104; Manufacturer_No3 (none) -> 223878715649; Manufacturer_No4 (none) -> GRM155R71C104KA88D
- C62, C69: Description (none) -> CAPACITOR CERAMIC, 100NF, +/-10%, 50V, X7R,0805; Item Number (none) -> 10022135; Manufacturer (none) -> YAGEO_RMS1; Manufacturer2 (none) -> MURATA MANUFACTURING CO., LTD.; Manufacturer3 (none) -> YAGEO_RMS1; Manufacturer4 (none) -> SAMSUNG_RMS1; Manufacturer5 (none) -> YAGEO_RMS1; Manufacturer6 (none) -> AVX_RMS1; Manufacturer_Desc (none) -> CAPACITOR, CERAMIC, MULTILAYER, 50 V, X7R, 0.1 UF, SURFACE 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; Manufacturer_Desc2 (none) -> MONOLITHIC CERAMIC CAPACITOR; Manufacturer_Desc3 (none) -> CAPACITOR, CERAMIC, MULTILAYER, 50 V, X7R, 0.1 UF, SURFACE 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; Manufacturer_Desc4 (none) -> MULTILAYER CERAMIC CAPACITOR; Manufacturer_Desc5 (none) -> CAP CER .1UF 50V 10% X7R 0805; Manufacturer_Desc6 (none) -> CAPACITOR CERAMIC, 100NF, +/-10%, 50V, X7R,0805, X7R DIELEC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; Manufacturer_No (none) -> 223858055649; Manufacturer_No2 (none) -> GRM21BR71H104KA01L; Manufacturer_No3 (none) -> 223858015649; Manufacturer_No4 (none) -> CL21B104KBCNNNC; Manufacturer_No5 (none) -> CC0805KRX7R9BB104; Manufacturer_No6 (none) -> 08055C104KAT2A
- IC15, IC17: Description (none) -> IC AIR FLOW SENSOR,(0-1 LITRE); Item Number (none) -> 10022706; Manufacturer (none) -> HONEYWELL_RMS1; Manufacturer2 (none) -> HONEYWELL_RMS1; Manufacturer_Desc (none) -> AIRFLOW SENSOR; Manufacturer_Desc2 (none) -> AIR FLOW SENSOR; Manufacturer_No (none) -> AWM3300V; Manufacturer_No2 (none) -> FBAL001DU
- IC16, IC18, IC22: Description (none) -> IC, PRESSURE TRANSDUCER,(-10/+100 MBAR); Item Number (none) -> 10023117; Manufacturer (none) -> SENSYM_RMS1; Manufacturer2 (none) -> HONEYWELL_RMS1; Manufacturer_Desc (none) -> PRESSURE TRANSDUCER; Manufacturer_Desc2 (none) -> IC DIFFERENTIAL PRESSURE SENSOR WITH ANALOGUE OUTPUT -10 TO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; Manufacturer_No (none) -> ASDX001D44R-SQ04689; Manufacturer_No2 (none) -> XZ209766-ASDX
- IC33: Description (none) -> IC, BAROMETRIC PRESSURE SENSOR; Item Number (none) -> 10023159; Manufacturer (none) -> HONEYWELL_RMS1; Manufacturer2 (none) -> SENSORTECHNICS; Manufacturer_Desc (none) -> IC ABSOLUTE PRESSURE SENSOR WITH ANALOGUE OUTPUT 600 TO 110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; Manufacturer_Desc2 (none) -> PRESSURE TRANSDUCER; Manufacturer_No (none) -> XZ209330-ASDX; Manufacturer_No2 (none) -> BSDX0611BARO-X
- R33, R34, R37, R38, R42, R51: Description (none) -> RESISTOR, 4.7 K OHM, 0.063W +/-5%; Item Number (none) -> 10022617; Manufacturer (none) -> ASJ; Manufacturer2 (none) -> YAGEO_RMS1; Manufacturer3 (none) -> YAGEO_RMS1; Manufacturer4 (none) -> YAGEO_RMS1; Manufacturer_Desc (none) -> THICK FILM CHIP RESISTOR; Manufacturer_Desc2 (none) -> RESISTOR, METAL GLAZE/THICK FILM, 0.1 W, 5 %, 100 PPM, 4700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; Manufacturer_Desc3 (none) -> RESISTOR, METAL GLAZE/THICK FILM, 0.1 W, 5 %, 100 PPM, 4700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; Manufacturer_Desc4 (none) -> RESISTOR, METAL GLAZE/THICK FILM, 0.1 W, 5 %, 100 PPM, 4700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; Manufacturer_No (none) -> CR16-472JL; Manufacturer_No2 (none) -> 232270260472L; Manufacturer_No3 (none) -> RC0603JR-074K7L; Manufacturer_No4 (none) -> 232270260472

Commit message: back anotate from cmp file
Parts:
- BL2: footprint 10125623A00:2XBL-AWM -> AllModules:B2CAP-RB0505_1
- BL4: footprint 10125623A00:3XBL-AWM -> AllModules:B3CAP-RB0505_1
- C102, C59, C65, C67, C94: footprint 10125623A00:C1206 -> AllModules:C0805_1
- C103, C109, C113, C40, C48, C57, C60, C63, C66, C70, C72, C95: footprint 10125623A00:C0805 -> AllModules:C0402_1
- C104, C61, C64, C68, C71, C73, C96: footprint 10125623A00:C0805 -> AllModules:C0603_1
- C62, C69: footprint 10125623A00:C0805 -> AllModules:C0805_1
- IC16, IC18, IC22: footprint 10125623A00:ASDX -> AllModules:ASDX001D44R_1
- IC19: footprint 10125623A00:ASDX -> AllModules:ASDX100D44R_1
- IC27, IC28, IC30, IC34, IC35: footprint 10125623A00:SQ276 -> AllModules:SQ276-05856_1
- IC33: footprint 10125623A00:ASDX -> AllModules:BSDX-A2_1
- JP2, JP3, JP4: footprint 10125623A00:0805 -> AllModules:R0603_1
- R33, R34, R37, R38, R39, R42, R51: footprint 10125623A00:R0805 -> AllModules:R0603_1

Commit message: fix typo
Other:
- note added: "Dual implantation of Analog and Digital sensor: If SPI sensors are used then the equivalent analog sensors will not be wired"
- note removed: "Dual implantation of Analog and Digital sensor:If SPI sensors are used then the equivalent analog sensors will not be wired"
Changed lines of the file:
@@
 SCLK-SPI-0
 Text Notes 9137 8075 0    59   ~ 0
-Dual implantation of Analog and Digital sensor:If SPI sensors are used then the equivalent analog sensors will not be wired
+Dual implantation of Analog and Digital sensor: If SPI sensors are used then the equivalent analog sensors will not be wired
 Wire Notes Line
 	15325 7838 9012 7838

Commit message: CPU schematic updated to Kicad resistor and cap symbols
Parts:
- C102, C59, C65, C67, C94: symbol cpu-board:C1206 -> Flipped_Devices:C_Small
- C103, C104, C109, C113, C40, C48, C57, C60, C61, C62, C63, C64, C66, C68, C69, C70, C71, C72, C73, C95, C96: symbol cpu-board:C0805 -> Flipped_Devices:C_Small
- R33, R34, R37, R38, R39, R42, R51: symbol cpu-board:R0805 -> Flipped_Devices:R
Connections:
- wire segments 314 -> 313
Other:
- moved on the sheet: BL3, IC17, IC18, IC22, IC34, JP3

Commit message: ran renameSchSyms.py
Parts:
- BL1, BL3: symbol cpu-board:BLIN-AWM33 -> BL:BLIN-AWM33
- BL2: symbol cpu-board:2XBL-AWM -> BL:2XBL-AWM
- BL4: symbol cpu-board:3XBL-ADSX -> BL:3XBL-ADSX
- C102, C59, C65, C94: symbol Flipped_Devices:C_Small -> Capacitor:C0805_220nF_25V_10%
- C103, C60, C63, C66, C70, C95: symbol Flipped_Devices:C_Small -> Capacitor:C0402_100nF_16V_10%
- C104, C61, C64, C68, C71, C96: symbol Flipped_Devices:C_Small -> Capacitor:C0603_4n7F_50V_10%
- C62, C69: symbol Flipped_Devices:C_Small -> Capacitor:C0805_100nF_50V_10%
- IC15, IC17: symbol cpu-board:AWM3300V -> IC:AWM3300V
- IC16, IC18, IC22: symbol cpu-board:ASDX -> IC:ASDX_10023117
- IC33: symbol cpu-board:ASDX -> IC:ASDX_10023159
- R33, R34, R37, R38, R42, R51: symbol Flipped_Devices:R -> Resistor:R_4k7_5%
Changed lines of the file:
@@
 CE\-FLOW-EXP-SENS
 $Comp
-L Flipped_Devices:C_Small C65
+L Capacitor:C0805_220nF_25V_10% C65
 U 1 1 6EB094ED
 P 1500 3350
@@
 $EndComp
 $Comp
-L Flipped_Devices:R R34
+L Resistor:R_4k7_5% R34
 U 1 1 EFB8A895
 P 4400 1900
@@
 $EndComp
 $Comp
-L Flipped_Devices:C_Small C63
+L Capacitor:C0402_100nF_16V_10% C63
 U 1 1 2FAB5BC8
 P 4650 2150
@@
 $EndComp
 $Comp
-L Flipped_Devices:C_Small C64
+L Capacitor:C0603_4n7F_50V_10% C64
 U 1 1 680B2917
 P 3550 2100
@@
 $EndComp
 $Comp
-L Flipped_Devices:R R38
+L Resistor:R_4k7_5% R38
 U 1 1 6C0A03D3
 P 4300 3700
@@
 $EndComp
 $Comp
-L Flipped_Devices:C_Small C70
+L Capacitor:C0402_100nF_16V_10% C70
 U 1 1 5F8D81F9
 P 4550 4000
@@
 $EndComp
 $Comp
-L Flipped_Devices:C_Small C71
+L Capacitor:C0603_4n7F_50V_10% C71
 U 1 1 13BC9B95
 P 3550 3900
@@
 $EndComp
 $Comp
-L cpu-board:ASDX IC18
+L IC:ASDX_10023117 IC18
 U 1 1 CEEB9070
 P 2550 3800
@@
 $EndComp
 $Comp
-L Flipped_Devices:C_Small C60
+L Capacitor:C0402_100nF_16V_10% C60
 U 1 1 74AE98EE
 P 11450 2300
@@
 $EndComp
 $Comp
-L Flipped_Devices:C_Small C61
+L Capacitor:C0603_4n7F_50V_10% C61
 U 1 1 4189E79D
 P 10900 2300
@@
 $EndComp
 $Comp
-L Flipped_Devices:C_Small C62
+L Capacitor:C0805_100nF_50V_10% C62
 U 1 1 3872CC01
 P 9500 2050
@@
 $EndComp
 $Comp
-L cpu-board:AWM3300V IC15
+L IC:AWM3300V IC15
 U 1 1 90D2B56F
 P 10050 2050
@@
 $EndComp
 $Comp
-L Flipped_Devices:R R37
+L Resistor:R_4k7_5% R37
 U 1 1 11FD54D7
 P 14550 2050
@@
 $EndComp
 $Comp
-L Flipped_Devices:C_Small C66
+L Capacitor:C0402_100nF_16V_10% C66
 U 1 1 5B12AA4C
 P 14750 2250
@@
 $EndComp
 $Comp
-L Flipped_Devices:C_Small C68
+L Capacitor:C0603_4n7F_50V_10% C68
 U 1 1 F44D85A5
 P 14200 2200
@@
 $EndComp
 $Comp
-L Flipped_Devices:C_Small C69
+L Capacitor:C0805_100nF_50V_10% C69
 U 1 1 1015ED7D
 P 12850 2000
@@
 $EndComp
 $Comp
-L cpu-board:AWM3300V IC17
+L IC:AWM3300V IC17
 U 1 1 93EF86A4
 P 13350 2050
@@
 $EndComp
 $Comp
-L cpu-board:BLIN-AWM33 BL1
+L BL:BLIN-AWM33 BL1
 U 1 1 AAFF44B7
 P 10450 2425
@@
 $EndComp
 $Comp
-L cpu-board:BLIN-AWM33 BL3
+L BL:BLIN-AWM33 BL3
 U 1 1 6617CE3C
 P 13800 2450
@@
 $EndComp
 $Comp
-L Flipped_Devices:C_Small C95
+L Capacitor:C0402_100nF_16V_10% C95
 U 1 1 A1AFAF59
 P 4300 9550
@@
 $EndComp
 $Comp
-L Flipped_Devices:R R51
+L Resistor:R_4k7_5% R51
 U 1 1 C00D2805
 P 3900 9400
@@
 $EndComp
 $Comp
-L Flipped_Devices:C_Small C94
+L Capacitor:C0805_220nF_25V_10% C94
 U 1 1 84DA4059
 P 1550 9050
@@
 Connection ~ 1800 8750
 $Comp
-L cpu-board:ASDX IC33
+L IC:ASDX_10023159 IC33
 U 1 1 B100278E
 P 2550 9500
@@
 Connection ~ 1550 10050
 $Comp
-L Flipped_Devices:C_Small C96
+L Capacitor:C0603_4n7F_50V_10% C96
 U 1 1 C9A1B3F0
 P 3600 9575
@@
 $EndComp
 $Comp
-L Flipped_Devices:R R42
+L Resistor:R_4k7_5% R42
 U 1 1 83169F00
 P 4300 5550
@@
 $EndComp
 $Comp
-L Flipped_Devices:C_Small C104
+L Capacitor:C0603_4n7F_50V_10% C104
 U 1 1 CA435796
 P 3550 5700
@@
 $EndComp
 $Comp
-L cpu-board:ASDX IC22
+L IC:ASDX_10023117 IC22
 U 1 1 2C1B848F
 P 2550 5650
@@
 $EndComp
 $Comp
-L Flipped_Devices:C_Small C102
+L Capacitor:C0805_220nF_25V_10% C102
 U 1 1 DC61BB42
 P 1500 5200
@@
 	4550 5550 4850 5550
 $Comp
-L Flipped_Devices:C_Small C103
+L Capacitor:C0402_100nF_16V_10% C103
 U 1 1 0E789015
 P 4550 5850
@@
 	2500 2950 2500 3050
 $Comp
-L cpu-board:ASDX IC16
+L IC:ASDX_10023117 IC16
 U 1 1 9EF2916C
 P 2500 2000
@@
 	14000 2450 14000 2650
 $Comp
-L Flipped_Devices:R R33
+L Resistor:R_4k7_5% R33
 U 1 1 05E5179D
 P 11200 2050
@@
 	1800 7500 2000 7500
 $Comp
-L cpu-board:2XBL-AWM BL2
+L BL:2XBL-AWM BL2
 U 1 1 04E96AC4
 P 3350 8400
@@
 Connection ~ 1500 2200
 $Comp
-L Flipped_Devices:C_Small C59
+L Capacitor:C0805_220nF_25V_10% C59
 U 1 1 079CFDA5
 P 1500 1600
@@
 	1500 1250 1500 1500
 $Comp
-L cpu-board:3XBL-ADSX BL4
+L BL:3XBL-ADSX BL4
 U 1 1 2C3F9162
 P 3300 1500
