File: CPU_RB0505/10125623A00_1.sch (KiCad schematic (older format))
At the start: 65 parts, among them IC3 K6R4016C1D-TI10, IC4 ST10F276, IC40 CD74HCT245M, IC41 74HCT1G04GW, IC42 74HCT1G32GW, IC43 74HCT1G32GW, IC44 NC7SZ66, Q1 8MHz, T6 2N7002

Commit message: back anotate from cmp file
Parts:
- C1, C3: footprint 10125623A00:C0603 -> AllModules:C0603_1
- C10, C110, C116, C120, C22, C23, C25, C26, C27, C28, C29, C36, C51, C9: footprint 10125623A00:C0805 -> AllModules:C0402_1
- C112, C114: footprint 10125623A00:C0603 -> AllModules:C0805_1
- C14: footprint 10125623A00:RESEAU2 -> AllModules:C0612-4_1
- C6: footprint 10125623A00:C0805 -> AllModules:C0805_1
- C7, C8: footprint 10125623A00:TANTALB -> AllModules:C3216_1
- D1, D2, D3, D5: footprint 10125623A00:5SOT23 -> AllModules:SC70-5_1
- D10, D8, D9: footprint 10125623A00:SOT23DIO -> AllModules:SOT23-1G_1
- IC3: footprint 10125623A00:TSOPIIZ4 -> AllModules:TSOP2-44_1
- IC4: footprint 10125623A00:TQFP144 -> AllModules:TQFP144_1
- IC40: footprint 10125623A00:SO20 -> AllModules:MX.A20_COMPOSANT_1
- IC41, IC42, IC43, IC44: footprint 10125623A00:SOT23-5 -> AllModules:SC70-5_1
- JP7, JP8: footprint 10125623A00:0805 -> AllModules:R0603_1
- PST1, PST3, PST4, PST6: footprint 10125623A00:1X01 -> AllModules:PT-1.0MM_TEST_1
- PT1, PT2: footprint 10125623A00:1X01 -> AllModules:C12000_1
- Q1: footprint 10125623A00:SM49 -> AllModules:HC49-4HSMX_1
- R1, R10, R14, R15, R3, R45, R46, R60, R61, R62, R72: footprint 10125623A00:R0805 -> AllModules:R0603_1
- RS1, RS2, RS3, RS4, RS5, RS6, RS7: footprint 10125623A00:BCN16_4_ -> AllModules:BCN16_1
- T6: footprint 10125623A00:SOT23MOS -> AllModules:SOT23-GSD_1

Commit message: fix erc errors, change many pin electrical types
Connections:
- net labels added: LED_PRESENCE_AC
- net labels removed: LED_PRESENCE_LED
- wire segments 552 -> 553
Changed lines of the file:
@@
 TX_UART_ST
 Text HLabel 12000 2350 2    50   Input ~ 0
-LED_PRESENCE_LED
+LED_PRESENCE_AC
 Text HLabel 12000 2450 2    50   Input ~ 0
 USB-BUSY
@@
 	14900 4850 14900 4950
 Wire Wire Line
-	15000 1950 15000 2150
+	15000 1950 15000 1975
 Wire Wire Line
 	15000 2150 14900 2150
@@
 Wire Wire Line
 	12000 2150 11850 2150
-Wire Wire Line
-	11850 2350 12000 2350
 Wire Wire Line
 	12000 2450 11850 2450
@@
 $EndComp
 NoConn ~ 8100 7550
+$Comp
+L power:PWR_FLAG #FLG0103
+U 1 1 5ED7A82D
+P 15000 1975
+F 0 "#FLG0103" H 15000 2050 50  0001 C CNN
+F 1 "PWR_FLAG" V 15000 2103 50  0000 L CNN
+F 2 "" H 15000 1975 50  0001 C CNN
+F 3 "~" H 15000 1975 50  0001 C CNN
+	1    15000 1975
+	0    1    1    0
+$EndComp
+Connection ~ 15000 1975
+Wire Wire Line
+	15000 1975 15000 2150
+Wire Wire Line
+	11850 2350 12000 2350
 Wire Bus Line
 	15950 2650 15950 4250
@@
 Wire Bus Line
 	8700 2050 8700 3650
+$Comp
+L power:PWR_FLAG #FLG0112
+U 1 1 600E17E9
+P 11700 3250
+F 0 "#FLG0112" H 11700 3325 50  0001 C CNN
+F 1 "PWR_FLAG" H 11700 3423 50  0000 C CNN
+F 2 "" H 11700 3250 50  0001 C CNN
+F 3 "~" H 11700 3250 50  0001 C CNN
+	1    11700 3250
+	1    0    0    -1
+$EndComp
+Connection ~ 11700 3250
 $EndSCHEMATC

Commit message: CPU schematic updated to Kicad resistor and cap symbols
Parts:
- C1, C112, C114, C3: symbol cpu-board:C0603 -> Flipped_Devices:C_Small
- C10, C110, C116, C120, C22, C23, C25, C26, C27, C28, C29, C36, C51, C6, C9: symbol cpu-board:C0805 -> Flipped_Devices:C_Small
- C7, C8: symbol cpu-board:TANTALB -> Flipped_Devices:CP_Small
- R1, R10, R14, R15, R3, R45, R46, R60, R61, R62, R72: symbol cpu-board:R0805 -> Flipped_Devices:R
Connections:
- wire segments 553 -> 558
Changed lines of the file:
@@
 $EndComp
 $Comp
-L cpu-board:C0805 C?
+L Flipped_Devices:C_Small C?
 U 1 1 CB1F8FE5
 P 14700 2150
@@
 $EndComp
 $Comp
-L cpu-board:C0805 C?
+L Flipped_Devices:C_Small C?
 U 1 1 A05C1986
 P 7350 9650
@@
 $EndComp
 $Comp
-L cpu-board:C0805 C?
+L Flipped_Devices:C_Small C?
 U 1 1 93AA069D
 P 7350 9800
@@
 $EndComp
 $Comp
-L cpu-board:C0805 C?
+L Flipped_Devices:C_Small C?
 U 1 1 5F5D481B
 P 7350 9950
@@
 $EndComp
 $Comp
-L cpu-board:C0805 C?
+L Flipped_Devices:C_Small C?
 U 1 1 0EABB629
 P 7350 10100
@@
 $EndComp
 $Comp
-L cpu-board:C0805 C?
+L Flipped_Devices:C_Small C?
 U 1 1 C9504634
 P 7350 10250
@@
 $EndComp
 $Comp
-L cpu-board:C0805 C?
+L Flipped_Devices:C_Small C?
 U 1 1 AB97CB13
 P 7350 10400
@@
 $EndComp
 $Comp
-L cpu-board:C0805 C?
+L Flipped_Devices:C_Small C?
 U 1 1 BCAFF6B0
 P 7350 10550
@@
 $EndComp
 $Comp
-L cpu-board:C0805 C?
+L Flipped_Devices:C_Small C?
 U 1 1 284AD347
 P 7350 10700
@@
 $EndComp
 $Comp
-L cpu-board:R0805 R?
+L Flipped_Devices:R R?
 U 1 1 E6C7F8B8
 P 5550 1350
@@
 $EndComp
 $Comp
-L cpu-board:C0805 C?
+L Flipped_Devices:C_Small C?
 U 1 1 967579EA
 P 6550 1300
@@
 $EndComp
 $Comp
-L cpu-board:TANTALB C?
+L Flipped_Devices:CP_Small C?
 U 1 1 6D37B6AD
 P 7400 1100
@@
 $EndComp
 $Comp
-L cpu-board:C0805 C?
+L Flipped_Devices:C_Small C?
 U 1 1 501DA122
 P 8450 1300
@@
 $EndComp
 $Comp
-L cpu-board:C0603 C?
+L Flipped_Devices:C_Small C?
 U 1 1 7EE2FFE3
 P 5750 1050
@@
 $EndComp
 $Comp
-L cpu-board:C0603 C?
+L Flipped_Devices:C_Small C?
 U 1 1 5ADCC44B
 P 5550 1050
@@
 $EndComp
 $Comp
-L cpu-board:R0805 R?
+L Flipped_Devices:R R?
 U 1 1 C54AB7D0
 P 2200 9550
@@
 $EndComp
 $Comp
-L cpu-board:R0805 R?
+L Flipped_Devices:R R?
 U 1 1 BAB36D42
 P 2200 9850
@@
 $EndComp
 $Comp
-L cpu-board:C0805 C?
+L Flipped_Devices:C_Small C?
 U 1 1 597E8BEF
 P 2200 10050
@@
 $EndComp
 $Comp
-L cpu-board:R0805 R?
+L Flipped_Devices:R R?
 U 1 1 D628991E
 P 3100 5950
@@
 $EndComp
 $Comp
-L cpu-board:C0805 C?
+L Flipped_Devices:C_Small C?
 U 1 1 662809D9
 P 11150 1200
@@
 $EndComp
 $Comp
-L cpu-board:R0805 R?
+L Flipped_Devices:R R?
 U 1 1 CEF2471C
 P 12650 4050
@@
 $EndComp
 $Comp
-L cpu-board:R0805 R?
+L Flipped_Devices:R R?
 U 1 1 CCBE402C
 P 12050 7250
@@
 $EndComp
 $Comp
-L cpu-board:C0603 C?
+L Flipped_Devices:C_Small C?
 U 1 1 9A495DAC
 P 12200 7250
@@
 $EndComp
 $Comp
-L cpu-board:R0805 R?
+L Flipped_Devices:R R?
 U 1 1 F7CB6097
 P 4800 10950
@@
 $EndComp
 $Comp
-L cpu-board:C0805 C?
+L Flipped_Devices:C_Small C?
 U 1 1 7614D321
 P 4800 10550
@@
 $EndComp
 $Comp
-L cpu-board:C0805 C?
+L Flipped_Devices:C_Small C?
 U 1 1 150190AD
 P 10200 3250
@@
 $EndComp
 $Comp
-L cpu-board:R0805 R?
+L Flipped_Devices:R R?
 U 1 1 C18C78EC
 P 8500 950
@@
 	7950 1500 7950 1100
 $Comp
-L cpu-board:TANTALB C?
+L Flipped_Devices:CP_Small C?
 U 1 1 6F4029DE
 P 8250 1300
@@
 	8250 1100 8250 950
 Wire Wire Line
-	8250 950  8300 950
-Wire Wire Line
 	7400 1250 7400 1200
 Wire Wire Line
@@
 	7400 950  7250 950
 Wire Wire Line
-	7150 950  7150 1000
-Wire Wire Line
 	7250 950  7250 1600
 Connection ~ 7250 950
@@
 Connection ~ 7150 1500
 Wire Wire Line
-	7150 1500 7150 1400
-Wire Wire Line
 	6450 1600 6450 1500
 Wire Wire Line
@@
 Wire Wire Line
 	6150 1500 6150 1250
-Connection ~ 5550 1150
-Wire Wire Line
-	5550 1600 5550 1550
 Wire Wire Line
 	5750 1600 5750 1150
@@
 	2600 5850 2800 5850
 Wire Wire Line
-	4300 5950 3300 5950
-Wire Wire Line
-	2900 5950 2800 5950
-Wire Wire Line
 	2800 5950 2800 5850
 Connection ~ 2800 5850
@@
 Connection ~ 12400 4050
 Wire Wire Line
-	12400 4050 12450 4050
-Wire Wire Line
 	12400 4400 12400 4450
 Wire Wire Line
@@
 	11700 3600 11700 3250
 Wire Wire Line
-	11700 3250 12050 3250
+	11700 3250 11950 3250
 Wire Wire Line
 	12000 3550 12000 3600
@@
 	4250 8300 4250 10450
 Wire Wire Line
-	2400 9550 2650 9550
-Wire Wire Line
 	2650 9550 2650 9850
 Wire Wire Line
 	2650 10050 2300 10050
-Wire Wire Line
-	2400 9850 2650 9850
 Connection ~ 2650 9850
 Wire Wire Line
 	2650 9850 2650 10050
 Wire Wire Line
-	1650 9550 2000 9550
-Wire Wire Line
 	1800 9950 1900 9950
 Wire Wire Line
 	1900 9950 1900 9850
 Wire Wire Line
-	1900 9850 2000 9850
-Wire Wire Line
 	1900 9950 1900 10050
 Wire Wire Line
@@
 	5050 10550 5050 10750
 Wire Wire Line
-	5050 10950 5000 10950
-Wire Wire Line
 	5050 10750 5100 10750
 Connection ~ 5050 10750
@@
 	4400 10550 4400 10950
 Wire Wire Line
-	4400 10950 4600 10950
-Wire Wire Line
 	11050 1200 10950 1200
 Wire Wire Line
@@
 	11750 7700 12050 7700
 Wire Wire Line
-	12050 7700 12050 7450
-Wire Wire Line
 	12050 7700 12050 7750
 Connection ~ 12050 7700
@@
 	-1   0    0    -1
 $EndComp
-Wire Wire Line
-	12050 7050 12050 6700
 $Comp
-L cpu-board:R0805 R?
+L Flipped_Devices:R R?
 U 1 1 CBBF32AF
 P 12450 6700
@@
 	12200 7150 12200 6700
 Wire Wire Line
-	12200 6700 12250 6700
-Wire Wire Line
 	12200 6700 12050 6700
 Connection ~ 12200 6700
@@
 Connection ~ 12650 6600
 Wire Wire Line
-	12650 6600 12650 6700
-Wire Wire Line
 	12850 5950 13000 5950
 Wire Wire Line
@@
 	14900 6850 14900 6800
 $Comp
-L cpu-board:C0603 C?
+L Flipped_Devices:C_Small C?
 U 1 1 C17297D4
 P 14150 7300
@@
 	13300 6900 13300 6850
 Wire Wire Line
-	12650 6700 12650 7350
-Wire Wire Line
 	12650 7350 12700 7350
-Connection ~ 12650 6700
 Wire Wire Line
 	13650 7300 13650 7150
@@
 Connection ~ 13650 7300
 $Comp
-L cpu-board:R0805 R?
+L Flipped_Devices:R R?
 U 1 1 CC254D70
 P 13800 7700
@@
 	13950 7950 13800 7950
 Connection ~ 13800 7950
-Wire Wire Line
-	13800 7950 13800 7900
-Wire Wire Line
-	13800 7500 13800 7300
 Connection ~ 13800 7300
 Wire Wire Line
@@
 	5950 1550 5950 1600
 $Comp
-L cpu-board:R0805 R?
+L Flipped_Devices:R R?
 U 1 1 E7C109B0
 P 7150 1200
@@
 Wire Wire Line
 	11850 2350 12000 2350
+$Comp
+L power:PWR_FLAG #FLG0112
+U 1 1 600E17E9
+P 11950 3250
+F 0 "#FLG0112" H 11950 3325 50  0001 C CNN
+F 1 "PWR_FLAG" H 12100 3400 50  0000 C CNN
+F 2 "" H 11950 3250 50  0001 C CNN
+F 3 "~" H 11950 3250 50  0001 C CNN
+	1    11950 3250
+	1    0    0    -1
+$EndComp
+Wire Wire Line
+	12650 6600 12650 6700
+Wire Wire Line
+	5550 1200 5550 1150
+Connection ~ 5550 1150
+Wire Wire Line
+	5550 1500 5550 1600
+Wire Wire Line
+	7150 950  7150 1050
+Wire Wire Line
+	7150 1350 7150 1500
+Wire Wire Line
+	8250 950  8350 950
+Wire Wire Line
+	8650 950  8700 950
+Wire Wire Line
+	12400 4050 12500 4050
+Wire Wire Line
+	12800 4050 12850 4050
+Connection ~ 11950 3250
+Wire Wire Line
+	11950 3250 12050 3250
+Wire Wire Line
+	2800 5950 2950 5950
+Wire Wire Line
+	3250 5950 4300 5950
+Wire Wire Line
+	2350 9550 2650 9550
+Wire Wire Line
+	1650 9550 2050 9550
+Wire Wire Line
+	1900 9850 2050 9850
+Wire Wire Line
+	2350 9850 2650 9850
+Wire Wire Line
+	4400 10950 4650 10950
+Wire Wire Line
+	4950 10950 5050 10950
+Wire Wire Line
+	12050 7400 12050 7700
+Wire Wire Line
+	12050 6700 12050 7100
+Wire Wire Line
+	12200 6700 12300 6700
+Wire Wire Line
+	12600 6700 12650 6700
+Connection ~ 12650 6700
+Wire Wire Line
+	12650 6700 12650 7350
+Wire Wire Line
+	13800 7300 13800 7550
+Wire Wire Line
+	13800 7850 13800 7950
 Wire Bus Line
 	15950 2650 15950 4250
@@
 Wire Bus Line
 	8700 2050 8700 3650
-$Comp
-L power:PWR_FLAG #FLG0112
-U 1 1 600E17E9
-P 11700 3250
-F 0 "#FLG0112" H 11700 3325 50  0001 C CNN
-F 1 "PWR_FLAG" H 11700 3423 50  0000 C CNN
-F 2 "" H 11700 3250 50  0001 C CNN
-F 3 "~" H 11700 3250 50  0001 C CNN
-	1    11700 3250
-	1    0    0    -1
-$EndComp
-Connection ~ 11700 3250
 $EndSCHEMATC

Commit message: CPU board diode and transistor symbols changed to Kicad symbols
Parts:
- D10, D9: symbol cpu-board:BAT54 -> Flipped_Devices:D_Schottky_A1K3
- D8: symbol cpu-board:BZX84CXX -> Flipped_Devices:D_Zener_A1K3
- Q1: symbol cpu-board:SM49 -> Device:Crystal_Small
- T6: symbol cpu-board:2N7002 -> Flipped_Devices:Q_NMOS_GSD
Changed lines of the file:
@@
 $EndComp
 $Comp
-L cpu-board:SM49 Q?
+L Device:Crystal_Small Q?
 U 1 1 F8782F37
 P 5650 1150
@@
 $EndComp
 $Comp
-L cpu-board:BZX84CXX D?
+L Flipped_Devices:D_Zener_A1K3 D?
 U 1 1 8A392F19
-P 12400 4300
+P 12400 4250
 AR Path="/8A392F19" Ref="D?"  Part="1"
 AR Path="/5E923584/8A392F19" Ref="D8"  Part="1"
-F 0 "D8" V 12441 4179 59  0000 R TNN
-F 1 "BZX84C4V7" V 12360 4176 59  0000 R TNN
-F 2 "AllModules:SOT23-1G_1" H 12400 4300 50  0001 C CNN
-F 3 "" H 12400 4300 50  0001 C CNN
-F 4 "DIODE ZENER, 0.35W,4.7V" H 12400 4300 50  0001 C CNN "Description"
-F 5 "10022655" H 12400 4300 50  0001 C CNN "Item Number"
-F 6 "NXP SEMICONDUCTORS_RMS1" H 12400 4300 50  0001 C CNN "Manufacturer"
-F 7 "BZX84-C4V7" H 12400 4300 50  0001 C CNN "Manufacturer_No"
-F 8 "VOLTAGE REGULATOR DIODE" H 12400 4300 50  0001 C CNN "Manufacturer_Desc"
-F 9 "NXP SEMICONDUCTORS_RMS1" H 12400 4300 50  0001 C CNN "Manufacturer2"
-F 10 "BZX84-C4V7,215" H 12400 4300 50  0001 C CNN "Manufacturer_No2"
-F 11 "" H 12400 4300 50  0001 C CNN "Manufacturer_Desc2"
-	1    12400 4300
+F 0 "D8" V 12441 4129 59  0000 R TNN
+F 1 "BZX84C4V7" V 12360 4126 59  0000 R TNN
+F 2 "AllModules:SOT23-1G_1" H 12400 4250 50  0001 C CNN
+F 3 "" H 12400 4250 50  0001 C CNN
+F 4 "DIODE ZENER, 0.35W,4.7V" H 12400 4250 50  0001 C CNN "Description"
+F 5 "10022655" H 12400 4250 50  0001 C CNN "Item Number"
+F 6 "NXP SEMICONDUCTORS_RMS1" H 12400 4250 50  0001 C CNN "Manufacturer"
+F 7 "BZX84-C4V7" H 12400 4250 50  0001 C CNN "Manufacturer_No"
+F 8 "VOLTAGE REGULATOR DIODE" H 12400 4250 50  0001 C CNN "Manufacturer_Desc"
+F 9 "NXP SEMICONDUCTORS_RMS1" H 12400 4250 50  0001 C CNN "Manufacturer2"
+F 10 "BZX84-C4V7,215" H 12400 4250 50  0001 C CNN "Manufacturer_No2"
+F 11 "" H 12400 4250 50  0001 C CNN "Manufacturer_Desc2"
+	1    12400 4250
 	0    -1   -1   0
 $EndComp
@@
 $EndComp
 $Comp
-L cpu-board:BAT54 D?
+L Flipped_Devices:D_Schottky_A1K3 D?
 U 1 1 59396773
-P 13950 7750
+P 13950 7700
 AR Path="/59396773" Ref="D?"  Part="1"
 AR Path="/5E923584/59396773" Ref="D9"  Part="1"
-F 0 "D9" V 14074 7531 59  0000 L BNN
-F 1 "BAT54" V 13932 7658 42  0000 R TNN
-F 2 "AllModules:SOT23-1G_1" H 13950 7750 50  0001 C CNN
-F 3 "" H 13950 7750 50  0001 C CNN
-F 4 "DIODE SCHOTTKY, 30V, 200MA" H 13950 7750 50  0001 C CNN "Description"
-F 5 "10022652" H 13950 7750 50  0001 C CNN "Item Number"
-F 6 "NXP SEMICONDUCTORS_RMS1" H 13950 7750 50  0001 C CNN "Manufacturer"
-F 7 "BAT54,215" H 13950 7750 50  0001 C CNN "Manufacturer_No"
-F 8 "" H 13950 7750 50  0001 C CNN "Manufacturer_Desc"
-F 9 "NXP SEMICONDUCTORS_RMS1" H 13950 7750 50  0001 C CNN "Manufacturer2"
-F 10 "BAT54" H 13950 7750 50  0001 C CNN "Manufacturer_No2"
-F 11 "SCHOTTKY BARRIER DOUBLE DIODE" H 13950 7750 50  0001 C CNN "Manufacturer_Desc2"
-	1    13950 7750
+F 0 "D9" V 14074 7481 59  0000 L BNN
+F 1 "BAT54" V 13932 7608 42  0000 R TNN
+F 2 "AllModules:SOT23-1G_1" H 13950 7700 50  0001 C CNN
+F 3 "" H 13950 7700 50  0001 C CNN
+F 4 "DIODE SCHOTTKY, 30V, 200MA" H 13950 7700 50  0001 C CNN "Description"
+F 5 "10022652" H 13950 7700 50  0001 C CNN "Item Number"
+F 6 "NXP SEMICONDUCTORS_RMS1" H 13950 7700 50  0001 C CNN "Manufacturer"
+F 7 "BAT54,215" H 13950 7700 50  0001 C CNN "Manufacturer_No"
+F 8 "" H 13950 7700 50  0001 C CNN "Manufacturer_Desc"
+F 9 "NXP SEMICONDUCTORS_RMS1" H 13950 7700 50  0001 C CNN "Manufacturer2"
+F 10 "BAT54" H 13950 7700 50  0001 C CNN "Manufacturer_No2"
+F 11 "SCHOTTKY BARRIER DOUBLE DIODE" H 13950 7700 50  0001 C CNN "Manufacturer_Desc2"
+	1    13950 7700
 	0    -1   -1   0
 $EndComp
@@
 	10400 6400 11750 6400
 Wire Wire Line
-	11750 6400 11750 6450
+	11750 6400 11750 6500
 Wire Wire Line
 	8100 7350 8300 7350
@@
 Connection ~ 12400 4050
 Wire Wire Line
-	12400 4400 12400 4450
-Wire Wire Line
 	11350 3350 11350 4050
 Wire Wire Line
@@
 	7650 9650 7650 9800
 Wire Wire Line
-	11750 6850 11750 7700
+	11750 6900 11750 7700
 Wire Wire Line
 	11750 7700 12050 7700
@@
 	12200 7700 12050 7700
 $Comp
-L cpu-board:2N7002 T?
+L Flipped_Devices:Q_NMOS_GSD T?
 U 1 1 78F4DB2D
-P 11850 6650
+P 11850 6700
 AR Path="/78F4DB2D" Ref="T?"  Part="1"
 AR Path="/5E923584/78F4DB2D" Ref="T6"  Part="1"
-F 0 "T6" H 11785 6919 64  0000 L BNN
-F 1 "2N7002" H 11564 6830 59  0000 L BNN
-F 2 "AllModules:SOT23-GSD_1" H 11850 6650 50  0001 C CNN
-F 3 "" H 11850 6650 50  0001 C CNN
-F 4 "TRANSISTOR MOSFET N CHANNEL 60V, 0.18A" H 11850 6650 50  0001 C CNN "Description"
-F 5 "10097274" H 11850 6650 50  0001 C CNN "Item Number"
-F 6 "ON SEMICONDUCTOR_RMS1" H 11850 6650 50  0001 C CNN "Manufacturer"
-F 7 "2N7002LT1G" H 11850 6650 50  0001 C CNN "Manufacturer_No"
-F 8 "SMALL SIGNAL MOSFET" H 11850 6650 50  0001 C CNN "Manufacturer_Desc"
-F 9 "NXP SEMICONDUCTORS_RMS1" H 11850 6650 50  0001 C CNN "Manufacturer2"
-F 10 "2N7002,215" H 11850 6650 50  0001 C CNN "Manufacturer_No2"
-F 11 "" H 11850 6650 50  0001 C CNN "Manufacturer_Desc2"
-F 12 "NXP SEMICONDUCTORS_RMS1" H 11850 6650 50  0001 C CNN "Manufacturer3"
-F 13 "2N7002" H 11850 6650 50  0001 C CNN "Manufacturer_No3"
-F 14 "N-CHANNEL TRENCHMOS FET" H 11850 6650 50  0001 C CNN "Manufacturer_Desc3"
-	1    11850 6650
+F 0 "T6" H 11785 6969 64  0000 L BNN
+F 1 "2N7002" H 11564 6880 59  0000 L BNN
+F 2 "AllModules:SOT23-GSD_1" H 11850 6700 50  0001 C CNN
+F 3 "" H 11850 6700 50  0001 C CNN
+F 4 "TRANSISTOR MOSFET N CHANNEL 60V, 0.18A" H 11850 6700 50  0001 C CNN "Description"
+F 5 "10097274" H 11850 6700 50  0001 C CNN "Item Number"
+F 6 "ON SEMICONDUCTOR_RMS1" H 11850 6700 50  0001 C CNN "Manufacturer"
+F 7 "2N7002LT1G" H 11850 6700 50  0001 C CNN "Manufacturer_No"
+F 8 "SMALL SIGNAL MOSFET" H 11850 6700 50  0001 C CNN "Manufacturer_Desc"
+F 9 "NXP SEMICONDUCTORS_RMS1" H 11850 6700 50  0001 C CNN "Manufacturer2"
+F 10 "2N7002,215" H 11850 6700 50  0001 C CNN "Manufacturer_No2"
+F 11 "" H 11850 6700 50  0001 C CNN "Manufacturer_Desc2"
+F 12 "NXP SEMICONDUCTORS_RMS1" H 11850 6700 50  0001 C CNN "Manufacturer3"
+F 13 "2N7002" H 11850 6700 50  0001 C CNN "Manufacturer_No3"
+F 14 "N-CHANNEL TRENCHMOS FET" H 11850 6700 50  0001 C CNN "Manufacturer_Desc3"
+	1    11850 6700
 	-1   0    0    -1
 $EndComp
@@
 Connection ~ 12050 6700
 $Comp
-L cpu-board:BAT54 D?
+L Flipped_Devices:D_Schottky_A1K3 D?
 U 1 1 13A4EF58
 P 12450 6400
@@
 	12200 6700 12200 6400
 Wire Wire Line
-	12200 6400 12250 6400
-Wire Wire Line
-	12550 6400 12650 6400
+	12200 6400 12300 6400
 Wire Wire Line
 	12650 6400 12650 6600
@@
 	13800 8000 13800 7950
 Wire Wire Line
-	13950 7850 13950 7950
-Wire Wire Line
 	13950 7950 13800 7950
 Connection ~ 13800 7950
@@
 Wire Wire Line
 	13800 7850 13800 7950
+Wire Wire Line
+	12400 4450 12400 4400
+Wire Wire Line
+	12600 6400 12650 6400
+Wire Wire Line
+	13950 7850 13950 7950
 Wire Bus Line
 	15950 2650 15950 4250
