File: 10096315 Blower Driver/10096315 Blower Driver.sch (KiCad schematic (older format))
At the start: 113 parts

Commit message: Finalizing reference designators per issue #12. Added missing C24-C26 (100 nF decoupling caps for +24V). Added no-connect symbols. Added some previously missing ground ties on a couple ICs. Added V-REF-M connection between pins 3 and 8 of IC1. TODO: ERC
Parts:
- added C24, C25, C26: Capacitor_100nF, Capacitors_SMD:C_0805, symbol Blower_Driver_Components:Capacitor_100nF
- gave numbers to parts that had none: 113
Connections:
- net +24V: now also C24.~, C25.~, C26.~
- net GND: now also IC4.3 (COM), IC5.3 (COM), J22.1
- net GNDPWR: now also C24.~, C25.~, C26.~
- net VREF-M: now also IC1.8 (VREF)
- net at IC2.7 (DISCH): now also R37.~, R50.~
- new net: C20.~, IC1.10 (OSC), R41.~
- new net: C18.~, IC1.11 (+ERROR_IN), R42.~
- new net: C21.~, IC1.15 (-SENSE), R39.~
- new net: FI7.~, R2.~, T1.1 (G)
- new net: FI5.~, R8.~, T6.3 (D)
- new net: FI6.~, R42.~, R7.~
- new net: C22.~, FI3.~, J2.10
- new net: C22.~, FI4.~, J2.9
- no-connect marks 0 -> 9
Other:
- note added: "NB: C18 here was (mis)labeled C16\nin original schematic."
- note added: "NB: Net-ties don't show refdes in original,\nso NT1 is original to this version of the\nschematic."
- note added: "TODO: test points (PT?)"
