File: 10096315 Blower Driver/ctrb0505-A.kicad_pcb (KiCad board)
At the start: 4 copper layers, 92.5 x 72 mm, 310 parts, among them IC1 L-BC-SO24, IC2 L-BC-SO08, IC3 L-BC-SO08, IC4 L-BC-SO08, IC5 L-BC-SO08, IC6 REG-BC-DPAK, J1 F-COCMS-MOL43650-0212, J11 F-CO-MOL5566-02, J2 F-CO-HE10-2010D, J22 F-CO-MOL7395M09, J3 F-CO-MOL7395M02, J6 F-CO-MOL7395M08, T1 Q-SOT23-IRLML2803, T10 Q-SOT23-IRLML2803, T2 Q-BC-DPAK-GDS, T3 Q-BC-DPAK-GDS, T4 Q-BC-DPAK-GDS, T5 Q-BC-DPAK-GDS, T6 Q-BC-DPAK-GDS, T7 Q-BC-DPAK-GDS, T8 Q-SOT23-IRLML2803, T9 Q-BC-DPAK-GDS

Commit message: newly generated pcb
Parts:
- removed the ? at (305.0, -181.5) (x2)
- removed the ? at (321.3, -188.9)
- removed the ? at (295.1, -160.1)
- removed the ? at (290.0, -160.1)
- removed the ? at (292.6, -160.1)
- removed the ? at (290.0, -151.2)
- removed the ? at (295.1, -151.2)
- removed the ? at (292.6, -151.2)
- removed the ? at (283.1, -160.1)
- removed the ? at (278.0, -160.1)
- removed the ? at (280.5, -160.1)
- removed the ? at (278.0, -151.2)
- removed the ? at (339.3, -160.7)
- removed the ? at (283.1, -151.2)
- removed the ? at (280.5, -151.2)
- removed the ? at (260.3, -192.2)
- removed the ? at (334.9, -192.2)
- removed the ? at (334.9, -138.0)
- removed the ? at (260.3, -138.0)
- removed the ? at (323.8, -166.4)
- removed the ? at (323.8, -169.0)
- removed the ? at (323.8, -171.5)
- removed the ? at (323.8, -174.0)
- removed the ? at (334.5, -149.2)
- removed the ? at (323.8, -176.6)
- removed the ? at (323.8, -179.1)
- removed the ? at (323.8, -181.7)
- removed the ? at (323.8, -184.2)
- removed the ? at (323.8, -186.7)
- removed the ? at (259.3, -184.2)
- removed the ? at (253.8, -184.2)
- removed the ? at (271.3, -167.4)
- removed the ? at (271.3, -164.8)
- removed the ? at (271.3, -162.3)
- removed the ? at (334.5, -155.3)
- removed the ? at (271.3, -159.8)
- removed the ? at (271.3, -157.2)
- removed the ? at (271.3, -154.7)
- removed the ? at (271.3, -152.1)
- removed the ? at (271.3, -149.6)
- removed the ? at (271.3, -147.1)
- removed the ? at (271.3, -144.5)
- removed the ? at (314.6, -194.4)
- removed the ? at (314.6, -196.9)
- removed the ? at (317.2, -194.4)
- removed the ? at (324.6, -150.2)
- removed the ? at (317.2, -196.9)
- removed the ? at (319.7, -194.4)
- removed the ? at (319.7, -196.9)
- removed the ? at (322.3, -194.4)
- removed the ? at (322.3, -196.9)
- removed the ? at (324.8, -194.4)
- removed the ? at (324.8, -196.9)
- removed the ? at (256.4, -177.5)
- removed the ? at (263.9, -175.0)
- removed the ? at (258.9, -175.0)
- removed the ? at (324.6, -151.5)
- removed the ? at (256.4, -172.5)
- removed the ? at (261.4, -172.5)
- removed the ? at (261.4, -177.5)
- removed the ? at (315.8, -184.2)
- removed the ? at (315.8, -179.1)
- removed the ? at (308.3, -194.5)
- removed the ? at (277.8, -194.5)
- removed the ? at (308.3, -181.5)
- removed the ? at (277.8, -181.5)
- removed the ? at (315.8, -173.4)
- removed the ? at (324.6, -152.8)
- removed the ? at (315.8, -168.3)
- removed the ? at (104.5, -105.5)
- removed the ? at (104.5, -90.2)
- removed the ? at (104.5, -95.3)
- removed the ? at (104.5, -100.4)
- removed the ? at (104.5, -110.5)
- removed the ? at (104.5, -115.6)
- removed the ? at (104.5, -120.7)
- removed the ? at (320.5, -150.1)
- removed the ? at (309.4, -139.2)
- removed the ? at (297.3, -139.2)
- removed the ? at (301.6, -181.0) (x2)
- removed the ? at (284.8, -145.5)
- removed the ? at (317.0, -148.7)
- removed the ? at (317.0, -151.1)
- removed the ? at (317.0, -153.7)
- removed the ? at (314.9, -191.6)
- removed the ? at (320.1, -187.0)
- removed the ? at (329.1, -191.5)
- removed the ? at (327.2, -191.5)
- removed the ? at (325.3, -191.5)
- removed the ? at (268.5, -183.4)
- removed the ? at (300.5, -164.4) (x2)
- removed the ? at (316.7, -187.4)
- removed the ? at (341.8, -199.0)
- removed the ? at (305.9, -197.2)
- removed the ? at (304.3, -197.2)
- removed the ? at (302.7, -197.2)
- removed the ? at (301.2, -197.2)
- removed the ? at (299.6, -197.2)
- removed the ? at (298.0, -197.2)
- removed the ? at (298.0, -195.6)
- removed the ? at (298.0, -194.0)
- removed the ? at (288.6, -164.4) (x2)
- removed the ? at (298.0, -192.5)
- removed the ? at (319.3, -191.6)
- removed the ? at (312.9, -191.5)
- removed the ? at (298.0, -190.9)
- removed the ? at (321.3, -190.4)
- removed the ? at (298.0, -189.3)
- removed the ? at (307.2, -188.9)
- removed the ? at (327.2, -187.6)
- removed the ? at (318.5, -187.0)
- removed the ? at (276.6, -164.4) (x2)
- removed the ? at (318.6, -167.4)
- removed the ? at (319.2, -166.4)
- removed the ? at (320.1, -165.4)
- removed the ? at (341.5, -162.9)
- removed the ? at (328.9, -161.6)
- removed the ? at (316.6, -160.9)
- removed the ? at (339.1, -158.5)
- removed the ? at (316.1, -158.0)
- removed the ? at (328.9, -156.6)
- removed the ? at (276.1, -183.7) (x2)
- removed the ? at (324.6, -156.6)
- removed the ? at (318.9, -155.3)
- removed the ? at (311.5, -155.7)
- removed the ? at (326.8, -154.9)
- removed the ? at (339.1, -154.4)
- removed the ? at (325.7, -153.6)
- removed the ? at (330.9, -151.5)
- removed the ? at (330.0, -150.2)
- removed the ? at (328.1, -149.0)
- removed the ? at (325.7, -149.0)
- removed the ? at (303.0, -149.6)
- removed the ? at (339.1, -148.2)
- removed the ? at (330.7, -147.7)
- removed the ? at (330.8, -146.3)
- removed the ? at (308.8, -145.5)
- removed the ? at (318.9, -144.6)
- removed the ? at (330.2, -144.0)
- removed the ? at (317.7, -143.2)
- removed the ? at (317.7, -141.4)
- removed the ? at (317.0, -139.2)
- removed the ? at (285.3, -139.2)
- removed the ? at (290.9, -149.6)
- removed the ? at (327.0, -138.4)
- removed the ? at (310.1, -135.9)
- removed the ? at (298.0, -135.1)
- removed the ? at (286.2, -132.0)
- removed the ? at (298.8, -145.7)
- removed the ? at (296.9, -145.5)
- removed the ? at (286.6, -145.8)
- removed the ? at (275.1, -146.1)
- removed the ? at (278.9, -149.6)
- removed the ? at (276.7, -179.1)
- removed the ? at (287.5, -179.1)
- removed the ? at (307.2, -160.1)
- removed the ? at (302.1, -160.1)
- removed the ? at (304.6, -160.1)
- removed the ? at (302.1, -151.2)
- removed the ? at (307.2, -151.2)
- removed the ? at (304.6, -151.2)
- removed cam1: COIN_EXTERNE, ctrb0505-A1_clean.PcbLib:cam1
- removed cam12: FABRICATION-FEE, ctrb0505-A1_clean.PcbLib:cam12
- removed cam13: PERCAGE_TABLEAU, ctrb0505-A1_clean.PcbLib:cam13
- removed cam14: FEE_COMP, ctrb0505-A1_clean.PcbLib:cam14
- removed cam15: FEE_COMP, ctrb0505-A1_clean.PcbLib:cam15
- removed cam2: COIN_EXTERNE, ctrb0505-A1_clean.PcbLib:cam2
- removed cam3: COIN_EXTERNE, ctrb0505-A1_clean.PcbLib:cam3
- removed cam4: COIN_EXTERNE, ctrb0505-A1_clean.PcbLib:cam4
- removed cam5: FILM18_HORIZONTAL, ctrb0505-A1_clean.PcbLib:cam5
- removed cam6: A3_PER_COVIDIEN, ctrb0505-A1_clean.PcbLib:cam6
- removed cam7: A3_EQFC_COVIDIEN, ctrb0505-A1_clean.PcbLib:cam7
- removed cam8: PER-COVIDIEN_TEXTE, ctrb0505-A1_clean.PcbLib:cam8
- removed cam9: A3_EQFS_COVIDIEN, ctrb0505-A1_clean.PcbLib:cam9
- added ? (x2): , , F.Cu at (295.2, 54.0)
- added ?: , , F.Cu at (311.4, 46.7)
- added ?: , , F.Cu at (285.3, 75.5)
- added ?: , , F.Cu at (280.2, 75.5)
- added ?: , , F.Cu at (282.7, 75.5)
- added ?: , , F.Cu at (280.2, 84.4)
- added ?: , , F.Cu at (285.3, 84.4)
- added ?: , , F.Cu at (282.7, 84.4)
- added ?: , , F.Cu at (273.2, 75.5)
- added ?: , , F.Cu at (268.1, 75.5)
- added ?: , , F.Cu at (270.7, 75.5)
- added ?: , , F.Cu at (268.1, 84.4)
- added ?: , , F.Cu at (329.5, 74.8)
- added ?: , , F.Cu at (273.2, 84.4)
- added ?: , , F.Cu at (270.7, 84.4)
- added ?: , , F.Cu at (250.5, 43.4)
- added ?: , , F.Cu at (325.1, 43.4)
- added ?: , , F.Cu at (325.1, 97.6)
- added ?: , , F.Cu at (250.5, 97.6)
- added ?: , , F.Cu at (314.0, 69.1)
- added ?: , , F.Cu at (314.0, 66.6)
- added ?: , , F.Cu at (314.0, 64.0)
- added ?: , , F.Cu at (314.0, 61.5)
- added ?: , , F.Cu at (324.6, 86.4)
- added ?: , , F.Cu at (314.0, 59.0)
- added ?: , , F.Cu at (314.0, 56.4)
- added ?: , , F.Cu at (314.0, 53.9)
- added ?: , , F.Cu at (314.0, 51.3)
- added ?: , , F.Cu at (314.0, 48.8)
- added ?: , , F.Cu at (249.5, 51.3)
- added ?: , , F.Cu at (244.0, 51.3)
- added ?: , , F.Cu at (261.5, 68.2)
- added ?: , , F.Cu at (261.5, 70.7)
- added ?: , , F.Cu at (261.5, 73.3)
- added ?: , , F.Cu at (324.6, 80.2)
- added ?: , , F.Cu at (261.5, 75.8)
- added ?: , , F.Cu at (261.5, 78.3)
- added ?: , , F.Cu at (261.5, 80.9)
- added ?: , , F.Cu at (261.5, 83.4)
- added ?: , , F.Cu at (261.5, 86.0)
- added ?: , , F.Cu at (261.5, 88.5)
- added ?: , , F.Cu at (261.5, 91.0)
- added ?: , , F.Cu at (304.8, 41.2)
- added ?: , , F.Cu at (304.8, 38.6)
- added ?: , , F.Cu at (307.3, 41.2)
- added ?: , , F.Cu at (314.7, 85.3)
- added ?: , , F.Cu at (307.3, 38.6)
- added ?: , , F.Cu at (309.9, 41.2)
- added ?: , , F.Cu at (309.9, 38.6)
- added ?: , , F.Cu at (312.4, 41.2)
- added ?: , , F.Cu at (312.4, 38.6)
- added ?: , , F.Cu at (315.0, 41.2)
- added ?: , , F.Cu at (315.0, 38.6)
- added ?: , , F.Cu at (246.6, 58.1)
- added ?: , , F.Cu at (254.1, 60.6)
- added ?: , , F.Cu at (249.1, 60.6)
- added ?: , , F.Cu at (314.7, 84.1)
- added ?: , , F.Cu at (246.6, 63.1)
- added ?: , , F.Cu at (251.6, 63.1)
- added ?: , , F.Cu at (251.6, 58.1)
- added ?: , , F.Cu at (305.9, 51.3)
- added ?: , , F.Cu at (305.9, 56.4)
- added ?: , , F.Cu at (298.4, 41.1)
- added ?: , , F.Cu at (268.0, 41.1)
- added ?: , , F.Cu at (298.4, 54.1)
- added ?: , , F.Cu at (268.0, 54.1)
- added ?: , , F.Cu at (305.9, 62.1)
- added ?: , , F.Cu at (314.7, 82.8)
- added ?: , , F.Cu at (305.9, 67.2)
- added ?: , , F.Cu at (94.6, 130.1)
- added ?: , , F.Cu at (94.6, 145.3)
- added ?: , , F.Cu at (94.6, 140.2)
- added ?: , , F.Cu at (94.6, 135.2)
- added ?: , , F.Cu at (94.6, 125.0)
- added ?: , , F.Cu at (94.6, 119.9)
- added ?: , , F.Cu at (94.6, 114.8)
- added ?: , , F.Cu at (310.7, 85.5)
- added ?: , , F.Cu at (299.6, 96.3)
- added ?: , , F.Cu at (287.5, 96.3)
- added ? (x2): , , F.Cu at (291.7, 54.5)
- added ?: , , F.Cu at (274.9, 90.1)
- added ?: , , F.Cu at (307.2, 86.8)
- added ?: , , F.Cu at (307.2, 84.4)
- added ?: , , F.Cu at (307.2, 81.8)
- added ?: , , F.Cu at (305.0, 44.0)
- added ?: , , F.Cu at (310.2, 48.5)
- added ?: , , F.Cu at (319.2, 44.1)
- added ?: , , F.Cu at (317.3, 44.1)
- added ?: , , F.Cu at (315.4, 44.1)
- added ?: , , F.Cu at (258.6, 52.1)
- added ? (x2): , , F.Cu at (290.6, 71.2)
- added ?: , , F.Cu at (306.8, 48.2)
- added ?: , , F.Cu at (331.9, 36.6)
- added ?: , , F.Cu at (296.1, 38.3)
- added ?: , , F.Cu at (294.5, 38.3)
- added ?: , , F.Cu at (292.9, 38.3)
- added ?: , , F.Cu at (291.3, 38.3)
- added ?: , , F.Cu at (289.7, 38.3)
- added ?: , , F.Cu at (288.1, 38.3)
- added ?: , , F.Cu at (288.1, 39.9)
- added ?: , , F.Cu at (288.1, 41.5)
- added ? (x2): , , F.Cu at (278.8, 71.2)
- added ?: , , F.Cu at (288.1, 43.1)
- added ?: , , F.Cu at (309.4, 43.9)
- added ?: , , F.Cu at (303.0, 44.1)
- added ?: , , F.Cu at (288.1, 44.7)
- added ?: , , F.Cu at (311.4, 45.2)
- added ?: , , F.Cu at (288.1, 46.3)
- added ?: , , F.Cu at (297.3, 46.7)
- added ?: , , F.Cu at (317.3, 48.0)
- added ?: , , F.Cu at (308.6, 48.5)
- added ? (x2): , , F.Cu at (266.7, 71.2)
- added ?: , , F.Cu at (308.7, 68.2)
- added ?: , , F.Cu at (309.3, 69.1)
- added ?: , , F.Cu at (310.3, 70.1)
- added ?: , , F.Cu at (331.7, 72.6)
- added ?: , , F.Cu at (319.0, 73.9)
- added ?: , , F.Cu at (306.7, 74.7)
- added ?: , , F.Cu at (329.3, 77.1)
- added ?: , , F.Cu at (306.2, 77.5)
- added ?: , , F.Cu at (319.0, 79.0)
- added ? (x2): , , F.Cu at (266.2, 51.9)
- added ?: , , F.Cu at (314.7, 79.0)
- added ?: , , F.Cu at (309.0, 80.2)
- added ?: , , F.Cu at (301.6, 79.9)
- added ?: , , F.Cu at (317.0, 80.7)
- added ?: , , F.Cu at (329.3, 81.2)
- added ?: , , F.Cu at (315.8, 82.0)
- added ?: , , F.Cu at (321.0, 84.1)
- added ?: , , F.Cu at (320.2, 85.3)
- added ?: , , F.Cu at (318.2, 86.6)
- added ?: , , F.Cu at (315.9, 86.6)
- added ?: , , F.Cu at (293.1, 86.0)
- added ?: , , F.Cu at (329.3, 87.3)
- added ?: , , F.Cu at (320.9, 87.9)
- added ?: , , F.Cu at (320.9, 89.2)
- added ?: , , F.Cu at (299.0, 90.1)
- added ?: , , F.Cu at (309.0, 91.0)
- added ?: , , F.Cu at (320.4, 91.6)
- added ?: , , F.Cu at (307.9, 92.4)
- added ?: , , F.Cu at (307.9, 94.1)
- added ?: , , F.Cu at (307.2, 96.3)
- added ?: , , F.Cu at (275.5, 96.3)
- added ?: , , F.Cu at (281.1, 86.0)
- added ?: , , F.Cu at (317.1, 97.2)
- added ?: , , F.Cu at (300.2, 99.6)
- added ?: , , F.Cu at (288.1, 100.4)
- added ?: , , F.Cu at (276.4, 103.5)
- added ?: , , F.Cu at (288.9, 89.8)
- added ?: , , F.Cu at (287.0, 90.1)
- added ?: , , F.Cu at (276.8, 89.7)
- added ?: , , F.Cu at (265.3, 89.4)
- added ?: , , F.Cu at (269.0, 86.0)
- added ?: , , F.Cu at (266.8, 56.5)
- added ?: , , F.Cu at (277.6, 56.5)
- added ?: , , F.Cu at (297.3, 75.5)
- added ?: , , F.Cu at (292.2, 75.5)
- added ?: , , F.Cu at (294.8, 75.5)
- added ?: , , F.Cu at (292.2, 84.4)
- added ?: , , F.Cu at (297.3, 84.4)
- added ?: , , F.Cu at (294.8, 84.4)
- added CAM1: COIN_EXTERNE, ctrb0505-A:COIN_EXTERNE_1, F.Cu at (241.4, 34.6)
- added CAM12: FABRICATION-FEE, ctrb0505-A:FABRICATION-FEE_1, F.Cu at (139.1, 0.01)
- added CAM13: PERCAGE_TABLEAU, ctrb0505-A:PERCAGE_TABLEAU_1, F.Cu at (130.2, 82.7)
- added CAM14: FEE_COMP, ctrb0505-A:FEE_COMP_2, B.Cu at (247.2, 105.6)
- added CAM15: FEE_COMP, ctrb0505-A:FEE_COMP_1, F.Cu at (315.1, 105.6)
- added CAM2: COIN_EXTERNE, ctrb0505-A:COIN_EXTERNE_1, F.Cu at (241.4, 106.6)
- added CAM3: COIN_EXTERNE, ctrb0505-A:COIN_EXTERNE_1, F.Cu at (334.0, 106.6)
- added CAM4: COIN_EXTERNE, ctrb0505-A:COIN_EXTERNE_1, F.Cu at (334.0, 34.6)
- added CAM5: FILM18_HORIZONTAL, ctrb0505-A:FILM18_HORIZONTAL_1, F.Cu at (288.5, 76.6)
- added CAM6: A3_PER_COVIDIEN, ctrb0505-A:A3_PER_COVIDIEN_1, F.Cu at (206.1, 96.0)
- added CAM7: A3_EQFC_COVIDIEN, ctrb0505-A:A3_EQFC_COVIDIEN_1, F.Cu at (287.0, 89.6)
- added CAM8: PER-COVIDIEN_TEXTE, ctrb0505-A:PER-COVIDIEN_TEXTE_1, F.Cu at (250.9, 137.6)
- added CAM9: A3_EQFS_COVIDIEN, ctrb0505-A:A3_EQFS_COVIDIEN_1, B.Cu at (287.4, 72.6)
- C1: footprint ctrb0505-A1_clean.PcbLib:C1 -> ctrb0505-A:C0805_1
- C10: footprint ctrb0505-A1_clean.PcbLib:C10 -> ctrb0505-A:RC1206_1
- C11: footprint ctrb0505-A1_clean.PcbLib:C11 -> ctrb0505-A:C0603_1
- C12: footprint ctrb0505-A1_clean.PcbLib:C12 -> ctrb0505-A:C0805_1
- C13: footprint ctrb0505-A1_clean.PcbLib:C13 -> ctrb0505-A:RC1206_1
- C14: footprint ctrb0505-A1_clean.PcbLib:C14 -> ctrb0505-A:C0603_1
- C15: footprint ctrb0505-A1_clean.PcbLib:C15 -> ctrb0505-A:C0805_1
- C16: footprint ctrb0505-A1_clean.PcbLib:C16 -> ctrb0505-A:RC1206_1
- C17: footprint ctrb0505-A1_clean.PcbLib:C17 -> ctrb0505-A:C0603_1
- C18: footprint ctrb0505-A1_clean.PcbLib:C18 -> ctrb0505-A:C0805_1
- C19: footprint ctrb0505-A1_clean.PcbLib:C19 -> ctrb0505-A:C0805_1
- C2: footprint ctrb0505-A1_clean.PcbLib:C2 -> ctrb0505-A:03515_1
- C20: footprint ctrb0505-A1_clean.PcbLib:C20 -> ctrb0505-A:C0603_1
- C21: footprint ctrb0505-A1_clean.PcbLib:C21 -> ctrb0505-A:C0805_1
- C22: footprint ctrb0505-A1_clean.PcbLib:C22 -> ctrb0505-A:C0612-4_1
- C23: footprint ctrb0505-A1_clean.PcbLib:C23 -> ctrb0505-A:C0612-4_1
- C24: footprint ctrb0505-A1_clean.PcbLib:C24 -> ctrb0505-A:C0805_1
- C25: footprint ctrb0505-A1_clean.PcbLib:C25 -> ctrb0505-A:C0805_1
- C26: footprint ctrb0505-A1_clean.PcbLib:C26 -> ctrb0505-A:C0805_1
- C27: footprint ctrb0505-A1_clean.PcbLib:C27 -> ctrb0505-A:03515_1
- C28: footprint ctrb0505-A1_clean.PcbLib:C28 -> ctrb0505-A:HT-13X27_1
- C29: footprint ctrb0505-A1_clean.PcbLib:C29 -> ctrb0505-A:HT-13X27_1
- C3: footprint ctrb0505-A1_clean.PcbLib:C3 -> ctrb0505-A:C0805_1
- C4: footprint ctrb0505-A1_clean.PcbLib:C4 -> ctrb0505-A:C7343_1
- C5: footprint ctrb0505-A1_clean.PcbLib:C5 -> ctrb0505-A:C0805_1
- C6: footprint ctrb0505-A1_clean.PcbLib:C6 -> ctrb0505-A:C0805_1
- C7: footprint ctrb0505-A1_clean.PcbLib:C7 -> ctrb0505-A:C0603_1
- C8: footprint ctrb0505-A1_clean.PcbLib:C8 -> ctrb0505-A:C0603_1
- C9: footprint ctrb0505-A1_clean.PcbLib:C9 -> ctrb0505-A:C0805_1
- D1: footprint ctrb0505-A1_clean.PcbLib:D1 -> ctrb0505-A:SMB_1
- D10: footprint ctrb0505-A1_clean.PcbLib:D10 -> ctrb0505-A:SMA_1
- D11: footprint ctrb0505-A1_clean.PcbLib:D11 -> ctrb0505-A:SOD80_1
- D12: footprint ctrb0505-A1_clean.PcbLib:D12 -> ctrb0505-A:SOD80_1
- D13: footprint ctrb0505-A1_clean.PcbLib:D13 -> ctrb0505-A:SOD80_1
- D14: footprint ctrb0505-A1_clean.PcbLib:D14 -> ctrb0505-A:SOT23-1G_1
- D15: footprint ctrb0505-A1_clean.PcbLib:D15 -> ctrb0505-A:SOT23-1G_1
- D16: footprint ctrb0505-A1_clean.PcbLib:D16 -> ctrb0505-A:SOT23-1G_1
- D17: footprint ctrb0505-A1_clean.PcbLib:D17 -> ctrb0505-A:DPAK-2ANODES_1
- D18: footprint ctrb0505-A1_clean.PcbLib:D18 -> ctrb0505-A:SMB_1
- D19: footprint ctrb0505-A1_clean.PcbLib:D19 -> ctrb0505-A:SMB_1
- D2: footprint ctrb0505-A1_clean.PcbLib:D2 -> ctrb0505-A:SOD323_1
- D20: footprint ctrb0505-A1_clean.PcbLib:D20 -> ctrb0505-A:SMB_1
- D21: footprint ctrb0505-A1_clean.PcbLib:D21 -> ctrb0505-A:SMB_1
- D22: footprint ctrb0505-A1_clean.PcbLib:D22 -> ctrb0505-A:SMB_1
- D23: footprint ctrb0505-A1_clean.PcbLib:D23 -> ctrb0505-A:SMB_1
- D24: footprint ctrb0505-A1_clean.PcbLib:D24 -> ctrb0505-A:SOT23-1G_1
- D3: footprint ctrb0505-A1_clean.PcbLib:D3 -> ctrb0505-A:SOD323_1
- D4: footprint ctrb0505-A1_clean.PcbLib:D4 -> ctrb0505-A:SOD323_1
- D5: footprint ctrb0505-A1_clean.PcbLib:D5 -> ctrb0505-A:SOD323_1
- D6: footprint ctrb0505-A1_clean.PcbLib:D6 -> ctrb0505-A:SOD323_1
- D7: footprint ctrb0505-A1_clean.PcbLib:D7 -> ctrb0505-A:SOD323_1
- D8: footprint ctrb0505-A1_clean.PcbLib:D8 -> ctrb0505-A:SMA_1
- D9: footprint ctrb0505-A1_clean.PcbLib:D9 -> ctrb0505-A:SMA_1
- F1: footprint ctrb0505-A1_clean.PcbLib:F1 -> ctrb0505-A:FU154000_1
- FI1: footprint ctrb0505-A1_clean.PcbLib:FI1 -> ctrb0505-A:BNX002_1
- FI3: footprint ctrb0505-A1_clean.PcbLib:FI3 -> ctrb0505-A:C0603_1
- FI4: footprint ctrb0505-A1_clean.PcbLib:FI4 -> ctrb0505-A:C0603_1
- FI5: footprint ctrb0505-A1_clean.PcbLib:FI5 -> ctrb0505-A:C0603_1
- FI6: footprint ctrb0505-A1_clean.PcbLib:FI6 -> ctrb0505-A:C0603_1
- FI7: footprint ctrb0505-A1_clean.PcbLib:FI7 -> ctrb0505-A:C0603_1
- FI8: footprint ctrb0505-A1_clean.PcbLib:FI8 -> ctrb0505-A:C0603_1
- FI9: footprint ctrb0505-A1_clean.PcbLib:FI9 -> ctrb0505-A:C0603_1
- IC1: footprint ctrb0505-A1_clean.PcbLib:IC1 -> ctrb0505-A:MX.A24_COMPOSANT_1
- IC2: footprint ctrb0505-A1_clean.PcbLib:IC2 -> ctrb0505-A:MX.A8_COMPOSANT_1
- IC3: footprint ctrb0505-A1_clean.PcbLib:IC3 -> ctrb0505-A:MX.A8_COMPOSANT_1
- IC4: footprint ctrb0505-A1_clean.PcbLib:IC4 -> ctrb0505-A:MX.A8_COMPOSANT_1
- IC5: footprint ctrb0505-A1_clean.PcbLib:IC5 -> ctrb0505-A:MX.A8_COMPOSANT_1
- IC6: footprint ctrb0505-A1_clean.PcbLib:IC6 -> ctrb0505-A:DPAK_1
- J1: footprint ctrb0505-A1_clean.PcbLib:J1 -> ctrb0505-A:MOL43650-02C_1
- J11: footprint ctrb0505-A1_clean.PcbLib:J11 -> ctrb0505-A:MOL5566-2_1
- J2: footprint ctrb0505-A1_clean.PcbLib:J2 -> ctrb0505-A:BP2X5D_1
- J22: footprint ctrb0505-A1_clean.PcbLib:J22 -> ctrb0505-A:MOL7395-9_1
- J3: footprint ctrb0505-A1_clean.PcbLib:J3 -> ctrb0505-A:MOL7395-2_1
- J6: footprint ctrb0505-A1_clean.PcbLib:J6 -> ctrb0505-A:MOL7395-8_1
- MIR1: footprint ctrb0505-A1_clean.PcbLib:MIR1 -> ctrb0505-A:MIRECMS-SAFT_1
- MIR2: footprint ctrb0505-A1_clean.PcbLib:MIR2 -> ctrb0505-A:MIRECMS-SAFT_1
- MIR3: footprint ctrb0505-A1_clean.PcbLib:MIR3 -> ctrb0505-A:MIRECMS-SAFT_1
- MIR4: footprint ctrb0505-A1_clean.PcbLib:MIR4 -> ctrb0505-A:MIRECMS-SAFT_1
- PT1: footprint ctrb0505-A1_clean.PcbLib:PT1 -> ctrb0505-A:C12000_1
- R1: footprint ctrb0505-A1_clean.PcbLib:R1 -> ctrb0505-A:R2512_1
- R10: footprint ctrb0505-A1_clean.PcbLib:R10 -> ctrb0505-A:R0603_1
- R11: footprint ctrb0505-A1_clean.PcbLib:R11 -> ctrb0505-A:R0603_1
- R12: footprint ctrb0505-A1_clean.PcbLib:R12 -> ctrb0505-A:R0603_1
- R13: footprint ctrb0505-A1_clean.PcbLib:R13 -> ctrb0505-A:R0603_1
- R2: footprint ctrb0505-A1_clean.PcbLib:R2 -> ctrb0505-A:R0603_1
- R20: footprint ctrb0505-A1_clean.PcbLib:R20 -> ctrb0505-A:R0603_1
- R3: footprint ctrb0505-A1_clean.PcbLib:R3 -> ctrb0505-A:R0603_1
- R30: footprint ctrb0505-A1_clean.PcbLib:R30 -> ctrb0505-A:R0603_1
- R31: footprint ctrb0505-A1_clean.PcbLib:R31 -> ctrb0505-A:R0603_1
- R32: footprint ctrb0505-A1_clean.PcbLib:R32 -> ctrb0505-A:R0603_1
- R33: footprint ctrb0505-A1_clean.PcbLib:R33 -> ctrb0505-A:R0603_1
- R35: footprint ctrb0505-A1_clean.PcbLib:R35 -> ctrb0505-A:R0603_1
- R37: footprint ctrb0505-A1_clean.PcbLib:R37 -> ctrb0505-A:R0603_1
- R38: footprint ctrb0505-A1_clean.PcbLib:R38 -> ctrb0505-A:R0603_1
- R39: footprint ctrb0505-A1_clean.PcbLib:R39 -> ctrb0505-A:R0603_1
- R4: footprint ctrb0505-A1_clean.PcbLib:R4 -> ctrb0505-A:R0603_1
- R40: footprint ctrb0505-A1_clean.PcbLib:R40 -> ctrb0505-A:R2512_1
- R41: footprint ctrb0505-A1_clean.PcbLib:R41 -> ctrb0505-A:R0603_1
- R42: footprint ctrb0505-A1_clean.PcbLib:R42 -> ctrb0505-A:R0603_1
- R5: footprint ctrb0505-A1_clean.PcbLib:R5 -> ctrb0505-A:R0603_1
- R50: footprint ctrb0505-A1_clean.PcbLib:R50 -> ctrb0505-A:R0603_1
- R58: footprint ctrb0505-A1_clean.PcbLib:R58 -> ctrb0505-A:RC1206_1
- R59: footprint ctrb0505-A1_clean.PcbLib:R59 -> ctrb0505-A:RC1206_1
- R6: footprint ctrb0505-A1_clean.PcbLib:R6 -> ctrb0505-A:R0603_1
- R60: footprint ctrb0505-A1_clean.PcbLib:R60 -> ctrb0505-A:RC1206_1
- R7: footprint ctrb0505-A1_clean.PcbLib:R7 -> ctrb0505-A:R0603_1
- R8: footprint ctrb0505-A1_clean.PcbLib:R8 -> ctrb0505-A:R0603_1
- R9: footprint ctrb0505-A1_clean.PcbLib:R9 -> ctrb0505-A:R0603_1
- T1: footprint ctrb0505-A1_clean.PcbLib:T1 -> ctrb0505-A:SOT23-GSD_1
- T10: footprint ctrb0505-A1_clean.PcbLib:T10 -> ctrb0505-A:SOT23-GSD_1
- T2: footprint ctrb0505-A1_clean.PcbLib:T2 -> ctrb0505-A:DPAK-GDS_1
- T3: footprint ctrb0505-A1_clean.PcbLib:T3 -> ctrb0505-A:DPAK-GDS_1
- T4: footprint ctrb0505-A1_clean.PcbLib:T4 -> ctrb0505-A:DPAK-GDS_1
- T5: footprint ctrb0505-A1_clean.PcbLib:T5 -> ctrb0505-A:DPAK-GDS_1
- T6: footprint ctrb0505-A1_clean.PcbLib:T6 -> ctrb0505-A:DPAK-GDS_1
- T7: footprint ctrb0505-A1_clean.PcbLib:T7 -> ctrb0505-A:DPAK-GDS_1
- T8: footprint ctrb0505-A1_clean.PcbLib:T8 -> ctrb0505-A:SOT23-GSD_1
- T9: footprint ctrb0505-A1_clean.PcbLib:T9 -> ctrb0505-A:DPAK-GDS_1
- ZC2: footprint ctrb0505-A1_clean.PcbLib:ZC21 -> ctrb0505-A:C-SC8_1
- ZC27: footprint ctrb0505-A1_clean.PcbLib:ZC22 -> ctrb0505-A:C-SC10_1
- ZM1: footprint ctrb0505-A1_clean.PcbLib:ZM1 -> ctrb0505-A:FIX35M_1
- ZM2: footprint ctrb0505-A1_clean.PcbLib:ZM2 -> ctrb0505-A:FIX35M_1
- ZM3: footprint ctrb0505-A1_clean.PcbLib:ZM3 -> ctrb0505-A:FIX35M_1
- ZM4: footprint ctrb0505-A1_clean.PcbLib:ZM4 -> ctrb0505-A:FIX35M_1
- ZT2: footprint ctrb0505-A1_clean.PcbLib:ZT2 -> ctrb0505-A:TO220ABGDS-INV_COUCHE_1
- ZT3: footprint ctrb0505-A1_clean.PcbLib:ZT3 -> ctrb0505-A:TO220ABGDS-INV_COUCHE_1
- ZT4: footprint ctrb0505-A1_clean.PcbLib:ZT4 -> ctrb0505-A:TO220ABGDS-INV_COUCHE_1
- ZT5: footprint ctrb0505-A1_clean.PcbLib:ZT5 -> ctrb0505-A:TO220ABGDS-INV_COUCHE_1
- ZT6: footprint ctrb0505-A1_clean.PcbLib:ZT6 -> ctrb0505-A:TO220ABGDS-INV_COUCHE_1
- ZT7: footprint ctrb0505-A1_clean.PcbLib:ZT7 -> ctrb0505-A:TO220ABGDS-INV_COUCHE_1
- moved C28 235.8 mm to (268.0, 54.1)
- moved C29 235.8 mm to (268.0, 41.1)
- moved J1 235.8 mm to (261.5, 54.3)
- moved C3 235.8 mm to (299.2, 58.7)
- moved D24 235.8 mm to (285.9, 63.1)
- moved FI1 235.8 mm to (249.1, 60.6)
- moved IC6 235.8 mm to (292.9, 44.7), turned to 0 degrees
- moved MIR1 235.8 mm to (244.0, 37.1)
- moved R11 235.8 mm to (267.5, 94.9)
- moved R12 235.8 mm to (279.5, 94.9)
- moved R13 235.8 mm to (291.6, 94.9)
- moved R40 235.8 mm to (305.6, 72.6)
- moved R7 235.8 mm to (329.7, 72.6)
- moved T10 235.8 mm to (282.1, 63.1)
- moved C10 235.8 mm to (271.9, 98.0)
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Connections:
- net BRAKE/ renamed BRAKE_
- net FAULT/ renamed FAULT_
Other:
- net class All Nets removed
- rule pad_to_mask_clearance: 0.05 -> 0.051
- board text removed: "(1)Fabrique suivant IPC A610 classe III. (1)Manufactured according to IPC A610 class III."
- board text removed: "0,3"
- board text removed: "0,8"
- board text removed: "0,9"
- board text removed: "0,95"
- board text removed: "1,2"
- board text removed: "1,4"
- board text removed: "3,5"
- board text removed: "35u"
- board text removed: "A"
- board text removed: "ATTENTION: Le circuit imprime doit etre UL94V-0. (2)Le fabricant doit etre reconnu UL et doit apposer le marquage correspondant."
- board text removed: "BLANCHE"
- board text removed: "Cote de pliage des TO220"
- board text removed: "Dimension folding of TO220"
- board text removed: "Fabrique suivant IPC A610 classe III. Manufactured according to IPC A610 class III."
- board text removed: "NOTA: C2 et C27 sont montes en double implantation.r Two assemblies possible for C2 and C27"
- board text removed: "NOTA: T2 a T7 montes en double implantation. r Plaquer les composants T2 a T7 r lorsqu'ils sont montes en boitier TO220 afin d'obtenir une coplaneite optimum."
- board text removed: "T2"
- board text removed: "T7"
- board text removed: "The printed circuit board must be UL94V-0 (2) The manufacturer must be recognized UL and must affix corresponding marking."
- board text removed: "Toutes les dimensions sonr en millimetres. All the dimensions are in millimeter."
- board text removed: "Two assemblies possible from T2 to T7.r To plate the T2 components in T7 r when they are assembled out of caseTO220 r in order to obtain an optimum co planarity."
- board text removed: "VERT"
- board text removed: "X"
- board text removed: "YES"

Commit message: remove unused text items
Parts:
- removed the ? at (295.2, 54.0) (x2)
- removed the ? at (311.4, 46.7)
- removed the ? at (285.3, 75.5)
- removed the ? at (280.2, 75.5)
- removed the ? at (282.7, 75.5)
- removed the ? at (280.2, 84.4)
- removed the ? at (285.3, 84.4)
- removed the ? at (282.7, 84.4)
- removed the ? at (273.2, 75.5)
- removed the ? at (268.1, 75.5)
- removed the ? at (270.7, 75.5)
- removed the ? at (268.1, 84.4)
- removed the ? at (329.5, 74.8)
- removed the ? at (273.2, 84.4)
- removed the ? at (270.7, 84.4)
- removed the ? at (250.5, 43.4)
- removed the ? at (325.1, 43.4)
- removed the ? at (325.1, 97.6)
- removed the ? at (250.5, 97.6)
- removed the ? at (314.0, 69.1)
- removed the ? at (314.0, 66.6)
- removed the ? at (314.0, 64.0)
- removed the ? at (314.0, 61.5)
- removed the ? at (324.6, 86.4)
- removed the ? at (314.0, 59.0)
- removed the ? at (314.0, 56.4)
- removed the ? at (314.0, 53.9)
- removed the ? at (314.0, 51.3)
- removed the ? at (314.0, 48.8)
- removed the ? at (249.5, 51.3)
- removed the ? at (244.0, 51.3)
- removed the ? at (261.5, 68.2)
- removed the ? at (261.5, 70.7)
- removed the ? at (261.5, 73.3)
- removed the ? at (324.6, 80.2)
- removed the ? at (261.5, 75.8)
- removed the ? at (261.5, 78.3)
- removed the ? at (261.5, 80.9)
- removed the ? at (261.5, 83.4)
- removed the ? at (261.5, 86.0)
- removed the ? at (261.5, 88.5)
- removed the ? at (261.5, 91.0)
- removed the ? at (304.8, 41.2)
- removed the ? at (304.8, 38.6)
- removed the ? at (307.3, 41.2)
- removed the ? at (314.7, 85.3)
- removed the ? at (307.3, 38.6)
- removed the ? at (309.9, 41.2)
- removed the ? at (309.9, 38.6)
- removed the ? at (312.4, 41.2)
- removed the ? at (312.4, 38.6)
- removed the ? at (315.0, 41.2)
- removed the ? at (315.0, 38.6)
- removed the ? at (246.6, 58.1)
- removed the ? at (254.1, 60.6)
- removed the ? at (249.1, 60.6)
- removed the ? at (314.7, 84.1)
- removed the ? at (246.6, 63.1)
- removed the ? at (251.6, 63.1)
- removed the ? at (251.6, 58.1)
- removed the ? at (305.9, 51.3)
- removed the ? at (305.9, 56.4)
- removed the ? at (298.4, 41.1)
- removed the ? at (268.0, 41.1)
- removed the ? at (298.4, 54.1)
- removed the ? at (268.0, 54.1)
- removed the ? at (305.9, 62.1)
- removed the ? at (314.7, 82.8)
- removed the ? at (305.9, 67.2)
- removed the ? at (94.6, 130.1)
- removed the ? at (94.6, 145.3)
- removed the ? at (94.6, 140.2)
- removed the ? at (94.6, 135.2)
- removed the ? at (94.6, 125.0)
- removed the ? at (94.6, 119.9)
- removed the ? at (94.6, 114.8)
- removed the ? at (310.7, 85.5)
- removed the ? at (299.6, 96.3)
- removed the ? at (287.5, 96.3)
- removed the ? at (291.7, 54.5) (x2)
- removed the ? at (274.9, 90.1)
- removed the ? at (307.2, 86.8)
- removed the ? at (307.2, 84.4)
- removed the ? at (307.2, 81.8)
- removed the ? at (305.0, 44.0)
- removed the ? at (310.2, 48.5)
- removed the ? at (319.2, 44.1)
- removed the ? at (317.3, 44.1)
- removed the ? at (315.4, 44.1)
- removed the ? at (258.6, 52.1)
- removed the ? at (290.6, 71.2) (x2)
- removed the ? at (306.8, 48.2)
- removed the ? at (331.9, 36.6)
- removed the ? at (296.1, 38.3)
- removed the ? at (294.5, 38.3)
- removed the ? at (292.9, 38.3)
- removed the ? at (291.3, 38.3)
- removed the ? at (289.7, 38.3)
- removed the ? at (288.1, 38.3)
- removed the ? at (288.1, 39.9)
- removed the ? at (288.1, 41.5)
- removed the ? at (278.8, 71.2) (x2)
- removed the ? at (288.1, 43.1)
- removed the ? at (309.4, 43.9)
- removed the ? at (303.0, 44.1)
- removed the ? at (288.1, 44.7)
- removed the ? at (311.4, 45.2)
- removed the ? at (288.1, 46.3)
- removed the ? at (297.3, 46.7)
- removed the ? at (317.3, 48.0)
- removed the ? at (308.6, 48.5)
- removed the ? at (266.7, 71.2) (x2)
- removed the ? at (308.7, 68.2)
- removed the ? at (309.3, 69.1)
- removed the ? at (310.3, 70.1)
- removed the ? at (331.7, 72.6)
- removed the ? at (319.0, 73.9)
- removed the ? at (306.7, 74.7)
- removed the ? at (329.3, 77.1)
- removed the ? at (306.2, 77.5)
- removed the ? at (319.0, 79.0)
- removed the ? at (266.2, 51.9) (x2)
- removed the ? at (314.7, 79.0)
- removed the ? at (309.0, 80.2)
- removed the ? at (301.6, 79.9)
- removed the ? at (317.0, 80.7)
- removed the ? at (329.3, 81.2)
- removed the ? at (315.8, 82.0)
- removed the ? at (321.0, 84.1)
- removed the ? at (320.2, 85.3)
- removed the ? at (318.2, 86.6)
- removed the ? at (315.9, 86.6)
- removed the ? at (293.1, 86.0)
- removed the ? at (329.3, 87.3)
- removed the ? at (320.9, 87.9)
- removed the ? at (320.9, 89.2)
- removed the ? at (299.0, 90.1)
- removed the ? at (309.0, 91.0)
- removed the ? at (320.4, 91.6)
- removed the ? at (307.9, 92.4)
- removed the ? at (307.9, 94.1)
- removed the ? at (307.2, 96.3)
- removed the ? at (275.5, 96.3)
- removed the ? at (281.1, 86.0)
- removed the ? at (317.1, 97.2)
- removed the ? at (300.2, 99.6)
- removed the ? at (288.1, 100.4)
- removed the ? at (276.4, 103.5)
- removed the ? at (288.9, 89.8)
- removed the ? at (287.0, 90.1)
- removed the ? at (276.8, 89.7)
- removed the ? at (265.3, 89.4)
- removed the ? at (269.0, 86.0)
- removed the ? at (266.8, 56.5)
- removed the ? at (277.6, 56.5)
- removed the ? at (297.3, 75.5)
- removed the ? at (292.2, 75.5)
- removed the ? at (294.8, 75.5)
- removed the ? at (292.2, 84.4)
- removed the ? at (297.3, 84.4)
- removed the ? at (294.8, 84.4)
- added ?: , , F.Cu at (295.2, 54.0)
- added ?: , , F.Cu at (291.7, 54.5)
- added ?: , , F.Cu at (290.6, 71.2)
- added ?: , , F.Cu at (278.8, 71.2)
- added ?: , , F.Cu at (266.7, 71.2)
- added ?: , , F.Cu at (266.2, 51.9)

Commit message: add holes as fprint
Parts:
- removed the ? at (295.2, 54.0)
- removed the ? at (291.7, 54.5)
- removed the ? at (290.6, 71.2)
- removed the ? at (278.8, 71.2)
- removed the ? at (266.7, 71.2)
- removed the ? at (266.2, 51.9)
- added ?: , ctrb0505-A:ThroughHole_36milx12mil_Pad_Cu_Mask, F.Cu at (295.2, 54.0)
- added ?: , ctrb0505-A:ThroughHole_36milx12mil_Pad_Cu_Mask, F.Cu at (291.7, 54.5)
- added ?: , ctrb0505-A:ThroughHole_36milx12mil_Pad_Cu_Mask, F.Cu at (290.6, 71.2)
- added ?: , ctrb0505-A:ThroughHole_36milx12mil_Pad_Cu_Mask, F.Cu at (278.8, 71.2)
- added ?: , ctrb0505-A:ThroughHole_36milx12mil_Pad_Cu_Mask, F.Cu at (266.7, 71.2)
- added ?: , ctrb0505-A:ThroughHole_36milx12mil_Pad_Cu_Mask, F.Cu at (266.2, 51.9)
Changed lines of the file:
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@@
     )
   )
-  (module "" (layer F.Cu)
+  (module ctrb0505-A:ThroughHole_36milx12mil_Pad_Cu_Mask (layer F.Cu)
     (at 295.191 54.0104)
     (fp_text reference "" (at 0 0) (layer F.SilkS)
@@
       (net 26 +24V))
   )
-  (module "" (layer F.Cu)
+  (module ctrb0505-A:ThroughHole_36milx12mil_Pad_Cu_Mask (layer F.Cu)
     (at 291.7366 54.5184)
     (fp_text reference "" (at 0 0) (layer F.SilkS)
@@
       (net 52 +15V))
   )
-  (module "" (layer F.Cu)
+  (module ctrb0505-A:ThroughHole_36milx12mil_Pad_Cu_Mask (layer F.Cu)
     (at 290.5936 71.1554)
     (fp_text reference "" (at 0 0) (layer F.SilkS)
@@
       (net 70 ISENS))
   )
-  (module "" (layer F.Cu)
+  (module ctrb0505-A:ThroughHole_36milx12mil_Pad_Cu_Mask (layer F.Cu)
     (at 278.7826 71.1554)
     (fp_text reference "" (at 0 0) (layer F.SilkS)
@@
       (net 70 ISENS))
   )
-  (module "" (layer F.Cu)
+  (module ctrb0505-A:ThroughHole_36milx12mil_Pad_Cu_Mask (layer F.Cu)
     (at 266.7176 71.1554)
     (fp_text reference "" (at 0 0) (layer F.SilkS)
@@
       (net 70 ISENS))
   )
-  (module "" (layer F.Cu)
+  (module ctrb0505-A:ThroughHole_36milx12mil_Pad_Cu_Mask (layer F.Cu)
     (at 266.2096 51.8514)
     (fp_text reference "" (at 0 0) (layer F.SilkS)
