File: 10096315 Blower Driver/ctrb0505-A.sch (KiCad schematic (older format))
At the start: 139 parts, among them IC1 MotorDriver, IC2 NE555D, IC3 IR2118S, IC4 IR2118S, IC5 IR2118S, IC6 LinearRegulator, J1 2pinConnector_Power, J11 DNP, J2 10pinConnector, J22 DNP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

Commit message: Blower: fields corrections on schematics
Parts:
- C2: Item Number 10022506 -> 10022506_TH
- C27: Description CAPACITOR,470UF, +/-20%,25V -> CAPACITOR,470UF, +/-20%,25V TH; Item Number 10095969 -> 10095969_TH; Manufacturer2 NICHICON_RMS1 -> (none); Manufacturer_No EEEFK1E471P -> ECA1EHG471; Manufacturer_No2 UCD1E471MNL1GS -> (none)
- TH3, TH4: value MountingHole -> ThroughHole
Changed lines of the file:
@@
 F 2 "AllModules:MOL5566-2_1" H 1400 2600 50  0001 C CNN
 F 3 "https://www.molex.com/pdm_docs/sd/039281023_sd.pdf" H 1400 2600 50  0001 C CNN
-F 4 "0039281023" H 1400 2600 50  0001 C CNN "Manufacturer_No"
-F 5 " CONN HEADER VERT 2 CONTACTS Mini Fit Jr  5.5PIN PITCH" H 1400 2600 50  0001 C CNN "Description"
-F 6 "MOLEX" H 1400 2600 50  0001 C CNN "Manufacturer"
+F 4 " CONN HEADER VERT 2 CONTACTS Mini Fit Jr  5.5PIN PITCH" H 1400 2600 50  0001 C CNN "Description"
+F 5 "MOLEX" H 1400 2600 50  0001 C CNN "Manufacturer"
+F 6 "0039281023" H 1400 2600 50  0001 C CNN "Manufacturer_No"
 	1    1400 2600
 	1    0    0    -1
@@
 F 1 "DNP" H 11150 2850 50  0001 C CNN
 F 2 "AllModules:03515_1" H 11200 1950 50  0001 C CNN
-F 3 "" H 11150 2850 50  0001 C CNN
-F 4 "CAPACITOR,470UF, +/-20%,25V" H 11150 2400 50  0001 C CNN "Description"
-F 5 "10095969" H 11150 2400 50  0001 C CNN "Item Number"
+F 3 "https://industrial.panasonic.com/ww/products/capacitors/aluminum-capacitors/aluminum-cap-lead/models/ECA1EHG471B" H 11150 2850 50  0001 C CNN
+F 4 "CAPACITOR,470UF, +/-20%,25V TH" H 11150 2400 50  0001 C CNN "Description"
+F 5 "10095969_TH" H 11150 2400 50  0001 C CNN "Item Number"
 F 6 "PANASONIC_RMS1" H 11150 2400 50  0001 C CNN "Manufacturer"
-F 7 "EEEFK1E471P" H 11150 2400 50  0001 C CNN "Manufacturer_No"
-F 8 "NICHICON_RMS1" H 0   0   50  0001 C CNN "Manufacturer2"
-F 9 "UCD1E471MNL1GS" H 0   0   50  0001 C CNN "Manufacturer_No2"
+F 7 "ECA1EHG471" H 11150 2400 50  0001 C CNN "Manufacturer_No"
 	1    11150 2400
 	1    0    0    -1
@@
 F 1 "470uF" H 11375 2325 50  0000 C CNN
 F 2 "AllModules:C-SC10_1" H 11200 1950 50  0001 C CNN
-F 3 "" H 11150 2850 50  0001 C CNN
-F 4 "EEEFK1E471P" H 11150 2400 50  0001 C CNN "Manufacturer_No"
-F 5 "CAPACITOR,470UF, +/-20%,25V" H 11150 2400 50  0001 C CNN "Description"
-F 6 "10095969" H 11150 2400 50  0001 C CNN "Item Number"
-F 7 "PANASONIC_RMS1" H 11150 2400 50  0001 C CNN "Manufacturer"
+F 3 "https://www.nichicon.co.jp/english/products/pdfs/e-ucd.pdf" H 11150 2850 50  0001 C CNN
+F 4 "CAPACITOR,470UF, +/-20%,25V" H 11150 2400 50  0001 C CNN "Description"
+F 5 "10095969" H 11150 2400 50  0001 C CNN "Item Number"
+F 6 "PANASONIC_RMS1" H 11150 2400 50  0001 C CNN "Manufacturer"
+F 7 "EEEFK1E471P" H 11150 2400 50  0001 C CNN "Manufacturer_No"
 F 8 "NICHICON_RMS1" H 0   0   50  0001 C CNN "Manufacturer2"
 F 9 "UCD1E471MNL1GS" H 0   0   50  0001 C CNN "Manufacturer_No2"
@@
 F 1 "DNP" H 19225 5150 50  0001 C CNN
 F 2 "AllModules:TO220ABGDS-INV_COUCHE_1" H 19275 4000 50  0001 C CNN
-F 3 "https://www.vishay.com/docs/91406/sihfz24.pdf" H 19225 5050 50  0001 C CNN
+F 3 "http://www.vishay.com/docs/91406/sihfz24.pdf" H 19225 5050 50  0001 C CNN
 F 4 "TRANSISTOR MOSFET, 60V, 16.7A,  N CHANNEL" H 19225 4650 50  0001 C CNN "Description"
 F 5 "10022559_TH" H 19225 4650 50  0001 C CNN "Item Number"
@@
 F 1 "DNP" H 19225 7350 50  0001 C CNN
 F 2 "AllModules:TO220ABGDS-INV_COUCHE_1" H 19275 6200 50  0001 C CNN
-F 3 "https://www.vishay.com/docs/91406/sihfz24.pdf" H 19225 7250 50  0001 C CNN
+F 3 "http://www.vishay.com/docs/91406/sihfz24.pdf" H 19225 7250 50  0001 C CNN
 F 4 "TRANSISTOR MOSFET, 60V, 16.7A,  N CHANNEL" H 19225 6850 50  0001 C CNN "Description"
 F 5 "10022559_TH" H 19225 6850 50  0001 C CNN "Item Number"
@@
 F 2 "AllModules:03515_1" H 8850 1950 50  0001 C CNN
 F 3 "" H 8800 2850 50  0001 C CNN
-F 4 "10022506" H 8800 2400 50  0001 C CNN "Item Number"
+F 4 "10022506_TH" H 8800 2400 50  0001 C CNN "Item Number"
 F 5 "NICHICON_RMS1" H 8800 2400 50  0001 C CNN "Manufacturer"
 F 6 "URZ1H101MPD" H 8800 2400 50  0001 C CNN "Manufacturer_No"
@@
 F 2 "AllModules:ThroughHole_36milx12mil_Pad_Cu_Mask" H 1000 6500 50  0001 C CNN
 F 3 "~" H 1000 6500 50  0001 C CNN
+F 4 "" H 1000 6500 50  0001 C CNN "Manufacturer"
 	1    1000 6500
 	1    0    0    -1
@@
 F 2 "AllModules:ThroughHole_36milx12mil_Pad_Cu_Mask" H 1000 7000 50  0001 C CNN
 F 3 "~" H 1000 7000 50  0001 C CNN
+F 4 "" H 1000 7000 50  0001 C CNN "Manufacturer"
 	1    1000 7000
 	1    0    0    -1
@@
 P 2000 6500
 F 0 "TH3" H 2100 6546 50  0000 L CNN
-F 1 "MountingHole" H 2100 6455 50  0000 L CNN
+F 1 "ThroughHole" H 2100 6455 50  0000 L CNN
 F 2 "AllModules:ThroughHole_36milx12mil_Pad_Cu_Mask" H 2000 6500 50  0001 C CNN
 F 3 "~" H 2000 6500 50  0001 C CNN
+F 4 "" H 2000 6500 50  0001 C CNN "Manufacturer"
 	1    2000 6500
 	1    0    0    -1
@@
 P 2000 7000
 F 0 "TH4" H 2100 7046 50  0000 L CNN
-F 1 "MountingHole" H 2100 6955 50  0000 L CNN
+F 1 "ThroughHole" H 2100 6955 50  0000 L CNN
 F 2 "AllModules:ThroughHole_36milx12mil_Pad_Cu_Mask" H 2000 7000 50  0001 C CNN
 F 3 "~" H 2000 7000 50  0001 C CNN
+F 4 "" H 2000 7000 50  0001 C CNN "Manufacturer"
 	1    2000 7000
 	1    0    0    -1
@@
 F 2 "AllModules:ThroughHole_36milx12mil_Pad_Cu_Mask" H 3000 6500 50  0001 C CNN
 F 3 "~" H 3000 6500 50  0001 C CNN
+F 4 "" H 3000 6500 50  0001 C CNN "Manufacturer"
 	1    3000 6500
 	1    0    0    -1
@@
 F 2 "AllModules:ThroughHole_36milx12mil_Pad_Cu_Mask" H 3000 7000 50  0001 C CNN
 F 3 "~" H 3000 7000 50  0001 C CNN
+F 4 "" H 3000 7000 50  0001 C CNN "Manufacturer"
 	1    3000 7000
 	1    0    0    -1

Commit message: Blower project update based on new layout and update lib
Parts:
- removed TH1, TH2, TH3, TH4, TH5, TH6: ThroughHole, AllModules:ThroughHole_36milx12mil_Pad_Cu_Mask, symbol V_Mechanical:MountingHole
- C1, C12, C15, C18, C19, C21, C24, C25, C26, C3, C5, C6, C9: footprint AllModules:C0805_1 -> AllModules:C0805
- C10, C13, C16, R58, R59, R60: footprint AllModules:RC1206_1 -> AllModules:RC1206
- C11, C14, C17, C20, C7, C8, FI3, FI4, FI5, FI6, FI7, FI8, FI9: footprint AllModules:C0603_1 -> AllModules:C0603
- C2, C27: footprint AllModules:03515_1 -> AllModules:03515_10111101
- C22, C23: footprint AllModules:C0612-4_1 -> AllModules:C0612-4
- C28: footprint AllModules:HT-13X27_1 -> AllModules:HT-13X27_10111011
- C29: footprint AllModules:HT-13X27_1 -> AllModules:HT-13X27_10011011
- C4: footprint AllModules:C7343_1 -> AllModules:C7343
- D1, D18, D19, D20, D21, D22, D23: footprint AllModules:SMB_1 -> AllModules:SMB
- D10, D8, D9: footprint AllModules:SMA_1 -> AllModules:SMA
- D11, D12, D13: footprint AllModules:SOD80_1 -> AllModules:SOD80
- D14, D15, D16, D24: footprint AllModules:SOT23-1G_1 -> AllModules:SOT23-1G
- D17: footprint AllModules:DPAK-2ANODES_1 -> AllModules:DPAK-2ANODES
- D2, D3, D4, D5, D6, D7: footprint AllModules:SOD323_1 -> AllModules:SOD323
- F1: footprint AllModules:FU154000_1 -> AllModules:FU154000
- FI1: footprint AllModules:BNX002_1 -> AllModules:BNX002_101110011011101110111011
- IC1: footprint AllModules:MX.A24_COMPOSANT_1 -> AllModules:MX.A24_COMPOSANT
- IC2, IC3, IC4, IC5: footprint AllModules:MX.A8_COMPOSANT_1 -> AllModules:MX.A8_COMPOSANT
- IC6: footprint AllModules:DPAK_1b -> AllModules:DPAK
- J1: footprint AllModules:MOL43650-02C_1 -> AllModules:MOL43650-02C
- J11: footprint AllModules:MOL5566-2_1 -> AllModules:MOL5566-2_10111011
- J2: footprint AllModules:BP2X5D_1 -> AllModules:BP2X5D_1101100110111011101110011001100110111011
- J22: footprint AllModules:MOL7395-9_1 -> AllModules:MOL7395-9_110110011001100110011001100110011011
- J3: footprint AllModules:MOL7395-2_1 -> AllModules:MOL7395-2_10011001
- J4: footprint AllModules:JUMPER2_NoCopper_1 -> AllModules:JUMPER2_NoCopper
- J6: footprint AllModules:MOL7395-8_1 -> AllModules:MOL7395-8_10111011101110111101101110111011
- L1: footprint AllModules:ELC09DxxxxF_NoCopper_1 -> AllModules:ELC09DxxxxF_NoCopper
- MIR1, MIR2, MIR3, MIR4: footprint AllModules:MIRECMS-SAFT_1 -> AllModules:MIRECMS-SAFT
- NT1: footprint AllModules:C12000_0 -> AllModules:NetTie-2_SMD_Pad_2.5x5mm
- PT1: footprint AllModules:C12000_1 -> AllModules:C12000
- R1, R40: footprint AllModules:R2512_1 -> AllModules:R2512
- R10, R11, R12, R13, R2, R20, R3, R30, R31, R32, R33, R35, R37, R38, R39, R4, R41, R42, R5, R50, R6, R7, R8, R9: footprint AllModules:R0603_1 -> AllModules:R0603
- T1, T10, T8: footprint AllModules:SOT23-GSD_1 -> AllModules:SOT23-GSD
- T2, T3, T4, T5, T6, T7, T9: footprint AllModules:DPAK-GDS_1 -> AllModules:DPAK-GDS
- ZC2: footprint AllModules:C-SC8_1 -> AllModules:C-SC8
- ZC27: footprint AllModules:C-SC10_1 -> AllModules:C-SC10
- ZM1, ZM2, ZM3, ZM4: footprint AllModules:FIX35M_1 -> AllModules:FIX35M_1101
- ZT2, ZT4, ZT6: footprint AllModules:TO220ABGDS-INV_COUCHE_1 -> AllModules:TO220ABGDS-INV_COUCHE_101110011001
- ZT3, ZT5, ZT7: footprint AllModules:TO220ABGDS-INV_COUCHE_1 -> AllModules:TO220ABGDS-INV_COUCHE_101110011011
Connections:
- net GND: now reaches C2.-, C27.-, C3.1, C5.1, IC6.2 (GND), ZC2.-, ZC27.-
- net N9: now reaches D17.A1, D17.A2, T9.D
- net GND-PUIS: now reaches D1.1, D24.1, FI1.CG1 (e), FI1.CG2, FI1.CG3, J4.2, T10.S

Commit message: Blower: revert blower project modifications only keep shared lib modifications in this branch
Parts:
- added TH1, TH2, TH3, TH4, TH5, TH6: ThroughHole, AllModules:ThroughHole_36milx12mil_Pad_Cu_Mask, symbol V_Mechanical:MountingHole
- C1, C12, C15, C18, C19, C21, C24, C25, C26, C3, C5, C6, C9: footprint AllModules:C0805 -> AllModules:C0805_1
- C10, C13, C16, R58, R59, R60: footprint AllModules:RC1206 -> AllModules:RC1206_1
- C11, C14, C17, C20, C7, C8, FI3, FI4, FI5, FI6, FI7, FI8, FI9: footprint AllModules:C0603 -> AllModules:C0603_1
- C2, C27: footprint AllModules:03515_10111101 -> AllModules:03515_1
- C22, C23: footprint AllModules:C0612-4 -> AllModules:C0612-4_1
- C28: footprint AllModules:HT-13X27_10111011 -> AllModules:HT-13X27_1
- C29: footprint AllModules:HT-13X27_10011011 -> AllModules:HT-13X27_1
- C4: footprint AllModules:C7343 -> AllModules:C7343_1
- D1, D18, D19, D20, D21, D22, D23: footprint AllModules:SMB -> AllModules:SMB_1
- D10, D8, D9: footprint AllModules:SMA -> AllModules:SMA_1
- D11, D12, D13: footprint AllModules:SOD80 -> AllModules:SOD80_1
- D14, D15, D16, D24: footprint AllModules:SOT23-1G -> AllModules:SOT23-1G_1
- D17: footprint AllModules:DPAK-2ANODES -> AllModules:DPAK-2ANODES_1
- D2, D3, D4, D5, D6, D7: footprint AllModules:SOD323 -> AllModules:SOD323_1
- F1: footprint AllModules:FU154000 -> AllModules:FU154000_1
- FI1: footprint AllModules:BNX002_101110011011101110111011 -> AllModules:BNX002_1
- IC1: footprint AllModules:MX.A24_COMPOSANT -> AllModules:MX.A24_COMPOSANT_1
- IC2, IC3, IC4, IC5: footprint AllModules:MX.A8_COMPOSANT -> AllModules:MX.A8_COMPOSANT_1
- IC6: footprint AllModules:DPAK -> AllModules:DPAK_1b
- J1: footprint AllModules:MOL43650-02C -> AllModules:MOL43650-02C_1
- J11: footprint AllModules:MOL5566-2_10111011 -> AllModules:MOL5566-2_1
- J2: footprint AllModules:BP2X5D_1101100110111011101110011001100110111011 -> AllModules:BP2X5D_1
- J22: footprint AllModules:MOL7395-9_110110011001100110011001100110011011 -> AllModules:MOL7395-9_1
- J3: footprint AllModules:MOL7395-2_10011001 -> AllModules:MOL7395-2_1
- J4: footprint AllModules:JUMPER2_NoCopper -> AllModules:JUMPER2_NoCopper_1
- J6: footprint AllModules:MOL7395-8_10111011101110111101101110111011 -> AllModules:MOL7395-8_1
- L1: footprint AllModules:ELC09DxxxxF_NoCopper -> AllModules:ELC09DxxxxF_NoCopper_1
- MIR1, MIR2, MIR3, MIR4: footprint AllModules:MIRECMS-SAFT -> AllModules:MIRECMS-SAFT_1
- NT1: footprint AllModules:NetTie-2_SMD_Pad_2.5x5mm -> AllModules:C12000_0
- PT1: footprint AllModules:C12000 -> AllModules:C12000_1
- R1, R40: footprint AllModules:R2512 -> AllModules:R2512_1
- R10, R11, R12, R13, R2, R20, R3, R30, R31, R32, R33, R35, R37, R38, R39, R4, R41, R42, R5, R50, R6, R7, R8, R9: footprint AllModules:R0603 -> AllModules:R0603_1
- T1, T10, T8: footprint AllModules:SOT23-GSD -> AllModules:SOT23-GSD_1
- T2, T3, T4, T5, T6, T7, T9: footprint AllModules:DPAK-GDS -> AllModules:DPAK-GDS_1
- ZC2: footprint AllModules:C-SC8 -> AllModules:C-SC8_1
- ZC27: footprint AllModules:C-SC10 -> AllModules:C-SC10_1
- ZM1, ZM2, ZM3, ZM4: footprint AllModules:FIX35M_1101 -> AllModules:FIX35M_1
- ZT2, ZT4, ZT6: footprint AllModules:TO220ABGDS-INV_COUCHE_101110011001 -> AllModules:TO220ABGDS-INV_COUCHE_1
- ZT3, ZT5, ZT7: footprint AllModules:TO220ABGDS-INV_COUCHE_101110011011 -> AllModules:TO220ABGDS-INV_COUCHE_1
Connections:
- net GND: no longer names the net of C2.-, C27.-, C3.1, C5.1, IC6.2 (GND), ZC2.-, ZC27.-
- net GND-PUIS: no longer names the net of D1.1, D24.1, FI1.CG1 (e), FI1.CG2, FI1.CG3, J4.2, T10.S
- net N9: no longer names the net of D17.A1, D17.A2, T9.D

Commit message: Bllower schematic updated with diodes A and K convention, name of Net 9 GND-PUIS and GND added
Parts:
- C1, C12, C15, C18, C19, C21, C24, C25, C26, C3, C5, C6, C9: footprint AllModules:C0805_1 -> save10096315 Blower Driver:C0805
- C10, C13, C16, R58, R59, R60: footprint AllModules:RC1206_1 -> save10096315 Blower Driver:RC1206
- C11, C14, C17, C20, C7, C8, FI3, FI4, FI5, FI6, FI7, FI8, FI9: footprint AllModules:C0603_1 -> save10096315 Blower Driver:C0603
- C2, C27: footprint AllModules:03515_1 -> save10096315 Blower Driver:03515
- C22, C23: footprint AllModules:C0612-4_1 -> save10096315 Blower Driver:C0612-4
- C28, C29: footprint AllModules:HT-13X27_1 -> save10096315 Blower Driver:HT-13X27
- C4: footprint AllModules:C7343_1 -> save10096315 Blower Driver:C7343
- D1, D18, D19, D20, D21, D22, D23: footprint AllModules:SMB_1 -> save10096315 Blower Driver:SMB
- D10, D8, D9: footprint AllModules:SMA_1 -> save10096315 Blower Driver:SMA
- D11, D12, D13: footprint AllModules:SOD80_1 -> save10096315 Blower Driver:SOD80
- D14, D15, D16, D24: footprint AllModules:SOT23-1G_1 -> save10096315 Blower Driver:SOT23-1G
- D17: footprint AllModules:DPAK-2ANODES_1 -> save10096315 Blower Driver:DPAK-2ANODES
- D2, D3, D4, D5, D6, D7: footprint AllModules:SOD323_1 -> save10096315 Blower Driver:SOD323
- F1: footprint AllModules:FU154000_1 -> save10096315 Blower Driver:FU154000
- FI1: footprint AllModules:BNX002_1 -> save10096315 Blower Driver:BNX002
- IC1: footprint AllModules:MX.A24_COMPOSANT_1 -> save10096315 Blower Driver:MX.A24_COMPOSANT
- IC2, IC3, IC4, IC5: footprint AllModules:MX.A8_COMPOSANT_1 -> save10096315 Blower Driver:MX.A8_COMPOSANT
- IC6: footprint AllModules:DPAK_1b -> save10096315 Blower Driver:DPAK
- J1: footprint AllModules:MOL43650-02C_1 -> save10096315 Blower Driver:MOL43650-02C
- J11: footprint AllModules:MOL5566-2_1 -> save10096315 Blower Driver:MOL5566-2
- J2: footprint AllModules:BP2X5D_1 -> save10096315 Blower Driver:BP2X5D
- J22: footprint AllModules:MOL7395-9_1 -> save10096315 Blower Driver:MOL7395-9
- J3: footprint AllModules:MOL7395-2_1 -> save10096315 Blower Driver:MOL7395-2
- J6: footprint AllModules:MOL7395-8_1 -> save10096315 Blower Driver:MOL7395-8
- MIR1, MIR2, MIR3, MIR4: footprint AllModules:MIRECMS-SAFT_1 -> save10096315 Blower Driver:MIRECMS-SAFT
- PT1: footprint AllModules:C12000_1 -> save10096315 Blower Driver:C12000
- R1, R40: footprint AllModules:R2512_1 -> save10096315 Blower Driver:R2512
- R10, R11, R12, R13, R2, R20, R3, R30, R31, R32, R33, R35, R37, R38, R39, R4, R41, R42, R5, R50, R6, R7, R8, R9: footprint AllModules:R0603_1 -> save10096315 Blower Driver:R0603
- T1, T10, T8: footprint AllModules:SOT23-GSD_1 -> save10096315 Blower Driver:SOT23-GSD
- T2, T3, T4, T5, T6, T7, T9: footprint AllModules:DPAK-GDS_1 -> save10096315 Blower Driver:DPAK-GDS
- ZC2: footprint AllModules:C-SC8_1 -> save10096315 Blower Driver:C-SC8
- ZC27: footprint AllModules:C-SC10_1 -> save10096315 Blower Driver:C-SC10
- ZM1, ZM2, ZM3, ZM4: footprint AllModules:FIX35M_1 -> save10096315 Blower Driver:FIX35M
- ZT2, ZT3, ZT4, ZT5, ZT6, ZT7: footprint AllModules:TO220ABGDS-INV_COUCHE_1 -> save10096315 Blower Driver:TO220ABGDS-INV_COUCHE
Connections:
- net GND: now reaches C2.-, C27.-, C3.1, C5.1, IC6.2 (GND), ZC2.-, ZC27.-
- net N9: now reaches D17.A1, D17.A2, T9.D
- net GND-PUIS: now reaches D1.1, D24.1, FI1.CG1 (e), FI1.CG2, FI1.CG3, J4.2, T10.S

Commit message: Blower schematic: vias added on a second page
Parts:
- removed TH1, TH2, TH3, TH4, TH5, TH6: ThroughHole, AllModules:ThroughHole_36milx12mil_Pad_Cu_Mask, symbol V_Mechanical:MountingHole
- ZM1, ZM2, ZM3, ZM4: footprint save10096315 Blower Driver:FIX35M -> AllModules:FIX35M
Changed lines of the file:
@@
 $Descr A2 23386 16535
 encoding utf-8
-Sheet 1 1
+Sheet 1 2
 Title ""
 Date ""
@@
 F 0 "ZM4" H 4100 6599 50  0000 L CNN
 F 1 "MountingHole_Pad" H 4100 6508 50  0000 L CNN
-F 2 "save10096315 Blower Driver:FIX35M" H 4000 6550 50  0001 C CNN
+F 2 "AllModules:FIX35M" H 4000 6550 50  0001 C CNN
 F 3 "~" H 4000 6550 50  0001 C CNN
 	1    4000 6550
@@
 F 0 "ZM3" H 5100 6599 50  0000 L CNN
 F 1 "MountingHole_Pad" H 5100 6508 50  0000 L CNN
-F 2 "save10096315 Blower Driver:FIX35M" H 5000 6550 50  0001 C CNN
+F 2 "AllModules:FIX35M" H 5000 6550 50  0001 C CNN
 F 3 "~" H 5000 6550 50  0001 C CNN
 	1    5000 6550
@@
 F 0 "ZM1" H 4100 7099 50  0000 L CNN
 F 1 "MountingHole_Pad" H 4100 7008 50  0000 L CNN
-F 2 "save10096315 Blower Driver:FIX35M" H 4000 7050 50  0001 C CNN
+F 2 "AllModules:FIX35M" H 4000 7050 50  0001 C CNN
 F 3 "~" H 4000 7050 50  0001 C CNN
 	1    4000 7050
@@
 F 0 "ZM2" H 5100 7099 50  0000 L CNN
 F 1 "MountingHole_Pad" H 5100 7008 50  0000 L CNN
-F 2 "save10096315 Blower Driver:FIX35M" H 5000 7050 50  0001 C CNN
+F 2 "AllModules:FIX35M" H 5000 7050 50  0001 C CNN
 F 3 "~" H 5000 7050 50  0001 C CNN
 	1    5000 7050
@@
 	1    0    0    -1
 $EndComp
-$Comp
-L V_Mechanical:MountingHole TH1
-U 1 1 5E9B8648
-P 1000 6500
-F 0 "TH1" H 1100 6546 50  0000 L CNN
-F 1 "ThroughHole" H 1100 6455 50  0000 L CNN
-F 2 "AllModules:ThroughHole_36milx12mil_Pad_Cu_Mask" H 1000 6500 50  0001 C CNN
-F 3 "~" H 1000 6500 50  0001 C CNN
-F 4 "" H 1000 6500 50  0001 C CNN "Manufacturer"
-	1    1000 6500
-	1    0    0    -1
-$EndComp
-$Comp
-L V_Mechanical:MountingHole TH2
-U 1 1 5E9C0F88
-P 1000 7000
-F 0 "TH2" H 1100 7046 50  0000 L CNN
-F 1 "ThroughHole" H 1100 6955 50  0000 L CNN
-F 2 "AllModules:ThroughHole_36milx12mil_Pad_Cu_Mask" H 1000 7000 50  0001 C CNN
-F 3 "~" H 1000 7000 50  0001 C CNN
-F 4 "" H 1000 7000 50  0001 C CNN "Manufacturer"
-	1    1000 7000
-	1    0    0    -1
-$EndComp
-$Comp
-L V_Mechanical:MountingHole TH3
-U 1 1 5EA021CD
-P 2000 6500
-F 0 "TH3" H 2100 6546 50  0000 L CNN
-F 1 "ThroughHole" H 2100 6455 50  0000 L CNN
-F 2 "AllModules:ThroughHole_36milx12mil_Pad_Cu_Mask" H 2000 6500 50  0001 C CNN
-F 3 "~" H 2000 6500 50  0001 C CNN
-F 4 "" H 2000 6500 50  0001 C CNN "Manufacturer"
-	1    2000 6500
-	1    0    0    -1
-$EndComp
-$Comp
-L V_Mechanical:MountingHole TH4
-U 1 1 5EA021D7
-P 2000 7000
-F 0 "TH4" H 2100 7046 50  0000 L CNN
-F 1 "ThroughHole" H 2100 6955 50  0000 L CNN
-F 2 "AllModules:ThroughHole_36milx12mil_Pad_Cu_Mask" H 2000 7000 50  0001 C CNN
-F 3 "~" H 2000 7000 50  0001 C CNN
-F 4 "" H 2000 7000 50  0001 C CNN "Manufacturer"
-	1    2000 7000
-	1    0    0    -1
-$EndComp
-$Comp
-L V_Mechanical:MountingHole TH5
-U 1 1 5EAC8D45
-P 3000 6500
-F 0 "TH5" H 3100 6546 50  0000 L CNN
-F 1 "ThroughHole" H 3100 6455 50  0000 L CNN
-F 2 "AllModules:ThroughHole_36milx12mil_Pad_Cu_Mask" H 3000 6500 50  0001 C CNN
-F 3 "~" H 3000 6500 50  0001 C CNN
-F 4 "" H 3000 6500 50  0001 C CNN "Manufacturer"
-	1    3000 6500
-	1    0    0    -1
-$EndComp
-$Comp
-L V_Mechanical:MountingHole TH6
-U 1 1 5EAC8D4F
-P 3000 7000
-F 0 "TH6" H 3100 7046 50  0000 L CNN
-F 1 "ThroughHole" H 3100 6955 50  0000 L CNN
-F 2 "AllModules:ThroughHole_36milx12mil_Pad_Cu_Mask" H 3000 7000 50  0001 C CNN
-F 3 "~" H 3000 7000 50  0001 C CNN
-F 4 "" H 3000 7000 50  0001 C CNN "Manufacturer"
-	1    3000 7000
-	1    0    0    -1
-$EndComp
 Connection ~ 8800 2550
 Wire Wire Line
@@
 Text Label 5225 2150 0    50   ~ 0
 N9
+$Sheet
+S 14100 14350 1825 975
+U 5EBEB280
+F0 "GND_Vias" 50
+F1 "ctrb0505-B.sch" 50
+$EndSheet
 $EndSCHEMATC
