File: 10005011 Power Management/10005011 Power Management.kicad_pcb (KiCad board)
At the start: 4 copper layers, 0 parts

Commit message: Initial Imported PCB & Paul's Work
Parts:
- added ?: , , F.Cu at (419.3, 127.0)
- added ?: , , F.Cu at (419.3, 172.1)
- added ?: , , F.Cu at (190.6, 128.1)
- added ?: , , F.Cu at (193.2, 125.6)
- added ?: , , F.Cu at (190.6, 125.6)
- added ?: , , F.Cu at (193.2, 123.0)
- added ?: , , F.Cu at (190.6, 123.0)
- added ?: , , F.Cu at (193.2, 120.5)
- added ?: , , F.Cu at (190.6, 120.5)
- added ?: , , F.Cu at (193.2, 117.9)
- added ?: , , F.Cu at (190.6, 117.9)
- added ?: , , F.Cu at (186.9, 84.2)
- added ?: , , F.Cu at (419.3, 177.2)
- added ?: , , F.Cu at (195.9, 84.2)
- added ?: , , F.Cu at (201.9, 84.2)
- added ?: , , F.Cu at (242.0, 237.2)
- added ?: , , F.Cu at (242.0, 234.7)
- added ?: , , F.Cu at (244.5, 237.2)
- added ?: , , F.Cu at (244.5, 234.7)
- added ?: , , F.Cu at (247.1, 237.2)
- added ?: , , F.Cu at (247.1, 234.7)
- added ?: , , F.Cu at (249.6, 237.2)
- added ?: , , F.Cu at (249.6, 234.7)
- added ?: , , F.Cu at (445.4, 126.4)
- added ?: , , F.Cu at (252.1, 237.2)
- added ?: , , F.Cu at (252.1, 234.7)
- added ?: , , F.Cu at (292.5, 21.4)
- added ?: , , F.Cu at (293.9, 21.4)
- added ?: , , F.Cu at (295.4, 21.4)
- added ?: , , F.Cu at (296.8, 21.4)
- added ?: , , F.Cu at (303.4, 21.4)
- added ?: , , F.Cu at (304.8, 21.4)
- added ?: , , F.Cu at (306.2, 21.4)
- added ?: , , F.Cu at (307.6, 21.4)
- added ?: , , F.Cu at (445.4, 131.5)
- added ?: , , F.Cu at (269.7, 214.1)
- added ?: , , F.Cu at (203.7, 189.1)
- added ?: , , F.Cu at (203.7, 38.1)
- added ?: , , F.Cu at (269.7, 38.1)
- added ?: , , F.Cu at (208.2, 152.9)
- added ?: , , F.Cu at (265.3, 152.9)
- added ?: , , F.Cu at (265.3, 44.9)
- added ?: , , F.Cu at (208.2, 44.9)
- added ?: , , F.Cu at (245.1, 34.6)
- added ?: , , F.Cu at (228.8, 52.1)
- added ?: , , F.Cu at (445.4, 136.6)
- added ?: , , F.Cu at (226.9, 52.1)
- added ?: , , F.Cu at (225.7, 50.8)
- added ?: , , F.Cu at (226.9, 49.6)
- added ?: , , F.Cu at (225.7, 48.3)
- added ?: , , F.Cu at (216.9, 56.5)
- added ?: , , F.Cu at (223.2, 44.4)
- added ?: , , F.Cu at (216.8, 43.9)
- added ?: , , F.Cu at (216.9, 42.7)
- added ?: , , F.Cu at (222.5, 32.4)
- added ?: , , F.Cu at (212.3, 32.4)
- added ?: , , F.Cu at (445.5, 147.1)
- added ?: , , F.Cu at (217.4, 32.4)
- added ?: , , F.Cu at (204.7, 27.3)
- added ?: , , F.Cu at (212.3, 26.1)
- added ?: , , F.Cu at (217.4, 26.1)
- added ?: , , F.Cu at (222.5, 26.1)
- added ?: , , F.Cu at (204.7, 22.3)
- added ?: , , F.Cu at (212.3, 21.0)
- added ?: , , F.Cu at (217.4, 21.0)
- added ?: , , F.Cu at (222.5, 21.0)
- added ?: , , F.Cu at (252.9, 231.5)
- added ?: , , F.Cu at (445.1, 141.1)
- added ?: , , F.Cu at (252.9, 232.6)
- added ?: , , F.Cu at (251.8, 232.6)
- added ?: , , F.Cu at (251.8, 231.5)
- added ?: , , F.Cu at (261.6, 232.8)
- added ?: , , F.Cu at (263.4, 229.3)
- added ?: , , F.Cu at (271.7, 228.9)
- added ?: , , F.Cu at (256.3, 228.3)
- added ?: , , F.Cu at (257.2, 226.7)
- added ?: , , F.Cu at (271.7, 227.4)
- added ?: , , F.Cu at (257.2, 224.7)
- added ?: , , F.Cu at (204.1, 120.5)
- added ?: , , F.Cu at (242.5, 222.6)
- added ?: , , F.Cu at (245.7, 222.6)
- added ?: , , F.Cu at (238.9, 219.1)
- added ?: , , F.Cu at (238.9, 221.0)
- added ?: , , F.Cu at (254.1, 220.7)
- added ?: , , F.Cu at (271.6, 219.7)
- added ?: , , F.Cu at (257.0, 213.7)
- added ?: , , F.Cu at (274.8, 214.4)
- added ?: , , F.Cu at (225.0, 212.8)
- added ?: , , F.Cu at (230.4, 212.8)
- added ?: , , F.Cu at (209.1, 123.5)
- added ?: , , F.Cu at (242.5, 212.4)
- added ?: , , F.Cu at (244.4, 212.4)
- added ?: , , F.Cu at (262.5, 213.1)
- added ?: , , F.Cu at (273.8, 211.3)
- added ?: , , F.Cu at (225.0, 210.2)
- added ?: , , F.Cu at (230.4, 210.2)
- added ?: , , F.Cu at (242.5, 210.5)
- added ?: , , F.Cu at (244.4, 210.5)
- added ?: , , F.Cu at (244.1, 207.0)
- added ?: , , F.Cu at (276.2, 206.4)
- added ?: , , F.Cu at (187.9, 46.4)
- added ?: , , F.Cu at (267.9, 192.0)
- added ?: , , F.Cu at (267.9, 185.5)
- added ?: , , F.Cu at (200.9, 183.8)
- added ?: , , F.Cu at (278.8, 184.9)
- added ?: , , F.Cu at (193.1, 181.5)
- added ?: , , F.Cu at (204.1, 180.4)
- added ?: , , F.Cu at (205.7, 180.4)
- added ?: , , F.Cu at (204.1, 179.1)
- added ?: , , F.Cu at (205.7, 179.1)
- added ?: , , F.Cu at (192.5, 167.6)
- added ?: , , F.Cu at (419.3, 131.5)
- added ?: , , F.Cu at (198.1, 46.4)
- added ?: , , F.Cu at (192.9, 169.6)
- added ?: , , F.Cu at (204.1, 168.3)
- added ?: , , F.Cu at (204.1, 169.6)
- added ?: , , F.Cu at (205.4, 169.6)
- added ?: , , F.Cu at (205.4, 168.3)
- added ?: , , F.Cu at (192.6, 164.6)
- added ?: , , F.Cu at (192.4, 161.6)
- added ?: , , F.Cu at (197.1, 159.1)
- added ?: , , F.Cu at (199.6, 156.4)
- added ?: , , F.Cu at (201.1, 150.5)
- added ?: , , F.Cu at (195.5, 51.5)
- added ?: , , F.Cu at (201.1, 148.6)
- added ?: , , F.Cu at (202.5, 146.7)
- added ?: , , F.Cu at (215.3, 147.0)
- added ?: , , F.Cu at (217.0, 146.9)
- added ?: , , F.Cu at (223.8, 147.5)
- added ?: , , F.Cu at (243.8, 147.0)
- added ?: , , F.Cu at (252.3, 148.2)
- added ?: , , F.Cu at (203.5, 145.8)
- added ?: , , F.Cu at (205.0, 145.9)
- added ?: , , F.Cu at (216.1, 146.1)
- added ?: , , F.Cu at (195.5, 56.5)
- added ?: , , F.Cu at (219.9, 145.8)
- added ?: , , F.Cu at (225.5, 146.0)
- added ?: , , F.Cu at (241.4, 144.2)
- added ?: , , F.Cu at (260.0, 144.9)
- added ?: , , F.Cu at (271.8, 144.4)
- added ?: , , F.Cu at (216.0, 141.9)
- added ?: , , F.Cu at (221.8, 141.9)
- added ?: , , F.Cu at (232.9, 143.2)
- added ?: , , F.Cu at (241.6, 141.7)
- added ?: , , F.Cu at (251.3, 143.2)
- added ?: , , F.Cu at (190.5, 56.5)
- added ?: , , F.Cu at (253.4, 141.8)
- added ?: , , F.Cu at (254.8, 141.6)
- added ?: , , F.Cu at (259.5, 143.3)
- added ?: , , F.Cu at (266.3, 141.7)
- added ?: , , F.Cu at (268.1, 143.3)
- added ?: , , F.Cu at (271.1, 143.5)
- added ?: , , F.Cu at (201.0, 141.0)
- added ?: , , F.Cu at (201.0, 139.1)
- added ?: , , F.Cu at (216.0, 139.2)
- added ?: , , F.Cu at (220.1, 141.1)
- added ?: , , F.Cu at (193.0, 54.0)
- added ?: , , F.Cu at (232.9, 140.4)
- added ?: , , F.Cu at (240.0, 140.0)
- added ?: , , F.Cu at (263.8, 141.4)
- added ?: , , F.Cu at (201.0, 137.2)
- added ?: , , F.Cu at (205.8, 136.9)
- added ?: , , F.Cu at (208.5, 137.5)
- added ?: , , F.Cu at (208.5, 138.8)
- added ?: , , F.Cu at (214.9, 138.4)
- added ?: , , F.Cu at (215.0, 137.2)
- added ?: , , F.Cu at (218.2, 137.1)
- added ?: , , F.Cu at (198.0, 54.0)
- added ?: , , F.Cu at (218.9, 138.1)
- added ?: , , F.Cu at (220.3, 138.1)
- added ?: , , F.Cu at (221.6, 138.5)
- added ?: , , F.Cu at (223.3, 138.4)
- added ?: , , F.Cu at (222.4, 137.6)
- added ?: , , F.Cu at (245.4, 138.6)
- added ?: , , F.Cu at (258.3, 137.5)
- added ?: , , F.Cu at (262.7, 136.5)
- added ?: , , F.Cu at (264.4, 138.3)
- added ?: , , F.Cu at (265.5, 136.5)
- added ?: , , F.Cu at (190.5, 51.5)
- added ?: , , F.Cu at (271.5, 136.5)
- added ?: , , F.Cu at (201.0, 135.3)
- added ?: , , F.Cu at (211.4, 135.6)
- added ?: , , F.Cu at (215.9, 135.4)
- added ?: , , F.Cu at (218.1, 134.6)
- added ?: , , F.Cu at (217.3, 136.4)
- added ?: , , F.Cu at (219.2, 134.2)
- added ?: , , F.Cu at (219.4, 135.5)
- added ?: , , F.Cu at (220.2, 136.4)
- added ?: , , F.Cu at (220.3, 134.7)
- added ?: , , F.Cu at (280.3, 24.8)
- added ?: , , F.Cu at (221.6, 134.1)
- added ?: , , F.Cu at (223.1, 134.5)
- added ?: , , F.Cu at (235.6, 136.3)
- added ?: , , F.Cu at (237.2, 134.1)
- added ?: , , F.Cu at (238.1, 135.8)
- added ?: , , F.Cu at (238.9, 134.1)
- added ?: , , F.Cu at (243.6, 136.4)
- added ?: , , F.Cu at (254.0, 136.4)
- added ?: , , F.Cu at (260.1, 136.4)
- added ?: , , F.Cu at (261.1, 135.5)
- added ?: , , F.Cu at (280.3, 29.8)
- added ?: , , F.Cu at (267.2, 135.7)
- added ?: , , F.Cu at (272.7, 134.7)
- added ?: , , F.Cu at (201.0, 131.5)
- added ?: , , F.Cu at (201.0, 133.4)
- added ?: , , F.Cu at (204.1, 132.1)
- added ?: , , F.Cu at (226.4, 131.4)
- added ?: , , F.Cu at (227.7, 133.2)
- added ?: , , F.Cu at (233.4, 133.6)
- added ?: , , F.Cu at (234.8, 133.8)
- added ?: , , F.Cu at (246.6, 133.7)
- added ?: , , F.Cu at (275.3, 29.8)
- added ?: , , F.Cu at (255.2, 131.5)
- added ?: , , F.Cu at (257.4, 133.4)
- added ?: , , F.Cu at (258.4, 133.1)
- added ?: , , F.Cu at (261.1, 133.0)
- added ?: , , F.Cu at (263.1, 131.7)
- added ?: , , F.Cu at (266.6, 132.5)
- added ?: , , F.Cu at (269.2, 133.8)
- added ?: , , F.Cu at (270.1, 132.8)
- added ?: , , F.Cu at (201.0, 129.6)
- added ?: , , F.Cu at (214.7, 129.4)
- added ?: , , F.Cu at (419.3, 136.6)
- added ?: , , F.Cu at (277.7, 27.3)
- added ?: , , F.Cu at (219.9, 130.9)
- added ?: , , F.Cu at (253.7, 130.7)
- added ?: , , F.Cu at (256.1, 130.6)
- added ?: , , F.Cu at (258.6, 129.9)
- added ?: , , F.Cu at (262.5, 129.9)
- added ?: , , F.Cu at (264.2, 130.8)
- added ?: , , F.Cu at (201.0, 127.7)
- added ?: , , F.Cu at (201.4, 126.5)
- added ?: , , F.Cu at (221.0, 126.7)
- added ?: , , F.Cu at (266.1, 127.5)
- added ?: , , F.Cu at (282.7, 27.3)
- added ?: , , F.Cu at (201.2, 123.9)
- added ?: , , F.Cu at (211.1, 125.1)
- added ?: , , F.Cu at (217.7, 123.8)
- added ?: , , F.Cu at (219.3, 123.8)
- added ?: , , F.Cu at (234.6, 123.9)
- added ?: , , F.Cu at (201.2, 122.0)
- added ?: , , F.Cu at (217.7, 122.0)
- added ?: , , F.Cu at (221.9, 122.3)
- added ?: , , F.Cu at (223.1, 122.3)
- added ?: , , F.Cu at (240.3, 121.6)
- added ?: , , F.Cu at (275.3, 24.8)
- added ?: , , F.Cu at (240.3, 122.8)
- added ?: , , F.Cu at (241.5, 122.7)
- added ?: , , F.Cu at (241.5, 121.6)
- added ?: , , F.Cu at (266.0, 122.6)
- added ?: , , F.Cu at (201.3, 120.1)
- added ?: , , F.Cu at (217.7, 120.7)
- added ?: , , F.Cu at (221.9, 121.0)
- added ?: , , F.Cu at (223.1, 121.0)
- added ?: , , F.Cu at (243.6, 119.0)
- added ?: , , F.Cu at (270.8, 120.7)
- added ?: , , F.Cu at (225.4, 123.8)
- added ?: , , F.Cu at (270.8, 119.4)
- added ?: , , F.Cu at (201.3, 118.1)
- added ?: , , F.Cu at (204.2, 117.8)
- added ?: , , F.Cu at (249.8, 114.1)
- added ?: , , F.Cu at (264.3, 113.1)
- added ?: , , F.Cu at (185.7, 109.9)
- added ?: , , F.Cu at (190.7, 109.9)
- added ?: , , F.Cu at (195.8, 109.9)
- added ?: , , F.Cu at (200.9, 109.9)
- added ?: , , F.Cu at (245.4, 109.2)
- added ?: , , F.Cu at (215.2, 123.8)
- added ?: , , F.Cu at (258.7, 109.1)
- added ?: , , F.Cu at (263.5, 108.3)
- added ?: , , F.Cu at (188.2, 107.4)
- added ?: , , F.Cu at (193.3, 107.4)
- added ?: , , F.Cu at (198.4, 107.4)
- added ?: , , F.Cu at (201.5, 106.1)
- added ?: , , F.Cu at (203.4, 107.4)
- added ?: , , F.Cu at (243.0, 107.4)
- added ?: , , F.Cu at (259.1, 107.9)
- added ?: , , F.Cu at (260.5, 107.5)
- added ?: , , F.Cu at (217.8, 118.7)
- added ?: , , F.Cu at (263.5, 106.2)
- added ?: , , F.Cu at (185.7, 104.8)
- added ?: , , F.Cu at (190.7, 104.8)
- added ?: , , F.Cu at (195.8, 104.8)
- added ?: , , F.Cu at (266.9, 103.5)
- added ?: , , F.Cu at (270.6, 104.8)
- added ?: , , F.Cu at (273.5, 104.8)
- added ?: , , F.Cu at (193.3, 102.3)
- added ?: , , F.Cu at (246.4, 100.7)
- added ?: , , F.Cu at (195.8, 99.7)
- added ?: , , F.Cu at (217.8, 113.6)
- added ?: , , F.Cu at (198.4, 100.4)
- added ?: , , F.Cu at (200.9, 99.7)
- added ?: , , F.Cu at (203.4, 100.4)
- added ?: , , F.Cu at (208.5, 99.7)
- added ?: , , F.Cu at (213.6, 99.7)
- added ?: , , F.Cu at (256.7, 99.0)
- added ?: , , F.Cu at (257.6, 98.1)
- added ?: , , F.Cu at (259.6, 98.4)
- added ?: , , F.Cu at (270.1, 99.9)
- added ?: , , F.Cu at (273.8, 99.7)
- added ?: , , F.Cu at (222.8, 113.6)
- added ?: , , F.Cu at (197.1, 95.9)
- added ?: , , F.Cu at (202.2, 95.9)
- added ?: , , F.Cu at (207.3, 95.9)
- added ?: , , F.Cu at (253.9, 97.0)
- added ?: , , F.Cu at (258.7, 97.6)
- added ?: , , F.Cu at (275.5, 95.5)
- added ?: , , F.Cu at (189.5, 94.7)
- added ?: , , F.Cu at (194.6, 94.7)
- added ?: , , F.Cu at (199.6, 94.7)
- added ?: , , F.Cu at (204.7, 94.7)
- added ?: , , F.Cu at (220.3, 116.1)
- added ?: , , F.Cu at (209.8, 94.7)
- added ?: , , F.Cu at (249.8, 93.0)
- added ?: , , F.Cu at (260.1, 93.5)
- added ?: , , F.Cu at (258.8, 93.7)
- added ?: , , F.Cu at (261.1, 92.9)
- added ?: , , F.Cu at (266.4, 92.9)
- added ?: , , F.Cu at (273.6, 94.0)
- added ?: , , F.Cu at (197.1, 92.1)
- added ?: , , F.Cu at (202.2, 92.1)
- added ?: , , F.Cu at (204.7, 90.8)
- added ?: , , F.Cu at (215.3, 116.1)
- added ?: , , F.Cu at (207.3, 92.1)
- added ?: , , F.Cu at (209.8, 90.8)
- added ?: , , F.Cu at (250.9, 92.2)
- added ?: , , F.Cu at (254.5, 92.4)
- added ?: , , F.Cu at (261.8, 92.0)
- added ?: , , F.Cu at (264.3, 91.3)
- added ?: , , F.Cu at (265.2, 92.7)
- added ?: , , F.Cu at (270.1, 92.5)
- added ?: , , F.Cu at (199.6, 89.6)
- added ?: , , F.Cu at (203.4, 88.3)
- added ?: , , F.Cu at (419.3, 141.6)
- added ?: , , F.Cu at (222.8, 118.7)
- added ?: , , F.Cu at (207.3, 88.3)
- added ?: , , F.Cu at (223.4, 89.5)
- added ?: , , F.Cu at (229.2, 87.9)
- added ?: , , F.Cu at (248.2, 89.1)
- added ?: , , F.Cu at (248.5, 87.8)
- added ?: , , F.Cu at (259.6, 88.0)
- added ?: , , F.Cu at (261.8, 87.8)
- added ?: , , F.Cu at (263.9, 90.0)
- added ?: , , F.Cu at (265.1, 89.4)
- added ?: , , F.Cu at (271.6, 88.0)
- added ?: , , F.Cu at (236.8, 34.6)
- added ?: , , F.Cu at (199.6, 85.8)
- added ?: , , F.Cu at (204.7, 85.8)
- added ?: , , F.Cu at (209.8, 85.8)
- added ?: , , F.Cu at (234.1, 86.9)
- added ?: , , F.Cu at (235.5, 87.7)
- added ?: , , F.Cu at (248.4, 85.2)
- added ?: , , F.Cu at (255.5, 85.7)
- added ?: , , F.Cu at (254.6, 86.8)
- added ?: , , F.Cu at (265.4, 87.0)
- added ?: , , F.Cu at (266.5, 87.7)
- added ?: , , F.Cu at (229.9, 22.1)
- added ?: , , F.Cu at (274.9, 85.3)
- added ?: , , F.Cu at (229.3, 82.6)
- added ?: , , F.Cu at (228.9, 83.8)
- added ?: , , F.Cu at (235.8, 83.5)
- added ?: , , F.Cu at (249.3, 84.0)
- added ?: , , F.Cu at (261.0, 83.9)
- added ?: , , F.Cu at (262.8, 83.3)
- added ?: , , F.Cu at (263.8, 82.8)
- added ?: , , F.Cu at (270.2, 82.9)
- added ?: , , F.Cu at (277.2, 83.3)
- added ?: , , F.Cu at (206.5, 19.1)
- added ?: , , F.Cu at (204.7, 82.0)
- added ?: , , F.Cu at (209.8, 82.0)
- added ?: , , F.Cu at (228.6, 81.6)
- added ?: , , F.Cu at (229.6, 80.2)
- added ?: , , F.Cu at (246.7, 80.2)
- added ?: , , F.Cu at (247.1, 81.2)
- added ?: , , F.Cu at (250.1, 82.0)
- added ?: , , F.Cu at (251.1, 81.1)
- added ?: , , F.Cu at (261.6, 81.9)
- added ?: , , F.Cu at (263.0, 81.9)
- added ?: , , F.Cu at (251.5, 19.1)
- added ?: , , F.Cu at (264.9, 82.3)
- added ?: , , F.Cu at (266.1, 81.9)
- added ?: , , F.Cu at (270.3, 81.1)
- added ?: , , F.Cu at (271.0, 80.2)
- added ?: , , F.Cu at (271.0, 82.0)
- added ?: , , F.Cu at (276.3, 80.7)
- added ?: , , F.Cu at (276.3, 82.4)
- added ?: , , F.Cu at (277.2, 81.5)
- added ?: , , F.Cu at (199.6, 79.4)
- added ?: , , F.Cu at (203.4, 79.4)
- added ?: , , F.Cu at (214.6, 29.1)
- added ?: , , F.Cu at (207.3, 79.4)
- added ?: , , F.Cu at (219.7, 78.0)
- added ?: , , F.Cu at (221.6, 79.0)
- added ?: , , F.Cu at (222.7, 79.0)
- added ?: , , F.Cu at (226.9, 78.7)
- added ?: , , F.Cu at (228.2, 78.4)
- added ?: , , F.Cu at (247.4, 79.3)
- added ?: , , F.Cu at (254.6, 77.6)
- added ?: , , F.Cu at (270.3, 79.3)
- added ?: , , F.Cu at (276.3, 79.0)
- added ?: , , F.Cu at (221.6, 29.1)
- added ?: , , F.Cu at (277.2, 79.8)
- added ?: , , F.Cu at (277.2, 78.2)
- added ?: , , F.Cu at (193.9, 76.2)
- added ?: , , F.Cu at (197.4, 76.2)
- added ?: , , F.Cu at (200.9, 76.9)
- added ?: , , F.Cu at (204.7, 76.9)
- added ?: , , F.Cu at (208.5, 76.9)
- added ?: , , F.Cu at (210.6, 76.7)
- added ?: , , F.Cu at (217.7, 76.1)
- added ?: , , F.Cu at (222.4, 77.3)
- added ?: , , F.Cu at (240.1, 25.3)
- added ?: , , F.Cu at (231.4, 77.0)
- added ?: , , F.Cu at (260.1, 77.0)
- added ?: , , F.Cu at (261.7, 77.1)
- added ?: , , F.Cu at (194.6, 74.3)
- added ?: , , F.Cu at (199.6, 74.3)
- added ?: , , F.Cu at (203.4, 74.3)
- added ?: , , F.Cu at (207.3, 74.3)
- added ?: , , F.Cu at (226.9, 73.1)
- added ?: , , F.Cu at (261.3, 73.2)
- added ?: , , F.Cu at (263.0, 73.3)
- added ?: , , F.Cu at (248.7, 25.3)
- added ?: , , F.Cu at (217.7, 71.5)
- added ?: , , F.Cu at (226.9, 70.5)
- added ?: , , F.Cu at (226.9, 71.8)
- added ?: , , F.Cu at (258.8, 71.8)
- added ?: , , F.Cu at (264.5, 70.3)
- added ?: , , F.Cu at (267.4, 70.2)
- added ?: , , F.Cu at (267.4, 71.7)
- added ?: , , F.Cu at (186.9, 69.3)
- added ?: , , F.Cu at (195.8, 69.3)
- added ?: , , F.Cu at (200.9, 69.3)
- added ?: , , F.Cu at (200.0, 19.1)
- added ?: , , F.Cu at (206.0, 69.3)
- added ?: , , F.Cu at (211.1, 69.3)
- added ?: , , F.Cu at (216.1, 69.3)
- added ?: , , F.Cu at (227.3, 67.7)
- added ?: , , F.Cu at (227.3, 68.9)
- added ?: , , F.Cu at (259.5, 68.8)
- added ?: , , F.Cu at (262.8, 67.6)
- added ?: , , F.Cu at (263.8, 68.2)
- added ?: , , F.Cu at (273.1, 68.5)
- added ?: , , F.Cu at (193.3, 66.7)
- added ?: , , F.Cu at (419.3, 146.7)
- added ?: , , F.Cu at (257.9, 19.1)
- added ?: , , F.Cu at (198.4, 66.7)
- added ?: , , F.Cu at (203.4, 66.7)
- added ?: , , F.Cu at (208.5, 66.7)
- added ?: , , F.Cu at (227.3, 66.1)
- added ?: , , F.Cu at (267.5, 66.7)
- added ?: , , F.Cu at (186.9, 64.2)
- added ?: , , F.Cu at (195.8, 64.2)
- added ?: , , F.Cu at (200.9, 64.2)
- added ?: , , F.Cu at (206.0, 64.2)
- added ?: , , F.Cu at (211.1, 64.2)
- added ?: , , F.Cu at (285.3, 17.0)
- added ?: , , F.Cu at (186.9, 60.4)
- added ?: , , F.Cu at (190.7, 61.6)
- added ?: , , F.Cu at (193.3, 60.4)
- added ?: , , F.Cu at (198.4, 60.4)
- added ?: , , F.Cu at (246.6, 60.7)
- added ?: , , F.Cu at (244.4, 58.3)
- added ?: , , F.Cu at (250.4, 57.8)
- added ?: , , F.Cu at (255.5, 57.8)
- added ?: , , F.Cu at (260.6, 57.8)
- added ?: , , F.Cu at (266.3, 57.8)
- added ?: , , F.Cu at (284.5, 15.8)
- added ?: , , F.Cu at (275.2, 57.8)
- added ?: , , F.Cu at (282.8, 57.8)
- added ?: , , F.Cu at (246.6, 54.6)
- added ?: , , F.Cu at (250.4, 54.6)
- added ?: , , F.Cu at (255.5, 54.6)
- added ?: , , F.Cu at (260.6, 54.6)
- added ?: , , F.Cu at (266.3, 54.6)
- added ?: , , F.Cu at (275.2, 54.6)
- added ?: , , F.Cu at (282.8, 54.6)
- added ?: , , F.Cu at (229.5, 54.0)
- added ?: , , F.Cu at (283.7, 17.0)
- added ?: , , F.Cu at (234.6, 54.0)
- added ?: , , F.Cu at (240.0, 54.0)
- added ?: , , F.Cu at (255.5, 52.1)
- added ?: , , F.Cu at (257.4, 52.1)
- added ?: , , F.Cu at (275.2, 52.1)
- added ?: , , F.Cu at (255.5, 50.2)
- added ?: , , F.Cu at (257.4, 50.2)
- added ?: , , F.Cu at (282.8, 51.5)
- added ?: , , F.Cu at (257.4, 48.3)
- added ?: , , F.Cu at (269.4, 46.7)
- added ?: , , F.Cu at (282.9, 15.8)
- added ?: , , F.Cu at (270.8, 46.7)
- added ?: , , F.Cu at (272.2, 46.7)
- added ?: , , F.Cu at (185.7, 42.6)
- added ?: , , F.Cu at (190.7, 42.6)
- added ?: , , F.Cu at (199.6, 42.6)
- added ?: , , F.Cu at (212.3, 43.9)
- added ?: , , F.Cu at (185.7, 37.5)
- added ?: , , F.Cu at (190.7, 37.5)
- added ?: , , F.Cu at (198.7, 34.6)
- added ?: , , F.Cu at (185.7, 32.4)
- added ?: , , F.Cu at (282.1, 17.0)
- added ?: , , F.Cu at (190.7, 32.4)
- added ?: , , F.Cu at (198.7, 32.1)
- added ?: , , F.Cu at (198.7, 33.4)
- added ?: , , F.Cu at (275.8, 33.7)
- added ?: , , F.Cu at (279.0, 33.7)
- added ?: , , F.Cu at (282.2, 33.7)
- added ?: , , F.Cu at (192.6, 30.5)
- added ?: , , F.Cu at (196.8, 30.5)
- added ?: , , F.Cu at (197.7, 31.2)
- added ?: , , F.Cu at (198.7, 30.5)
- added ?: , , F.Cu at (214.8, 154.1)
- added ?: , , F.Cu at (199.6, 27.3)
- added ?: , , F.Cu at (199.6, 22.3)
- added ?: , , F.Cu at (283.8, 21.6)
- added ?: , , F.Cu at (281.0, 20.3)
- added ?: , , F.Cu at (294.3, 16.6)
- added ?: , , F.Cu at (305.0, 16.2)
- added ?: , , F.Cu at (198.9, 154.8)
- added ?: , , F.Cu at (284.8, 48.0)
- added ?: , , F.Cu at (185.5, 121.9)
- added ?: , , F.Cu at (185.5, 127.4)
- added ?: , , F.Cu at (218.7, 154.1)
- added ?: , , F.Cu at (185.5, 132.9)
- added ?: , , F.Cu at (185.5, 138.4)
- added ?: , , F.Cu at (185.5, 143.9)
- added ?: , , F.Cu at (193.3, 155.2)
- added ?: , , F.Cu at (203.1, 160.0)
- added ?: , , F.Cu at (196.2, 164.6)
- added ?: , , F.Cu at (199.6, 169.8)
- added ?: , , F.Cu at (199.0, 173.8)
- added ?: , , F.Cu at (202.8, 171.4)
- added ?: , , F.Cu at (204.1, 175.8)
- added ?: , , F.Cu at (222.7, 154.1)
- added ?: , , F.Cu at (205.7, 175.8)
- added ?: , , F.Cu at (200.3, 178.0)
- added ?: , , F.Cu at (195.9, 181.1)
- added ?: , , F.Cu at (193.9, 178.3)
- added ?: , , F.Cu at (187.9, 179.9)
- added ?: , , F.Cu at (196.4, 189.7)
- added ?: , , F.Cu at (204.1, 183.6)
- added ?: , , F.Cu at (205.7, 183.6)
- added ?: , , F.Cu at (192.3, 163.1)
- added ?: , , F.Cu at (207.4, 139.4)
- added ?: , , F.Cu at (226.6, 154.1)
- added ?: , , F.Cu at (202.9, 137.8)
- added ?: , , F.Cu at (208.1, 134.3)
- added ?: , , F.Cu at (209.4, 136.1)
- added ?: , , F.Cu at (211.8, 134.1)
- added ?: , , F.Cu at (211.4, 130.8)
- added ?: , , F.Cu at (214.6, 131.0)
- added ?: , , F.Cu at (209.9, 129.6)
- added ?: , , F.Cu at (216.1, 129.7)
- added ?: , , F.Cu at (232.7, 137.9)
- added ?: , , F.Cu at (212.7, 147.4)
- added ?: , , F.Cu at (419.3, 151.8)
- added ?: , , F.Cu at (230.6, 154.1)
- added ?: , , F.Cu at (212.1, 144.7)
- added ?: , , F.Cu at (218.4, 147.2)
- added ?: , , F.Cu at (239.4, 143.2)
- added ?: , , F.Cu at (250.4, 140.0)
- added ?: , , F.Cu at (255.0, 140.2)
- added ?: , , F.Cu at (256.4, 136.4)
- added ?: , , F.Cu at (261.9, 141.7)
- added ?: , , F.Cu at (264.7, 140.2)
- added ?: , , F.Cu at (267.6, 137.5)
- added ?: , , F.Cu at (270.8, 141.7)
- added ?: , , F.Cu at (234.6, 154.1)
- added ?: , , F.Cu at (273.6, 140.1)
- added ?: , , F.Cu at (276.4, 137.5)
- added ?: , , F.Cu at (240.9, 125.6)
- added ?: , , F.Cu at (243.6, 125.6)
- added ?: , , F.Cu at (238.4, 125.6)
- added ?: , , F.Cu at (236.4, 116.8)
- added ?: , , F.Cu at (236.0, 89.8)
- added ?: , , F.Cu at (236.0, 92.1)
- added ?: , , F.Cu at (217.5, 90.6)
- added ?: , , F.Cu at (226.3, 87.0)
- added ?: , , F.Cu at (238.5, 154.1)
- added ?: , , F.Cu at (229.6, 86.1)
- added ?: , , F.Cu at (229.6, 84.7)
- added ?: , , F.Cu at (227.9, 87.7)
- added ?: , , F.Cu at (228.2, 85.3)
- added ?: , , F.Cu at (227.1, 81.3)
- added ?: , , F.Cu at (220.0, 81.3)
- added ?: , , F.Cu at (217.9, 84.1)
- added ?: , , F.Cu at (219.2, 90.4)
- added ?: , , F.Cu at (195.4, 33.8)
- added ?: , , F.Cu at (217.0, 52.6)
- added ?: , , F.Cu at (242.5, 154.1)
- added ?: , , F.Cu at (223.8, 38.3)
- added ?: , , F.Cu at (221.2, 38.3)
- added ?: , , F.Cu at (222.5, 38.3)
- added ?: , , F.Cu at (221.2, 41.4)
- added ?: , , F.Cu at (222.5, 41.4)
- added ?: , , F.Cu at (223.8, 41.4)
- added ?: , , F.Cu at (221.6, 49.1)
- added ?: , , F.Cu at (222.8, 49.1)
- added ?: , , F.Cu at (224.1, 49.1)
- added ?: , , F.Cu at (221.6, 52.2)
- added ?: , , F.Cu at (246.4, 154.1)
- added ?: , , F.Cu at (222.8, 52.2)
- added ?: , , F.Cu at (221.7, 44.4)
- added ?: , , F.Cu at (224.1, 52.2)
- added ?: , , F.Cu at (285.9, 19.1)
- added ?: , , F.Cu at (291.2, 31.5)
- added ?: , , F.Cu at (262.8, 64.9)
- added ?: , , F.Cu at (256.2, 62.5)
- added ?: , , F.Cu at (250.9, 66.8)
- added ?: , , F.Cu at (252.0, 70.5)
- added ?: , , F.Cu at (252.0, 68.6)
- added ?: , , F.Cu at (250.4, 154.1)
- added ?: , , F.Cu at (252.0, 72.4)
- added ?: , , F.Cu at (265.3, 74.6)
- added ?: , , F.Cu at (268.8, 74.7)
- added ?: , , F.Cu at (250.1, 83.1)
- added ?: , , F.Cu at (251.1, 83.7)
- added ?: , , F.Cu at (255.3, 90.7)
- added ?: , , F.Cu at (254.6, 89.7)
- added ?: , , F.Cu at (254.4, 93.5)
- added ?: , , F.Cu at (255.5, 93.8)
- added ?: , , F.Cu at (261.6, 97.0)
- added ?: , , F.Cu at (254.4, 154.1)
- added ?: , , F.Cu at (258.4, 100.7)
- added ?: , , F.Cu at (260.3, 100.4)
- added ?: , , F.Cu at (263.1, 102.1)
- added ?: , , F.Cu at (264.0, 101.3)
- added ?: , , F.Cu at (276.9, 95.5)
- added ?: , , F.Cu at (234.7, 121.7)
- added ?: , , F.Cu at (271.4, 158.8)
- added ?: , , F.Cu at (275.5, 212.9)
- added ?: , , F.Cu at (278.7, 231.2)
- added ?: , , F.Cu at (266.6, 231.2)
- added ?: , , F.Cu at (258.3, 154.1)
- added ?: , , F.Cu at (260.1, 209.4)
- added ?: , , F.Cu at (251.8, 209.3)
- added ?: , , F.Cu at (252.9, 209.2)
- added ?: , , F.Cu at (250.4, 211.2)
- added ?: , , F.Cu at (254.2, 206.4)
- added ?: , , F.Cu at (242.2, 217.2)
- added ?: , , F.Cu at (254.1, 222.3)
- added ?: , , F.Cu at (253.7, 223.6)
- added ?: , , F.Cu at (249.8, 225.8)
- added ?: , , F.Cu at (250.6, 232.1)
- added ?: , , F.Cu at (244.9, 43.6)
- added ?: , , F.Cu at (242.2, 229.9)
- added ?: , , F.Cu at (242.2, 228.0)
- added ?: , , F.Cu at (244.7, 226.7)
- added ?: , , F.Cu at (248.2, 226.7)
- added ?: , , F.Cu at (246.0, 228.0)
- added ?: , , F.Cu at (246.0, 229.9)
- added ?: , , F.Cu at (251.8, 229.7)
- added ?: , , F.Cu at (224.1, 234.2)
- added ?: , , F.Cu at (223.3, 235.0)
- added ?: , , F.Cu at (231.4, 236.6)
- added ?: , , F.Cu at (241.0, 43.6)
- added ?: , , F.Cu at (246.6, 63.5)
- added ?: , , F.Cu at (199.3, 180.7)
- added ?: , , F.Cu at (221.9, 232.1)
- added ?: , , F.Cu at (198.4, 166.3)
- added ?: , , F.Cu at (192.9, 74.3)
- added ?: , , F.Cu at (192.2, 75.9)
- added ?: , , F.Cu at (188.6, 75.9)
- added ?: , , F.Cu at (194.6, 92.1)
- added ?: , , F.Cu at (188.6, 92.1)
- added ?: , , F.Cu at (192.2, 92.1)
- added ?: , , F.Cu at (419.3, 156.9)
- added ?: , , F.Cu at (237.0, 43.6)
- added ?: , , F.Cu at (192.2, 93.4)
- added ?: , , F.Cu at (188.6, 93.4)
- added ?: , , F.Cu at (188.6, 72.8)
- added ?: , , F.Cu at (192.2, 72.8)
- added ?: , , F.Cu at (289.2, 12.6)
- added ?: , , F.Cu at (259.1, 83.7)
- added ?: , , F.Cu at (258.6, 84.8)
- added ?: , , F.Cu at (254.7, 83.3)
- added ?: , , F.Cu at (255.5, 82.5)
- added ?: , , F.Cu at (271.6, 86.5)
- added ?: , , F.Cu at (265.7, 31.2)
- added ?: , , F.Cu at (221.9, 36.9)
- added ?: , , F.Cu at (220.1, 79.1)
- added ?: , , F.Cu at (219.7, 80.2)
- added ?: , , F.Cu at (220.6, 147.9)
- added ?: , , F.Cu at (228.8, 237.7)
- added ?: , , F.Cu at (254.4, 74.8)
- added ?: , , F.Cu at (235.8, 234.9)
- added ?: , , F.Cu at (276.7, 143.6)
- added ?: , , F.Cu at (194.4, 171.8)
- added ?: , , F.Cu at (275.7, 158.1)
- added ?: , , F.Cu at (265.7, 28.6)
- added ?: , , F.Cu at (257.4, 59.9)
- added ?: , , F.Cu at (277.4, 156.0)
- added ?: , , F.Cu at (273.7, 151.5)
- added ?: , , F.Cu at (276.8, 151.5)
- added ?: , , F.Cu at (219.3, 142.0)
- added ?: , , F.Cu at (240.0, 112.7)
- added ?: , , F.Cu at (242.5, 116.8)
- added ?: , , F.Cu at (260.5, 128.1)
- added ?: , , F.Cu at (278.0, 186.5)
- added ?: , , F.Cu at (272.3, 187.9)
- added ?: , , F.Cu at (265.7, 26.1)
- added ?: , , F.Cu at (269.5, 113.6)
- added ?: , , F.Cu at (271.0, 113.6)
- added ?: , , F.Cu at (269.5, 114.8)
- added ?: , , F.Cu at (271.0, 114.8)
- added ?: , , F.Cu at (272.7, 120.7)
- added ?: , , F.Cu at (272.7, 119.4)
- added ?: , , F.Cu at (225.8, 232.4)
- added ?: , , F.Cu at (238.1, 224.3)
- added ?: , , F.Cu at (238.1, 223.0)
- added ?: , , F.Cu at (278.2, 209.2)
- added ?: , , F.Cu at (263.2, 31.2)
- added ?: , , F.Cu at (226.9, 100.5)
- added ?: , , F.Cu at (226.9, 101.8)
- added ?: , , F.Cu at (228.5, 100.5)
- added ?: , , F.Cu at (228.5, 101.8)
- added ?: , , F.Cu at (208.5, 104.9)
- added ?: , , F.Cu at (273.3, 166.5)
- added ?: , , F.Cu at (273.3, 165.3)
- added ?: , , F.Cu at (231.8, 227.9)
- added ?: , , F.Cu at (232.4, 230.0)
- added ?: , , F.Cu at (238.4, 230.0)
- added ?: , , F.Cu at (263.2, 28.6)
- added ?: , , F.Cu at (234.9, 218.6)
- added ?: , , F.Cu at (236.3, 217.4)
- added ?: , , F.Cu at (236.3, 218.6)
- added ?: , , F.Cu at (234.9, 217.4)
- added ?: , , F.Cu at (211.1, 102.3)
- added ?: , , F.Cu at (211.1, 107.4)
- added ?: , , F.Cu at (213.6, 104.8)
- added ?: , , F.Cu at (207.3, 107.4)
- added ?: , , F.Cu at (206.0, 109.9)
- added ?: , , F.Cu at (211.1, 109.9)
- added ?: , , F.Cu at (263.2, 26.1)
- added ?: , , F.Cu at (213.6, 66.7)
- added ?: , , F.Cu at (216.1, 64.2)
- added ?: , , F.Cu at (228.9, 95.5)
- added ?: , , F.Cu at (229.7, 93.4)
- added ?: , , F.Cu at (232.9, 94.4)
- added ?: , , F.Cu at (220.3, 90.4)
- added ?: , , F.Cu at (262.5, 98.7)
- added ?: , , F.Cu at (270.3, 98.6)
- added ?: , , F.Cu at (281.3, 21.8)
- added ?: , , F.Cu at (285.7, 13.2)
- added ?: , , F.Cu at (268.3, 31.2)
- added ?: , , F.Cu at (282.6, 13.0)
- added ?: , , F.Cu at (270.2, 203.6)
- added ?: , , F.Cu at (270.2, 202.3)
- added ?: , , F.Cu at (285.1, 21.9)
- added ?: , , F.Cu at (285.6, 22.9)
- added ?: , , F.Cu at (285.8, 20.9)
- added ?: , , F.Cu at (290.3, 18.5)
- added ?: , , F.Cu at (298.1, 21.9)
- added ?: , , F.Cu at (298.0, 20.5)
- added ?: , , F.Cu at (287.3, 22.6)
- added ?: , , F.Cu at (268.3, 23.5)
- added ?: , , F.Cu at (227.3, 226.3)
- added ?: , , F.Cu at (225.8, 226.3)
- added ?: , , F.Cu at (225.8, 227.7)
- added ?: , , F.Cu at (227.3, 227.7)
- added ?: , , F.Cu at (258.7, 64.9)
- added ?: , , F.Cu at (263.0, 76.1)
- added ?: , , F.Cu at (267.2, 68.4)
- added ?: , , F.Cu at (243.6, 113.3)
- added ?: , , F.Cu at (211.8, 137.9)
- added ?: , , F.Cu at (214.7, 140.5)
- added ?: , , F.Cu at (260.6, 23.5)
- added ?: , , F.Cu at (226.4, 139.7)
- added ?: , , F.Cu at (226.3, 134.7)
- added ?: , , F.Cu at (226.3, 136.4)
- added ?: , , F.Cu at (301.2, 18.9)
- added ?: , , F.Cu at (299.7, 12.4)
- added ?: , , F.Cu at (191.3, 177.8)
- added ?: , , F.Cu at (215.0, 52.7)
- added ?: , , F.Cu at (258.6, 234.7)
- added ?: , , F.Cu at (260.1, 234.7)
- added ?: , , F.Cu at (247.9, 63.0)
- added ?: , , F.Cu at (419.3, 162.0)
- added ?: , , F.Cu at (260.6, 31.2)
- added ?: , , F.Cu at (244.5, 63.2)
- added ?: , , F.Cu at (245.5, 63.2)
- added ?: , , F.Cu at (210.4, 53.1)
- added ?: , , F.Cu at (275.5, 175.3)
- added ?: , , F.Cu at (275.5, 177.8)
- added ?: , , F.Cu at (193.2, 148.4)
- added ?: , , F.Cu at (190.6, 148.4)
- added ?: , , F.Cu at (193.2, 145.9)
- added ?: , , F.Cu at (190.6, 145.9)
- added ?: , , F.Cu at (193.2, 143.3)
- added ?: , , F.Cu at (190.6, 143.3)
- added ?: , , F.Cu at (193.2, 140.8)
- added ?: , , F.Cu at (419.3, 167.0)
- added ?: , , F.Cu at (190.6, 140.8)
- added ?: , , F.Cu at (193.2, 138.3)
- added ?: , , F.Cu at (190.6, 138.3)
- added ?: , , F.Cu at (193.2, 135.7)
- added ?: , , F.Cu at (190.6, 135.7)
- added ?: , , F.Cu at (193.2, 133.2)
- added ?: , , F.Cu at (190.6, 133.2)
- added ?: , , F.Cu at (193.2, 130.6)
- added ?: , , F.Cu at (190.6, 130.6)
- added ?: , , F.Cu at (193.2, 128.1)
- added C1: C-BC-C0402, C0402_1, F.Cu at (263.1, 63.8)
- added C10: C-BC-C2220, C2220_1, B.Cu at (272.0, 114.6)
- added C100: CC-BC-C0612, C0612-4_5, B.Cu at (187.7, 143.9)
- added C101: C-BC-C0402, C0402_37, F.Cu at (253.6, 137.5)
- added C102: C-BC-C0402, C0402_38, F.Cu at (271.1, 137.5)
- added C103: C-BC-C0402, C0402_39, F.Cu at (274.9, 137.5)
- added C104: C-BC-C0402, C0402_40, F.Cu at (256.8, 137.5)
- added C105: C-BC-C0402, C0402_41, F.Cu at (266.0, 137.5)
- added C106: C-BC-C0805, C0805_11, F.Cu at (259.7, 36.5)
- added C107: C-BC-C2220, C2220_16, F.Cu at (206.5, 52.6)
- added C108: C-BC-C0402, C0402_42, F.Cu at (191.1, 185.5)
- added C109: C-BC-C0805, C0805_12, F.Cu at (247.9, 232.1)
- added C11: C-BC-C2220, C2220_2, F.Cu at (232.4, 228.9)
- added C110: C-BC-C0805, C0805_13, F.Cu at (269.8, 117.2)
- added C111: C-BC-C0603, C0603_21, F.Cu at (275.8, 180.7)
- added C112: C-BC-C0805, C0805_14, B.Cu at (278.4, 189.6)
- added C113: C-BC-C0805, C0805_15, B.Cu at (267.9, 189.3)
- added C114: C-BC-C2220, C2220_17, B.Cu at (273.0, 184.8)
- added C115: C-BC-C0603, C0603_22, B.Cu at (193.0, 58.1)
- added C116: C-BC-C0603, C0603_23, B.Cu at (191.1, 46.4)
- added C117: C-BC-C0603, C0603_24, F.Cu at (218.4, 104.5)
- added C118: C-BC-C0603, C0603_25, B.Cu at (220.0, 121.0)
- added C119: C-BC-C0603, C0603_26, F.Cu at (211.7, 127.7)
- added C12: C-BC-C0402, C0402_8, F.Cu at (218.4, 146.1)
- added C120: C-BC-C0402, C0402_43, B.Cu at (305.7, 19.7)
- added C121: C-BC-C0402, C0402_44, B.Cu at (300.3, 15.6)
- added C122: C-BC-C0402, C0402_44, B.Cu at (299.7, 18.8)
- added C123: C-BC-C0402, C0402_45, B.Cu at (288.9, 18.8)
- added C124: C-BC-C0402, C0402_46, B.Cu at (287.0, 16.2)
- added C125: C-BCP-WX10, C-SC10_2, B.Cu at (190.4, 70.2)
- added C126: C-BC-C0402, C0402_47, F.Cu at (272.7, 69.6)
- added C127: C-BC-C0402, C0402_48, B.Cu at (280.3, 16.2)
- added C128: C-BC-C0402, C0402_49, B.Cu at (284.1, 13.7)
- added C129: C-BC-C0402, C0402_50, B.Cu at (289.5, 15.6)
- added C13: C-BC-C0402, C0402_9, F.Cu at (218.4, 130.8)
- added C130: C-BC-C0402, C0402_51, B.Cu at (294.9, 19.7)
- added C131: C-BC-C0805, C0805_16, F.Cu at (220.9, 88.8)
- added C132: C-BC-C0805, C0805_17, B.Cu at (249.2, 77.5)
- added C133: C-BC-C0805, C0805_18, B.Cu at (244.7, 77.5)
- added C134: C-BC-C1210, C1210_6, B.Cu at (222.2, 70.8)
- added C135: C-BC-C1210, C1210_7, B.Cu at (229.2, 63.2)
- added C136: C-BC-C2220, C2220_18, F.Cu at (223.8, 105.4)
- added C137: C-BC-C2220, C2220_19, B.Cu at (225.7, 107.0)
- added C138: C-BC-C2220, C2220_20, B.Cu at (232.0, 102.6)
- added C139: C-BC-C1210, C1210_8, B.Cu at (276.8, 162.0)
- added C14: C-BC-C2220, C2220_3, B.Cu at (270.1, 176.2)
- added C140: C-BC-C0805, C0805_19, B.Cu at (190.4, 179.7)
- added C141: C-BC-C0805, C0805_20, B.Cu at (211.4, 54.6)
- added C15: C-BC-C0402, C0402_10, F.Cu at (210.1, 138.8)
- added C16: C-BC-C0402, C0402_10, F.Cu at (247.9, 229.9)
- added C17: C-BC-C0402, C0402_11, F.Cu at (194.6, 169.6)
- added C18: C-BC-C0603, C0603_2, F.Cu at (210.1, 140.4)
- added C19: C-BC-C0603, C0603_3, F.Cu at (209.8, 127.7)
- added C2: C-BC-C0805, C0805-AIROX-KEMET-C0805C106KA3, B.Cu at (286.0, 25.7)
- added C20: C-BC-C2220, C2220_4, F.Cu at (224.4, 220.7)
- added C21: C-BC-C1210, C1210_1, F.Cu at (235.5, 222.0)
- added C22: C-BC-C0603, C0603_4, F.Cu at (219.7, 127.7)
- added C23: C-BC-C0805, C0805_1, F.Cu at (252.3, 225.8)
- added C24: C-BC-C0603, C0603_5, F.Cu at (260.0, 227.4)
- added C25: C-BC-C0402, C0402_12, B.Cu at (231.1, 94.7)
- added C26: C-BC-C2220, C2220_5, F.Cu at (222.2, 69.6)
- added C27: C-BC-C2220, C2220_6, F.Cu at (222.2, 63.5)
- added C28: C-BC-C2220, C2220_7, B.Cu at (222.2, 65.7)
- added C29: C-BC-C1210, C1210_2, B.Cu at (222.2, 75.0)
- added C3: C-BC-C0402, C0402_2, F.Cu at (272.7, 67.3)
- added C30: C-BC-C0805, C0805_2, F.Cu at (220.9, 84.4)
- added C31: C-BC-C0805, C0805_3, F.Cu at (222.2, 73.7)
- added C32: C-BC-C0805, C0805_4, F.Cu at (220.9, 86.6)
- added C33: C-BC-C1206, RC1206_1, F.Cu at (229.7, 98.4)
- added C34: C-BC-C1210, C1210_3, F.Cu at (261.9, 125.8)
- added C35: C-BC-C0402, C0402_13, F.Cu at (263.8, 122.6)
- added C36: C-BC-C0402, C0402_14, F.Cu at (260.0, 122.6)
- added C37: C-BC-C0603, C0603_6, F.Cu at (230.4, 92.1)
- added C38: C-BC-C0603, C0603_7, F.Cu at (225.7, 89.6)
- added C39: C-BC-C0603, C0603_8, F.Cu at (225.0, 78.7)
- added C4: C-BC-C0402, C0402_3, F.Cu at (240.9, 143.2)
- added C40: C-BC-C2220, C2220_8, B.Cu at (222.2, 94.0)
- added C41: C-BC-C2220, C2220_9, B.Cu at (222.2, 100.0)
- added C42: C-BCP-WX10, C-SC10_1, B.Cu at (190.4, 95.6)
- added C43: C-BC-C2220, C2220_10, F.Cu at (222.2, 99.4)
- added C44: C-BCP-WX8, C-SC8_1, F.Cu at (240.5, 115.0)
- added C45: C-BC-C0805, C0805-AIROX-KEMET-C0805C106KA0, B.Cu at (240.9, 115.3)
- added C46: C-BC-C0402, C0402_15, B.Cu at (238.1, 118.1)
- added C47: C-BC-C0603, C0603_9, B.Cu at (240.6, 124.2)
- added C48: C-BC-C0402, C0402_16, F.Cu at (234.3, 83.5)
- added C49: C-BC-C0603, C0603_10, F.Cu at (234.3, 77.8)
- added C5: C-BC-C0402, C0402_4, F.Cu at (258.1, 63.8)
- added C50: C-BC-C1206, RC1206_2, F.Cu at (233.0, 89.8)
- added C51: C-BC-C2220, C2220_11, B.Cu at (275.2, 205.1)
- added C52: C-BC-C0603, C0603_11, F.Cu at (234.3, 80.0)
- added C53: CC-BC-C0612, C0612-4_1, B.Cu at (187.7, 121.9)
- added C54: C-BCP-WX8, C-SC8_2, F.Cu at (232.9, 123.9)
- added C55: C-BC-C0805, C0805_5, B.Cu at (232.9, 124.2)
- added C56: C-BC-C0603, C0603_12, F.Cu at (234.3, 85.4)
- added C57: C-BC-C0805, C0805_6, F.Cu at (205.7, 134.0)
- added C58: C-BC-C0402, C0402_17, F.Cu at (205.7, 132.1)
- added C59: C-BC-C0402, C0402_18, F.Cu at (205.7, 139.4)
- added C6: C-BC-C0402, C0402_5, F.Cu at (227.3, 137.8)
- added C60: C-BC-C2220, C2220_12, B.Cu at (270.1, 166.4)
- added C61: CC-BC-C0612, C0612-4_2, B.Cu at (187.7, 127.4)
- added C62: CC-BC-C0612, C0612-4_3, B.Cu at (187.7, 138.4)
- added C63: C-BC-C0402, C0402_19, F.Cu at (210.1, 137.5)
- added C64: C-BC-C0402, C0402_20, F.Cu at (213.0, 130.8)
- added C65: C-BC-C1210, C1210_4, F.Cu at (187.6, 176.9)
- added C66: C-BC-C2220, C2220_13, F.Cu at (230.4, 220.7)
- added C67: C-BC-C2220, C2220_14, F.Cu at (238.4, 228.9)
- added C68: C-BC-C0603, C0603_13, F.Cu at (244.1, 217.2)
- added C69: C-BC-C0402, C0402_21, F.Cu at (244.1, 219.1)
- added C7: C-BC-C0603, C0603_1, F.Cu at (253.9, 70.5)
- added C70: C-BC-C0805, C0805_7, F.Cu at (260.3, 219.7)
- added C71: C-BC-C0402, C0402_22, F.Cu at (259.7, 208.3)
- added C72: C-BC-C0603, C0603_14, F.Cu at (244.1, 220.7)
- added C73: C-BC-C2220, C2220_15, F.Cu at (275.1, 205.6)
- added C74: C-BC-C0603, C0603_15, F.Cu at (240.9, 219.1)
- added C75: C-BC-C0402, C0402_23, F.Cu at (257.4, 207.0)
- added C76: C-BC-C0805, C0805_8, F.Cu at (256.2, 215.3)
- added C77: C-BC-C0402, C0402_24, F.Cu at (244.1, 222.6)
- added C78: C-BC-C0402, C0402_25, F.Cu at (257.4, 208.3)
- added C79: C-BC-C0805, C0805_9, F.Cu at (260.3, 222.0)
- added C8: C-BC-C0402, C0402_6, F.Cu at (213.9, 55.3)
- added C80: C-BC-C0805, C0805_10, F.Cu at (260.3, 224.2)
- added C81: C-BC-C0402, C0402_26, F.Cu at (244.1, 224.8)
- added C82: C-BC-C0402, C0402_27, F.Cu at (224.1, 232.1)
- added C83: C-BC-C0603, C0603_16, F.Cu at (252.3, 211.5)
- added C84: C-BC-C0603, C0603_17, F.Cu at (277.4, 215.3)
- added C85: C-BC-C0402, C0402_28, F.Cu at (249.8, 88.6)
- added C86: C-BC-C0402, C0402_29, F.Cu at (261.9, 100.4)
- added C87: C-BC-C0402, C0402_30, F.Cu at (270.5, 88.0)
- added C88: C-BC-C0402, C0402_31, F.Cu at (261.2, 78.1)
- added C89: C-BC-C1206, RC1206-AIROX-KEMET-C1206C107A6, F.Cu at (288.2, 32.1)
- added C9: C-BC-C0402, C0402_7, F.Cu at (275.2, 151.5)
- added C90: C-BC-C1210, C1210_5, B.Cu at (268.2, 206.4)
- added C91: C-BC-C0402, C0402_32, B.Cu at (253.0, 87.7)
- added C92: C-BC-C0402, C0402_33, B.Cu at (270.5, 87.7)
- added C93: C-BC-C0402, C0402_34, F.Cu at (268.9, 99.1)
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Routing:
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- added copper zone on B.Cu, net (none)
- added copper zone on F.Cu, net (none)
- added copper zone on In1.Cu, net (none)
- added copper zone on In2.Cu, net (none)
- added copper zone on In3.Cu, net (none)
- added copper zone on In4.Cu, net (none)
Other:
- board outline added: 126 x 231.2 mm
- copper layers 4 -> 6
- net class Default: clearance 0.1524 -> 0.2; trace_width 0.254 -> 0.25; via_dia 0.6858 -> 0.8; via_drill 0.3302 -> 0.4
- rule pad_to_mask_clearance: 0 -> 0.051
- rule solder_mask_min_width: 0.1016 -> 0.25
- rule trace_clearance: 0.1524 -> 0.2
- rule trace_min: 0.127 -> 0.2
- rule via_min_drill: 0.254 -> 0.3
- rule via_min_size: 0.4572 -> 0.4
- board text added: "+"
- board text added: "+/-0,1"
- board text added: "+0,1 -0,05"
- board text added: "+0,10 -0,05"
- board text added: "+0,10 -0,10"
- board text added: "+0,125 -0,125"
- board text added: "+0,15 -0,10"
- board text added: "+10% -10%"
- board text added: "+24V"
- board text added: "+33V"
- board text added: "-"
- board text added: "0,3"
- board text added: "0,7"
- board text added: "0,8"
- board text added: "0,9"
- board text added: "0,95"
- board text added: "06/09"
- board text added: "08/10"
- board text added: "0V"
- board text added: "1"
- board text added: "1,1"
- board text added: "1,2"
- board text added: "1,3"
- board text added: "1,5"
- board text added: "1,6"
- board text added: "1/1"
- board text added: "2"
- board text added: "2 trous oblongs metallises de 0,7 x 1,9"
- board text added: "2,5"
- board text added: "220V"
- board text added: "25"
- board text added: "26"
- board text added: "3"
- board text added: "3,0"
- board text added: "3,2"
- board text added: "3,6"
- board text added: "4"
- board text added: "4,0"
- board text added: "4,6"
- board text added: "4096600 E07 002 C"
- board text added: "4096600 E07 005 C"
- board text added: "4096600 E07 006 C"
- board text added: "4096600 E07 007 C"
- board text added: "5"
- board text added: "6"
- board text added: "70u"
- board text added: "8 trous oblongs metallises de 1,1 x 2,0"
- board text added: "A"
- board text added: "AC"
- board text added: "ATTENTION / WARNING:"
- board text added: "B"
- board text added: "BATTERIE"
- board text added: "BLANCHE"
- board text added: "C"
- board text added: "DC"
- board text added: "DC EXT"
- board text added: "EEP"
- board text added: "FEE"
- board text added: "Fabrique suivant IPC A610D classe III 2005. Manufactured according to IPC A610D class III 2005."
- board text added: "ICSP"
- board text added: "LUMIERE"
- board text added: "Le circuit imprime doit etre UL94V-0. The printed circuit board must be UL94V-0 Le fabricant doit etre reconnu UL et doitxxx"
- board text added: "NAPPE"
- board text added: "O1"
- board text added: "O2"
- board text added: "PB540/560"
- board text added: "PLAN DE PERCAGE DRILL DRAWING"
- board text added: "POWER SUPPLY (Tantalum less) RB0505"
- board text added: "PROG EEP"
- board text added: "Power Management Board"
- board text added: "T"
- board text added: "TURBINE"
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