File: 10005011 Power Management/10005011 3V Reference.sch (KiCad schematic (older format))
At the start: 4 parts, among them IC12 LM4120AIM5-3.0

Commit message: added power flags to library and PIC to schematic
Parts:
- renumbered C59 to C?, C57 to C?, C58 to C?, IC12 to IC?
Connections:
- net labels added: +3.0VREF
- net labels removed: +3V0
- wire segments 22 -> 20
Changed lines of the file:
@@
-EESchema Schematic File Version 5
-EELAYER 33 0
+EESchema Schematic File Version 4
+LIBS:10005011 Power Management-cache
+EELAYER 26 0
 EELAYER END
 $Descr USLetter 11000 8500
 encoding utf-8
-Sheet 2 2
+Sheet 2 3
 Title ""
 Date ""
@@
 Comment3 ""
 Comment4 ""
-Comment5 ""
-Comment6 ""
-Comment7 ""
-Comment8 ""
-Comment9 ""
 $EndDescr
 Connection ~ 4950 4175
@@
 Connection ~ 4500 3625
 Connection ~ 6950 3625
-Wire Wire Line
-	4150 3625 4500 3625
 Wire Wire Line
 	4500 3275 4500 3625
@@
 	6250 4075 6950 4075
 Wire Wire Line
-	6950 3275 6950 3625
-Wire Wire Line
 	6950 3625 6950 3725
 Wire Wire Line
@@
 Wire Wire Line
 	6950 4075 6950 4250
-Text HLabel 4150 3625 0    50   Input ~ 0
-+5V
-Text HLabel 7500 3625 2    50   Input ~ 0
-+3V0
+Text HLabel 7500 3625 2    50   Output ~ 0
++3.0VREF
 $Comp
 L power:+5V #PWR?
 U 1 1 5E9171D8
 P 4500 3275
+AR Path="/5E88D608/5E9171D8" Ref="#PWR?"  Part="1"
+AR Path="/5E8E2802/5E9171D8" Ref="#PWR?"  Part="1"
 F 0 "#PWR?" H 4500 3125 50  0001 C CNN
 F 1 "+5V" H 4550 3475 50  0000 C CNN
@@
 $EndComp
 $Comp
-L power:+3V0 #PWR?
-U 1 1 5E917646
-P 6950 3275
-F 0 "#PWR?" H 6950 3125 50  0001 C CNN
-F 1 "+3V0" H 7000 3500 50  0000 C CNN
-F 2 "" H 6950 3275 50  0001 C CNN
-F 3 "" H 6950 3275 50  0001 C CNN
-	1    6950 3275
-	1    0    0    -1
-$EndComp
-$Comp
 L power:GNDA #PWR?
 U 1 1 5E91A751
 P 4950 4250
+AR Path="/5E88D608/5E91A751" Ref="#PWR?"  Part="1"
+AR Path="/5E8E2802/5E91A751" Ref="#PWR?"  Part="1"
 F 0 "#PWR?" H 4950 4000 50  0001 C CNN
 F 1 "GNDA" H 5000 4025 50  0000 C CNN
@@
 U 1 1 5E91B4CA
 P 6950 4250
+AR Path="/5E88D608/5E91B4CA" Ref="#PWR?"  Part="1"
+AR Path="/5E8E2802/5E91B4CA" Ref="#PWR?"  Part="1"
 F 0 "#PWR?" H 6950 4000 50  0001 C CNN
 F 1 "GNDA" H 7000 4025 50  0000 C CNN
@@
 $EndComp
 $Comp
-L Device:C C59
+L Device:C C?
 U 1 1 5E911F09
 P 4500 3975
-F 0 "C59" H 4650 4050 50  0000 L CNN
+AR Path="/5E88D608/5E911F09" Ref="C?"  Part="1"
+AR Path="/5E8E2802/5E911F09" Ref="C?"  Part="1"
+F 0 "C?" H 4650 4050 50  0000 L CNN
 F 1 "100nF" H 4650 3950 50  0000 L CNN
 F 2 "Capacitor_SMD:C_0402_1005Metric" H 4538 3825 50  0001 C CNN
@@
 $EndComp
 $Comp
-L Device:C C57
+L Device:C C?
 U 1 1 5E912A33
 P 6250 3875
-F 0 "C57" H 6375 3950 50  0000 L CNN
+AR Path="/5E88D608/5E912A33" Ref="C?"  Part="1"
+AR Path="/5E8E2802/5E912A33" Ref="C?"  Part="1"
+F 0 "C?" H 6375 3950 50  0000 L CNN
 F 1 "1uF" H 6375 3850 50  0000 L CNN
 F 2 "Capacitor_SMD:C_0805_2012Metric" H 6288 3725 50  0001 C CNN
@@
 $EndComp
 $Comp
-L Device:C C58
+L Device:C C?
 U 1 1 5E91C190
 P 6950 3875
-F 0 "C58" H 7100 3950 50  0000 L CNN
+AR Path="/5E88D608/5E91C190" Ref="C?"  Part="1"
+AR Path="/5E8E2802/5E91C190" Ref="C?"  Part="1"
+F 0 "C?" H 7100 3950 50  0000 L CNN
 F 1 "100nF" H 7100 3850 50  0000 L CNN
 F 2 "Capacitor_SMD:C_0402_1005Metric" H 6988 3725 50  0001 C CNN
@@
 $EndComp
 $Comp
-L Reference_Voltage:LM4120AIM5-3.0 IC12
+L Reference_Voltage:LM4120AIM5-3.0 IC?
 U 1 1 5E911405
 P 5475 3825
-F 0 "IC12" H 5500 4350 50  0000 C CNN
+AR Path="/5E88D608/5E911405" Ref="IC?"  Part="1"
+AR Path="/5E8E2802/5E911405" Ref="IC?"  Part="1"
+F 0 "IC?" H 5500 4350 50  0000 C CNN
 F 1 "LM4120AIM5-3.0" H 5500 4250 50  0000 C CNN
 F 2 "Package_TO_SOT_SMD:SOT-23-5" H 5175 3325 50  0001 L CIN

Commit message: added UART schematics from pages 1 and 3
Parts:
- removed IC?: LM4120AIM5-3.0, Package_TO_SOT_SMD:SOT-23-5, symbol Reference_Voltage:LM4120AIM5-3.0
- added U?: Reference_Voltage_LM4120AIM5-3.0, Package_TO_SOT_SMD:SOT-23-5, symbol page3:Reference_Voltage_LM4120AIM5-3.0
Other:
- moved on the sheet: C?
Changed lines of the file:
@@
 EESchema Schematic File Version 4
-LIBS:10005011 Power Management-cache
-EELAYER 26 0
+EELAYER 30 0
 EELAYER END
 $Descr USLetter 11000 8500
 encoding utf-8
-Sheet 2 3
+Sheet 2 6
 Title ""
 Date ""
@@
 Comment4 ""
 $EndDescr
-Connection ~ 4950 4175
-Connection ~ 4950 3625
-Connection ~ 6250 3625
-Connection ~ 6950 4075
-Connection ~ 4500 3625
-Connection ~ 6950 3625
+Connection ~ 3975 5050
+Connection ~ 3975 4500
+Connection ~ 5275 4500
+Connection ~ 5975 4950
+Connection ~ 3525 4500
+Connection ~ 5975 4500
 Wire Wire Line
-	4500 3275 4500 3625
+	3525 4150 3525 4500
 Wire Wire Line
-	4500 3625 4500 3825
+	3525 4500 3525 4700
 Wire Wire Line
-	4500 4125 4500 4175
+	3525 5000 3525 5050
 Wire Wire Line
-	4500 4175 4950 4175
+	3525 5050 3975 5050
 Wire Wire Line
-	4950 3625 4500 3625
+	3975 4500 3525 4500
 Wire Wire Line
-	4950 3625 5075 3625
+	3975 4500 4100 4500
 Wire Wire Line
-	4950 3825 4950 3625
+	3975 4700 3975 4500
 Wire Wire Line
-	4950 4025 4950 4175
+	3975 4900 3975 5050
 Wire Wire Line
-	4950 4175 4950 4250
+	3975 5050 3975 5125
 Wire Wire Line
-	5075 3825 4950 3825
+	4100 4700 3975 4700
 Wire Wire Line
-	5075 4025 4950 4025
+	4100 4900 3975 4900
 Wire Wire Line
-	5875 3625 6250 3625
+	4900 4500 5275 4500
 Wire Wire Line
-	6250 3625 6250 3725
+	5275 4500 5275 4600
 Wire Wire Line
-	6250 3625 6950 3625
+	5275 4500 5975 4500
 Wire Wire Line
-	6250 4025 6250 4075
+	5275 4900 5275 4950
 Wire Wire Line
-	6250 4075 6950 4075
+	5275 4950 5975 4950
 Wire Wire Line
-	6950 3625 6950 3725
+	5975 4500 5975 4600
 Wire Wire Line
-	6950 3625 7500 3625
+	5975 4500 6525 4500
 Wire Wire Line
-	6950 4075 6950 4025
+	5975 4950 5975 4900
 Wire Wire Line
-	6950 4075 6950 4250
-Text HLabel 7500 3625 2    50   Output ~ 0
+	5975 4950 5975 5125
+Text HLabel 6525 4500 2    50   Output ~ 0
 +3.0VREF
 $Comp
 L power:+5V #PWR?
 U 1 1 5E9171D8
-P 4500 3275
+P 3525 4150
 AR Path="/5E88D608/5E9171D8" Ref="#PWR?"  Part="1"
 AR Path="/5E8E2802/5E9171D8" Ref="#PWR?"  Part="1"
-F 0 "#PWR?" H 4500 3125 50  0001 C CNN
-F 1 "+5V" H 4550 3475 50  0000 C CNN
-F 2 "" H 4500 3275 50  0001 C CNN
-F 3 "" H 4500 3275 50  0001 C CNN
-	1    4500 3275
+AR Path="/5E8F17C0/5E9171D8" Ref="#PWR?"  Part="1"
+F 0 "#PWR?" H 3525 4000 50  0001 C CNN
+F 1 "+5V" H 3575 4350 50  0000 C CNN
+F 2 "" H 3525 4150 50  0001 C CNN
+F 3 "" H 3525 4150 50  0001 C CNN
+	1    3525 4150
 	1    0    0    -1
 $EndComp
@@
 L power:GNDA #PWR?
 U 1 1 5E91A751
-P 4950 4250
+P 3975 5125
 AR Path="/5E88D608/5E91A751" Ref="#PWR?"  Part="1"
 AR Path="/5E8E2802/5E91A751" Ref="#PWR?"  Part="1"
-F 0 "#PWR?" H 4950 4000 50  0001 C CNN
-F 1 "GNDA" H 5000 4025 50  0000 C CNN
-F 2 "" H 4950 4250 50  0001 C CNN
-F 3 "" H 4950 4250 50  0001 C CNN
-	1    4950 4250
+AR Path="/5E8F17C0/5E91A751" Ref="#PWR?"  Part="1"
+F 0 "#PWR?" H 3975 4875 50  0001 C CNN
+F 1 "GNDA" H 4025 4900 50  0000 C CNN
+F 2 "" H 3975 5125 50  0001 C CNN
+F 3 "" H 3975 5125 50  0001 C CNN
+	1    3975 5125
 	1    0    0    -1
 $EndComp
@@
 L power:GNDA #PWR?
 U 1 1 5E91B4CA
-P 6950 4250
+P 5975 5125
 AR Path="/5E88D608/5E91B4CA" Ref="#PWR?"  Part="1"
 AR Path="/5E8E2802/5E91B4CA" Ref="#PWR?"  Part="1"
-F 0 "#PWR?" H 6950 4000 50  0001 C CNN
-F 1 "GNDA" H 7000 4025 50  0000 C CNN
-F 2 "" H 6950 4250 50  0001 C CNN
-F 3 "" H 6950 4250 50  0001 C CNN
-	1    6950 4250
+AR Path="/5E8F17C0/5E91B4CA" Ref="#PWR?"  Part="1"
+F 0 "#PWR?" H 5975 4875 50  0001 C CNN
+F 1 "GNDA" H 6025 4900 50  0000 C CNN
+F 2 "" H 5975 5125 50  0001 C CNN
+F 3 "" H 5975 5125 50  0001 C CNN
+	1    5975 5125
 	1    0    0    -1
 $EndComp
@@
 L Device:C C?
 U 1 1 5E911F09
-P 4500 3975
+P 3525 4850
 AR Path="/5E88D608/5E911F09" Ref="C?"  Part="1"
 AR Path="/5E8E2802/5E911F09" Ref="C?"  Part="1"
-F 0 "C?" H 4650 4050 50  0000 L CNN
-F 1 "100nF" H 4650 3950 50  0000 L CNN
-F 2 "Capacitor_SMD:C_0402_1005Metric" H 4538 3825 50  0001 C CNN
-F 3 "~" H 4500 3975 50  0001 C CNN
-F 4 "Murata" H 4500 3975 50  0001 C CNN "Mnf"
-F 5 "GRM155R71C104JA88J" H 4500 3975 50  0001 C CNN "Mnf PN"
-	1    4500 3975
+AR Path="/5E8F17C0/5E911F09" Ref="C?"  Part="1"
+F 0 "C?" H 3675 4925 50  0000 L CNN
+F 1 "100nF" H 3675 4825 50  0000 L CNN
+F 2 "Capacitor_SMD:C_0402_1005Metric" H 3563 4700 50  0001 C CNN
+F 3 "~" H 3525 4850 50  0001 C CNN
+F 4 "Murata" H 3525 4850 50  0001 C CNN "Mnf"
+F 5 "GRM155R71C104JA88J" H 3525 4850 50  0001 C CNN "Mnf PN"
+	1    3525 4850
 	1    0    0    -1
 $EndComp
@@
 L Device:C C?
 U 1 1 5E912A33
-P 6250 3875
+P 5275 4750
 AR Path="/5E88D608/5E912A33" Ref="C?"  Part="1"
 AR Path="/5E8E2802/5E912A33" Ref="C?"  Part="1"
-F 0 "C?" H 6375 3950 50  0000 L CNN
-F 1 "1uF" H 6375 3850 50  0000 L CNN
-F 2 "Capacitor_SMD:C_0805_2012Metric" H 6288 3725 50  0001 C CNN
-F 3 "~" H 6250 3875 50  0001 C CNN
-F 4 "AVX" H 6250 3875 50  0001 C CNN "Mnf"
-F 5 "0805YC105KAT2A" H 6250 3875 50  0001 C CNN "Mnf PN"
-	1    6250 3875
+AR Path="/5E8F17C0/5E912A33" Ref="C?"  Part="1"
+F 0 "C?" H 5400 4825 50  0000 L CNN
+F 1 "1uF" H 5400 4725 50  0000 L CNN
+F 2 "Capacitor_SMD:C_0805_2012Metric" H 5313 4600 50  0001 C CNN
+F 3 "~" H 5275 4750 50  0001 C CNN
+F 4 "AVX" H 5275 4750 50  0001 C CNN "Mnf"
+F 5 "0805YC105KAT2A" H 5275 4750 50  0001 C CNN "Mnf PN"
+	1    5275 4750
 	1    0    0    -1
 $EndComp
@@
 L Device:C C?
 U 1 1 5E91C190
-P 6950 3875
+P 5975 4750
 AR Path="/5E88D608/5E91C190" Ref="C?"  Part="1"
 AR Path="/5E8E2802/5E91C190" Ref="C?"  Part="1"
-F 0 "C?" H 7100 3950 50  0000 L CNN
-F 1 "100nF" H 7100 3850 50  0000 L CNN
-F 2 "Capacitor_SMD:C_0402_1005Metric" H 6988 3725 50  0001 C CNN
-F 3 "~" H 6950 3875 50  0001 C CNN
-F 4 "Murata" H 6950 3875 50  0001 C CNN "Mnf"
-F 5 "GRM155R71C104JA88J" H 6950 3875 50  0001 C CNN "Mnf PN"
-	1    6950 3875
+AR Path="/5E8F17C0/5E91C190" Ref="C?"  Part="1"
+F 0 "C?" H 6125 4825 50  0000 L CNN
+F 1 "100nF" H 6125 4725 50  0000 L CNN
+F 2 "Capacitor_SMD:C_0402_1005Metric" H 6013 4600 50  0001 C CNN
+F 3 "~" H 5975 4750 50  0001 C CNN
+F 4 "Murata" H 5975 4750 50  0001 C CNN "Mnf"
+F 5 "GRM155R71C104JA88J" H 5975 4750 50  0001 C CNN "Mnf PN"
+	1    5975 4750
 	1    0    0    -1
 $EndComp
 $Comp
-L Reference_Voltage:LM4120AIM5-3.0 IC?
-U 1 1 5E911405
-P 5475 3825
-AR Path="/5E88D608/5E911405" Ref="IC?"  Part="1"
-AR Path="/5E8E2802/5E911405" Ref="IC?"  Part="1"
-F 0 "IC?" H 5500 4350 50  0000 C CNN
-F 1 "LM4120AIM5-3.0" H 5500 4250 50  0000 C CNN
-F 2 "Package_TO_SOT_SMD:SOT-23-5" H 5175 3325 50  0001 L CIN
-F 3 "http://www.ti.com/lit/ds/symlink/lm4120.pdf" H 6075 3225 50  0001 C CIN
-F 4 "TI" H 5275 3125 50  0001 C CNN "MNF"
-F 5 "LM4120AIM5-3.0" H 5575 3025 50  0001 C CNN "MNF PN"
-	1    5475 3825
+L page3:Reference_Voltage_LM4120AIM5-3.0 U?
+U 1 1 5E8F18F5
+P 4500 4700
+F 0 "U?" H 4200 5100 50  0000 L CNN
+F 1 "Reference_Voltage_LM4120AIM5-3.0" H 4200 4300 50  0000 L CNN
+F 2 "Package_TO_SOT_SMD:SOT-23-5" H 4200 4200 50  0001 L CIN
+F 3 "http://www.ti.com/lit/ds/symlink/lm4120.pdf" H 5100 4100 50  0001 C CIN
+F 4 "TI" H 4300 4000 50  0001 C CNN "MNF"
+F 5 "LM4120AIM5-3.0" H 4600 3900 50  0001 C CNN "MNF PN"
+	1    4500 4700
 	1    0    0    -1
 $EndComp
