File: 10005011 Power Management/10005011 3V Reference.sch (KiCad schematic (older format))
At the start: 4 parts

Commit message: adding sheets according to the pdf
Parts:
- removed C?: 100nF, Capacitor_SMD:C_0402_1005Metric, symbol Device:C
- added C?: 100nF, Capacitor_SMD:C_0402_1005Metric, symbol Device:C
Connections:
- net +5V: now also C?.1
- net GNDA: now also C?.2
Changed lines of the file:
@@
 $Descr USLetter 11000 8500
 encoding utf-8
-Sheet 2 8
+Sheet 2 13
 Title ""
 Date ""
@@
 $Comp
 L Device:C C?
-U 1 1 5E911F09
+U 1 1 5FB06048
 P 3525 4850
-AR Path="/5E88D608/5E911F09" Ref="C?"  Part="1"
-AR Path="/5E8E2802/5E911F09" Ref="C?"  Part="1"
-AR Path="/5E8F17C0/5E911F09" Ref="C?"  Part="1"
+AR Path="/5E88D608/5FB06048" Ref="C?"  Part="1"
+AR Path="/5E8E2802/5FB06048" Ref="C?"  Part="1"
+AR Path="/5E8F17C0/5FB06048" Ref="C?"  Part="1"
 F 0 "C?" H 3675 4925 50  0000 L CNN
 F 1 "100nF" H 3675 4825 50  0000 L CNN
