File: 10005011 Power Management/10005011 5V Regulator.sch (KiCad schematic (older format))
At the start: 13 parts

Commit message: adding sheets according to the pdf
Parts:
- removed C?: 100nF, Capacitor_SMD:C_0805_2012Metric, symbol Device:C
- removed C?: 10nF, Capacitor_SMD:C_0603_1608Metric, symbol Device:C
- removed C?: 10uF, Capacitor_SMD:C_0805_2012Metric, symbol Device:C
- removed R?: 10k, Capacitor_SMD:C_0603_1608Metric, symbol Device:R
- added C?: 100nF, Capacitor_SMD:C_0805_2012Metric, symbol Device:C
- added C?: 10nF, Capacitor_SMD:C_0603_1608Metric, symbol Device:C
- added C?: 10uF, Capacitor_SMD:C_0805_2012Metric, symbol Device:C
- added R?: 10k, Capacitor_SMD:C_0603_1608Metric, symbol Device:R
Changed lines of the file:
@@
 $Descr USLetter 11000 8500
 encoding utf-8
-Sheet 4 8
+Sheet 4 13
 Title ""
 Date ""
@@
 $Comp
 L power:GND #PWR0123
-U 1 1 5E96F757
+U 1 1 5FDD6129
 P 6450 4050
 F 0 "#PWR0123" H 6450 3800 50  0001 C CNN
@@
 $Comp
 L Device:R R?
-U 1 1 5E973040
+U 1 1 5FDD612B
 P 7425 3950
 F 0 "R?" H 7500 4000 50  0000 L CNN
@@
 $Comp
 L Device:C C?
-U 1 1 5E9651FC
+U 1 1 5FDD6125
 P 3675 3875
 F 0 "C?" H 3800 3925 50  0000 L CNN
@@
 $Comp
 L Device:C C?
-U 1 1 5E96B757
+U 1 1 5FDD6128
 P 6025 3900
 F 0 "C?" H 5900 3850 50  0000 R CNN
@@
 $Comp
 L Device:C C?
-U 1 1 5E978E52
+U 1 1 5FDD6130
 P 8625 3900
 F 0 "C?" H 8750 3950 50  0000 L CNN
