File: 10005011 Power Management/10005011 Micro Controller.sch (KiCad schematic (older format))
At the start: 38 parts

Commit message: adding sheets according to the pdf
Parts:
- removed C? (x3): 100nF, symbol Device:C
- removed IC?: LM393D, symbol Comparator:LM393
- removed IC?: LM393, symbol Comparator:LM393
- removed R? (x2): 10k, symbol Device:R
- removed R?: 33k, symbol Device:R
- removed R?: 27k, symbol Device:R
- removed R?: 10.2k, symbol Device:R
- removed R?: 100k, symbol Device:R
- removed R?: 4.7k, symbol Device:R
- removed TP?: PST2, symbol Connector:TestPoint_Alt
- removed TP?: PST3, symbol Connector:TestPoint_Alt
- removed TP?: PST8, symbol Connector:TestPoint_Alt
- removed TP?: PST7, symbol Connector:TestPoint_Alt
- added C? (x3): 100nF, symbol Device:C
- added IC?: LM393D, symbol Comparator:LM393
- added IC?: LM393, symbol Comparator:LM393
- added R? (x2): 10k, symbol Device:R
- added R?: 33k, symbol Device:R
- added R?: 27k, symbol Device:R
- added R?: 10.2k, symbol Device:R
- added R?: 100k, symbol Device:R
- added R?: 4.7k, symbol Device:R
- added TP?: PST2, symbol Connector:TestPoint_Alt
- added TP?: PST3, symbol Connector:TestPoint_Alt
- added TP?: PST8, symbol Connector:TestPoint_Alt
- added TP?: PST7, symbol Connector:TestPoint_Alt
Connections:
- net +3.0VREF: now also R?.1, R?.1
- net +5V: now also IC?.8 (V+), R?.1
- net 5VPIC: now also C?.1, C?.1, R?.1
- net AMB-TEMP: now also R?.2
- net CMP-IN-VACDC: now also IC?.3 (+)
- net CMP-OUT-VACDC: now also IC?.1, R?.2
- net GND: now also C?.2, C?.2, C?.2, IC?.4 (V-), R?.2, R?.2, R?.2
- net ICSP-PWR: now also R?.1, R?.2
- net MES-VACDC: now also IC?.2 (-)
- net PST2: now also TP?.1
- net PST3: now also TP?.1
- net PST7: now also TP?.1
- net PST8: now also TP?.1
- net VACDCREF: now also R?.1
- net VDCREF: now also R?.1, R?.2
- net at R?.1, R?.2: now also C?.1
Changed lines of the file:
@@
 $Descr A4 11693 8268
 encoding utf-8
-Sheet 3 8
+Sheet 3 13
 Title ""
 Date ""
@@
 $Comp
 L Device:C C?
-U 1 1 5E97C0C4
+U 1 1 5FEC9555
 P 2150 6850
 F 0 "C?" H 2175 6950 50  0000 L CNN
@@
 $Comp
 L Device:C C?
-U 1 1 5E97C0D9
+U 1 1 5FEC9558
 P 3350 6850
 F 0 "C?" H 3375 6950 50  0000 L CNN
@@
 $Comp
 L Connector:TestPoint_Alt TP?
-U 1 1 5E97C137
+U 1 1 5FEC955D
 P 4500 1700
 F 0 "TP?" V 4454 1888 50  0000 L CNN
@@
 $Comp
 L Connector:TestPoint_Alt TP?
-U 1 1 5E97C13E
+U 1 1 5FEC955E
 P 4500 1900
 F 0 "TP?" V 4454 2088 50  0000 L CNN
@@
 $Comp
 L Connector:TestPoint_Alt TP?
-U 1 1 5E97C164
+U 1 1 5FEC955F
 P 1200 2100
 F 0 "TP?" H 1258 2218 50  0000 L CNN
@@
 $Comp
 L Connector:TestPoint_Alt TP?
-U 1 1 5E97C16B
+U 1 1 5FEC9560
 P 1300 2300
 F 0 "TP?" H 1358 2418 50  0000 L CNN
@@
 $Comp
 L power:GND #PWR0106
-U 1 1 5E97C1AA
+U 1 1 5FEC9563
 P 2000 5800
 F 0 "#PWR0106" H 2000 5550 50  0001 C CNN
@@
 $Comp
 L Device:R R?
-U 1 1 5E97C1B4
+U 1 1 5FEC9564
 P 1300 5650
 F 0 "R?" H 1370 5696 50  0000 L CNN
@@
 $Comp
 L power:GND #PWR0107
-U 1 1 5E97C1CF
+U 1 1 5FEC9566
 P 1800 6400
 F 0 "#PWR0107" H 1800 6150 50  0001 C CNN
@@
 $Comp
 L Comparator:LM393 IC?
-U 1 1 5E97C1FC
+U 1 1 5FEC9568
 P 4900 3800
 F 0 "IC?" H 4900 3433 50  0000 C CNN
@@
 $Comp
 L Device:R R?
-U 1 1 5E97C203
+U 1 1 5FEC9569
 P 4400 3550
 F 0 "R?" H 4470 3596 50  0000 L CNN
@@
 $Comp
 L Device:R R?
-U 1 1 5E97C22E
+U 1 1 5FEC956E
 P 5800 4250
 F 0 "R?" H 5870 4296 50  0000 L CNN
@@
 $Comp
 L Device:R R?
-U 1 1 5E97C26D
+U 1 1 5FEC9574
 P 6050 2900
 F 0 "R?" V 6150 2900 50  0000 C CNN
@@
 $Comp
 L Device:R R?
-U 1 1 5E97C274
+U 1 1 5FEC9575
 P 5850 3250
 F 0 "R?" H 5920 3296 50  0000 L CNN
@@
 $Comp
 L power:GND #PWR0112
-U 1 1 5E97C291
+U 1 1 5FEC9577
 P 5850 3450
 F 0 "#PWR0112" H 5850 3200 50  0001 C CNN
@@
 $Comp
 L Comparator:LM393 IC?
-U 3 1 5E97C2AB
+U 3 1 5FEC9578
 P 5700 1800
 F 0 "IC?" H 5658 1846 50  0000 L CNN
@@
 $Comp
 L Device:C C?
-U 1 1 5E97C2EA
+U 1 1 5FEC957F
 P 4300 6950
 F 0 "C?" H 4325 7050 50  0000 L CNN
@@
 $Comp
 L Device:R R?
-U 1 1 5E97C326
+U 1 1 5FEC9586
 P 6200 5950
 F 0 "R?" H 6270 5996 50  0000 L CNN
@@
 $Comp
 L Device:R R?
-U 1 1 5E97C32D
+U 1 1 5FEC9587
 P 5600 6450
 F 0 "R?" H 5670 6496 50  0000 L CNN
@@
 $Comp
 L power:GND #PWR0119
-U 1 1 5E97C334
+U 1 1 5FEC9588
 P 5600 6700
 F 0 "#PWR0119" H 5600 6450 50  0001 C CNN
