File: 10005011 Power Management/10005011_USB-2UARTS.sch (KiCad schematic (older format))
At the start: 26 parts, among them IC26 NC7SZ66, IC27 NC7SZ66, IC4 FT2232, J1 USB Mini B, Q1 6 MHz

Commit message: adding sheets according to the pdf
Parts:
- removed C?: 33pF, symbol Device:C
- removed D?: BAT54C, Package_TO_SOT_SMD:SOT-23, symbol Diode:BAT54C
- removed R?: 470, symbol Device:R
- removed R? (x2): 27, symbol Device:R
- removed R?: 1.5k, symbol Device:R
- added C?: 33pF, symbol Device:C
- added D?: BAT54C, Package_TO_SOT_SMD:SOT-23, symbol Diode:BAT54C
- added R?: 470, symbol Device:R
- added R? (x2): 27, symbol Device:R
- added R?: 1.5k, symbol Device:R
Connections:
- net +5V: now also D?.1
- net DMF: now also R?.2
- net DMR: now also R?.1
- net DPF: now also R?.2
- net DPR: now also R?.1, R?.1
- net FTDI-3V3: now also C?.1
- net FTDI-AVCC: now also R?.1
- net GND: now also C?.2
- net TX-SW-PWR: now also D?.3
- net V-USB: now also D?.2, R?.2
- net at IC4.5 (~RSTOUT): now also R?.2
Changed lines of the file:
@@
 $Descr A4 11693 8268
 encoding utf-8
-Sheet 6 8
+Sheet 6 13
 Title "USB/2UARTS CONVERTER"
 Date "2020-04-09"
@@
 $Comp
 L Interface_USB:FT2232D IC4
-U 1 1 5EC37C32
+U 1 1 5FDBBAB8
 P 5800 3100
 F 0 "IC4" H 5150 4850 50  0000 C CNN
@@
 $Comp
 L power:GND #PWR0134
-U 1 1 5EC37C76
+U 1 1 5FDBBAB9
 P 3600 3200
 F 0 "#PWR0134" H 3600 2950 50  0001 C CNN
@@
 $Comp
 L Device:R R?
-U 1 1 5EC37C9E
+U 1 1 5FDBBABA
 P 3950 1200
 F 0 "R?" V 4050 1200 50  0000 C CNN
@@
 $Comp
 L power:GND #PWR0135
-U 1 1 5EC37CAA
+U 1 1 5FDBBABB
 P 4200 1800
 F 0 "#PWR0135" H 4200 1550 50  0001 C CNN
@@
 $Comp
 L Device:R R?
-U 1 1 5EC37CB0
+U 1 1 5FDBBABC
 P 4550 2200
 F 0 "R?" V 4650 2200 50  0000 C CNN
@@
 $Comp
 L Device:R R?
-U 1 1 5EC37CB6
+U 1 1 5FDBBABD
 P 4550 2400
 F 0 "R?" V 4650 2400 50  0000 C CNN
@@
 $Comp
 L Device:R R?
-U 1 1 5EC37CC6
+U 1 1 5FDBBABE
 P 4800 2650
 F 0 "R?" H 4870 2696 50  0000 L CNN
@@
 $Comp
 L power:GND #PWR0136
-U 1 1 5EC37CF8
+U 1 1 5FDBBABF
 P 6000 5100
 F 0 "#PWR0136" H 6000 4850 50  0001 C CNN
@@
 $Comp
 L Device:Crystal_GND2 Q1
-U 1 1 5EC37D14
+U 1 1 5FDBBAC1
 P 4200 3600
 F 0 "Q1" V 4050 3400 50  0000 C CNN
@@
 $Comp
 L power:GND #PWR0139
-U 1 1 5EC37D47
+U 1 1 5FDBBAC4
 P 3300 1900
 F 0 "#PWR0139" H 3300 1650 50  0001 C CNN
@@
 $Comp
 L Device:C C?
-U 1 1 5EC37D5F
+U 1 1 5FDBBAC5
 P 4600 1550
 F 0 "C?" H 4625 1650 50  0000 L CNN
@@
 $Comp
 L power:GND #PWR0140
-U 1 1 5EC37D6A
+U 1 1 5FDBBAC6
 P 4600 1800
 F 0 "#PWR0140" H 4600 1550 50  0001 C CNN
@@
 $Comp
 L Diode:BAT54C D?
-U 1 1 5EC37D84
+U 1 1 5FDBBAC7
 P 7300 1100
 F 0 "D?" H 7325 950 50  0000 L CNN
@@
 $Comp
 L power:+5V #PWR0144
-U 1 1 5EC52E27
+U 1 1 5FDBBACE
 P 6300 1000
 F 0 "#PWR0144" H 6300 850 50  0001 C CNN
@@
 $Comp
 L 10005011_Power_Management_Schematic_Symbols:47pF C127
-U 1 1 5EC6D582
+U 1 1 5FDBBAD1
 P 2250 2750
 F 0 "C127" H 2275 2850 50  0000 L CNN
@@
 $Comp
 L 10005011_Power_Management_Schematic_Symbols:47pF C128
-U 1 1 5EC70266
+U 1 1 5FDBBAD2
 P 2900 2750
 F 0 "C128" H 2925 2850 50  0000 L CNN
@@
 $Comp
 L page3:USB_B_Mini_2shield J1
-U 1 1 5EC715D8
+U 1 1 5FDBBAD3
 P 1400 2400
 F 0 "J1" H 1200 2750 50  0000 L CNN
@@
 $Comp
 L 10005011_Power_Management_Schematic_Symbols:82356050050 PG2
-U 1 1 5EC6C643
+U 1 1 5FDBBAD0
 P 2700 2750
 F 0 "PG2" V 2550 2850 50  0000 C CNN
@@
 $Comp
 L 10005011_Power_Management_Schematic_Symbols:0.1uF C1
-U 1 1 5ECCEFCD
+U 1 1 5FDBBAD7
 P 3100 1550
 F 0 "C1" H 3125 1650 50  0000 L CNN
@@
 $Comp
 L 10005011_Power_Management_Schematic_Symbols:0.1uF C3
-U 1 1 5ECD3814
+U 1 1 5FDBBAD8
 P 3700 1550
 F 0 "C3" H 3725 1650 50  0000 L CNN
@@
 $Comp
 L 10005011_Power_Management_Schematic_Symbols:0.1uF C5
-U 1 1 5ECD5E01
+U 1 1 5FDBBADA
 P 4200 1550
 F 0 "C5" H 4225 1650 50  0000 L CNN
@@
 $Comp
 L 10005011_Power_Management_Schematic_Symbols:0.01uF C2
-U 1 1 5ECD751C
+U 1 1 5FDBBADB
 P 3400 1550
 F 0 "C2" H 3425 1650 50  0000 L CNN
