File: 10005011 Power Management/10005011 PIC-MIcro.sch (KiCad schematic (older format))
At the start: 41 parts, among them IC1 LM393D, IC3 PIC18F6622, IC5 DS2480B, T2 IRLML5103

Commit message: changed to global nets
Parts:
- gave numbers to parts that had none: 1
Connections:
- wire segments 247 -> 238
Other:
- note removed: "TODO: J2 Missing"
