File: 10005011 Power Management/10005011 USB HOST.sch (KiCad schematic (older format))
At the start: 59 parts, among them IC15 CY7C67300-100AXI, IC16 CY7C1021DV33, IC17 24LC512, IC18 SN74LVC2T45, IC19 SN74LVC2T45, IC2 SN74AHC1G08, IC20 SN74LVC2T45, J12 USB_A, J13 USB_A, J14 Conn_01x04_Male, Q3 12MHz

Commit message: extracted footprints of sheet7, and association in sch
Parts:
- C101, C102, C103, C104, C105, C120, C121, C122, C123, C129, C130, C85, C86, C87, C88, C91, C92, C93, C96, C97: footprint (none) -> 10005011 Power Management:C0402_1
- C94, C95: footprint (none) -> 10005011 Power Management:C0603_1
Changed lines of the file:
@@
 F 0 "C97" V 1698 2250 50  0000 C CNN
 F 1 "100nF" V 1789 2250 50  0000 C CNN
-F 2 "" H 1988 2100 50  0001 C CNN
+F 2 "10005011 Power Management:C0402_1" H 1988 2100 50  0001 C CNN
 F 3 "~" H 1950 2250 50  0001 C CNN
 F 4 "CAPACITOR,100NF,16V,+/-10%,X7R,0402" V 1950 2250 50  0001 C CNN "Description"
@@
 F 0 "C105" V 2798 2250 50  0000 C CNN
 F 1 "100nF" V 2889 2250 50  0000 C CNN
-F 2 "" H 3088 2100 50  0001 C CNN
+F 2 "10005011 Power Management:C0402_1" H 3088 2100 50  0001 C CNN
 F 3 "~" H 3050 2250 50  0001 C CNN
 F 4 "CAPACITOR,100NF,16V,+/-10%,X7R,0402" V 3050 2250 50  0001 C CNN "Description"
@@
 F 0 "C101" V 1698 4050 50  0000 C CNN
 F 1 "100nF" V 1789 4050 50  0000 C CNN
-F 2 "" H 1988 3900 50  0001 C CNN
+F 2 "10005011 Power Management:C0402_1" H 1988 3900 50  0001 C CNN
 F 3 "~" H 1950 4050 50  0001 C CNN
 F 4 "CAPACITOR,100NF,16V,+/-10%,X7R,0402" V 1950 4050 50  0001 C CNN "Description"
@@
 F 0 "C104" V 2798 4050 50  0000 C CNN
 F 1 "100nF" V 2889 4050 50  0000 C CNN
-F 2 "" H 3088 3900 50  0001 C CNN
+F 2 "10005011 Power Management:C0402_1" H 3088 3900 50  0001 C CNN
 F 3 "~" H 3050 4050 50  0001 C CNN
 F 4 "CAPACITOR,100NF,16V,+/-10%,X7R,0402" V 3050 4050 50  0001 C CNN "Description"
@@
 F 0 "C102" V 1698 5900 50  0000 C CNN
 F 1 "100nF" V 1789 5900 50  0000 C CNN
-F 2 "" H 1988 5750 50  0001 C CNN
+F 2 "10005011 Power Management:C0402_1" H 1988 5750 50  0001 C CNN
 F 3 "~" H 1950 5900 50  0001 C CNN
 F 4 "CAPACITOR,100NF,16V,+/-10%,X7R,0402" V 1950 5900 50  0001 C CNN "Description"
@@
 F 0 "C103" V 2798 5900 50  0000 C CNN
 F 1 "100nF" V 2889 5900 50  0000 C CNN
-F 2 "" H 3088 5750 50  0001 C CNN
+F 2 "10005011 Power Management:C0402_1" H 3088 5750 50  0001 C CNN
 F 3 "~" H 3050 5900 50  0001 C CNN
 F 4 "CAPACITOR,100NF,16V,+/-10%,X7R,0402" V 3050 5900 50  0001 C CNN "Description"
@@
 F 0 "C85" H 4385 1154 50  0000 R CNN
 F 1 "100nF" H 4385 1245 50  0000 R CNN
-F 2 "" H 4538 1050 50  0001 C CNN
+F 2 "10005011 Power Management:C0402_1" H 4538 1050 50  0001 C CNN
 F 3 "~" H 4500 1200 50  0001 C CNN
 F 4 "CAPACITOR,100NF,16V,+/-10%,X7R,0402" V 4500 1200 50  0001 C CNN "Description"
@@
 F 0 "C86" H 4885 1154 50  0000 R CNN
 F 1 "100nF" H 4885 1245 50  0000 R CNN
-F 2 "" H 5038 1050 50  0001 C CNN
+F 2 "10005011 Power Management:C0402_1" H 5038 1050 50  0001 C CNN
 F 3 "~" H 5000 1200 50  0001 C CNN
 F 4 "CAPACITOR,100NF,16V,+/-10%,X7R,0402" V 5000 1200 50  0001 C CNN "Description"
@@
 F 0 "C87" H 5385 1154 50  0000 R CNN
 F 1 "100nF" H 5385 1245 50  0000 R CNN
-F 2 "" H 5538 1050 50  0001 C CNN
+F 2 "10005011 Power Management:C0402_1" H 5538 1050 50  0001 C CNN
 F 3 "~" H 5500 1200 50  0001 C CNN
 F 4 "CAPACITOR,100NF,16V,+/-10%,X7R,0402" V 5500 1200 50  0001 C CNN "Description"
@@
 F 0 "C88" H 5885 1154 50  0000 R CNN
 F 1 "100nF" H 5885 1245 50  0000 R CNN
-F 2 "" H 6038 1050 50  0001 C CNN
+F 2 "10005011 Power Management:C0402_1" H 6038 1050 50  0001 C CNN
 F 3 "~" H 6000 1200 50  0001 C CNN
 F 4 "CAPACITOR,100NF,16V,+/-10%,X7R,0402" V 6000 1200 50  0001 C CNN "Description"
@@
 F 0 "C94" H 6715 10096 50  0000 L CNN
 F 1 "22pF" H 6715 10005 50  0000 L CNN
-F 2 "" H 6638 9900 50  0001 C CNN
+F 2 "10005011 Power Management:C0603_1" H 6638 9900 50  0001 C CNN
 F 3 "~" H 6600 10050 50  0001 C CNN
 F 4 "CAPACITOR CERAMIC,22PF,+/-5%,50V,0603" V 6600 10050 50  0001 C CNN "Description"
@@
 F 0 "C95" H 7115 10096 50  0000 L CNN
 F 1 "22pF" H 7115 10005 50  0000 L CNN
-F 2 "" H 7038 9900 50  0001 C CNN
+F 2 "10005011 Power Management:C0603_1" H 7038 9900 50  0001 C CNN
 F 3 "~" H 7000 10050 50  0001 C CNN
 F 4 "CAPACITOR CERAMIC,22PF,+/-5%,50V,0603" V 7000 10050 50  0001 C CNN "Description"
@@
 F 0 "C93" V 2598 9150 50  0000 C CNN
 F 1 "100nF" V 2689 9150 50  0000 C CNN
-F 2 "" H 2888 9000 50  0001 C CNN
+F 2 "10005011 Power Management:C0402_1" H 2888 9000 50  0001 C CNN
 F 3 "~" H 2850 9150 50  0001 C CNN
 F 4 "CAPACITOR,100NF,16V,+/-10%,X7R,0402" V 2850 9150 50  0001 C CNN "Description"
@@
 F 0 "C96" V 11152 7950 50  0000 C CNN
 F 1 "100nF" V 11061 7950 50  0000 C CNN
-F 2 "" H 10938 7800 50  0001 C CNN
+F 2 "10005011 Power Management:C0402_1" H 10938 7800 50  0001 C CNN
 F 3 "~" H 10900 7950 50  0001 C CNN
 F 4 "CAPACITOR,100NF,16V,+/-10%,X7R,0402" V 10900 7950 50  0001 C CNN "Description"
@@
 F 0 "C92" V 13602 5800 50  0000 C CNN
 F 1 "100nF" V 13511 5800 50  0000 C CNN
-F 2 "" H 13388 5650 50  0001 C CNN
+F 2 "10005011 Power Management:C0402_1" H 13388 5650 50  0001 C CNN
 F 3 "~" H 13350 5800 50  0001 C CNN
 F 4 "CAPACITOR,100NF,16V,+/-10%,X7R,0402" V 13350 5800 50  0001 C CNN "Description"
@@
 F 0 "C91" V 13602 5350 50  0000 C CNN
 F 1 "100nF" V 13511 5350 50  0000 C CNN
-F 2 "" H 13388 5200 50  0001 C CNN
+F 2 "10005011 Power Management:C0402_1" H 13388 5200 50  0001 C CNN
 F 3 "~" H 13350 5350 50  0001 C CNN
 F 4 "CAPACITOR,100NF,16V,+/-10%,X7R,0402" V 13350 5350 50  0001 C CNN "Description"
@@
 F 0 "C123" H 14215 1896 50  0000 L CNN
 F 1 "100nF" H 14215 1805 50  0000 L CNN
-F 2 "" H 14138 1700 50  0001 C CNN
+F 2 "10005011 Power Management:C0402_1" H 14138 1700 50  0001 C CNN
 F 3 "~" H 14100 1850 50  0001 C CNN
 F 4 "CAPACITOR,100NF,16V,+/-10%,X7R,0402" V 14100 1850 50  0001 C CNN "Description"
@@
 F 0 "C130" H 12415 1896 50  0000 L CNN
 F 1 "47pF" H 12415 1805 50  0000 L CNN
-F 2 "" H 12338 1700 50  0001 C CNN
+F 2 "10005011 Power Management:C0402_1" H 12338 1700 50  0001 C CNN
 F 3 "~" H 12300 1850 50  0001 C CNN
 F 4 "CAPACITOR,47 PF,+/-5%,50V,0402" V 12300 1850 50  0001 C CNN "Description"
@@
 F 0 "C129" H 13315 1896 50  0000 L CNN
 F 1 "47pF" H 13315 1805 50  0000 L CNN
-F 2 "" H 13238 1700 50  0001 C CNN
+F 2 "10005011 Power Management:C0402_1" H 13238 1700 50  0001 C CNN
 F 3 "~" H 13200 1850 50  0001 C CNN
 F 4 "CAPACITOR,47 PF,+/-5%,50V,0402" V 13200 1850 50  0001 C CNN "Description"
@@
 F 0 "C122" H 14215 3796 50  0000 L CNN
 F 1 "100nF" H 14215 3705 50  0000 L CNN
-F 2 "" H 14138 3600 50  0001 C CNN
+F 2 "10005011 Power Management:C0402_1" H 14138 3600 50  0001 C CNN
 F 3 "~" H 14100 3750 50  0001 C CNN
 F 4 "CAPACITOR,100NF,16V,+/-10%,X7R,0402" V 14100 3750 50  0001 C CNN "Description"
@@
 F 0 "C120" H 12415 3796 50  0000 L CNN
 F 1 "47pF" H 12415 3705 50  0000 L CNN
-F 2 "" H 12338 3600 50  0001 C CNN
+F 2 "10005011 Power Management:C0402_1" H 12338 3600 50  0001 C CNN
 F 3 "~" H 12300 3750 50  0001 C CNN
 F 4 "CAPACITOR,47 PF,+/-5%,50V,0402" V 12300 3750 50  0001 C CNN "Description"
@@
 F 0 "C121" H 13315 3796 50  0000 L CNN
 F 1 "47pF" H 13315 3705 50  0000 L CNN
-F 2 "" H 13238 3600 50  0001 C CNN
+F 2 "10005011 Power Management:C0402_1" H 13238 3600 50  0001 C CNN
 F 3 "~" H 13200 3750 50  0001 C CNN
 F 4 "CAPACITOR,47 PF,+/-5%,50V,0402" V 13200 3750 50  0001 C CNN "Description"

Commit message: footprints and sch sheet6 association and orientation
Parts:
- added C89: 100uF, 10005011 Power Management:RC1206-AIROX-KEMET-C1206C107A6, symbol Device:C
- D15: renamed from D?; footprint Package_TO_SOT_SMD:SOT-23 -> 10005011 Power Management:SOT23-1G_1
- IC15: footprint TQFP-100 -> 10005011 Power Management:TQFP100_1
- IC16: footprint TSOP-44 -> 10005011 Power Management:TSOP2-44_1
- IC17: footprint (none) -> 10005011 Power Management:MX.A8M_1
- IC18, IC19, IC20: footprint (none) -> 10005011 Power Management:uSO08_1
- IC2: footprint (none) -> 10005011 Power Management:SOT23-5_1
- J12, J13: footprint (none) -> 10005011 Power Management:MOL47500-0001_1
- J14: symbol Connector:Conn_01x04_Male -> Connector:Conn_01x06_Male
- L10, L24, L26: footprint (none) -> 10005011 Power Management:C0805-AIROX-MURATA-BLM21PG221D
- L11, L9: footprint (none) -> 10005011 Power Management:DLP31S-AIROX_1
- L13, L14: footprint (none) -> 10005011 Power Management:C1210_1
- L25: renamed from L?; footprint (none) -> 10005011 Power Management:C0805-AIROX-MURATA-BLM21PG221D
- ML6, ML8, PG3, PG4, PG5, PG6: footprint Resistor_SMD:R_0603_1608Metric -> 10005011 Power Management:R0603_1
- PCT1: footprint Resistor_SMD:R_1812_4532Metric -> 10005011 Power Management:C1812_1
- Q3: footprint (none) -> 10005011 Power Management:HC49-4HSMX_1
- R102, R103, R104, R40, R68: footprint (none) -> 10005011 Power Management:R0603_1
- R105, R106: footprint (none) -> 10005011 Power Management:C0603_1
- SW2: renamed from SW?; footprint (none) -> 10005011 Power Management:MCDMR-02T_1
Connections:
- net +3V3: now also C103.1, C104.1, C105.1, C91.1, C92.1, C96.2, R102.1; no longer C103.2, C104.2, C105.2, C91.2, C92.2, C96.1, R102.2
- net +5V: now also C97.2, PCT1.1; no longer C97.1, PCT1.2
- net A15: now also R102.2; no longer R102.1
- net GND: now also C103.2, C104.2, C105.2, C120.2, C121.2, C122.2, C123.2, C129.2, C130.2, C91.2, C92.2, C93.1, C94.1, C95.1, C96.1, C97.1, L25.2, L26.2, ML6.2, ML8.2, PG3.2 (A2), PG4.2 (A2), PG5.2 (A2), PG6.2 (A2), R40.2, R68.1, C89.2; no longer C103.1, C104.1, C105.1, C91.1, C92.1, C93.2, C94.2, C95.2, C96.2, C97.2, R40.1, R68.2
- net USB-RESET: now also R40.1; no longer R40.2
- net at IC15.28 (XTALOUT): now also R103.2; no longer R103.1
- net at IC15.29 (XTALIN), Q3.2: now also C95.2, R104.1; no longer C95.1, R104.2
- net at D15.3, IC17.8 (VCC): now also C93.2, R68.2; no longer C93.1, R68.1
- net at J12.1 (VBUS): now also L10.2; no longer L10.1
- net at C123.1, L13.2, ML6.1: now also L10.1; no longer L10.2
- net at L13.1, L14.1: now also PCT1.2, C89.1; no longer PCT1.1
- new net: C94.2, Q3.1, R103.1, R104.2
- no-connect marks 27 -> 36
Other:
- moved on the sheet: PCT1, R104

Commit message: Merge branch powermanagement-dev_DotMatrix2
Parts:
- removed C89: 100uF, 10005011 Power Management:RC1206-AIROX-KEMET-C1206C107A6, symbol Device:C
- C101, C102, C103, C104, C105, C120, C121, C122, C123, C129, C130, C85, C86, C87, C88, C91, C92, C93, C96, C97: footprint 10005011 Power Management:C0402_1 -> (none)
- C94, C95, R105, R106: footprint 10005011 Power Management:C0603_1 -> (none)
- D15: footprint 10005011 Power Management:SOT23-1G_1 -> Package_TO_SOT_SMD:SOT-23
- IC15: footprint 10005011 Power Management:TQFP100_1 -> TQFP-100
- IC16: footprint 10005011 Power Management:TSOP2-44_1 -> TSOP-44
- IC17: footprint 10005011 Power Management:MX.A8M_1 -> (none)
- IC18, IC19, IC20: footprint 10005011 Power Management:uSO08_1 -> (none)
- IC2: footprint 10005011 Power Management:SOT23-5_1 -> (none)
- J12, J13: footprint 10005011 Power Management:MOL47500-0001_1 -> (none)
- J14: symbol Connector:Conn_01x06_Male -> Connector:Conn_01x04_Male
- L10, L24, L26: footprint 10005011 Power Management:C0805-AIROX-MURATA-BLM21PG221D -> (none)
- L11, L9: footprint 10005011 Power Management:DLP31S-AIROX_1 -> (none)
- L13, L14: footprint 10005011 Power Management:C1210_1 -> (none)
- L?: renamed from L25; footprint 10005011 Power Management:C0805-AIROX-MURATA-BLM21PG221D -> (none)
- ML6, ML8, PG3, PG4, PG5, PG6: footprint 10005011 Power Management:R0603_1 -> Resistor_SMD:R_0603_1608Metric
- PCT1: footprint 10005011 Power Management:C1812_1 -> Resistor_SMD:R_1812_4532Metric
- Q3: footprint 10005011 Power Management:HC49-4HSMX_1 -> (none)
- R102, R103, R104, R40, R68: footprint 10005011 Power Management:R0603_1 -> (none)
- SW?: renamed from SW2; footprint 10005011 Power Management:MCDMR-02T_1 -> (none)
Connections:
- net +3V3: now also C103.2, C104.2, C105.2, C91.2, C92.2, C96.1, R102.2; no longer C103.1, C104.1, C105.1, C91.1, C92.1, C96.2, R102.1
- net +5V: now also C97.1, PCT1.2; no longer C97.2, PCT1.1
- net A15: now also R102.1; no longer R102.2
- net GND: now also C103.1, C104.1, C105.1, C91.1, C92.1, C93.2, C94.2, C95.2, C96.2, C97.2, R40.1, R68.2; no longer C103.2, C104.2, C105.2, C120.2, C121.2, C122.2, C123.2, C129.2, C130.2, C91.2, C92.2, C93.1, C94.1, C95.1, C96.1, C97.1, L26.2, L?.2, ML6.2, ML8.2, PG3.2 (A2), PG4.2 (A2), PG5.2 (A2), PG6.2 (A2), R40.2, R68.1
- net USB-RESET: now also R40.2; no longer R40.1
- net at IC15.28 (XTALOUT): now also R103.1; no longer R103.2
- net at IC15.29 (XTALIN), Q3.2: now also C95.1, R104.2; no longer C95.2, R104.1
- net at D15.3, IC17.8 (VCC): now also C93.1, R68.1; no longer C93.2, R68.2
- net at J12.1 (VBUS): now also L10.1; no longer L10.2
- net at L13.1, L14.1: now also PCT1.1; no longer PCT1.2
- net at C123.1, L13.2, ML6.1: now also L10.2; no longer L10.1
- new net: C94.1, Q3.1, R103.2, R104.1
- new net: C123.2, C129.2, C130.2, L?.2, ML6.2, PG3.2 (A2), PG4.2 (A2)
- new net: C120.2, C121.2, C122.2, L26.2, ML8.2, PG5.2 (A2), PG6.2 (A2)
- no-connect marks 36 -> 27
Other:
- moved on the sheet: PCT1, R104

Commit message: all components with refdes
Parts:
- gave numbers to parts that had none: 1
Changed lines of the file:
@@
 	6850 8450 7000 8450
 $Comp
-L 10005011_Power_Management:MCDM(R)-02-T SW?
+L 10005011_Power_Management:MCDM(R)-02-T SW2
 U 1 1 5ED2A4CB
 P 6200 9200
-F 0 "SW?" V 6246 9430 50  0000 L CNN
+F 0 "SW2" V 6246 9430 50  0000 L CNN
 F 1 "MCDM(R)-02-T" V 6155 9430 50  0000 L CNN
 F 2 "" H 6200 9200 50  0001 C CNN

Commit message: footprints sheet6 and small fix to sheet7
Parts:
- C101, C102, C103, C104, C105, C120, C121, C122, C123, C129, C130, C85, C86, C87, C88, C91, C92, C93, C96, C97: footprint (none) -> 10005011 Power Management:C0402_1
- C94, C95: footprint (none) -> 10005011 Power Management:C0603_1
- IC15: footprint TQFP-100 -> 10005011 Power Management:TQFP100_1
- IC16: footprint TSOP-44 -> 10005011 Power Management:TSOP2-44_1
- IC17: footprint (none) -> 10005011 Power Management:MX.A8M_1
- IC18, IC19, IC20: footprint (none) -> 10005011 Power Management:uSO08_1
- IC2: footprint (none) -> 10005011 Power Management:SOT23-5_1
- J12, J13: footprint (none) -> 10005011 Power Management:MOL47500-0001_1
- J14: footprint (none) -> 10005011 Power Management:B4BZR-SM3TF_1; symbol Connector:Conn_01x04_Male -> Connector:Conn_01x06_Male
- L10, L24, L26: footprint (none) -> 10005011 Power Management:C0805-AIROX-MURATA-BLM21PG221D
- L11, L9: footprint (none) -> 10005011 Power Management:DLP31S-AIROX_1
- L13, L14: footprint (none) -> 10005011 Power Management:C1210_1
- L25: renamed from L?; footprint (none) -> 10005011 Power Management:C0805-AIROX-MURATA-BLM21PG221D
- Q3: footprint (none) -> 10005011 Power Management:HC49-4HSMX_1
- R102, R103, R104, R105, R106, R40, R68: footprint (none) -> 10005011 Power Management:R0603_1
- SW2: footprint (none) -> 10005011 Power Management:MCDMR-02T_1
Connections:
- no-connect marks 27 -> 29

Commit message: updating footprints
Parts:
- ML6, ML8: footprint Resistor_SMD:R_0603_1608Metric -> 10005011 Power Management:R0603_1
Changed lines of the file:
@@
 F 0 "ML6" H 14703 1850 50  0000 L CNN
 F 1 "B72500T0040M060" H 14703 1850 50  0001 L CNN
-F 2 "Resistor_SMD:R_0603_1608Metric" V 14530 1850 50  0001 C CNN
+F 2 "10005011 Power Management:R0603_1" V 14530 1850 50  0001 C CNN
 F 3 "https://www.tdk-electronics.tdk.com/inf/75/db/CTVS_14/Standard_series.pdf" H 14600 1850 50  0001 C CNN
 F 4 "Digi-Key" H 14600 1850 50  0001 C CNN "Source"
@@
 F 0 "ML8" H 14703 3750 50  0000 L CNN
 F 1 "B72500T0040M060" H 14703 3750 50  0001 L CNN
-F 2 "Resistor_SMD:R_0603_1608Metric" V 14530 3750 50  0001 C CNN
+F 2 "10005011 Power Management:R0603_1" V 14530 3750 50  0001 C CNN
 F 3 "https://www.tdk-electronics.tdk.com/inf/75/db/CTVS_14/Standard_series.pdf" H 14600 3750 50  0001 C CNN
 F 4 "Digi-Key" H 14600 3750 50  0001 C CNN "Source"

Commit message: assigned footprints with cmp file
Parts:
- D15: footprint Package_TO_SOT_SMD:SOT-23 -> 10005011 Power Management:SOT23-1G_1
- J12: footprint 10005011 Power Management:MOL47500-0001_1 -> 10005011 Power Management:MOL47500-0001_2
- PCT1: footprint Resistor_SMD:R_1812_4532Metric -> 10005011 Power Management:C1812_1
- PG3, PG4, PG5, PG6: footprint Resistor_SMD:R_0603_1608Metric -> 10005011 Power Management:R0603_1
- PST10, PST11: footprint (none) -> 10005011 Power Management:TEST-CMS-0.8_1
Changed lines of the file:
@@
 F 0 "PST10" V 8500 2650 50  0000 C CNN
 F 1 "TestPoint" H 8500 2584 50  0001 C CNN
-F 2 "" H 8700 2350 50  0001 C CNN
+F 2 "10005011 Power Management:TEST-CMS-0.8_1" H 8700 2350 50  0001 C CNN
 F 3 "~" H 8700 2350 50  0001 C CNN
 	1    8500 2350
@@
 F 0 "PST11" V 8600 2650 50  0000 C CNN
 F 1 "TestPoint" H 8658 2377 50  0001 L CNN
-F 2 "" H 8800 2350 50  0001 C CNN
+F 2 "10005011 Power Management:TEST-CMS-0.8_1" H 8800 2350 50  0001 C CNN
 F 3 "~" H 8800 2350 50  0001 C CNN
 	1    8600 2350
@@
 F 0 "D15" V 3059 9038 50  0000 L CNN
 F 1 "BAT54C" V 3150 9038 50  0000 L CNN
-F 2 "Package_TO_SOT_SMD:SOT-23" H 2925 8375 50  0001 L CNN
+F 2 "10005011 Power Management:SOT23-1G_1" H 2925 8375 50  0001 L CNN
 F 3 "https://media.digikey.com/pdf/Data%20Sheets/ON%20Semiconductor%20PDFs/BAT54(A,C,S).pdf" H 3120 8950 50  0001 C CNN
 F 4 "SOT23" V 3241 9038 50  0000 L CNN "BOM_Footprint"
@@
 F 0 "J12" H 15270 1239 50  0000 R CNN
 F 1 "USB_A" H 15270 1148 50  0000 R CNN
-F 2 "10005011 Power Management:MOL47500-0001_1" H 15650 1200 50  0001 C CNN
+F 2 "10005011 Power Management:MOL47500-0001_2" H 15650 1200 50  0001 C CNN
 F 3 " ~" H 15650 1200 50  0001 C CNN
 F 4 "CONNECTOR USB A" H 15500 1250 50  0001 C CNN "Description"
@@
 F 0 "PG4" V 12800 1929 50  0000 L CNN
 F 1 "82356050050" V 12845 1929 50  0001 L CNN
-F 2 "Resistor_SMD:R_0603_1608Metric" H 12800 1850 50  0001 C CNN
+F 2 "10005011 Power Management:R0603_1" H 12800 1850 50  0001 C CNN
 F 3 "https://katalog.we-online.de/pbs/datasheet/82356050050.pdf" H 12800 1850 50  0001 C CNN
 F 4 "Würth Elektronik" H 12800 1850 50  0001 C CNN "Mfgr"
@@
 F 0 "PG3" V 13700 1929 50  0000 L CNN
 F 1 "82356050050" V 13745 1929 50  0001 L CNN
-F 2 "Resistor_SMD:R_0603_1608Metric" H 13700 1850 50  0001 C CNN
+F 2 "10005011 Power Management:R0603_1" H 13700 1850 50  0001 C CNN
 F 3 "https://katalog.we-online.de/pbs/datasheet/82356050050.pdf" H 13700 1850 50  0001 C CNN
 F 4 "Würth Elektronik" H 13700 1850 50  0001 C CNN "Mfgr"
@@
 F 0 "PCT1" V 10085 1050 50  0000 C CNN
 F 1 "MS-MSMF110" V 10176 1050 50  0000 C CNN
-F 2 "Resistor_SMD:R_1812_4532Metric" H 10450 850 50  0001 L CNN
+F 2 "10005011 Power Management:C1812_1" H 10450 850 50  0001 L CNN
 F 3 "https://www.bourns.com/docs/Product-Datasheets/mfmsmf.pdf" H 10400 1050 50  0001 C CNN
 F 4 "Bourns Inc." H 10400 1050 50  0001 C CNN "Mfgr"
@@
 F 0 "PG6" V 12800 3829 50  0000 L CNN
 F 1 "82356050050" V 12845 3829 50  0001 L CNN
-F 2 "Resistor_SMD:R_0603_1608Metric" H 12800 3750 50  0001 C CNN
+F 2 "10005011 Power Management:R0603_1" H 12800 3750 50  0001 C CNN
 F 3 "https://katalog.we-online.de/pbs/datasheet/82356050050.pdf" H 12800 3750 50  0001 C CNN
 F 4 "Würth Elektronik" H 12800 3750 50  0001 C CNN "Mfgr"
@@
 F 0 "PG5" V 13700 3829 50  0000 L CNN
 F 1 "82356050050" V 13745 3829 50  0001 L CNN
-F 2 "Resistor_SMD:R_0603_1608Metric" H 13700 3750 50  0001 C CNN
+F 2 "10005011 Power Management:R0603_1" H 13700 3750 50  0001 C CNN
 F 3 "https://katalog.we-online.de/pbs/datasheet/82356050050.pdf" H 13700 3750 50  0001 C CNN
 F 4 "Würth Elektronik" H 13700 3750 50  0001 C CNN "Mfgr"
