File: 10005011 Power Management/10005011 USB HOST.sch (KiCad schematic (older format))
At the start: 61 parts, among them IC15 CY7C67300-100AXI, IC16 CY7C1021DV33, IC17 24LC512, IC18 SN74LVC2T45, IC19 SN74LVC2T45, IC2 SN74AHC1G08, IC20 SN74LVC2T45, J12 USB_A, J13 USB_A, J14 Conn_01x04_Male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

Commit message: change CR1-BIS to ZCR1 so that kicad does not think it is missing annotation, do the same in the PCB to be able to read netlist without components getting erased and placed new
Connections:
- net labels added: +3.3V
- net labels removed: +3V3
- no-connect marks 29 -> 36
Changed lines of the file:
@@
 	0    -1   1    0
-$EndComp
-$Comp
-L power:+3V3 #PWR0102
-U 1 1 5E9D4587
-P 2700 2150
-F 0 "#PWR0102" H 2700 2000 50  0001 C CNN
-F 1 "+3V3" H 2715 2323 50  0000 C CNN
-F 2 "" H 2700 2150 50  0001 C CNN
-F 3 "" H 2700 2150 50  0001 C CNN
-	1    2700 2150
-	1    0    0    -1
 $EndComp
 Wire Wire Line
@@
 	0    1    1    0
 $EndComp
-$Comp
-L power:+3V3 #PWR0108
-U 1 1 5E9DD937
-P 2700 3950
-F 0 "#PWR0108" H 2700 3800 50  0001 C CNN
-F 1 "+3V3" H 2715 4123 50  0000 C CNN
-F 2 "" H 2700 3950 50  0001 C CNN
-F 3 "" H 2700 3950 50  0001 C CNN
-	1    2700 3950
-	1    0    0    -1
-$EndComp
 Wire Wire Line
 	2100 4050 2300 4050
@@
 	0    1    1    0
 $EndComp
-$Comp
-L power:+3V3 #PWR0113
-U 1 1 5E9E0D45
-P 2700 5800
-F 0 "#PWR0113" H 2700 5650 50  0001 C CNN
-F 1 "+3V3" H 2715 5973 50  0000 C CNN
-F 2 "" H 2700 5800 50  0001 C CNN
-F 3 "" H 2700 5800 50  0001 C CNN
-	1    2700 5800
-	1    0    0    -1
-$EndComp
 Wire Wire Line
 	2100 5900 2300 5900
@@
 Wire Wire Line
 	6100 2400 6100 2550
-$Comp
-L power:+3V3 #PWR0119
-U 1 1 5EA3D6AE
-P 7300 2350
-F 0 "#PWR0119" H 7300 2200 50  0001 C CNN
-F 1 "+3V3" H 7315 2523 50  0000 C CNN
-F 2 "" H 7300 2350 50  0001 C CNN
-F 3 "" H 7300 2350 50  0001 C CNN
-	1    7300 2350
-	1    0    0    -1
-$EndComp
 Wire Wire Line
 	7500 2550 7500 2450
@@
 	1    6000 1200
 	-1   0    0    1
-$EndComp
-$Comp
-L power:+3V3 #PWR0121
-U 1 1 5EA69E3A
-P 5300 950
-F 0 "#PWR0121" H 5300 800 50  0001 C CNN
-F 1 "+3V3" H 5315 1123 50  0000 C CNN
-F 2 "" H 5300 950 50  0001 C CNN
-F 3 "" H 5300 950 50  0001 C CNN
-	1    5300 950
-	1    0    0    -1
 $EndComp
 $Comp
@@
 Wire Wire Line
 	12300 8000 12500 8000
-$Comp
-L power:+3V3 #PWR0132
-U 1 1 5EFD979D
-P 10550 7850
-F 0 "#PWR0132" H 10550 7700 50  0001 C CNN
-F 1 "+3V3" H 10565 8023 50  0000 C CNN
-F 2 "" H 10550 7850 50  0001 C CNN
-F 3 "" H 10550 7850 50  0001 C CNN
-	1    10550 7850
-	1    0    0    -1
-$EndComp
-$Comp
-L power:+3V3 #PWR0133
-U 1 1 5F0E0F8C
-P 11800 8050
-F 0 "#PWR0133" H 11800 7900 50  0001 C CNN
-F 1 "+3V3" H 11815 8223 50  0000 C CNN
-F 2 "" H 11800 8050 50  0001 C CNN
-F 3 "" H 11800 8050 50  0001 C CNN
-	1    11800 8050
-	1    0    0    -1
-$EndComp
 Wire Wire Line
 	11800 8200 11900 8200
@@
 	12750 5800 13050 5800
 Connection ~ 13050 5800
-$Comp
-L power:+3V3 #PWR0135
-U 1 1 5F2CE059
-P 13800 5750
-F 0 "#PWR0135" H 13800 5600 50  0001 C CNN
-F 1 "+3V3" H 13815 5923 50  0000 C CNN
-F 2 "" H 13800 5750 50  0001 C CNN
-F 3 "" H 13800 5750 50  0001 C CNN
-	1    13800 5750
-	1    0    0    -1
-$EndComp
 Wire Wire Line
 	13800 5750 13800 5800
@@
 U 1 1 5F2EF52D
 P 15500 1250
+AR Path="/5F2EF52D" Ref="J12"  Part="1"
+AR Path="/5E9C3EF6/5F2EF52D" Ref="J12"  Part="1"
 F 0 "J12" H 15270 1239 50  0000 R CNN
 F 1 "USB_A" H 15270 1148 50  0000 R CNN
@@
 U 1 1 5F94AF33
 P 15500 3150
+AR Path="/5F94AF33" Ref="J13"  Part="1"
+AR Path="/5E9C3EF6/5F94AF33" Ref="J13"  Part="1"
 F 0 "J13" H 15270 3139 50  0000 R CNN
 F 1 "USB_A" H 15270 3048 50  0000 R CNN
@@
 Wire Wire Line
 	10250 8350 8400 8350
+$Comp
+L 10005011_Power_Management:+3.3V #PWR0102
+U 1 1 5E994D31
+P 2700 2150
+F 0 "#PWR0102" H 2700 2000 50  0001 C CNN
+F 1 "+3.3V" H 2715 2323 50  0000 C CNN
+F 2 "" H 2700 2150 50  0001 C CNN
+F 3 "" H 2700 2150 50  0001 C CNN
+	1    2700 2150
+	1    0    0    -1
+$EndComp
+$Comp
+L 10005011_Power_Management:+3.3V #PWR0108
+U 1 1 5E99836C
+P 5300 950
+F 0 "#PWR0108" H 5300 800 50  0001 C CNN
+F 1 "+3.3V" H 5315 1123 50  0000 C CNN
+F 2 "" H 5300 950 50  0001 C CNN
+F 3 "" H 5300 950 50  0001 C CNN
+	1    5300 950
+	1    0    0    -1
+$EndComp
+$Comp
+L 10005011_Power_Management:+3.3V #PWR0113
+U 1 1 5E99D785
+P 2700 5800
+F 0 "#PWR0113" H 2700 5650 50  0001 C CNN
+F 1 "+3.3V" H 2715 5973 50  0000 C CNN
+F 2 "" H 2700 5800 50  0001 C CNN
+F 3 "" H 2700 5800 50  0001 C CNN
+	1    2700 5800
+	1    0    0    -1
+$EndComp
+$Comp
+L 10005011_Power_Management:+3.3V #PWR0119
+U 1 1 5E99E15A
+P 10550 7850
+F 0 "#PWR0119" H 10550 7700 50  0001 C CNN
+F 1 "+3.3V" H 10565 8023 50  0000 C CNN
+F 2 "" H 10550 7850 50  0001 C CNN
+F 3 "" H 10550 7850 50  0001 C CNN
+	1    10550 7850
+	1    0    0    -1
+$EndComp
+$Comp
+L 10005011_Power_Management:+3.3V #PWR0121
+U 1 1 5E9A4B97
+P 11800 8050
+F 0 "#PWR0121" H 11800 7900 50  0001 C CNN
+F 1 "+3.3V" H 11815 8223 50  0000 C CNN
+F 2 "" H 11800 8050 50  0001 C CNN
+F 3 "" H 11800 8050 50  0001 C CNN
+	1    11800 8050
+	1    0    0    -1
+$EndComp
+$Comp
+L 10005011_Power_Management:+3.3V #PWR0132
+U 1 1 5E9A6F6A
+P 13800 5750
+F 0 "#PWR0132" H 13800 5600 50  0001 C CNN
+F 1 "+3.3V" H 13815 5923 50  0000 C CNN
+F 2 "" H 13800 5750 50  0001 C CNN
+F 3 "" H 13800 5750 50  0001 C CNN
+	1    13800 5750
+	1    0    0    -1
+$EndComp
+$Comp
+L 10005011_Power_Management:+3.3V #PWR0133
+U 1 1 5E9A7D15
+P 7300 2350
+F 0 "#PWR0133" H 7300 2200 50  0001 C CNN
+F 1 "+3.3V" H 7315 2523 50  0000 C CNN
+F 2 "" H 7300 2350 50  0001 C CNN
+F 3 "" H 7300 2350 50  0001 C CNN
+	1    7300 2350
+	1    0    0    -1
+$EndComp
+NoConn ~ 6200 2550
+NoConn ~ 6300 2550
+NoConn ~ 6400 2550
+NoConn ~ 6500 2550
+NoConn ~ 6600 2550
+NoConn ~ 6700 2550
+NoConn ~ 6800 2550
+$Comp
+L 10005011_Power_Management:+3.3V #PWR0135
+U 1 1 5E99B62E
+P 2700 3950
+F 0 "#PWR0135" H 2700 3800 50  0001 C CNN
+F 1 "+3.3V" H 2715 4123 50  0000 C CNN
+F 2 "" H 2700 3950 50  0001 C CNN
+F 3 "" H 2700 3950 50  0001 C CNN
+	1    2700 3950
+	1    0    0    -1
+$EndComp
 Wire Bus Line
 	9750 5850 9750 7350

Commit message: Powermanagement dev, ERC
Parts:
- IC16: value CY7C1021DV33 -> CY7C1021CV33
- J14: value Conn_01x04_Male -> EEPROM LOADER
Connections:
- net MRSR-SPI-1 renamed MTSR-SPI-1
Changed lines of the file:
@@
 U 1 1 5EA0D50B
 P 7250 5600
+AR Path="/5EA0D50B" Ref="IC15"  Part="1"
+AR Path="/5E9C3EF6/5EA0D50B" Ref="IC15"  Part="1"
 F 0 "IC15" H 8650 3100 60  0000 C CNN
 F 1 "CY7C67300-100AXI" H 9000 3000 60  0000 C CNN
@@
 SCLK-SPI-1
 Text GLabel 1750 4750 0    50   Input ~ 0
-MRSR-SPI-1
+MTSR-SPI-1
 Wire Wire Line
 	1750 4550 2100 4550
@@
 	4400 10000 3600 10000
 Wire Wire Line
-	4100 8550 3600 8550
-Wire Wire Line
 	3600 6600 3600 8550
 Connection ~ 3600 8550
@@
 Connection ~ 3200 9150
 Wire Wire Line
-	3200 9150 3200 9550
+	3200 9150 3200 9300
 Connection ~ 2600 9550
 $Comp
@@
 P 1550 9650
 F 0 "J14" H 1523 9578 50  0000 R CNN
-F 1 "Conn_01x04_Male" H 1522 9623 50  0001 R CNN
+F 1 "EEPROM LOADER" H 1522 9623 50  0001 R CNN
 F 2 "10005011 Power Management:B4BZR-SM3TF_1" H 1550 9650 50  0001 C CNN
 F 3 "~" H 1550 9650 50  0001 C CNN
@@
 P 13350 7150
 F 0 "IC16" H 13800 8150 50  0000 C CNN
-F 1 "CY7C1021DV33" H 14000 8050 50  0000 C CNN
+F 1 "CY7C1021CV33" H 14000 8050 50  0000 C CNN
 F 2 "10005011 Power Management:TSOP2-44_1" H 13350 6990 50  0001 C CNN
-F 3 "https://www.cypress.com/file/42751/download" H 12500 7300 50  0001 C CNN
+F 3 "https://www.cypress.com/file/38801/download" H 12500 7300 50  0001 C CNN
 F 4 "IC,RAM,3V3,64KX16,10NS,TSOP" H 14600 3400 50  0001 C CNN "Description"
 F 5 "10022899" H 14500 3500 50  0001 C CNN "Item Number"
@@
 	15100 2350 15500 2350
 Wire Wire Line
-	15500 2350 15500 1850
+	15500 2350 15500 2000
 Wire Wire Line
 	15600 1650 15600 1850
@@
 	15500 1850 15500 1650
 Wire Wire Line
-	15200 1050 15100 1050
+	15200 1050 15150 1050
 Wire Wire Line
 	14800 1050 14600 1050
@@
 	15100 4250 15500 4250
 Wire Wire Line
-	15500 4250 15500 3750
+	15500 4250 15500 3900
 Wire Wire Line
 	15600 3550 15600 3750
@@
 	15500 3750 15500 3550
 Wire Wire Line
-	15200 2950 15100 2950
+	15200 2950 15150 2950
 Wire Wire Line
 	14800 2950 14600 2950
@@
 	1    0    0    -1
 $EndComp
+$Comp
+L power:PWR_FLAG #FLG0119
+U 1 1 5F150EFA
+P 3500 9100
+F 0 "#FLG0119" H 3500 9175 50  0001 C CNN
+F 1 "PWR_FLAG" H 3500 9250 50  0000 C CNN
+F 2 "" H 3500 9100 50  0001 C CNN
+F 3 "~" H 3500 9100 50  0001 C CNN
+	1    3500 9100
+	1    0    0    -1
+$EndComp
+Wire Wire Line
+	3500 9100 3500 9300
+Wire Wire Line
+	3600 8550 4100 8550
+Wire Wire Line
+	3500 9300 3200 9300
+Connection ~ 3200 9300
+Wire Wire Line
+	3200 9300 3200 9550
+$Comp
+L power:PWR_FLAG #FLG0122
+U 1 1 5F23A015
+P 15200 1850
+F 0 "#FLG0122" H 15200 1925 50  0001 C CNN
+F 1 "PWR_FLAG" H 15200 2000 50  0000 C CNN
+F 2 "" H 15200 1850 50  0001 C CNN
+F 3 "~" H 15200 1850 50  0001 C CNN
+	1    15200 1850
+	1    0    0    -1
+$EndComp
+$Comp
+L power:PWR_FLAG #FLG0123
+U 1 1 5F2421C3
+P 15150 800
+F 0 "#FLG0123" H 15150 875 50  0001 C CNN
+F 1 "PWR_FLAG" H 15150 950 50  0000 C CNN
+F 2 "" H 15150 800 50  0001 C CNN
+F 3 "~" H 15150 800 50  0001 C CNN
+	1    15150 800
+	1    0    0    -1
+$EndComp
+$Comp
+L power:PWR_FLAG #FLG0124
+U 1 1 5F2428E5
+P 15150 2750
+F 0 "#FLG0124" H 15150 2825 50  0001 C CNN
+F 1 "PWR_FLAG" H 15150 2900 50  0000 C CNN
+F 2 "" H 15150 2750 50  0001 C CNN
+F 3 "~" H 15150 2750 50  0001 C CNN
+	1    15150 2750
+	1    0    0    -1
+$EndComp
+$Comp
+L power:PWR_FLAG #FLG0125
+U 1 1 5F243226
+P 15200 3750
+F 0 "#FLG0125" H 15200 3825 50  0001 C CNN
+F 1 "PWR_FLAG" H 15200 3900 50  0000 C CNN
+F 2 "" H 15200 3750 50  0001 C CNN
+F 3 "~" H 15200 3750 50  0001 C CNN
+	1    15200 3750
+	1    0    0    -1
+$EndComp
+Wire Wire Line
+	15200 1850 15200 2000
+Wire Wire Line
+	15200 2000 15500 2000
+Connection ~ 15500 2000
+Wire Wire Line
+	15500 2000 15500 1850
+Wire Wire Line
+	15150 800  15150 1050
+Connection ~ 15150 1050
+Wire Wire Line
+	15150 1050 15100 1050
+Wire Wire Line
+	15150 2750 15150 2950
+Connection ~ 15150 2950
+Wire Wire Line
+	15150 2950 15100 2950
+Wire Wire Line
+	15200 3750 15200 3900
+Wire Wire Line
+	15200 3900 15500 3900
+Connection ~ 15500 3900
+Wire Wire Line
+	15500 3900 15500 3750
 Wire Bus Line
 	9750 5850 9750 7350

Commit message: merge duplicated symbol
Parts:
- J12: footprint 10005011 Power Management:MOL47500-0001_2 -> 10005011 Power Management:MOL47500-0001_1

Commit message: update fp path
Parts:
- C101, C102, C103, C104, C105, C120, C121, C122, C123, C129, C130, C85, C86, C87, C88, C91, C92, C93, C96, C97: footprint 10005011 Power Management:C0402_1 -> AllModules:C0402_1
- C89: footprint 10005011 Power Management:RC1206-AIROX-KEMET-C1206C107A6 -> AllModules:RC1206-AIROX-KEMET-C1206C107A6
- C94, C95: footprint 10005011 Power Management:C0603_1 -> AllModules:C0603_1
- D15: footprint 10005011 Power Management:SOT23-1G_1 -> AllModules:SOT23-1G_1
- IC15: footprint 10005011 Power Management:TQFP100_1 -> AllModules:TQFP100_1
- IC16: footprint 10005011 Power Management:TSOP2-44_1 -> AllModules:TSOP2-44_1
- IC17: footprint 10005011 Power Management:MX.A8M_1 -> AllModules:MX.A8M_1
- IC18, IC19, IC20: footprint 10005011 Power Management:uSO08_1 -> AllModules:uSO08_1
- IC2: footprint 10005011 Power Management:SOT23-5_1 -> AllModules:SOT23-5_1
- J12, J13: footprint 10005011 Power Management:MOL47500-0001_1 -> AllModules:MOL47500-0001_1
- J14: footprint 10005011 Power Management:B4BZR-SM3TF_1 -> AllModules:B4BZR-SM3TF_1
- L10, L24, L25, L26: footprint 10005011 Power Management:C0805-AIROX-MURATA-BLM21PG221D -> AllModules:C0805-AIROX-MURATA-BLM21PG221D
- L11, L9: footprint 10005011 Power Management:DLP31S-AIROX_1 -> AllModules:DLP31S-AIROX_1
- L13, L14: footprint 10005011 Power Management:C1210_1 -> AllModules:C1210_1
- ML6, ML8, PG3, PG4, PG5, PG6, R102, R103, R104, R105, R106, R40, R68, R8: footprint 10005011 Power Management:R0603_1 -> AllModules:R0603_1
- PCT1: footprint 10005011 Power Management:C1812_1 -> AllModules:C1812_1
- PST10, PST11: footprint 10005011 Power Management:TEST-CMS-0.8_1 -> AllModules:TEST-CMS-0.8_1
- Q3: footprint 10005011 Power Management:HC49-4HSMX_1 -> AllModules:HC49-4HSMX_1
- SW2: footprint 10005011 Power Management:MCDMR-02T_1 -> AllModules:MCDMR-02T_1
