File: 10005011 Power Management/10005011 PIC-Micro.sch (KiCad schematic (older format))
At the start: 41 parts, among them IC1 LM393D, IC3 PIC18F6622, IC5 DS2480B, J2 ICSP, T2 IRLML5103

Commit message: Merge branch powermanagement-dev_DotMatrix2
Parts:
- renumbered TP2 to PST2, TP3 to PST3, TP4 to PST4, TP5 to PST5, TP6 to PST6, TP7 to PST7, TP8 to PST8
Other:
- note added: "Notes:\n2. ML5 not populated? Was marked "NC" on original schematic.\n3. TX and RX labels are transposed from original."
- note removed: "Notes:\n1. DS2480B needs to be updated with all required fields.\n2. ML5 not populated? Was marked "NC" on original schematic.\n3. TX and RX labels are transposed from original."
Changed lines of the file:
@@
 	4100 8050 3700 8050
 $Comp
-L Connector:TestPoint_Alt TP4
+L Connector:TestPoint_Alt PST4
 U 1 1 5FEC955B
 P 5650 3050
-F 0 "TP4" V 5604 3238 50  0000 L CNN
+F 0 "PST4" V 5604 3238 50  0000 L CNN
 F 1 "PST4" V 5695 3238 50  0000 L CNN
 F 2 "" H 5850 3050 50  0001 C CNN
@@
 $EndComp
 $Comp
-L Connector:TestPoint_Alt TP5
+L Connector:TestPoint_Alt PST5
 U 1 1 5FEC955C
 P 5650 3250
-F 0 "TP5" V 5604 3438 50  0000 L CNN
+F 0 "PST5" V 5604 3438 50  0000 L CNN
 F 1 "PST5" V 5695 3438 50  0000 L CNN
 F 2 "" H 5850 3250 50  0001 C CNN
@@
 	5050 2450 5250 2450
 $Comp
-L Connector:TestPoint_Alt TP2
+L Connector:TestPoint_Alt PST2
 U 1 1 5E97C137
 P 5650 2650
-F 0 "TP2" V 5604 2838 50  0000 L CNN
+F 0 "PST2" V 5604 2838 50  0000 L CNN
 F 1 "PST2" V 5695 2838 50  0000 L CNN
 F 2 "" H 5850 2650 50  0001 C CNN
@@
 $EndComp
 $Comp
-L Connector:TestPoint_Alt TP3
+L Connector:TestPoint_Alt PST3
 U 1 1 5E97C13E
 P 5650 2850
-F 0 "TP3" V 5604 3038 50  0000 L CNN
+F 0 "PST3" V 5604 3038 50  0000 L CNN
 F 1 "PST3" V 5695 3038 50  0000 L CNN
 F 2 "" H 5850 2850 50  0001 C CNN
@@
 	2900 2250 2750 2250
 $Comp
-L Connector:TestPoint_Alt TP8
+L Connector:TestPoint_Alt PST8
 U 1 1 5E97C164
 P 2350 3050
-F 0 "TP8" H 2408 3168 50  0000 L CNN
+F 0 "PST8" H 2408 3168 50  0000 L CNN
 F 1 "PST8" H 2408 3077 50  0000 L CNN
 F 2 "" H 2550 3050 50  0001 C CNN
@@
 $EndComp
 $Comp
-L Connector:TestPoint_Alt TP7
+L Connector:TestPoint_Alt PST7
 U 1 1 5E97C16B
 P 2450 3250
-F 0 "TP7" H 2508 3368 50  0000 L CNN
+F 0 "PST7" H 2508 3368 50  0000 L CNN
 F 1 "PST7" H 2508 3277 50  0000 L CNN
 F 2 "" H 2650 3250 50  0001 C CNN
@@
 $EndComp
 $Comp
-L Connector:TestPoint_Alt TP6
+L Connector:TestPoint_Alt PST6
 U 1 1 5FEC9561
 P 2550 3450
-F 0 "TP6" H 2608 3568 50  0000 L CNN
+F 0 "PST6" H 2608 3568 50  0000 L CNN
 F 1 "PST6" H 2608 3477 50  0000 L CNN
 F 2 "" H 2750 3450 50  0001 C CNN
@@
 $EndComp
 Text Notes 9850 8650 0    118  ~ 0
-Notes:\n1. DS2480B needs to be updated with all required fields.\n2. ML5 not populated?  Was marked "NC" on original schematic.\n3. TX and RX labels are transposed from original.
-$Comp
-L power:GND #PWR?
+Notes:\n2. ML5 not populated?  Was marked "NC" on original schematic.\n3. TX and RX labels are transposed from original.
+$Comp
+L power:GND #PWR?

Commit message: updating footprints
Parts:
- C16, C82: footprint Capacitor_SMD:C_0402_1005Metric -> 10005011 Power Management:C0402_1
- ML5, R11: footprint Resistor_SMD:R_0603_1608Metric -> 10005011 Power Management:R0603_1
Changed lines of the file:
@@
 F 0 "R11" V 12153 7050 50  0000 C CNN
 F 1 "100" V 12244 7050 50  0000 C CNN
-F 2 "Resistor_SMD:R_0603_1608Metric" V 12380 7050 50  0001 C CNN
+F 2 "10005011 Power Management:R0603_1" V 12380 7050 50  0001 C CNN
 F 3 "https://www.bourns.com/docs/Product-Datasheets/CHPREZTR.pdf" H 12450 7050 50  0001 C CNN
 F 4 "Bourns Inc." H 12450 7050 50  0001 C CNN "Mfgr"
@@
 F 0 "C16" H 12215 7391 50  0000 L CNN
 F 1 "470pF" H 12215 7300 50  0000 L CNN
-F 2 "Capacitor_SMD:C_0402_1005Metric" H 12138 7150 50  0001 C CNN
+F 2 "10005011 Power Management:C0402_1" H 12138 7150 50  0001 C CNN
 F 3 "https://psearch.en.murata.com/capacitor/product/GCM155R71H471KA37%23.pdf" H 12100 7300 50  0001 C CNN
 F 4 "Murata Electronics" H 12100 7300 50  0001 C CNN "Mfgr"
@@
 F 0 "C82" H 12886 6637 50  0000 R CNN
 F 1 "0.1uF" H 12886 6546 50  0000 R CNN
-F 2 "Capacitor_SMD:C_0402_1005Metric" H 13038 6350 50  0001 C CNN
+F 2 "10005011 Power Management:C0402_1" H 13038 6350 50  0001 C CNN
 F 3 "https://psearch.en.murata.com/capacitor/product/GCM155R71C104KA55%23.pdf" H 13000 6500 50  0001 C CNN
 F 4 "Murata Electronics" H 13000 6500 50  0001 C CNN "Mfgr"
@@
 F 0 "ML5" H 12903 7491 50  0000 L CNN
 F 1 "NC" H 12903 7400 50  0000 L CNN
-F 2 "Resistor_SMD:R_0603_1608Metric" V 12730 7400 50  0001 C CNN
+F 2 "10005011 Power Management:R0603_1" V 12730 7400 50  0001 C CNN
 F 3 "https://www.tdk-electronics.tdk.com/inf/75/db/CTVS_14/Standard_series.pdf" H 12800 7400 50  0001 C CNN
 F 4 "Digi-Key" H 12800 7400 50  0001 C CNN "Source"

Commit message: assigned footprints with cmp file
Parts:
- C12, C13, C15, C17, C4, C6, C63, C64: footprint (none) -> 10005011 Power Management:C0402_1
- CT1: footprint Resistor_SMD:R_0603_1608Metric -> 10005011 Power Management:K164_1
- D1: footprint (none) -> 10005011 Power Management:SOT23-1G_1
- IC1: footprint (none) -> 10005011 Power Management:MX.A8_COMPOSANT_1
- IC3: footprint Package_QFP:TQFP-64_10x10mm_P0.5mm -> 10005011 Power Management:TQFP64_1
- IC5: footprint Package_SO:SOIC-8_3.9x4.9mm_P1.27mm -> 10005011 Power Management:MX.A8_COMPOSANT_1
- J2: footprint (none) -> 10005011 Power Management:B6BZR-SM3TF_1; symbol Connector:Conn_01x06_Female -> Connector:Conn_01x08_Female
- PST2, PST3, PST4, PST5, PST6, PST7, PST8: footprint (none) -> 10005011 Power Management:TEST-CMS-0.8_1
- R1, R10, R108, R109, R110, R111, R112, R14, R15, R16, R17, R2, R4, R9, R98: footprint (none) -> 10005011 Power Management:R0603_1
- T2: footprint (none) -> 10005011 Power Management:SOT23-GSD_1
Connections:
- no-connect marks 9 -> 11
Other:
- note added: "TODO: T2 symbol pin names"

Commit message: remove text
Other:
- note removed: "TODO: T2 symbol pin names"
Changed lines of the file:
@@
 Text GLabel 5350 4350 2    50   Output ~ 0
 LED-BATTERY-STATUS
-Text Notes 4900 9950 0    197  ~ 0
-TODO: T2 symbol pin names
 NoConn ~ 1950 9000
 NoConn ~ 1950 8900
