File: 10005011 Power Management/10005011 Switching-ExtPWR.sch (KiCad schematic (older format))
At the start: 98 parts, among them IC21 LT1716IS5, IC22 LT1716IS5, IC23 LM4040DIM3-5.0, IC24 LM4040DIM3-5.0, IC28 L78M05CDT, IC7 INA170, J3 DC, J4 AC, J5 EXT DC, SW1 CMF2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

Commit message: conflict solved, two FLTR2
Parts:
- FLTR2: value BNX002-11 -> BNX002-1
Changed lines of the file:
@@
-	1    0    0    -1
-$EndComp
-$Comp
-L 10005011_Power_Management:BNX002-11 FLTR?
-U 1 1 5F74A76D
-P 13100 5550
-AR Path="/5E92767C/5F74A76D" Ref="FLTR?"  Part="1"
-AR Path="/5FEC5422/5F74A76D" Ref="FLTR2"  Part="1"
-F 0 "FLTR2" H 13075 5923 50  0000 C CNN
-F 1 "BNX002-11" H 13075 5832 50  0000 C CNN
-F 2 "10005011 Power Management:BNX002_1" H 12990 5570 50  0001 C CNN
-F 3 "https://www.murata.com/en-us/api/pdfdownloadapi?cate=luNoiseSupprFilteBlockType&partno=BNX002-11" H 12990 5570 50  0001 C CNN
-F 4 "10022532" H 12990 5570 50  0001 C CNN "Item Number"
-F 5 "Murata" H 12990 5570 50  0001 C CNN "Manufacturer"
-F 6 "BNX002-11" H 13100 5550 50  0001 C CNN "MPN"
-F 7 "BNX002-11" H 13100 5550 50  0001 C CNN "Manufacturer_No"
-F 8 "FILTER CC, 1MHZ-1GHZ, 10A, 50V" H 13100 5550 50  0001 C CNN "Description"
-	1    13100 5550
 	1    0    0    -1
 $EndComp
@@
 Wire Wire Line
 	13500 5450 13850 5450
+$Comp
+L 10005011_Power_Management:BNX002-11 FLTR?
+U 1 1 5F74A76D
+P 13100 5550
+AR Path="/5E92767C/5F74A76D" Ref="FLTR?"  Part="1"
+AR Path="/5FEC5422/5F74A76D" Ref="FLTR2"  Part="1"
+F 0 "FLTR2" H 13075 5923 50  0000 C CNN
+F 1 "BNX002-1" H 13075 5832 50  0000 C CNN
+F 2 "10005011 Power Management:BNX002_1" H 12990 5570 50  0001 C CNN
+F 3 "https://www.murata.com/en-us/api/pdfdownloadapi?cate=luNoiseSupprFilteBlockType&partno=BNX002-11" H 12990 5570 50  0001 C CNN
+F 4 "10022532" H 12990 5570 50  0001 C CNN "Item Number"
+F 5 "Murata" H 12990 5570 50  0001 C CNN "Manufacturer"
+F 6 "BNX002-11" H 13100 5550 50  0001 C CNN "MPN"
+F 7 "BNX002-11" H 13100 5550 50  0001 C CNN "Manufacturer_No"
+F 8 "FILTER CC, 1MHZ-1GHZ, 10A, 50V" H 13100 5550 50  0001 C CNN "Description"
+	1    13100 5550
+	1    0    0    -1
+$EndComp
 $EndSCHEMATC

Commit message: solved repeated Res and Ind
Parts:
- renumbered R31 to R30
Changed lines of the file:
@@
 	3200 2000 3550 2000
 $Comp
-L Device:R R31
+L Device:R R30
 U 1 1 5EA66D0F
 P 3750 3050
-F 0 "R31" H 3820 3096 50  0000 L CNN
+F 0 "R30" H 3820 3096 50  0000 L CNN
 F 1 "10k" H 3820 3005 50  0000 L CNN
 F 2 "10005011 Power Management:R0603_1" V 3680 3050 50  0001 C CNN

Commit message: Powermanagement dev sheet2
Parts:
- added ML4: Varistor, 10005011 Power Management:RC1206_1, symbol Device:Varistor
- D17, D18: footprint 10005011 Power Management:SOT23-1G_1 -> Package_TO_SOT_SMD:SOT-23; symbol Device:D_Schottky -> 10005011_Power_Management:BAT54; Description (none) -> DIODE SCHOTTKY 30V 200MA SOT23-3; Item Number (none) -> 10022652; Mfgr (none) -> ON Semiconductor; Mfgr_PN (none) -> BAT54LT1G; Source (none) -> Digi-Key; Source_PN (none) -> BAT54LT1GOSTR-ND
- D19: symbol 10005011_Power_Management_Schematic_Symbols:1N5819 -> 10005011_Power_Management:1N5819; Item Number (none) -> 10022650
- D3: symbol 10005011_Power_Management_Schematic_Symbols:SZ1SMB -> 10005011_Power_Management:SZ1SMB
- IC23, IC24: symbol Reference_Voltage:LM4040DBZ-5 -> 10005011_Power_Management:LM4040DIM3-5.0; Description (none) -> IC,VOLTAGE REFERENCE,SHUNT, 5V,SOT23; Item Number (none) -> 10022903; Manufacturer (none) -> NATIONAL SEMICONDUCTOR; Manufacturer_No (none) -> LM4040DIM3-5.0
- J5: symbol Connector:Conn_01x06_Male -> Connector:Conn_01x10_Male
- R45: value .015 1% -> 0.015; Description (none) -> RESISTOR, 0.015 OHM, 1W,+/-1%,2010; Item Number (none) -> 10022710; Tolerance (none) -> 1%
- T10, T15, T3, T4, T5: symbol Transistor_FET:SUD50P06-15 -> 10005011_Power_Management:SUD50P06-15L-E3
- T11, T6: symbol Device:Q_PMOS_GSD -> 10005011_Power_Management:IRLML5103TRPBF
- T12, T13, T17, T7, T8: symbol Transistor_FET:2N7002 -> 10005011_Power_Management:2N7002
- T14: symbol Transistor_FET:SUD50P06-15 -> 10005011_Power_Management:SUD50P06-15L-E3; BOM_Footprint (none) -> DPAK; Description (none) -> MOSFET P-CH 60V 50A TO252; Item Number (none) -> 10022560; Mfgr (none) -> Vishay Siliconix; Mfgr_PN (none) -> SUD50P06-15L-E3; Source (none) -> Digi-Key; Source_PN (none) -> SUD50P06-15L-E3CT-ND
- T16: symbol Device:Q_PMOS_GSD -> 10005011_Power_Management:IRLML5103TRPBF; Description (none) -> MOSFET P-CH 30V 760MA SOT-23; Item Number (none) -> 10022933; Mfgr (none) -> Infineon Technologies; Mfgr_PN (none) -> IRLML5103TRPBF; Source (none) -> Digi-Key; Source_PN (none) -> IRLML5103PBFCT-ND
- T18: symbol Transistor_FET:2N7002 -> 10005011_Power_Management:2N7002; Description (none) -> MOSFET N-CH 60V 350MA SOT23; Item Number (none) -> 10022882; Mfgr (none) -> Diodes Incorporated; Mfgr_PN (none) -> 2N7002AQ-7; Source (none) -> Digi-Key; Source_PN (none) -> 2N7002AQ-7DICT-ND
- T9: symbol Transistor_FET:SUD50P06-15 -> 10005011_Power_Management:SUD50P06-15L-E3; Description (none) -> MOSFET P-CH 60V 50A TO252; Item Number (none) -> 10022560; Mfgr (none) -> Vishay Siliconix; Mfgr_PN (none) -> SUD50P06-15L-E3; Source (none) -> Digi-Key; Source_PN (none) -> SUD50P06-15L-E3CT-ND
Connections:
- wire segments 394 -> 398
Other:
- moved on the sheet: C106, C107, C108, C132, C133, C140, C141, C18, C19, C22, C23, C24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

Commit message: use standard kicad library for C and R in sheets1-3
Parts:
- C106: value 0.1uF_0805 -> 0.1uF; symbol 10005011_Power_Management_Schematic_Symbols:0.1uF_0805 -> Device:C
- D2: symbol 10005011_Power_Management_Schematic_Symbols:BAT54C -> 10005011_Power_Management:BAT54C
- R107: symbol 10005011_Power_Management_Schematic_Symbols:66.5k -> Device:R
Changed lines of the file:
@@
 Connection ~ 11600 5000
 $Comp
-L 10005011_Power_Management_Schematic_Symbols:0.1uF_0805 C106
+L Device:C C106
 U 1 1 5E9BAE39
 P 12500 5150
 F 0 "C106" H 12615 5059 50  0000 L CNN
-F 1 "0.1uF_0805" H 12615 5150 50  0000 L CNN
+F 1 "0.1uF" H 12615 5150 50  0000 L CNN
 F 2 "10005011 Power Management:C0805_1" H 12538 5000 50  0001 C CNN
 F 3 "https://www.yageo.com/upload/media/product/productsearch/datasheet/mlcc/UPY-GPHC_X7R_6.3V-to-50V_18.pdf" H 12500 5150 50  0001 C CNN
@@
 F 6 "Digi-Key" H 12500 5150 50  0001 C CNN "Source"
 F 7 "311-1140-1-ND" H 12500 5150 50  0001 C CNN "Source_PN"
-F 8 "0805" H 12615 5241 50  0000 L CNN "Bom_Footprint"
+F 8 "0805" H 12615 5241 50  0001 L CNN "Bom_Footprint"
 F 9 "CAP CER 0.1UF 50V X7R 0805" H 12500 5150 50  0001 C CNN "Description"
 F 10 "X7R" H 12500 5150 50  0001 C CNN "Dielectric"
@@
 ON-OFF
 $Comp
-L 10005011_Power_Management_Schematic_Symbols:66.5k R107
+L Device:R R107
 U 1 1 5F290125
 P 1800 10200
@@
 	7350 1950 7350 1900
 $Comp
-L 10005011_Power_Management_Schematic_Symbols:BAT54C D2
+L 10005011_Power_Management:BAT54C D2
 U 1 1 5F1F8D7E
 P 7350 1700

Commit message: Powermanagement dev library
Parts:
- C106: value 0.1uF -> 100nF; Bom_Footprint 0805 -> (none); Description CAP CER 0.1UF 50V X7R 0805 -> CAPACITOR CERAMIC, 100NF, +/-10%, 50V, X7R,0805; Item Number (none) -> 10022135
- C132, C133, C140, C141, C23: Description (none) -> CAPACITOR CERAMIC, 100NF, +/-10%, 50V, X7R,0805; Item Number (none) -> 10022135
- D13: symbol 10005011_Power_Management_Schematic_Symbols:SMCJ33C -> Device:D_TVS; Description TRANSIENT VOLTAGE SUPPRESSOR,SMC -> DIODE, 33V, VCL 53.3V, 1500W; Item Number (none) -> 10022658
- D17, D18: footprint Package_TO_SOT_SMD:SOT-23 -> 10005011 Power Management:SOT23-1G_1
- D2: BOM_Footprint SOT23 -> (none); Item Number (none) -> 10022653
- D3: Item Number (none) -> 10022654
- IC7: symbol page2:INA170 -> 10005011_Power_Management:INA170; Description (none) -> IC,CURRENT SHUNT MONITOR,MSOP; Item Number (none) -> 10022891; Manufacturer (none) -> TEXAS INSTRUMENTS; Manufacturer_No (none) -> INA170EA
- SW1: symbol page2:CMF2 -> 10005011_Power_Management:CMF2; Description (none) -> SWITCH SOCKET 2 POLES; Item Number (none) -> 10022930; Manufacturer (none) -> SCHURTER; Manufacturer_No (none) -> CMF2.1011.12
Changed lines of the file:
@@
 F 2 "10005011 Power Management:C0805_1" H 838 9150 50  0001 C CNN
 F 3 "~" H 800 9300 50  0001 C CNN
+F 4 "CAPACITOR CERAMIC, 100NF, +/-10%, 50V, X7R,0805" H 800 9300 50  0001 C CNN "Description"
+F 5 "10022135" H 800 9300 50  0001 C CNN "Item Number"
 	1    800  9300
 	1    0    0    -1
@@
 Connection ~ 6500 7900
 $Comp
-L page2:INA170 IC7
+L 10005011_Power_Management:INA170 IC7
 U 1 1 5EADCC7F
 P 1700 9550
@@
 F 2 "10005011 Power Management:uSO08_1" H 1700 8900 50  0001 C CNN
 F 3 "https://www.ti.com/lit/ds/symlink/ina170.pdf" H 1850 9700 50  0001 C CNN
+F 4 "IC,CURRENT SHUNT MONITOR,MSOP" H 1700 9550 50  0001 C CNN "Description"
+F 5 "10022891" H 1700 9550 50  0001 C CNN "Item Number"
+F 6 "TEXAS INSTRUMENTS" H 1700 9550 50  0001 C CNN "Manufacturer"
+F 7 "INA170EA" H 1700 9550 50  0001 C CNN "Manufacturer_No"
 	1    1700 9550
 	1    0    0    -1
@@
 P 12500 5150
 F 0 "C106" H 12615 5059 50  0000 L CNN
-F 1 "0.1uF" H 12615 5150 50  0000 L CNN
+F 1 "100nF" H 12615 5150 50  0000 L CNN
 F 2 "10005011 Power Management:C0805_1" H 12538 5000 50  0001 C CNN
 F 3 "https://www.yageo.com/upload/media/product/productsearch/datasheet/mlcc/UPY-GPHC_X7R_6.3V-to-50V_18.pdf" H 12500 5150 50  0001 C CNN
@@
 F 6 "Digi-Key" H 12500 5150 50  0001 C CNN "Source"
 F 7 "311-1140-1-ND" H 12500 5150 50  0001 C CNN "Source_PN"
-F 8 "0805" H 12615 5241 50  0001 L CNN "Bom_Footprint"
-F 9 "CAP CER 0.1UF 50V X7R 0805" H 12500 5150 50  0001 C CNN "Description"
+F 8 "" H 12615 5241 50  0001 L CNN "Bom_Footprint"
+F 9 "CAPACITOR CERAMIC, 100NF, +/-10%, 50V, X7R,0805" H 12500 5150 50  0001 C CNN "Description"
 F 10 "X7R" H 12500 5150 50  0001 C CNN "Dielectric"
 F 11 "50V" H 12500 5150 50  0001 C CNN "Voltage"
+F 12 "10022135" H 12500 5150 50  0001 C CNN "Item Number"
 	1    12500 5150
 	1    0    0    1
@@
 $EndComp
 $Comp
-L 10005011_Power_Management_Schematic_Symbols:SMCJ33C D13
+L Device:D_TVS D13
 U 1 1 5E9C7BFC
 P 14900 5250
@@
 F 6 "Digi-Key" H 14900 5250 50  0001 C CNN "Source"
 F 7 "SMCJ33CAQ-13-FDICT-ND" H 14900 5250 50  0001 C CNN "Source_PN"
-F 8 "TRANSIENT VOLTAGE SUPPRESSOR,SMC" H 14900 5250 50  0001 C CNN "Description"
+F 8 "DIODE, 33V, VCL 53.3V, 1500W" H 14900 5250 50  0001 C CNN "Description"
+F 9 "10022658" V 14900 5250 50  0001 C CNN "Item Number"
 	1    14900 5250
 	0    1    -1   0
@@
 	14900 5000 14900 5100
 $Comp
-L page2:ALIM1 #ALIM1
+L 10005011_Power_Management:ECM100US33>2413 #ALIM1
 U 1 1 5E985667
 P 13950 2150
@@
 F 2 "" H 13950 1800 100 0001 C CNN
 F 3 "" H 13950 1700 100 0001 C CNN
+F 4 "POWER SUPPLY, 220VAC, 33VDC, 100W" H 13950 2150 50  0001 C CNN "Description"
+F 5 "10022932" H 13950 2150 50  0001 C CNN "Item Number"
+F 6 "XP POWER PLC" H 13950 2150 50  0001 C CNN "Manufacturer"
+F 7 "ECM100US33>2413" H 13950 2150 50  0001 C CNN "Manufacturer_No"
 	1    13950 2150
 	1    0    0    -1
 $EndComp
 $Comp
-L page2:CMF2 SW1
+L 10005011_Power_Management:CMF2 SW1
 U 1 1 5E986E8B
 P 11350 2400
 F 0 "SW1" H 11433 3265 50  0000 C CNN
 F 1 "CMF2" H 11433 3174 50  0000 C CNN
-F 2 "10005011 Power Management:CMF1_1" H 11200 2450 50  0001 C CNN
-F 3 "https://www.schurter.com/en/datasheet/typ_CMF2__CMF5.pdf" H 11200 2450 50  0001 C CNN
+F 2 "10005011 Power Management:CMF1_1" H 11200 2450 100 0001 C CNN
+F 3 "https://www.schurter.com/en/datasheet/typ_CMF2__CMF5.pdf" H 11200 2450 100 0001 C CNN
+F 4 "SWITCH SOCKET 2 POLES" H 11350 2400 50  0001 C CNN "Description"
+F 5 "10022930" H 11350 2400 50  0001 C CNN "Item Number"
+F 6 "SCHURTER" H 11350 2400 50  0001 C CNN "Manufacturer"
+F 7 "CMF2.1011.12" H 11350 2400 50  0001 C CNN "Manufacturer_No"
 	1    11350 2400
 	1    0    0    -1
@@
 U 1 1 5FEEEA48
 P 10300 8250
-F 0 "D18" H 10250 8483 50  0000 C CNN
-F 1 "BAT54" H 10250 8574 50  0000 C CNN
-F 2 "Package_TO_SOT_SMD:SOT-23" H 10070 8088 50  0001 L CNN
+F 0 "D18" H 10250 8069 50  0000 C CNN
+F 1 "BAT54" H 10250 8160 50  0000 C CNN
+F 2 "10005011 Power Management:SOT23-1G_1" H 10070 8088 50  0001 L CNN
 F 3 "http://www.onsemi.com/pub/Collateral/BAT54LT1-D.PDF" H 10220 8350 50  0001 C CNN
 F 4 "DIODE SCHOTTKY 30V 200MA SOT23-3" H 10625 8075 60  0001 C CNN "Description"
@@
 F 2 "10005011 Power Management:C0805_1" H 9788 7500 50  0001 C CNN
 F 3 "~" H 9750 7650 50  0001 C CNN
+F 4 "CAPACITOR CERAMIC, 100NF, +/-10%, 50V, X7R,0805" H 9750 7650 50  0001 C CNN "Description"
+F 5 "10022135" H 9750 7650 50  0001 C CNN "Item Number"
 	1    9750 7650
 	0    -1   1    0
@@
 Wire Wire Line
 	12200 8450 12200 8550
-$Comp
-L 10005011_Power_Management:BAT54 D17
-U 1 1 60B18780
-P 14750 8350
-F 0 "D17" H 14700 8583 50  0000 C CNN
-F 1 "BAT54" H 14700 8674 50  0000 C CNN
-F 2 "Package_TO_SOT_SMD:SOT-23" H 14520 8188 50  0001 L CNN
-F 3 "http://www.onsemi.com/pub/Collateral/BAT54LT1-D.PDF" H 14670 8450 50  0001 C CNN
-F 4 "DIODE SCHOTTKY 30V 200MA SOT23-3" H 15075 8175 60  0001 C CNN "Description"
-F 5 "10022652" H 14750 8300 50  0001 C CNN "Item Number"
-F 6 "ON Semiconductor" H 15075 8175 60  0001 C CNN "Mfgr"
-F 7 "BAT54LT1G" H 15075 8175 60  0001 C CNN "Mfgr_PN"
-F 8 "Digi-Key" H 14925 8175 60  0001 C CNN "Source"
-F 9 "BAT54LT1GOSTR-ND" H 14900 8175 60  0001 C CNN "Source_PN"
-	1    14750 8350
-	-1   0    0    1
-$EndComp
 $Comp
 L Device:R R123
@@
 F 2 "10005011 Power Management:C0805_1" H 14238 7600 50  0001 C CNN
 F 3 "~" H 14200 7750 50  0001 C CNN
+F 4 "CAPACITOR CERAMIC, 100NF, +/-10%, 50V, X7R,0805" H 14200 7750 50  0001 C CNN "Description"
+F 5 "10022135" H 14200 7750 50  0001 C CNN "Item Number"
 	1    14200 7750
 	0    1    1    0
@@
 F 2 "10005011 Power Management:SOT23-1G_1" H 7075 1225 50  0001 L CNN
 F 3 "https://media.digikey.com/pdf/Data%20Sheets/ON%20Semiconductor%20PDFs/BAT54(A,C,S).pdf" H 7270 1800 50  0001 C CNN
-F 4 "SOT23" V 7391 1888 50  0000 L CNN "BOM_Footprint"
-F 5 "DIODE ARRAY SCHOTTKY 30V SOT23-3" H 7675 1525 60  0001 C CNN "Description"
-F 6 "ON Semiconductor" H 7675 1525 60  0001 C CNN "Mfgr"
-F 7 "BAT54C" H 7675 1525 60  0001 C CNN "Mfgr_PN"
-F 8 "Digi-Key" H 7525 1525 60  0001 C CNN "Source"
-F 9 "BAT54CFSCT-ND" H 7500 1525 60  0001 C CNN "Source_PN"
+F 4 "DIODE ARRAY SCHOTTKY 30V SOT23-3" H 7675 1525 60  0001 C CNN "Description"
+F 5 "ON Semiconductor" H 7675 1525 60  0001 C CNN "Mfgr"
+F 6 "BAT54C" H 7675 1525 60  0001 C CNN "Mfgr_PN"
+F 7 "Digi-Key" H 7525 1525 60  0001 C CNN "Source"
+F 8 "BAT54CFSCT-ND" H 7500 1525 60  0001 C CNN "Source_PN"
+F 9 "10022653" H 7350 1700 50  0001 C CNN "Item Number"
 	1    7350 1700
 	0    1    1    0
@@
 F 7 "F11561CT-ND" H 5450 1650 50  0001 C CNN "Source_PN"
 F 8 "TVS DIODE 36V 58.1V SMB" H 5450 1650 50  0001 C CNN "Description"
+F 9 "10022654" H 5450 1650 50  0001 C CNN "Item Number"
 	1    5450 1650
 	0    1    1    0
@@
 F 2 "10005011 Power Management:C0805_1" H 7388 4250 50  0001 C CNN
 F 3 "~" H 7350 4400 50  0001 C CNN
+F 4 "CAPACITOR CERAMIC, 100NF, +/-10%, 50V, X7R,0805" H 7350 4400 50  0001 C CNN "Description"
+F 5 "10022135" H 7350 4400 50  0001 C CNN "Item Number"
 	1    7350 4400
 	1    0    0    1
@@
 F 2 "10005011 Power Management:C0805_1" H 6388 4250 50  0001 C CNN
 F 3 "~" H 6350 4400 50  0001 C CNN
+F 4 "CAPACITOR CERAMIC, 100NF, +/-10%, 50V, X7R,0805" H 6350 4400 50  0001 C CNN "Description"
+F 5 "10022135" H 6350 4400 50  0001 C CNN "Item Number"
 	1    6350 4400
 	1    0    0    1
@@
 Wire Notes Line width 39
 	9300 3700 16050 3700
+$Comp
+L 10005011_Power_Management:BAT54 D17
+U 1 1 60B18780
+P 14750 8350
+F 0 "D17" H 14700 8169 50  0000 C CNN
+F 1 "BAT54" H 14700 8260 50  0000 C CNN
+F 2 "10005011 Power Management:SOT23-1G_1" H 14520 8188 50  0001 L CNN
+F 3 "http://www.onsemi.com/pub/Collateral/BAT54LT1-D.PDF" H 14670 8450 50  0001 C CNN
+F 4 "DIODE SCHOTTKY 30V 200MA SOT23-3" H 15075 8175 60  0001 C CNN "Description"
+F 5 "10022652" H 14750 8300 50  0001 C CNN "Item Number"
+F 6 "ON Semiconductor" H 15075 8175 60  0001 C CNN "Mfgr"
+F 7 "BAT54LT1G" H 15075 8175 60  0001 C CNN "Mfgr_PN"
+F 8 "Digi-Key" H 14925 8175 60  0001 C CNN "Source"
+F 9 "BAT54LT1GOSTR-ND" H 14900 8175 60  0001 C CNN "Source_PN"
+	1    14750 8350
+	-1   0    0    1
+$EndComp
 $EndSCHEMATC

Commit message: item 10022607
Parts:
- C108, C8: Description (none) -> CAPACITOR,100NF,16V,+/-10%,X7R,0402; Item Number (none) -> 10022607; Manufacturer (none) -> MURATA; Manufacturer_No (none) -> GRM155R71C104JA88J
Changed lines of the file:
@@
 F 2 "10005011 Power Management:C0402_1" H 8288 8550 50  0001 C CNN
 F 3 "~" H 8250 8700 50  0001 C CNN
+F 4 "CAPACITOR,100NF,16V,+/-10%,X7R,0402" H 8250 8700 50  0001 C CNN "Description"
+F 5 "10022607" H 8250 8700 50  0001 C CNN "Item Number"
+F 6 "MURATA" H 8250 8700 50  0001 C CNN "Manufacturer"
+F 7 "GRM155R71C104JA88J" H 8250 8700 50  0001 C CNN "Manufacturer_No"
 	1    8250 8700
 	-1   0    0    1
@@
 F 2 "10005011 Power Management:C0402_1" H 12738 8650 50  0001 C CNN
 F 3 "~" H 12700 8800 50  0001 C CNN
+F 4 "CAPACITOR,100NF,16V,+/-10%,X7R,0402" H 12700 8800 50  0001 C CNN "Description"
+F 5 "10022607" H 12700 8800 50  0001 C CNN "Item Number"
+F 6 "MURATA" H 12700 8800 50  0001 C CNN "Manufacturer"
+F 7 "GRM155R71C104JA88J" H 12700 8800 50  0001 C CNN "Manufacturer_No"
 	1    12700 8800
 	1    0    0    1

Commit message: IC21 and IC22 library included
Parts:
- IC21, IC22: symbol Comparator:MCP6561-OT -> 10005011_Power_Management:LT1716IS5; Description (none) -> IC,RAIL TO RAIL COMPARATOR, 44V, SOT23; Item Number (none) -> 10022902; Manufacturer (none) -> LINEAR TECHNOLOGY; Manufacturer_No (none) -> LT1716IS5#TRPBF
Changed lines of the file:
@@
 $EndComp
 $Comp
-L Comparator:MCP6561-OT IC21
+L 10005011_Power_Management:LT1716IS5 IC21
 U 1 1 5FF785A2
 P 9600 8350
@@
 F 2 "10005011 Power Management:SOT23-5_1" H 9500 8150 50  0001 L CNN
 F 3 "https://www.analog.com/media/en/technical-documentation/data-sheets/LT1716.pdf" H 9600 8550 50  0001 C CNN
+F 4 "IC,RAIL TO RAIL COMPARATOR, 44V, SOT23" H 9600 8350 50  0001 C CNN "Description"
+F 5 "10022902" H 9600 8350 50  0001 C CNN "Item Number"
+F 6 "LINEAR TECHNOLOGY" H 9600 8350 50  0001 C CNN "Manufacturer"
+F 7 "LT1716IS5#TRPBF" H 9600 8350 50  0001 C CNN "Manufacturer_No"
 	1    9600 8350
 	1    0    0    -1
@@
 $EndComp
 $Comp
-L Comparator:MCP6561-OT IC22
+L 10005011_Power_Management:LT1716IS5 IC22
 U 1 1 60B1879E
 P 14050 8450
@@
 F 2 "10005011 Power Management:SOT23-5_1" H 13950 8250 50  0001 L CNN
 F 3 "https://www.analog.com/media/en/technical-documentation/data-sheets/LT1716.pdf" H 14050 8650 50  0001 C CNN
+F 4 "IC,RAIL TO RAIL COMPARATOR, 44V, SOT23" H 14050 8450 50  0001 C CNN "Description"
+F 5 "10022902" H 14050 8450 50  0001 C CNN "Item Number"
+F 6 "LINEAR TECHNOLOGY" H 14050 8450 50  0001 C CNN "Manufacturer"
+F 7 "LT1716IS5#TRPBF" H 14050 8450 50  0001 C CNN "Manufacturer_No"
 	1    14050 8450
 	1    0    0    -1
