File: 10005011 Power Management/10005011 Buck-Boost 24V.sch (KiCad schematic (older format))
At the start: 63 parts, among them IC10 LTC3780, IC9 LT1620CMS8, T19 SI7884BDP, T20 SI7884BDP, T21 SI7884BDP, T22 SI7884BDP

Commit message: Powermanagement dev library
Parts:
- D12: symbol 10005011_Power_Management_Schematic_Symbols:BZX84C5V1 -> 10005011_Power_Management:BZX84C5V1; Description DIODE ZENER 5.1V 300MW SOT23-3 -> DIODE ZENER, 0.35,5.1V, SOT23; Item Number (none) -> 10022657
Other:
- moved on the sheet: T19, T20, T21, T22
Changed lines of the file:
@@
 L 10005011_Power_Management:SI7884BDP T20
 U 1 1 5EA1F704
-P 7800 2300
-F 0 "T20" H 7600 2550 50  0000 L CNN
-F 1 "SI7884BDP" H 7300 2450 50  0000 L CNN
-F 2 "10005011 Power Management:SO08-PPAD_SI7884_1" H 8650 2225 50  0001 C CIN
-F 3 "http://www.vishay.com/docs/68395/si7884bd.pdf" H 8125 2000 50  0001 L CNN
-F 4 "Digi-Key" H 8200 2225 50  0001 C CNN "Source"
-F 5 "SI7884BDP-T1-E3CT-ND" H 8450 2225 50  0001 C CNN "Source_PN"
-F 6 "MOSFET TRANS N CHANNEL,40V,12A,0.007 OHM, SO8" H 8600 2225 50  0001 C CNN "Description"
-F 7 "10022883" H 7800 2300 50  0001 C CNN "Item Number"
-F 8 "VISHAY" H 7800 2300 50  0001 C CNN "Manufacturer"
-F 9 "SI7848BDP-T1-E3" H 7800 2300 50  0001 C CNN "Manufacturer_No"
-	1    7800 2300
+P 7900 2300
+F 0 "T20" H 7700 2550 50  0000 L CNN
+F 1 "SI7884BDP" H 7400 2450 50  0000 L CNN
+F 2 "10005011 Power Management:SO08-PPAD_SI7884_1" H 8750 2225 50  0001 C CIN
+F 3 "http://www.vishay.com/docs/68395/si7884bd.pdf" H 8225 2000 50  0001 L CNN
+F 4 "Digi-Key" H 8300 2225 50  0001 C CNN "Source"
+F 5 "SI7884BDP-T1-E3CT-ND" H 8550 2225 50  0001 C CNN "Source_PN"
+F 6 "MOSFET TRANS N CHANNEL,40V,12A,0.007 OHM, SO8" H 8700 2225 50  0001 C CNN "Description"
+F 7 "10022883" H 7900 2300 50  0001 C CNN "Item Number"
+F 8 "VISHAY" H 7900 2300 50  0001 C CNN "Manufacturer"
+F 9 "SI7848BDP-T1-E3" H 7900 2300 50  0001 C CNN "Manufacturer_No"
+	1    7900 2300
 	-1   0    0    -1
 $EndComp
@@
 $EndComp
 $Comp
-L 10005011_Power_Management_Schematic_Symbols:BZX84C5V1 D12
+L 10005011_Power_Management:BZX84C5V1 D12
 U 1 1 5F0182BA
 P 10900 4800
@@
 F 6 "Digi-Key" H 10900 4800 50  0001 C CNN "Source"
 F 7 "BZX84C5V1-FDITR-ND" H 10900 4800 50  0001 C CNN "Source_PN"
-F 8 "DIODE ZENER 5.1V 300MW SOT23-3" H 10900 4800 50  0001 C CNN "Description"
+F 8 "DIODE ZENER, 0.35,5.1V, SOT23" H 10900 4800 50  0001 C CNN "Description"
+F 9 "10022657" H 10900 4800 50  0001 C CNN "Item Number"
 	1    10900 4800
 	0    1    1    0
@@
 L 10005011_Power_Management:SI7884BDP T19
 U 1 1 5E98B2EE
-P 6400 2300
-F 0 "T19" H 6200 2550 50  0000 L CNN
-F 1 "SI7884BDP" H 5900 2450 50  0000 L CNN
-F 2 "10005011 Power Management:SO08-PPAD_SI7884_1" H 7250 2225 50  0001 C CIN
-F 3 "http://www.vishay.com/docs/68395/si7884bd.pdf" H 6725 2000 50  0001 L CNN
-F 4 "Digi-Key" H 6800 2225 50  0001 C CNN "Source"
-F 5 "SI7884BDP-T1-E3CT-ND" H 7050 2225 50  0001 C CNN "Source_PN"
-F 6 "MOSFET TRANS N CHANNEL,40V,12A,0.007 OHM, SO8" H 7200 2225 50  0001 C CNN "Description"
-F 7 "10022883" H 6400 2300 50  0001 C CNN "Item Number"
-F 8 "VISHAY" H 6400 2300 50  0001 C CNN "Manufacturer"
-F 9 "SI7848BDP-T1-E3" H 6400 2300 50  0001 C CNN "Manufacturer_No"
-	1    6400 2300
+P 6300 2300
+F 0 "T19" H 6100 2550 50  0000 L CNN
+F 1 "SI7884BDP" H 5800 2450 50  0000 L CNN
+F 2 "10005011 Power Management:SO08-PPAD_SI7884_1" H 7150 2225 50  0001 C CIN
+F 3 "http://www.vishay.com/docs/68395/si7884bd.pdf" H 6625 2000 50  0001 L CNN
+F 4 "Digi-Key" H 6700 2225 50  0001 C CNN "Source"
+F 5 "SI7884BDP-T1-E3CT-ND" H 6950 2225 50  0001 C CNN "Source_PN"
+F 6 "MOSFET TRANS N CHANNEL,40V,12A,0.007 OHM, SO8" H 7100 2225 50  0001 C CNN "Description"
+F 7 "10022883" H 6300 2300 50  0001 C CNN "Item Number"
+F 8 "VISHAY" H 6300 2300 50  0001 C CNN "Manufacturer"
+F 9 "SI7848BDP-T1-E3" H 6300 2300 50  0001 C CNN "Manufacturer_No"
+	1    6300 2300
 	1    0    0    -1
 $EndComp
@@
 L 10005011_Power_Management:SI7884BDP T22
 U 1 1 5E98C0C9
-P 7800 3200
-F 0 "T22" H 7600 3450 50  0000 L CNN
-F 1 "SI7884BDP" H 7300 3350 50  0000 L CNN
-F 2 "10005011 Power Management:SO08-PPAD_SI7884_1" H 8650 3125 50  0001 C CIN
-F 3 "http://www.vishay.com/docs/68395/si7884bd.pdf" H 8125 2900 50  0001 L CNN
-F 4 "Digi-Key" H 8200 3125 50  0001 C CNN "Source"
-F 5 "SI7884BDP-T1-E3CT-ND" H 8450 3125 50  0001 C CNN "Source_PN"
-F 6 "MOSFET TRANS N CHANNEL,40V,12A,0.007 OHM, SO8" H 8600 3125 50  0001 C CNN "Description"
-F 7 "10022883" H 7800 3200 50  0001 C CNN "Item Number"
-F 8 "VISHAY" H 7800 3200 50  0001 C CNN "Manufacturer"
-F 9 "SI7848BDP-T1-E3" H 7800 3200 50  0001 C CNN "Manufacturer_No"
-	1    7800 3200
+P 7900 3200
+F 0 "T22" H 7700 3450 50  0000 L CNN
+F 1 "SI7884BDP" H 7400 3350 50  0000 L CNN
+F 2 "10005011 Power Management:SO08-PPAD_SI7884_1" H 8750 3125 50  0001 C CIN
+F 3 "http://www.vishay.com/docs/68395/si7884bd.pdf" H 8225 2900 50  0001 L CNN
+F 4 "Digi-Key" H 8300 3125 50  0001 C CNN "Source"
+F 5 "SI7884BDP-T1-E3CT-ND" H 8550 3125 50  0001 C CNN "Source_PN"
+F 6 "MOSFET TRANS N CHANNEL,40V,12A,0.007 OHM, SO8" H 8700 3125 50  0001 C CNN "Description"
+F 7 "10022883" H 7900 3200 50  0001 C CNN "Item Number"
+F 8 "VISHAY" H 7900 3200 50  0001 C CNN "Manufacturer"
+F 9 "SI7848BDP-T1-E3" H 7900 3200 50  0001 C CNN "Manufacturer_No"
+	1    7900 3200
 	-1   0    0    -1
 $EndComp
@@
 L 10005011_Power_Management:SI7884BDP T21
 U 1 1 5E98C9D5
-P 6400 3200
-F 0 "T21" H 6200 3450 50  0000 L CNN
-F 1 "SI7884BDP" H 5900 3350 50  0000 L CNN
-F 2 "10005011 Power Management:SO08-PPAD_SI7884_1" H 7250 3125 50  0001 C CIN
-F 3 "http://www.vishay.com/docs/68395/si7884bd.pdf" H 6725 2900 50  0001 L CNN
-F 4 "Digi-Key" H 6800 3125 50  0001 C CNN "Source"
-F 5 "SI7884BDP-T1-E3CT-ND" H 7050 3125 50  0001 C CNN "Source_PN"
-F 6 "MOSFET TRANS N CHANNEL,40V,12A,0.007 OHM, SO8" H 7200 3125 50  0001 C CNN "Description"
-F 7 "10022883" H 6400 3200 50  0001 C CNN "Item Number"
-F 8 "VISHAY" H 6400 3200 50  0001 C CNN "Manufacturer"
-F 9 "SI7848BDP-T1-E3" H 6400 3200 50  0001 C CNN "Manufacturer_No"
-	1    6400 3200
-	1    0    0    -1
-$EndComp
+P 6300 3200
+F 0 "T21" H 6100 3450 50  0000 L CNN
+F 1 "SI7884BDP" H 5800 3350 50  0000 L CNN
+F 2 "10005011 Power Management:SO08-PPAD_SI7884_1" H 7150 3125 50  0001 C CIN
+F 3 "http://www.vishay.com/docs/68395/si7884bd.pdf" H 6625 2900 50  0001 L CNN
+F 4 "Digi-Key" H 6700 3125 50  0001 C CNN "Source"
+F 5 "SI7884BDP-T1-E3CT-ND" H 6950 3125 50  0001 C CNN "Source_PN"
+F 6 "MOSFET TRANS N CHANNEL,40V,12A,0.007 OHM, SO8" H 7100 3125 50  0001 C CNN "Description"
+F 7 "10022883" H 6300 3200 50  0001 C CNN "Item Number"
+F 8 "VISHAY" H 6300 3200 50  0001 C CNN "Manufacturer"
+F 9 "SI7848BDP-T1-E3" H 6300 3200 50  0001 C CNN "Manufacturer_No"
+	1    6300 3200
+	1    0    0    -1
+$EndComp

Commit message: change CR1-BIS to ZCR1 so that kicad does not think it is missing annotation, do the same in the PCB to be able to read netlist without components getting erased and placed new
Parts:
- added ZCR1, ZCR2: ??SOD87C, 10005011 Power Management:SOD87_1, symbol 10005011_Power_Management:1N5819
Connections:
- net INTVCC-1: now also ZCR1.A, ZCR2.A
- net OS+: now reaches C136.1, C137.1, C138.1, C37.1, C40.1, C41.1, C42.+, C43.1, D5.K, IC9.5 (IN+), R62.2, T20.D, T20.D1 (D), T20.D2 (D), T20.D3 (D)
- net at C39.2, CR2.K, IC10.13 (BOOST2): now also ZCR2.K
- net at C38.2, CR1.K, IC10.24 (BOOST1): now also ZCR1.K
- net MES-24V-UTIL: now reaches C119.2, R64.1, R66.1
Other:
- moved on the sheet: R60
Changed lines of the file:
@@
 	7800 1250 7800 1850
 Wire Wire Line
-	7800 1250 8900 1250
+	7800 1250 8000 1250
 Wire Wire Line
 	7550 2150 7550 1850
@@
 Wire Wire Line
 	7550 2750 7800 2750
-Text Label 5750 2750 0    50   ~ 0
-SW2
-Text Label 8450 2750 2    50   ~ 0
-SW1
 Text Label 5750 3200 0    50   ~ 0
 BG2
@@
 Text Label 4800 7400 2    50   ~ 0
 BG1
-Text Label 4800 7200 2    50   ~ 0
-SW1
 Wire Wire Line
 	4500 8000 4500 8200
@@
 Text Label 2250 7400 0    50   ~ 0
 BG2
-Text Label 2250 7200 0    50   ~ 0
-SW2
 Wire Wire Line
 	2250 7400 2750 7400
@@
 Text Label 3050 5150 0    50   ~ 0
 VIN
-Text Label 5500 1050 2    50   ~ 0
-VIN
 Wire Wire Line
 	5500 1050 5300 1050
@@
 Wire Wire Line
 	3500 5150 3900 5150
-$Comp
-L Device:R R60
-U 1 1 5EE9A75C
-P 4800 6400
-F 0 "R60" H 4730 6354 50  0000 R CNN
-F 1 "10k" H 4730 6445 50  0000 R CNN
-F 2 "10005011 Power Management:R0603_1" V 4730 6400 50  0001 C CNN
-F 3 "~" H 4800 6400 50  0001 C CNN
-F 4 "RESISTOR,10K OHM.0.063W,+/-1%,0603" V 4800 6400 50  0001 C CNN "Description"
-F 5 "10022548" V 4800 6400 50  0001 C CNN "Item Number"
-F 6 "" V 4800 6400 50  0001 C CNN "Manufacturer"
-F 7 "" V 4800 6400 50  0001 C CNN "Manufacturer_No"
-	1    4800 6400
-	-1   0    0    1
-$EndComp
-Wire Wire Line
-	4800 6550 4800 6600
-Wire Wire Line
-	4800 6600 4300 6600
 Text Label 5200 5900 2    50   ~ 0
 INTVCC-1
 Wire Wire Line
-	4800 5900 5200 5900
-Wire Wire Line
-	4800 5900 4800 6150
-Wire Wire Line
-	4800 6150 5200 6150
+	4650 5900 5200 5900
+Wire Wire Line
+	4650 5900 4650 6150
+Wire Wire Line
+	4650 6150 5200 6150
 Wire Wire Line
 	5200 6150 5200 6450
 Wire Wire Line
 	5200 6750 5200 6800
-Connection ~ 4800 6150
-Wire Wire Line
-	4800 6150 4800 6250
+Connection ~ 4650 6150
 Connection ~ 5200 6800
 Wire Wire Line
@@
 	-1   0    0    -1
 $EndComp
+$Comp
+L 10005011_Power_Management:1N5819 D19-BIS?
+U 1 1 5E9EC701
+P 1200 6600
+AR Path="/5FEC5422/5E9EC701" Ref="D19-BIS?"  Part="1"
+AR Path="/5E92767C/5E9EC701" Ref="ZCR2"  Part="1"
+F 0 "ZCR2" V 1250 6900 50  0000 C CNN
+F 1 "??SOD87C" V 1150 6900 50  0000 C CNN
+F 2 "10005011 Power Management:SOD87_1" H 1150 6300 50  0001 C CNN
+F 3 "" H 1200 6600 50  0001 C CNN
+F 4 "" H 1200 5900 50  0001 C CNN "Mfgr"
+F 5 "" H 1250 6100 50  0001 C CNN "Mfgr_PN"
+F 6 "" H 1200 6000 50  0001 C CNN "Source"
+F 7 "" H 1150 6200 50  0001 C CNN "Source_PN"
+F 8 "" H 1150 6400 50  0001 C CNN "Description"
+F 9 "" H 1200 6600 50  0001 C CNN "Item Number"
+	1    1200 6600
+	0    -1   -1   0
+$EndComp
+Connection ~ 1200 6450
+Connection ~ 1200 6750
+$Comp
+L 10005011_Power_Management:1N5819 CR2-BIS?
+U 1 1 5EA4E9A7
+P 5200 6600
+AR Path="/5FEC5422/5EA4E9A7" Ref="CR2-BIS?"  Part="1"
+AR Path="/5E92767C/5EA4E9A7" Ref="ZCR1"  Part="1"
+F 0 "ZCR1" V 5250 6850 50  0000 C CNN
+F 1 "??SOD87C" V 5150 6850 50  0000 C CNN
+F 2 "10005011 Power Management:SOD87_1" H 5150 6300 50  0001 C CNN
+F 3 "" H 5200 6600 50  0001 C CNN
+F 4 "" H 5200 5900 50  0001 C CNN "Mfgr"
+F 5 "" H 5250 6100 50  0001 C CNN "Mfgr_PN"
+F 6 "" H 5200 6000 50  0001 C CNN "Source"
+F 7 "" H 5150 6200 50  0001 C CNN "Source_PN"
+F 8 "" H 5150 6400 50  0001 C CNN "Description"
+F 9 "" H 5200 6600 50  0001 C CNN "Item Number"
+	1    5200 6600
+	0    -1   -1   0
+$EndComp
+Connection ~ 5200 6450
+Connection ~ 5200 6750
+Wire Wire Line
+	4650 6600 4300 6600
+Wire Wire Line
+	4650 6150 4650 6250
+Wire Wire Line
+	4650 6550 4650 6600
+$Comp
+L Device:R R60
+U 1 1 5EE9A75C
+P 4650 6400
+F 0 "R60" H 4580 6354 50  0000 R CNN
+F 1 "10k" H 4580 6445 50  0000 R CNN
+F 2 "10005011 Power Management:R0603_1" V 4580 6400 50  0001 C CNN
+F 3 "~" H 4650 6400 50  0001 C CNN
+F 4 "RESISTOR,10K OHM.0.063W,+/-1%,0603" V 4650 6400 50  0001 C CNN "Description"
+F 5 "10022548" V 4650 6400 50  0001 C CNN "Item Number"
+F 6 "" V 4650 6400 50  0001 C CNN "Manufacturer"
+F 7 "" V 4650 6400 50  0001 C CNN "Manufacturer_No"
+	1    4650 6400
+	-1   0    0    1
+$EndComp
+Text GLabel 15150 2400 0    50   Input ~ 0
+MES-24V-UTIL
+Wire Wire Line
+	15150 2400 15250 2400
+Connection ~ 15250 2400
+Text Label 5500 1050 2    50   ~ 0
+VIN
+Text Label 4800 7200 2    50   ~ 0
+SW1
+Text Label 2250 7200 0    50   ~ 0
+SW2
+Text Label 8450 2750 2    50   ~ 0
+SW1
+Text Label 5750 2750 0    50   ~ 0
+SW2
+Text Label 8200 1050 2    50   ~ 0
+OS+
+Wire Wire Line
+	8200 1050 8000 1050
+Wire Wire Line
+	8000 1050 8000 1250
+Connection ~ 8000 1250
+Wire Wire Line
+	8000 1250 8900 1250
 $EndSCHEMATC

Commit message: Powermanagement dev, ERC
Changed lines of the file:
@@
 Connection ~ 5300 1300
 Wire Wire Line
-	5300 1300 6400 1300
+	5300 1300 5900 1300
 $Comp
 L Device:C C31
@@
 Wire Wire Line
 	8000 1250 8900 1250
+$Comp
+L power:PWR_FLAG #FLG0107
+U 1 1 5ED2132B
+P 2400 9000
+F 0 "#FLG0107" H 2400 9075 50  0001 C CNN
+F 1 "PWR_FLAG" H 2400 9150 50  0000 C CNN
+F 2 "" H 2400 9000 50  0001 C CNN
+F 3 "~" H 2400 9000 50  0001 C CNN
+	1    2400 9000
+	1    0    0    -1
+$EndComp
+Wire Wire Line
+	2400 9000 2400 9200
+Wire Wire Line
+	2400 9200 2650 9200
+Connection ~ 2650 9200
+$Comp
+L power:PWR_FLAG #FLG0108
+U 1 1 5ED37A93
+P 5900 1600
+F 0 "#FLG0108" H 5900 1675 50  0001 C CNN
+F 1 "PWR_FLAG" H 5900 1750 50  0000 C CNN
+F 2 "" H 5900 1600 50  0001 C CNN
+F 3 "~" H 5900 1600 50  0001 C CNN
+	1    5900 1600
+	1    0    0    -1
+$EndComp
+Wire Wire Line
+	5300 1700 5900 1700
+Wire Wire Line
+	5900 1700 5900 1600
+Connection ~ 5300 1700
+$Comp
+L power:PWR_FLAG #FLG0109
+U 1 1 5ED6C771
+P 5900 1000
+F 0 "#FLG0109" H 5900 1075 50  0001 C CNN
+F 1 "PWR_FLAG" H 5900 1150 50  0000 C CNN
+F 2 "" H 5900 1000 50  0001 C CNN
+F 3 "~" H 5900 1000 50  0001 C CNN
+	1    5900 1000
+	1    0    0    -1
+$EndComp
+Wire Wire Line
+	5900 1000 5900 1300
+Connection ~ 5900 1300
+Wire Wire Line
+	5900 1300 6400 1300
+$Comp
+L power:PWR_FLAG #FLG0118
+U 1 1 5EF9BB30
+P 12500 4300
+F 0 "#FLG0118" H 12500 4375 50  0001 C CNN
+F 1 "PWR_FLAG" H 12500 4450 50  0000 C CNN
+F 2 "" H 12500 4300 50  0001 C CNN
+F 3 "~" H 12500 4300 50  0001 C CNN
+	1    12500 4300
+	1    0    0    -1
+$EndComp
+Wire Wire Line
+	12500 4300 12500 4500
+Wire Wire Line
+	12500 4500 12250 4500
+Connection ~ 12250 4500
 $EndSCHEMATC

Commit message: update fp path
Parts:
- C115, C116, C117, C118, C119, C37, C38, C39, C49, C52, C56: footprint 10005011 Power Management:C0603_1 -> AllModules:C0603_1
- C125, C42: footprint 10005011 Power Management:C-SC10_1 -> AllModules:C-SC10_1
- C131, C30, C31, C32: footprint 10005011 Power Management:C0805_1 -> AllModules:C0805_1
- C134, C135, C29: footprint 10005011 Power Management:C1210_1 -> AllModules:C1210_1
- C136, C137, C138, C26, C27, C28, C40, C41, C43: footprint 10005011 Power Management:C2220_1 -> AllModules:C2220_1
- C25, C48: footprint 10005011 Power Management:C0402_1 -> AllModules:C0402_1
- C33, C50, R62: footprint 10005011 Power Management:RC1206_1 -> AllModules:RC1206_1
- CR1, CR2: footprint 10005011 Power Management:SOD123-AK_1 -> AllModules:SOD123-AK_1
- D12, D4: footprint 10005011 Power Management:SOT23-1DIODE_1 -> AllModules:SOT23-1DIODE_1
- D5, D6: footprint 10005011 Power Management:SMB_1 -> AllModules:SMB_1
- FLTR1, FLTR3: footprint 10005011 Power Management:BNX002+SF-AIROX_1 -> AllModules:BNX002+SF-AIROX_1
- IC10: footprint 10005011 Power Management:SSOP24_1 -> AllModules:SSOP24_1
- IC9: footprint 10005011 Power Management:uSO08_1 -> AllModules:uSO08_1
- JPL1: footprint 10005011 Power Management:GDCAFE-F_FERME_1 -> AllModules:GDCAFE-F_FERME_1
- L3: footprint 10005011 Power Management:SF-3863-WESI_1 -> AllModules:SF-3863-WESI_1
- R117: footprint 10005011 Power Management:R0805_1 -> AllModules:R0805_1
- R58, R59, R60, R61, R63, R64, R65, R66, R67, R74, R76: footprint 10005011 Power Management:R0603_1 -> AllModules:R0603_1
- R75: footprint 10005011 Power Management:R2512_1 -> AllModules:R2512_1
- T19, T20, T21, T22: footprint 10005011 Power Management:SO08-PPAD_SI7884_1 -> AllModules:SO08-PPAD_SI7884_1
- ZCR1, ZCR2: footprint 10005011 Power Management:SOD87_1 -> AllModules:SOD87_1

Commit message: fix L3 manufacturer and partnumber
Parts:
- L3: Manufacturer YAGEO -> WURTH ELEKTRONIK GMBH; Manufacturer_No 232272461001L -> P01/00004
Changed lines of the file:
@@
 F 4 "INDUCTOR, POWER CHOKE, 47UH, 8A" V 7150 2750 50  0001 C CNN "Description"
 F 5 "10022741" V 7150 2750 50  0001 C CNN "Item Number"
-F 6 "YAGEO" V 7150 2750 50  0001 C CNN "Manufacturer"
-F 7 "232272461001L" V 7150 2750 50  0001 C CNN "Manufacturer_No"
+F 6 "WURTH ELEKTRONIK GMBH" V 7150 2750 50  0001 C CNN "Manufacturer"
+F 7 "P01/00004" V 7150 2750 50  0001 C CNN "Manufacturer_No"
 	1    7150 2750
 	0    -1   -1   0
