File: 10005011 Power Management/10005011 Connectors-FAN.sch (KiCad schematic (older format))
At the start: 63 parts, among them IC25 L78M24CDT, IC6 TLV3012AIDBV, J10 BATTERY, J6 FAN, J7 CPU BOARD, J9 TURBINE, T23 IRLML2803, T31 IRLML5103

Commit message: Power Mgt board: update local symbols to global Update N°2
Parts:
- C139: value NC -> DNP; symbol Device:C -> Capacitor:C_4u7F_10%; Description (none) -> CAPACITOR CERAMIC, 4.7UF,+/-10%,50V; Item Number (none) -> 10039582; Manufacturer (none) -> KEMET; Manufacturer2 (none) -> TDK; Manufacturer3 (none) -> KEMET_RMS1; Manufacturer_No (none) -> C1210C475K5RACAUTO; Manufacturer_No2 (none) -> CNA6P1X7R1H475K250AE; Manufacturer_No3 (none) -> C1210C475K5RAC
Changed lines of the file:
@@
 Connection ~ 7700 7150
 $Comp
-L Device:C C139
+L Capacitor:C_4u7F_10% C139
 U 1 1 5EAE819F
 P 9150 7500
 F 0 "C139" H 9264 7454 50  0000 L CNN
-F 1 "NC" H 9264 7545 50  0000 L CNN
+F 1 "DNP" H 9264 7545 50  0000 L CNN
 F 2 "AllModules:C1210_1" H 9188 7350 50  0001 C CNN
 F 3 "~" H 9150 7500 50  0001 C CNN
+F 4 "CAPACITOR CERAMIC, 4.7UF,+/-10%,50V" H 9150 7500 50  0001 C CNN "Description"
+F 5 "10039582" H 9150 7500 50  0001 C CNN "Item Number"
+F 6 "KEMET" H 9150 7500 50  0001 C CNN "Manufacturer"
+F 7 "TDK" H 9150 7500 50  0001 C CNN "Manufacturer2"
+F 8 "KEMET_RMS1" H 9150 7500 50  0001 C CNN "Manufacturer3"
+F 9 "C1210C475K5RACAUTO" H 9150 7500 50  0001 C CNN "Manufacturer_No"
+F 10 "CNA6P1X7R1H475K250AE" H 9150 7500 50  0001 C CNN "Manufacturer_No2"
+F 11 "C1210C475K5RAC" H 9150 7500 50  0001 C CNN "Manufacturer_No3"
 	1    9150 7500
 	-1   0    0    1

Commit message: Power Mgt board: update local symbols to global Update N°3
Parts:
- JPL2, JPL3: symbol Device:Jumper_NC_Small -> Jumper:JUMP_0U
- R13: value NC -> DNP; symbol Device:R -> Resistor:R0603_100k_1%_10022549; Description (none) -> RESISTOR,100KOHM,0.063W,+/-1%,0603; Item Number (none) -> 10022549; Manufacturer (none) -> YAGEO_RMS1; Manufacturer2 (none) -> BOURNS_RMS1; Manufacturer3 (none) -> YAGEO_RMS1; Manufacturer_No (none) -> RC0603FR-07100KL; Manufacturer_No2 (none) -> CR0603-FX-1003ELF; Manufacturer_No3 (none) -> RC0603FR-07100KL
Other:
- moved on the sheet: PT1
Changed lines of the file:
@@
 	-1   0    0    1
 $EndComp
-$Comp
-L Power:PGND #PWR0167
-U 1 1 5EA7422F
-P 3200 7900
-F 0 "#PWR0167" H 3200 7650 50  0001 C CNN
-F 1 "PGND" H 3200 7750 50  0000 C CNN
-F 2 "" H 3200 7900 50  0001 C CNN
-F 3 "" H 3200 7900 50  0001 C CNN
-	1    3200 7900
-	1    0    0    -1
-$EndComp
-Wire Wire Line
-	3450 7200 3450 7450
-Wire Wire Line
-	3450 7450 3200 7450
-Wire Wire Line
-	3200 7450 3200 7000
+Wire Wire Line
+	3450 7200 3450 7300
 Connection ~ 3200 7000
-Connection ~ 3450 7450
-$Comp
-L Device:Jumper_NC_Small JPL2
-U 1 1 5EA74230
-P 3550 7600
-F 0 "JPL2" V 3504 7674 50  0000 L CNN
-F 1 "LINK" V 3595 7674 50  0000 L CNN
-F 2 "AllModules:GDCAFE-F_FERME_1" H 3550 7600 50  0001 C CNN
-F 3 "~" H 3550 7600 50  0001 C CNN
-	1    3550 7600
-	0    1    1    0
-$EndComp
-Connection ~ 3200 7450
-$Comp
-L Power:GND #PWR0168
-U 1 1 5EA74232
-P 3550 7900
-F 0 "#PWR0168" H 3550 7650 50  0001 C CNN
-F 1 "GND" H 3550 7750 50  0000 C CNN
-F 2 "" H 3550 7900 50  0001 C CNN
-F 3 "" H 3550 7900 50  0001 C CNN
-	1    3550 7900
-	1    0    0    -1
-$EndComp
-Wire Wire Line
-	3450 7450 3550 7450
-Wire Wire Line
-	3550 7450 3550 7500
-Wire Wire Line
-	3550 7700 3550 7900
-Wire Wire Line
-	3200 7450 3200 7900
 Wire Wire Line
 	3100 6600 3450 6600
@@
 	14200 8650 13950 8650
 $Comp
-L Device:R R13
+L Resistor:R0603_100k_1%_10022549 R13
 U 1 1 5EAE8193
 P 13300 7150
 F 0 "R13" V 13093 7150 50  0000 C CNN
-F 1 "NC" V 13184 7150 50  0000 C CNN
+F 1 "DNP" V 13184 7150 50  0000 C CNN
 F 2 "AllModules:R0603_1" V 13230 7150 50  0001 C CNN
 F 3 "~" H 13300 7150 50  0001 C CNN
+F 4 "RESISTOR,100KOHM,0.063W,+/-1%,0603" H 13300 7150 50  0001 C CNN "Description"
+F 5 "10022549" H 13300 7150 50  0001 C CNN "Item Number"
+F 6 "YAGEO_RMS1" H 13300 7150 50  0001 C CNN "Manufacturer"
+F 7 "BOURNS_RMS1" H 13300 7150 50  0001 C CNN "Manufacturer2"
+F 8 "YAGEO_RMS1" H 13300 7150 50  0001 C CNN "Manufacturer3"
+F 9 "RC0603FR-07100KL" H 13300 7150 50  0001 C CNN "Manufacturer_No"
+F 10 "CR0603-FX-1003ELF" H 13300 7150 50  0001 C CNN "Manufacturer_No2"
+F 11 "RC0603FR-07100KL" H 13300 7150 50  0001 C CNN "Manufacturer_No3"
 	1    13300 7150
 	0    1    1    0
@@
 	4850 7200 4850 7300
 Wire Wire Line
-	4200 7300 4200 7200
-Connection ~ 4200 7300
-Wire Wire Line
 	5500 7300 5500 7200
-Wire Wire Line
-	4200 7300 4850 7300
 $Comp
 L Diode:SZ1SMB D21
@@
 	0    1    1    0
 $EndComp
-$Comp
-L Connector:TestPoint PT1
-U 1 1 5EB70271
-P 4500 7700
-F 0 "PT1" H 4500 7970 50  0000 C CNN
-F 1 "TestPoint" H 4500 7900 50  0000 C CNN
-F 2 "AllModules:C12000_1" H 4700 7700 50  0001 C CNN
-F 3 "~" H 4700 7700 50  0001 C CNN
-	1    4500 7700
-	1    0    0    -1
-$EndComp
-Wire Wire Line
-	4200 7800 4200 7900
-Connection ~ 4200 7800
-Wire Wire Line
-	4500 7800 4500 7700
-Wire Wire Line
-	4200 7800 4500 7800
-Wire Wire Line
-	4200 7700 4200 7800
-Connection ~ 4200 7450
-Wire Wire Line
-	4200 7450 4200 7500
-Wire Wire Line
-	3550 7450 4200 7450
-$Comp
-L Power:0VANA #PWR0169
-U 1 1 5EB2DA0B
-P 4200 7900
-F 0 "#PWR0169" H 4200 7650 50  0001 C CNN
-F 1 "0VANA" H 4200 7750 50  0000 C CNN
-F 2 "" H 4200 7900 50  0001 C CNN
-F 3 "" H 4200 7900 50  0001 C CNN
-	1    4200 7900
-	1    0    0    -1
-$EndComp
-Wire Wire Line
-	4200 7450 4200 7300
-Connection ~ 3550 7450
 $Comp
 L Capacitor:C0805_100nF_50V_10% C109
@@
 	13850 7250 13850 7350
 $Comp
-L Diode:BAT54 D20
-U 1 1 5EAE8195
-P 12450 8350
-F 0 "D20" V 12450 8300 50  0000 R CNN
-F 1 "BAT54" V 12350 8300 50  0000 R CNN
-F 2 "AllModules:SOT23-1G_1" H 12220 8188 50  0001 L CNN
-F 3 "http://www.onsemi.com/pub/Collateral/BAT54LT1-D.PDF" H 12370 8450 50  0001 C CNN
-F 4 "DIODE SCHOTTKY 30V 200MA SOT23-3" H 12775 8175 60  0001 C CNN "Description"
-F 5 "ON Semiconductor" H 12775 8175 60  0001 C CNN "Mfgr"
-F 6 "BAT54LT1G" H 12775 8175 60  0001 C CNN "Mfgr_PN"
-F 7 "Digi-Key" H 12625 8175 60  0001 C CNN "Source"
-F 8 "BAT54LT1GOSTR-ND" H 12600 8175 60  0001 C CNN "Source_PN"
-F 9 "10022652" H 12450 8300 50  0001 C CNN "Item Number"
-	1    12450 8350
-	0    -1   -1   0
-$EndComp
-$Comp
 L Connector:Conn_01x02_Male J6
 U 1 1 5E94A06E
@@
 	1    0    0    -1
 $EndComp
-$Comp
-L Device:Jumper_NC_Small JPL3
-U 1 1 5EB10713
-P 4200 7600
-F 0 "JPL3" V 4154 7552 50  0000 R CNN
-F 1 "LINK" V 4245 7552 50  0000 R CNN
-F 2 "AllModules:GDCAFE-F_FERME_1" H 4200 7600 50  0001 C CNN
-F 3 "~" H 4200 7600 50  0001 C CNN
-	1    4200 7600
-	0    1    1    0
-$EndComp
 Text Notes 3700 1050 0    50   ~ 0
 ideally, a couple of the pins might be bypassed to PGND instead of GND,\nbut it doesn't really matter because the CPU board combines the grounds.
@@
 Wire Notes Line
 	2700 5650 2700 8150
+Wire Wire Line
+	4200 7300 4850 7300
+Wire Wire Line
+	4200 7300 4200 7200
+Connection ~ 4200 7300
+Wire Wire Line
+	4200 7300 3450 7300
+Connection ~ 3450 7300
+Wire Wire Line
+	3450 7300 3200 7300
+Connection ~ 3200 7300
+Wire Wire Line
+	3200 7300 3200 7000
+Wire Wire Line
+	3200 7300 3200 7400
+$Comp
+L Power:PGND #PWR?
+U 1 1 5EE6252B
+P 5500 7350
+F 0 "#PWR?" H 5500 7100 50  0001 C CNN
+F 1 "PGND" H 5500 7200 50  0000 C CNN
+F 2 "" H 5500 7350 50  0001 C CNN
+F 3 "" H 5500 7350 50  0001 C CNN
+	1    5500 7350
+	1    0    0    -1
+$EndComp
+Wire Wire Line
+	5500 7350 5500 7300
+Connection ~ 5500 7300
+$Comp
+L Diode:BAT54 D20
+U 1 1 5EAE8195
+P 12450 8350
+F 0 "D20" V 12450 8300 50  0000 R CNN
+F 1 "BAT54" V 12350 8300 50  0000 R CNN
+F 2 "AllModules:SOT23-1G_1" H 12220 8188 50  0001 L CNN
+F 3 "http://www.onsemi.com/pub/Collateral/BAT54LT1-D.PDF" H 12370 8450 50  0001 C CNN
+F 4 "DIODE SCHOTTKY 30V 200MA SOT23-3" H 12775 8175 60  0001 C CNN "Description"
+F 5 "ON Semiconductor" H 12775 8175 60  0001 C CNN "Mfgr"
+F 6 "BAT54LT1G" H 12775 8175 60  0001 C CNN "Mfgr_PN"
+F 7 "Digi-Key" H 12625 8175 60  0001 C CNN "Source"
+F 8 "BAT54LT1GOSTR-ND" H 12600 8175 60  0001 C CNN "Source_PN"
+F 9 "10022652" H 12450 8300 50  0001 C CNN "Item Number"
+	1    12450 8350
+	0    -1   -1   0
+$EndComp
+Wire Wire Line
+	4200 7875 4300 7875
+Wire Wire Line
+	3550 7850 3550 7900
+Wire Wire Line
+	3550 7400 4200 7400
+Connection ~ 3550 7400
+Wire Wire Line
+	3550 7450 3550 7400
+Wire Wire Line
+	3200 7400 3550 7400
+$Comp
+L Jumper:JUMP_0U JPL2
+U 1 1 5EA74230
+P 3550 7650
+F 0 "JPL2" V 3504 7724 50  0000 L CNN
+F 1 "LINK" V 3595 7724 50  0000 L CNN
+F 2 "AllModules:GDCAFE-F_FERME_1" H 3550 7650 50  0001 C CNN
+F 3 "~" H 3550 7650 50  0001 C CNN
+	1    3550 7650
+	0    1    1    0
+$EndComp
+Wire Wire Line
+	4200 7875 4200 7900
+Connection ~ 4200 7875
+$Comp
+L Jumper:JUMP_0U JPL3
+U 1 1 5EB10713
+P 4200 7650
+F 0 "JPL3" V 4154 7602 50  0000 R CNN
+F 1 "LINK" V 4245 7602 50  0000 R CNN
+F 2 "AllModules:GDCAFE-F_FERME_1" H 4200 7650 50  0001 C CNN
+F 3 "~" H 4200 7650 50  0001 C CNN
+	1    4200 7650
+	0    1    1    0
+$EndComp
+Wire Wire Line
+	4200 7450 4200 7400
+Wire Wire Line
+	4200 7850 4200 7875
+$Comp
+L Power:0VANA #PWR0169
+U 1 1 5EB2DA0B
+P 4200 7900
+F 0 "#PWR0169" H 4200 7650 50  0001 C CNN
+F 1 "0VANA" H 4200 7750 50  0000 C CNN
+F 2 "" H 4200 7900 50  0001 C CNN
+F 3 "" H 4200 7900 50  0001 C CNN
+	1    4200 7900
+	1    0    0    -1
+$EndComp
+$Comp
+L Connector:TestPoint PT1
+U 1 1 5EB70271
+P 4300 7875
+F 0 "PT1" V 4300 8125 50  0000 C CNN
+F 1 "TestPoint" H 4300 8075 50  0001 C CNN
+F 2 "AllModules:C12000_1" H 4500 7875 50  0001 C CNN
+F 3 "~" H 4500 7875 50  0001 C CNN
+	1    4300 7875
+	0    1    1    0
+$EndComp
+$Comp
+L Power:GND #PWR0168
+U 1 1 5EA74232
+P 3550 7900
+F 0 "#PWR0168" H 3550 7650 50  0001 C CNN
+F 1 "GND" H 3550 7750 50  0000 C CNN
+F 2 "" H 3550 7900 50  0001 C CNN
+F 3 "" H 3550 7900 50  0001 C CNN
+	1    3550 7900
+	1    0    0    -1
+$EndComp
 $EndSCHEMATC

Commit message: Libraries nicknames update in Kicad projects
Parts:
- C10, C114, C14, C60: symbol Capacitor:C_10uF_50V_10% -> V_Capacitor:C_10uF_50V_10%
- C100, C53, C61, C62, C98: symbol Capacitor:47pF_array -> V_Capacitor:47pF_array
- C109, C110, C112, C113: symbol Capacitor:C0805_100nF_50V_10% -> V_Capacitor:C0805_100nF_50V_10%
- C111: symbol Capacitor:C0603_10nF_50V_10% -> V_Capacitor:C0603_10nF_50V_10%
- C139: symbol Capacitor:C_4u7F_10% -> V_Capacitor:C_4u7F_10%
- C9: symbol Capacitor:C0402_100nF_16V_10% -> V_Capacitor:C0402_100nF_16V_10%
- D10: symbol Diode:BZX84C5V1_10022657 -> V_Diode:BZX84C5V1_10022657
- D14, D7: symbol Diode:BAT54C -> V_Diode:BAT54C
- D20: symbol Diode:BAT54 -> V_Diode:BAT54
- D21: symbol Diode:SZ1SMB -> V_Diode:SZ1SMB
- IC25: symbol IC:LM78M05_TO252 -> V_IC:LM78M05_TO252
- IC6: symbol IC:TLV3012AIDBV -> V_IC:TLV3012AIDBV
- J10: symbol Connector:Conn_01x10_Female -> V_Connector:Conn_01x10_Female
- J6: symbol Connector:Conn_01x02_Male -> V_Connector:Conn_01x02_Male
- J7: symbol Connector:Conn_02x13_Odd_Even -> V_Connector:Conn_02x13_Odd_Even
- J9: symbol Connector:Conn_01x04_Male -> V_Connector:Conn_01x04_Male
- JPL2, JPL3: symbol Jumper:JUMP_0U -> V_Jumper:JUMP_0U
- L15, L16, L17, L18, L19, L20, L21, L22, L23, L43, L44, L45, L46, L47, L48, L49, L50, L6: symbol Inductor:Ferrite_Bead_Small_10022907 -> V_Inductor:Ferrite_Bead_Small_10022907
- L4: symbol Inductor:L_Core_Iron_10022910 -> V_Inductor:L_Core_Iron_10022910
- L5, L61: symbol Inductor:Ferrite_Bead_Small_10022911 -> V_Inductor:Ferrite_Bead_Small_10022911
- ML2, ML3: symbol Varistor:Varistor_10022926 -> V_Varistor:Varistor_10022926
- PT1: symbol Connector:TestPoint -> V_Connector:TestPoint
- R114: symbol Resistor:R1206_1k5_1% -> V_Resistor:R1206_1k5_1%
- R115: symbol Resistor:R1206_1k_1%_10022557 -> V_Resistor:R1206_1k_1%_10022557
- R116: symbol Resistor:R1206_100R_1% -> V_Resistor:R1206_100R_1%
- R12, R77: symbol Resistor:R0603_10k_1%_10022548 -> V_Resistor:R0603_10k_1%_10022548
- R13, R20: symbol Resistor:R0603_100k_1%_10022549 -> V_Resistor:R0603_100k_1%_10022549
- R78: symbol Resistor:R0603_10k_0.1%_10022701 -> V_Resistor:R0603_10k_0.1%_10022701
- T23: symbol Transistor:IRLML2803TRPBF -> V_Transistor:IRLML2803TRPBF
- T31: symbol Transistor:IRLML5103TRPBF -> V_Transistor:IRLML5103TRPBF
Connections:
- net GND: now reaches IC6.2 (V-)
- net GND: now also C100.1, C100.2, C100.3, C100.4, C112.1, C113.1, C114.1, C139.1, C14.1, C53.1, C53.2, C53.3, C53.4, C60.1, C61.1, C61.2, C61.3, C61.4, C62.1, C62.2, C62.3, C62.4, C9.2, C98.1, C98.2, C98.3, C98.4, D10.A, D20.1 (A), D7.1, D7.2, IC25.2 (GND), J7.24 (Pin_24), J7.4 (Pin_4), JPL2.2, R116.2, R77.2, T23.S
- net +5V: now reaches C9.1, IC6.6 (V+)
- net +5V: now also L46.2
- net PGND: now reaches J7.1 (Pin_1)
- net PGND: now also C10.1, C109.1, C110.1, D21.A, J10.1 (Pin_1), J10.2 (Pin_2), J10.3 (Pin_3), J10.4 (Pin_4), J7.25 (Pin_25), J9.1 (Pin_1), JPL2.1, JPL3.1, ML2.1, ML3.1
- net 0VANA: now reaches J7.2 (Pin_2)
- net 0VANA: now also J7.26 (Pin_26), JPL3.2, PT1.1
