File: GR106768 Buzzer/GR106768_buzzer_charger.sch (KiCad schematic (older format))
At the start: 142 parts, among them IC5 LM317L_SO8, IC6 BQ2002C, IC7 TLV3011, IC8 LT3471, IC9 TLV3011, SW1 SW_SPDT, T10 Si2312BDS, T11 Si2315BDS, T12 Si2315BDS, T13 Si2312BDS, T5 Si2312BDS, T6 Si2315BDS, T7 Si2312BDS, T8 Si2315BDS, T9 Si2312BDS

Commit message: fix merge conflicts
Parts:
- removed C33 (x2): 100nF, GR106768 Buzzer:C0402_2, symbol Device:C
- removed C34 (x2): NC, GR106768 Buzzer:C0402_2, symbol Device:C
- removed D16, D17: BAT54C, GR106768 Buzzer:SOT23-1G_1, symbol Diode:BAT54C
- removed IC7: TLV3011, GR106768 Buzzer:SOT23-6_1, symbol GR106768_Buzzer:TLV3011
- removed IC9: TLV3011, GR106768 Buzzer:SOT23-6_2, symbol GR106768_Buzzer:TLV3011
- removed R30, R31: 0, GR106768 Buzzer:R0402_1, symbol Device:R
- removed R32, R34, R49, R51, R52, R61, R62, R66, R68, R70: 10k, GR106768 Buzzer:R0402_1, symbol Device:R
- removed R33: 1k, GR106768 Buzzer:R0402_1, symbol Device:R
- removed R35: 33k, GR106768 Buzzer:R0402_1, symbol Device:R
- removed R36: 33, GR106768 Buzzer:R0805_1, symbol Device:R
- removed R37: 220, GR106768 Buzzer:R0402_1, symbol Device:R
- removed R38, R39, R42, R47, R63, R64, R67: 100k, GR106768 Buzzer:R0402_1, symbol Device:R
- removed R40: 4.7K, GR106768 Buzzer:R0402_1, symbol Device:R
- removed R41: 180k, GR106768 Buzzer:R0402_1, symbol Device:R
- removed R43: 1.5M, GR106768 Buzzer:R0402_1, symbol Device:R
- removed R44: 680k, GR106768 Buzzer:R0402_1, symbol Device:R
- removed R45: 59k, GR106768 Buzzer:R0402_1, symbol Device:R
- removed R46: 1M, GR106768 Buzzer:R0402_1, symbol Device:R
- removed R53, R54: 47k, GR106768 Buzzer:R0402_1, symbol Device:R
- removed R55: 15k, GR106768 Buzzer:R0402_1, symbol Device:R
- removed R56: 182k, GR106768 Buzzer:R0402_1, symbol Device:R
- removed R57: 54.9k, GR106768 Buzzer:R0402_1, symbol Device:R
- removed R58: 4.99k, GR106768 Buzzer:R0402_1, symbol Device:R
- removed R65: 2.2k, GR106768 Buzzer:R0402_1, symbol Device:R
- removed R71: 470, GR106768 Buzzer:R0805_1, symbol Device:R
- removed T10 (x2), T13 (x2), T9 (x2): Si2312BDS, GR106768 Buzzer:SOT23-GSD_1, symbol GR106768_Buzzer:Si2312BDS
- removed T11 (x2), T12 (x2): Si2315BDS, GR106768 Buzzer:SOT23-GSD_1, symbol GR106768_Buzzer:Si2315BDS
- added C33: 100nF, GR106768 Buzzer:C0402_2, symbol Device:C
- added C34: NC, GR106768 Buzzer:C0402_2, symbol Device:C
- added T10, T13, T9: Si2312BDS, GR106768 Buzzer:SOT23-GSD_1, symbol GR106768_Buzzer:Si2312BDS
- added T11, T12: Si2315BDS, GR106768 Buzzer:SOT23-GSD_1, symbol GR106768_Buzzer:Si2315BDS
Connections:
- wire segments 715 -> 356
- no-connect marks 2 -> 1
Other:
- moved on the sheet: C33, C34, T10, T11, T12, T13, T9

Commit message: backannotate
Parts:
- D16, D17, D6: footprint 10005011 Power Management:SOT23-1G_1 -> GR106768 Buzzer:SOT23-1G_1
- IC7: footprint GR106768 Buzzer:SOT23-6_1 -> GR106768 Buzzer:SOT23-6_2
- IC9: footprint GR106768 Buzzer:SOT23-6_2 -> GR106768 Buzzer:SOT23-6_1
Changed lines of the file:
@@
 F 0 "D6" H 1300 4700 50  0000 L CNN
 F 1 "BAT54C" H 1150 4625 50  0000 L CNN
-F 2 "10005011 Power Management:SOT23-1G_1" H 1125 3925 50  0001 L CNN
+F 2 "GR106768 Buzzer:SOT23-1G_1" H 1125 3925 50  0001 L CNN
 F 3 "https://media.digikey.com/pdf/Data%20Sheets/ON%20Semiconductor%20PDFs/BAT54(A,C,S).pdf" H 1320 4500 50  0001 C CNN
 F 4 "DIODE ARRAY SCHOTTKY 30V SOT23-3" H 1725 4225 60  0001 C CNN "Description"
@@
 F 0 "D16" H 5600 8000 50  0000 L CNN
 F 1 "BAT54C" H 5450 7925 50  0000 L CNN
-F 2 "10005011 Power Management:SOT23-1G_1" H 5425 7225 50  0001 L CNN
+F 2 "GR106768 Buzzer:SOT23-1G_1" H 5425 7225 50  0001 L CNN
 F 3 "https://media.digikey.com/pdf/Data%20Sheets/ON%20Semiconductor%20PDFs/BAT54(A,C,S).pdf" H 5620 7800 50  0001 C CNN
 F 4 "DIODE ARRAY SCHOTTKY 30V SOT23-3" H 6025 7525 60  0001 C CNN "Description"
@@
 F 0 "D17" H 1800 6750 50  0000 L CNN
 F 1 "BAT54C" H 1650 6675 50  0000 L CNN
-F 2 "10005011 Power Management:SOT23-1G_1" H 1625 5975 50  0001 L CNN
+F 2 "GR106768 Buzzer:SOT23-1G_1" H 1625 5975 50  0001 L CNN
 F 3 "https://media.digikey.com/pdf/Data%20Sheets/ON%20Semiconductor%20PDFs/BAT54(A,C,S).pdf" H 1820 6550 50  0001 C CNN
 F 4 "DIODE ARRAY SCHOTTKY 30V SOT23-3" H 2225 6275 60  0001 C CNN "Description"
@@
 F 0 "IC9" H 13300 8400 50  0000 C CNN
 F 1 "TLV3011" H 13500 8075 50  0000 C CNN
-F 2 "GR106768 Buzzer:SOT23-6_2" H 13350 8200 50  0001 C CNN
+F 2 "GR106768 Buzzer:SOT23-6_1" H 13350 8200 50  0001 C CNN
 F 3 "http://www.ti.com/lit/ds/symlink/tlv3012.pdf" H 13150 8200 50  0001 C CNN
 F 4 "IC, COMPARATOR, SOT23-6" H 13150 8200 50  0001 C CNN "Description"
@@
 F 0 "IC7" H 7900 3375 50  0000 C CNN
 F 1 "TLV3011" H 8100 3050 50  0000 C CNN
-F 2 "GR106768 Buzzer:SOT23-6_1" H 7950 3175 50  0001 C CNN
+F 2 "GR106768 Buzzer:SOT23-6_2" H 7950 3175 50  0001 C CNN
 F 3 "http://www.ti.com/lit/ds/symlink/tlv3012.pdf" H 7750 3175 50  0001 C CNN
 F 4 "IC, COMPARATOR, SOT23-6" H 7750 3175 50  0001 C CNN "Description"

Commit message: update corresponding fp fields
Parts:
- C15, C16, C17, C18, C19, C25, C27, C28, C31, C32, C33, C34: footprint GR106768 Buzzer:C0402_2 -> GR106768 Buzzer:C0402_1
- IC7: footprint GR106768 Buzzer:SOT23-6_2 -> GR106768 Buzzer:SOT23-6_1

Commit message: rename c0402 as it differs from global fp library
Parts:
- C15, C16, C17, C18, C19, C25, C27, C28, C31, C32, C33, C34, C35: footprint GR106768 Buzzer:C0402_1 -> GR106768 Buzzer:C0402_1b
Changed lines of the file:
@@
 F 0 "C15" H 1300 2800 50  0000 L CNN
 F 1 "100nF" H 1275 2600 50  0000 L CNN
-F 2 "GR106768 Buzzer:C0402_1" H 1288 2550 50  0001 C CNN
+F 2 "GR106768 Buzzer:C0402_1b" H 1288 2550 50  0001 C CNN
 F 3 "~" H 1250 2700 50  0001 C CNN
     1    1250 2700
@@
 F 0 "C31" H 15500 3825 50  0000 L CNN
 F 1 "100nF" H 15500 3600 50  0000 L CNN
-F 2 "GR106768 Buzzer:C0402_1" H 15513 3550 50  0001 C CNN
+F 2 "GR106768 Buzzer:C0402_1b" H 15513 3550 50  0001 C CNN
 F 3 "~" H 15475 3700 50  0001 C CNN
     1    15475 3700
@@
 F 0 "C28" H 14925 3800 50  0000 L CNN
 F 1 "100pF" H 14925 3600 50  0000 L CNN
-F 2 "GR106768 Buzzer:C0402_1" H 14938 3550 50  0001 C CNN
+F 2 "GR106768 Buzzer:C0402_1b" H 14938 3550 50  0001 C CNN
 F 3 "~" H 14900 3700 50  0001 C CNN
     1    14900 3700
@@
 F 0 "C16" H 2350 5175 50  0000 L CNN
 F 1 "100nF" H 2325 4950 50  0000 L CNN
-F 2 "GR106768 Buzzer:C0402_1" H 2338 4900 50  0001 C CNN
+F 2 "GR106768 Buzzer:C0402_1b" H 2338 4900 50  0001 C CNN
 F 3 "~" H 2300 5050 50  0001 C CNN
     1    2300 5050
@@
 F 0 "C17" H 4775 5000 50  0000 L CNN
 F 1 "100nF" H 4775 4800 50  0000 L CNN
-F 2 "GR106768 Buzzer:C0402_1" H 4788 4750 50  0001 C CNN
+F 2 "GR106768 Buzzer:C0402_1b" H 4788 4750 50  0001 C CNN
 F 3 "~" H 4750 4900 50  0001 C CNN
     1    4750 4900
@@
 F 0 "C18" H 6975 3600 50  0000 L CNN
 F 1 "100nF" H 6950 3400 50  0000 L CNN
-F 2 "GR106768 Buzzer:C0402_1" H 6963 3350 50  0001 C CNN
+F 2 "GR106768 Buzzer:C0402_1b" H 6963 3350 50  0001 C CNN
 F 3 "~" H 6925 3500 50  0001 C CNN
     1    6925 3500
@@
 F 0 "C19" V 7875 2650 50  0000 L CNN
 F 1 "100nF" V 8150 2800 50  0000 L CNN
-F 2 "GR106768 Buzzer:C0402_1" H 8088 2575 50  0001 C CNN
+F 2 "GR106768 Buzzer:C0402_1b" H 8088 2575 50  0001 C CNN
 F 3 "~" H 8050 2725 50  0001 C CNN
     1    8050 2725
@@
 F 0 "C35" H 9725 5450 50  0000 L CNN
 F 1 "4.7nF" H 9725 5250 50  0000 L CNN
-F 2 "GR106768 Buzzer:C0402_1" H 9713 5200 50  0001 C CNN
+F 2 "GR106768 Buzzer:C0402_1b" H 9713 5200 50  0001 C CNN
 F 3 "~" H 9675 5350 50  0001 C CNN
     1    9675 5350
@@
 F 0 "C34" H 12325 8450 50  0000 L CNN
 F 1 "NC" H 12300 8250 50  0000 L CNN
-F 2 "GR106768 Buzzer:C0402_1" H 12313 8200 50  0001 C CNN
+F 2 "GR106768 Buzzer:C0402_1b" H 12313 8200 50  0001 C CNN
 F 3 "~" H 12275 8350 50  0001 C CNN
     1    12275 8350
@@
 F 0 "C33" V 13650 7625 50  0000 L CNN
 F 1 "100nF" V 13300 7600 50  0000 L CNN
-F 2 "GR106768 Buzzer:C0402_1" H 13513 7550 50  0001 C CNN
+F 2 "GR106768 Buzzer:C0402_1b" H 13513 7550 50  0001 C CNN
 F 3 "~" H 13475 7700 50  0001 C CNN
     1    13475 7700
@@
 F 0 "C32" H 15100 6425 50  0000 L CNN
 F 1 "100nF" H 15100 6200 50  0000 L CNN
-F 2 "GR106768 Buzzer:C0402_1" H 15063 6150 50  0001 C CNN
+F 2 "GR106768 Buzzer:C0402_1b" H 15063 6150 50  0001 C CNN
 F 3 "~" H 15025 6300 50  0001 C CNN
     1    15025 6300
@@
 F 0 "C27" H 11950 4025 50  0000 L CNN
 F 1 "100pF" H 11925 3825 50  0000 L CNN
-F 2 "GR106768 Buzzer:C0402_1" H 11938 3775 50  0001 C CNN
+F 2 "GR106768 Buzzer:C0402_1b" H 11938 3775 50  0001 C CNN
 F 3 "~" H 11900 3925 50  0001 C CNN
     1    11900 3925
@@
 F 0 "C25" H 13775 5050 50  0000 L CNN
 F 1 "100nF" H 13775 4850 50  0000 L CNN
-F 2 "GR106768 Buzzer:C0402_1" H 13788 4800 50  0001 C CNN
+F 2 "GR106768 Buzzer:C0402_1b" H 13788 4800 50  0001 C CNN
 F 3 "~" H 13750 4950 50  0001 C CNN
     1    13750 4950

Commit message: rename c0603 as it differs from global fp library
Parts:
- C20: footprint GR106768 Buzzer:C0603_1 -> GR106768 Buzzer:C0603_1b
Changed lines of the file:
@@
 F 0 "C20" V 7875 4875 50  0000 L CNN
 F 1 "330nF" V 8200 4875 50  0000 L CNN
-F 2 "GR106768 Buzzer:C0603_1" H 8088 4800 50  0001 C CNN
+F 2 "GR106768 Buzzer:C0603_1b" H 8088 4800 50  0001 C CNN
 F 3 "~" H 8050 4950 50  0001 C CNN
     1    8050 4950

Commit message: rename rc0805 as it differs from global fp library
Parts:
- C24: footprint GR106768 Buzzer:C0805_1 -> GR106768 Buzzer:C0805_1b
- R36, R71: footprint GR106768 Buzzer:R0805_1 -> GR106768 Buzzer:R0805_1b
Changed lines of the file:
@@
 F 0 "C24" V 13650 5925 50  0000 L CNN
 F 1 "1uF" V 13300 5900 50  0000 L CNN
-F 2 "GR106768 Buzzer:C0805_1" H 13513 5850 50  0001 C CNN
+F 2 "GR106768 Buzzer:C0805_1b" H 13513 5850 50  0001 C CNN
 F 3 "~" H 13475 6000 50  0001 C CNN
     1    13475 6000
@@
 F 0 "R36" H 3475 2525 50  0000 C CNN
 F 1 "33" H 3475 2425 50  0000 C CNN
-F 2 "GR106768 Buzzer:R0805_1" H 3475 2625 50  0001 C CNN
+F 2 "GR106768 Buzzer:R0805_1b" H 3475 2625 50  0001 C CNN
 F 3 "~" H 3475 2425 50  0001 C CNN
 F 4 "RESISTOR 33 OHM +/- 1% 0,125W,0805" H 3475 2625 50  0001 C CNN "Description"
@@
 F 0 "R71" H 2450 6550 50  0000 C CNN
 F 1 "470" H 2450 6450 50  0000 C CNN
-F 2 "GR106768 Buzzer:R0805_1" H 2450 6650 50  0001 C CNN
+F 2 "GR106768 Buzzer:R0805_1b" H 2450 6650 50  0001 C CNN
 F 3 "~" H 2450 6450 50  0001 C CNN
 F 4 "RESISTOR,470 OHM, 0.125W,+/-1%, 0805" H 2450 6650 50  0001 C CNN "Description"

Commit message: update fp libpaths
Parts:
- BAT1: footprint GR106768 Buzzer:BT-4-V150H-4.8V_1 -> AllModules:BT-4-V150H-4.8V_1
- C15, C16, C17, C18, C19, C25, C27, C28, C31, C32, C33, C34, C35: footprint GR106768 Buzzer:C0402_1b -> AllModules:C0402_1b
- C20: footprint GR106768 Buzzer:C0603_1b -> AllModules:C0603_1b
- C21, C23: footprint GR106768 Buzzer:C1210_1 -> AllModules:C1210_1
- C22, C26, C29: footprint GR106768 Buzzer:RC1206_1 -> AllModules:RC1206_1
- C24: footprint GR106768 Buzzer:C0805_1b -> AllModules:C0805_1b
- D10, D11, D12, D13, D14, D8: footprint GR106768 Buzzer:DO216AA_1 -> AllModules:DO216AA_1
- D15, D16, D17, D6, D7, D9: footprint GR106768 Buzzer:SOT23-1G_1 -> AllModules:SOT23-1G_1
- IC5, IC6: footprint GR106768 Buzzer:MX.A8_COMPOSANT_1 -> AllModules:MX.A8_COMPOSANT_1
- IC7, IC9: footprint GR106768 Buzzer:SOT23-6_1 -> AllModules:SOT23-6_1
- IC8: footprint GR106768 Buzzer:DFN10_1 -> AllModules:DFN10_1
- JP1: footprint GR106768 Buzzer:TB-CMS-AIROX_1 -> AllModules:TB-CMS-AIROX_1
- L2, L3, L4: footprint GR106768 Buzzer:WETPC-S_1 -> AllModules:WETPC-S_1
- LD1: footprint GR106768 Buzzer:D0603_1 -> AllModules:D0603_1
- R30, R31, R32, R33, R34, R35, R37, R38, R39, R40, R41, R42, R43, R44, R45, R46, R47, R48, R49, R50, R51, R52, R53, R54, R55, R56, R57, R58, R60, R61, R62, R63, R64, R65, R66, R67, R68, R70: footprint GR106768 Buzzer:R0402_1 -> AllModules:R0402_1
- R36, R71: footprint GR106768 Buzzer:R0805_1b -> AllModules:R0805_1b
- SJ1: footprint GR106768 Buzzer:TB-CMS-AIROX-2_1 -> AllModules:TB-CMS-AIROX-2_1
- SW1: footprint GR106768 Buzzer:NK236_1_1 -> AllModules:NK236_1_1
- T10, T11, T12, T13, T5, T6, T7, T8, T9: footprint GR106768 Buzzer:SOT23-GSD_1 -> AllModules:SOT23-GSD_1
