File: GR106768 Buzzer/old.kicad_pcb (KiCad board)
At the start: 4 copper layers, 76 x 58 mm, 232 parts, among them IC1 L-BC-SOT23-5, IC2 L-BC-SO08, IC3 L-BC-SO08, IC4 L-BC-SOT23-5, IC5 L-BC-SO08, IC6 L-BC-SO08, IC7 L-BC-SOT23-6, IC8 L-BC-DFN10, IC9 L-BC-SOT23-6, J1 BAR-10-1007, J2 MIRECMS, J3 MIRECMS, SW1 SI-10-NK236, T1 Q-BC-SOT23-BEC, T10 Q-BC-SOT23-GSD, T11 Q-BC-SOT23-GSD, T12 Q-BC-SOT23-GSD, T13 Q-BC-SOT23-GSD, T2 Q-BC-SOT23-BEC, T3 Q-BC-SOT23-BEC, T4 Q-BC-SOT23-BEC, T5 Q-BC-SOT23-GSD, T6 Q-BC-SOT23-GSD, T7 Q-BC-SOT23-GSD, T8 Q-BC-SOT23-GSD, T9 Q-BC-SOT23-GSD

Commit message: PCB and schematic updates
Parts:
- removed L2-2: SF-BC-NR4018, NR4018_1
- removed L3-2, L4-2: SF-BC-NR4012, NR4012_1
- added V100: Val**, AllModules:Via_12x32-1._.3.4, F.Cu at (174.7, 75.2)
- added V101: Val**, AllModules:Via_12x32, F.Cu at (111.7, 73.5)
- added V102: Val**, AllModules:Via_12x32-1._.3.4, F.Cu at (132.6, 72.6)
- added V103: Val**, AllModules:Via_12x32, F.Cu at (158.8, 71.7)
- added V104: Val**, AllModules:Via_12x32-1._.3.4, F.Cu at (165.1, 71.9)
- added V105: Val**, AllModules:Via_12x32-1._.3.4, F.Cu at (132.6, 70.9)
- added V106: Val**, AllModules:Via_12x32-1._.3.4, F.Cu at (151.4, 71.2)
- added V107: Val**, AllModules:Via_12x32, F.Cu at (184.4, 71.0)
- added V108: Val**, AllModules:Via_12x32-1._.3.4, F.Cu at (125.9, 70.2)
- added V109: Val**, AllModules:Via_12x32-1._.3.4, F.Cu at (177.4, 70.5)
- added V110: Val**, AllModules:Via_12x32-1._.3.4, F.Cu at (132.6, 69.6)
- added V111: Val**, AllModules:Via_12x32, F.Cu at (111.7, 68.5)
- added V112: Val**, AllModules:Via_12x32-1._.3.4, F.Cu at (158.8, 68.3)
- added V113: Val**, AllModules:Via_12x32, F.Cu at (165.1, 68.3)
- added V114: Val**, AllModules:Via_12x32-1._.3.4, F.Cu at (167.5, 68.6)
- added V115: Val**, AllModules:Via_12x32-1._.3.4, F.Cu at (132.6, 67.8)
- added V116: Val**, AllModules:Via_12x32, F.Cu at (116.5, 67.5)
- added V117: Val**, AllModules:Via_12x32, F.Cu at (123.3, 67.5)
- added V118: Val**, AllModules:Via_12x32-1._.3.4, F.Cu at (127.5, 67.0)
- added V119: Val**, AllModules:Via_12x32-1._.3.4, F.Cu at (174.9, 67.0)
- added V120: Val**, AllModules:Via_12x32-1._.3.4, F.Cu at (132.6, 66.5)
- added V121: Val**, AllModules:Via_12x32-1._.3.4, F.Cu at (151.4, 66.4)
- added V122: Val**, AllModules:Via_12x32-1._.3.4, F.Cu at (181.9, 66.2)
- added V123: Val**, AllModules:Via_12x32-1._.3.4, F.Cu at (132.6, 64.8)
- added V124: Val**, AllModules:Via_12x32, F.Cu at (111.7, 63.6)
- added V125: Val**, AllModules:Via_12x32, F.Cu at (124.0, 63.6)
- added V126: Val**, AllModules:Via_12x32, F.Cu at (129.0, 63.6)
- added V127: Val**, AllModules:Via_12x32, F.Cu at (134.0, 63.6)
- added V128: Val**, AllModules:Via_12x32, F.Cu at (139.0, 63.6)
- added V129: Val**, AllModules:Via_12x32, F.Cu at (144.0, 63.6)
- added V130: Val**, AllModules:Via_12x32, F.Cu at (149.0, 63.6)
- added V131: Val**, AllModules:Via_12x32, F.Cu at (154.0, 63.6)
- added V132: Val**, AllModules:Via_12x32, F.Cu at (159.0, 63.6)
- added V133: Val**, AllModules:Via_12x32, F.Cu at (164.0, 63.6)
- added V134: Val**, AllModules:Via_12x32, F.Cu at (174.0, 63.6)
- added V135: Val**, AllModules:Via_12x32, F.Cu at (179.0, 63.6)
- added V136: Val**, AllModules:Via_12x32, F.Cu at (184.4, 63.6)
- added V137: Val**, AllModules:Via_12x32, F.Cu at (184.4, 66.5)
- added V138: Val**, AllModules:Via_12x32, F.Cu at (171.3, 86.0)
- added V139: Val**, AllModules:Via_12x32-1._.3.4, F.Cu at (122.2, 101.2)
- added V140: Val**, AllModules:Via_12x32, F.Cu at (129.1, 100.3)
- added V141: Val**, AllModules:Via_12x32-1._.3.4, F.Cu at (156.1, 81.1)
- added V142: Val**, AllModules:Via_12x32-1._.3.4, F.Cu at (178.3, 79.7)
- added V143: Val**, AllModules:Via_12x32, F.Cu at (173.2, 76.2)
- added V144: Val**, AllModules:Via_12x32, F.Cu at (161.9, 89.3)
- added V145: Val**, AllModules:Via_12x32-1._.3.4, F.Cu at (143.0, 70.8)
- added V146: Val**, AllModules:Via_12x32-1._.3.4, F.Cu at (123.3, 103.7)
- added V147: Val**, AllModules:Via_12x32, F.Cu at (134.0, 83.6)
- added V148: Val**, AllModules:Via_12x32, F.Cu at (123.3, 71.7)
- added V149: Val**, AllModules:Via_12x32-1._.3.4, F.Cu at (147.0, 68.6)
- added V150: Val**, AllModules:Via_12x32-1._.3.4, F.Cu at (141.2, 68.7)
- added V151: Val**, AllModules:Via_12x32-1._.3.4, F.Cu at (135.9, 68.6)
- added V152: Val**, AllModules:Via_12x32-1._.3.4, F.Cu at (139.5, 70.8)
- added V153: Val**, AllModules:Via_12x32-1._.3.4, F.Cu at (139.5, 71.7)
- added V154: Val**, AllModules:Via_12x32-1._.3.4, F.Cu at (143.0, 71.7)
- added V155: Val**, AllModules:Via_12x32-1._._.4, F.Cu at (140.5, 73.3)
- added V156: Val**, AllModules:Via_12x32-1._._.4, F.Cu at (142.1, 73.3)
- added V157: Val**, AllModules:Via_12x32, F.Cu at (152.5, 94.5)
- added V158: Val**, AllModules:Via_12x32, F.Cu at (158.3, 94.6)
- added V159: Val**, AllModules:Via_12x32-1._._.4, F.Cu at (159.3, 96.7)
- added V160: Val**, AllModules:Via_12x32-1._._.4, F.Cu at (155.7, 90.7)
- added V161: Val**, AllModules:Via_12x32-1._._.4, F.Cu at (150.3, 90.7)
- added V162: Val**, AllModules:Via_12x32, F.Cu at (126.6, 79.4)
- added V163: Val**, AllModules:Via_12x32, F.Cu at (134.0, 99.8)
- added V164: Val**, AllModules:Via_12x32-1._.3.4, F.Cu at (134.1, 98.2)
- added V165: Val**, AllModules:Via_12x32-1._.3.4, F.Cu at (134.6, 104.0)
- added V166: Val**, AllModules:Via_12x32-1._.3.4, F.Cu at (139.1, 102.2)
- added V167: Val**, AllModules:Via_12x32-1._.3.4, F.Cu at (138.2, 96.3)
- added V168: Val**, AllModules:Via_12x32-1._.3.4, F.Cu at (139.1, 110.6)
- added V169: Val**, AllModules:Via_12x32, F.Cu at (162.3, 104.0)
- added V170: Val**, AllModules:Via_12x32, F.Cu at (162.3, 102.5)
- added V171: Val**, AllModules:Via_12x32-1._.3.4, F.Cu at (161.4, 101.1)
- added V172: Val**, AllModules:Via_12x32-1._._.4, F.Cu at (130.4, 103.8)
- added V173: Val**, AllModules:Via_12x32-1._._.4, F.Cu at (132.8, 83.7)
- added V69: Val**, AllModules:Via_12x32, F.Cu at (123.1, 85.5)
- added V70: Val**, AllModules:Via_12x32, F.Cu at (139.5, 86.0)
- added V71: Val**, AllModules:Via_12x32, F.Cu at (126.1, 85.3)
- added V72: Val**, AllModules:Via_12x32, F.Cu at (166.6, 84.9)
- added V73: Val**, AllModules:Via_12x32, F.Cu at (159.1, 84.7)
- added V74: Val**, AllModules:Via_12x32, F.Cu at (111.7, 83.5)
- added V75: Val**, AllModules:Via_12x32, F.Cu at (116.0, 83.5)
- added V76: Val**, AllModules:Via_12x32-1._.3.4, F.Cu at (119.5, 83.8)
- added V77: Val**, AllModules:Via_12x32-1._.3.4, F.Cu at (154.3, 83.8)
- added V78: Val**, AllModules:Via_12x32-1._.3.4, F.Cu at (161.2, 83.8)
- added V79: Val**, AllModules:Via_12x32-1._.3.4, F.Cu at (168.3, 83.2)
- added V80: Val**, AllModules:Via_12x32-1._.3.4, F.Cu at (135.4, 82.2)
- added V81: Val**, AllModules:Via_12x32, F.Cu at (140.2, 82.2)
- added V82: Val**, AllModules:Via_12x32, F.Cu at (184.4, 81.0)
- added V83: Val**, AllModules:Via_12x32-1._.3.4, F.Cu at (144.4, 80.8)
- added V84: Val**, AllModules:Via_12x32, F.Cu at (111.7, 78.5)
- added V85: Val**, AllModules:Via_12x32, F.Cu at (134.0, 78.0)
- added V86: Val**, AllModules:Via_12x32, F.Cu at (143.3, 78.2)
- added V87: Val**, AllModules:Via_12x32, F.Cu at (140.4, 77.3)
- added V88: Val**, AllModules:Via_12x32, F.Cu at (141.2, 77.3)
- added V89: Val**, AllModules:Via_12x32, F.Cu at (142.1, 77.3)
- added V90: Val**, AllModules:Via_12x32-1._.3.4, F.Cu at (169.5, 77.2)
- added V91: Val**, AllModules:Via_12x32, F.Cu at (139.1, 76.7)
- added V92: Val**, AllModules:Via_12x32, F.Cu at (140.4, 76.4)
- added V93: Val**, AllModules:Via_12x32, F.Cu at (141.2, 76.4)
- added V94: Val**, AllModules:Via_12x32, F.Cu at (142.1, 76.4)
- added V95: Val**, AllModules:Via_12x32, F.Cu at (184.4, 76.0)
- added V96: Val**, AllModules:Via_12x32, F.Cu at (159.4, 75.8)
- added V97: Val**, AllModules:Via_12x32, F.Cu at (117.2, 74.7)
- added V98: Val**, AllModules:Via_12x32-1._.3.4, F.Cu at (120.7, 74.8)
- added V99: Val**, AllModules:Via_12x32, F.Cu at (165.6, 74.8)
- added ZL2: SF-BC-NR4018, NR4018, F.Cu at (136.4, 71.7)
- added ZL3: SF-BC-NR4012, NR4012, F.Cu at (146.2, 71.7)
- added ZL4: SF-BC-NR4012, NR4012, F.Cu at (147.7, 79.5)
- added cam2: PER-COVIDIEN_TEXTE, AllModules:PER-COVIDIEN_TEXTE, F.Cu at (15.0, 175.0)
- added cam6: COIN_EXTERNE, COIN_EXTERNE, F.Cu at (110.0, 62.0)
- added cam7: COIN_EXTERNE, COIN_EXTERNE, F.Cu at (110.0, 120.0)
- added cam8: COIN_EXTERNE, COIN_EXTERNE, F.Cu at (186.0, 120.0)
- added cam9: COIN_EXTERNE, COIN_EXTERNE, F.Cu at (186.0, 62.0)
- BAT1: footprint BT-4-V150H-4.8V_1 -> BT-4-V150H-4.8V_100110011001
- BUZ1: footprint PKM33EPH-1201C_1 -> AllModules:PKM33EPH-1201C_101110111001
- BUZ2: footprint PKM33EPH-1201C_1 -> AllModules:PKM33EPH-1201C_100110111001
- C1: footprint C0612-4_1 -> C0612-4
- C10, C11, C15, C16, C17, C18, C19, C2, C25, C27, C28, C30, C31, C32, C33, C34, C35, C4, C5, C6, C7, C8, C9: footprint C0402_1 -> C0402
- C12: footprint AX10X30_1 -> AX10X30_10111011
- C13, C14, C20: footprint C0603_1 -> C0603
- C21, C23: footprint C1210_1 -> C1210
- C22, C26, C29, L1: footprint RC1206_1 -> RC1206
- C24, C3: footprint C0805_1 -> C0805
- D1, D10, D11, D12, D13, D14, D8: footprint DO216AA_1 -> DO216AA
- D15, D16, D17, D2, D3, D4, D5, D6, D7, D9: footprint SOT23-1G_1 -> SOT23-1G
- FI1: footprint WE-FA_1 -> WE-FA
- FU1: footprint F6126_1 -> F6126
- IC1, IC4: footprint SOT23-5_1 -> SOT23-5
- IC2, IC3, IC5, IC6: footprint MX.A8_COMPOSANT_1 -> MX.A8_COMPOSANT
- IC7, IC9: footprint SOT23-6_1 -> SOT23-6
- IC8: footprint DFN10_1 -> DFN10
- J1: footprint BAR7-3-2-COVIDIEN_1 -> BAR7-3-2-COVIDIEN_1111100110011001100110011001
- J2, J3: footprint MIRECMS-SAFT_1 -> MIRECMS-SAFT
- JP1: footprint TB-CMS-AIROX_1 -> AllModules:TB-CMS-AIROX_1
- L2, L3, L4: footprint WETPC-S_1 -> WETPC-S
- LD1: footprint D0603_1 -> D0603
- R1, R10, R11, R12, R13, R14, R15, R16, R17, R18, R19, R2, R20, R21, R22, R23, R24, R25, R26, R27, R28, R29, R3, R30, R31, R32, R33, R34, R35, R37, R38, R39, R4, R40, R41, R42, R43, R44, R45, R46, R47, R48, R49, R5, R50, R51, R52, R53, R54, R55, R56, R57, R58, R59, R6, R60, R61, R62, R63, R64, R65, R66, R67, R68, R69, R7, R70, R8, R9: footprint R0402_1 -> R0402
- R36, R71: footprint R0805_1 -> R0805
- SJ1: footprint TB-CMS-AIROX-2_1 -> TB-CMS-AIROX-2
- SW1: footprint NK236_1_1 -> NK236_1_100110011111
- T1, T2, T3, T4: footprint SOT23-BEC_1 -> SOT23-BEC
- T10, T11, T12, T13, T5, T6, T7, T8, T9: footprint SOT23-GSD_1 -> SOT23-GSD
- V1, V2, V3, V4, V5: value +5V -> Val**; footprint AllModules:Via_12x32-1._.3.4 -> AllModules:Via_12x32
- V10, V11: value SUPPLY-BUZ-CPU -> Val**; footprint AllModules:Via_12x32-1._.3.4 -> AllModules:Via_12x32
- V12, V13, V14: value -12V -> Val**; footprint AllModules:Via_12x32-1._.3.4 -> AllModules:Via_12x32
- V15: value -12V -> Val**
- V16: value N$78 -> Val**
- V17: value N$78 -> Val**; footprint AllModules:Via_12x32-1._.3.4 -> AllModules:Via_12x32
- V18, V19: value N$58 -> Val**; footprint AllModules:Via_12x32-1._.3.4 -> AllModules:Via_12x32
- V20: value N$31 -> Val**; footprint AllModules:Via_12x32-1._.3.4 -> AllModules:Via_12x32
- V21, V22: value GT1 -> Val**; footprint AllModules:Via_12x32-1._.3.4 -> AllModules:Via_12x32
- V23, V24, V25, V26, V28: value +12V -> Val**; footprint AllModules:Via_12x32-1._.3.4 -> AllModules:Via_12x32
- V27: value +12V -> Val**
- V29: value BATTV -> Val**; footprint AllModules:Via_12x32-1._._.4 -> AllModules:Via_12x32
- V30: value N$19 -> Val**
- V31: value N$18 -> Val**
- V32: value N$18 -> Val**; footprint AllModules:Via_12x32-1._.3.4 -> AllModules:Via_12x32
- V33: value N$10 -> Val**; footprint AllModules:Via_12x32-1._._.4 -> AllModules:Via_12x32
- V34, V36, V39, V40, V41, V42, V43, V44, V45, V46: value N$10 -> Val**; footprint AllModules:Via_12x32-1._.3.4 -> AllModules:Via_12x32
- V35, V37, V38: value N$10 -> Val**
- V47, V48: value STOP-INV -> Val**; footprint AllModules:Via_12x32-1._.3.4 -> AllModules:Via_12x32
- V49, V51: value VCHARG -> Val**
- V50: value VCHARG -> Val**; footprint AllModules:Via_12x32-1._.3.4 -> AllModules:Via_12x32
- V52: value VCHARG -> Val**; footprint AllModules:Via_12x32-1._._.4 -> AllModules:Via_12x32-1._.3.4
- V53, V54: value VBAT -> Val**
- V55: value VBAT -> Val**; footprint AllModules:Via_12x32-1._.3.4 -> AllModules:Via_12x32
- V56, V57, V59: value SUPPLY-BUZ -> Val**; footprint AllModules:Via_12x32-1._.3.4 -> AllModules:Via_12x32
- V58, V60: value SUPPLY-BUZ -> Val**
- V6, V7, V8, V9: value BUZ-ACT -> Val**; footprint AllModules:Via_12x32-1._.3.4 -> AllModules:Via_12x32
- V61, V62: value SHDN2 -> Val**; footprint AllModules:Via_12x32-1._._.4 -> AllModules:Via_12x32-1._.3.4
- V63, V64: value SHDN1 -> Val**; footprint AllModules:Via_12x32-1._._.4 -> AllModules:Via_12x32-1._.3.4
- V65, V66, V67, V68: value INHIB-STOP-INV -> Val**; footprint AllModules:Via_12x32-1._.3.4 -> AllModules:Via_12x32
- moved V13 63.2 mm to (120.7, 114.5)
- moved V47 61.0 mm to (121.0, 90.9)
- moved V23 59.2 mm to (111.7, 108.5)
- moved V57 57.4 mm to (116.0, 88.5)
- moved V10 57.3 mm to (166.5, 118.3)
- moved V3 56.5 mm to (131.5, 118.3)
- moved V11 56.3 mm to (171.5, 118.3)
- moved V41 54.5 mm to (184.4, 96.0)
- moved V33 52.7 mm to (111.7, 98.5)
- moved V2 48.3 mm to (126.5, 118.3)
- moved V12 46.5 mm to (175.4, 117.0)
- moved V60 46.0 mm to (176.2, 88.0)
- moved V36 41.5 mm to (178.5, 98.0)
- moved V16 40.6 mm to (164.9, 111.1)
- moved V24 40.1 mm to (161.5, 106.0)
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Connections:
- net +5V_CPU renamed /+5V_CPU
- net INHIB-STOP-INV-CPU renamed /INHIB-STOP-INV-CPU
- net N$1 renamed /N$1
- net N$11 renamed /N$11
- net N$12 renamed /N$12
- net N$13 renamed /N$13
- net N$14 renamed /N$14
- net N$15 renamed /N$15
- net N$16 renamed /N$16
- net N$17 renamed /N$17
- net N$2 renamed /N$2
- net N$20 renamed /N$20
- net N$21 renamed /N$21
- net N$22 renamed /N$22
- net N$23 renamed /N$23
- net N$24 renamed /N$24
- net N$25 renamed /N$25
- net N$26 renamed /N$26
- net N$27 renamed /N$27
- net N$28 renamed /N$28
- net N$29 renamed /N$29
- net N$3 renamed /N$3
- net N$30 renamed /N$30
- net N$32 renamed /N$32
- net N$33 renamed /N$33
- net N$34 renamed /N$34
- net N$35 renamed /N$35
- net N$36 renamed /N$36
- net N$37 renamed /N$37
- net N$38 renamed /N$38
- net N$39 renamed /N$39
- net N$4 renamed /N$4
- net N$40 renamed /N$40
- net N$41 renamed /N$41
- net N$42 renamed /N$42
- net N$43 renamed /N$43
- net N$44 renamed /N$44
- net N$45 renamed /N$45
- net N$46 renamed /N$46
- net N$47 renamed /N$47
- net N$48 renamed /N$48
- net N$49 renamed /N$49
- net N$5 renamed /N$5
- net N$50 renamed /N$50
- net N$51 renamed /N$51
- net N$52 renamed /N$52
- net N$53 renamed /N$53
- net N$54 renamed /N$54
- net N$55 renamed /N$55
- net N$56 renamed /N$56
- net N$57 renamed /N$57
- net N$59 renamed /N$59
- net N$6 renamed /N$6
- net N$7 renamed /N$7
- net N$8 renamed /N$8
- net N$9 renamed /N$9
- net PWM-BUZ renamed /PWM-BUZ
- net PWM-BUZZER-CPU renamed /PWM-BUZZER-CPU
- net STOP-INV-CPU renamed /STOP-INV-CPU
- net TEST-BUZZER-CPU renamed /TEST-BUZZER-CPU
- net TESTBUZ renamed /TESTBUZ
- BAT1 pad +: BATTV -> /BATTV
- BUZ1 pad 1: N$19 -> /N$19
- BUZ1 pad 2: N$31 -> /N$31
- BUZ2 pad 1: N$19 -> /N$19
- BUZ2 pad 2: N$31 -> /N$31
- C10 pad 2: +12V -> /+12V
- C11 pad 2: -12V -> /-12V
- C12 pad +: +12V -> /+12V
- C12 pad -: -12V -> /-12V
- C15 pad 2: +12V -> /+12V
- C16 pad 1: N$58 -> /N$58
- C19 pad 1: VCHARG -> /VCHARG
- C2 pad 2: +5V -> /+5V
- C20 pad 1: GT1 -> /GT1
- C20 pad 2: STOP-INV -> /STOP-INV
- C21 pad 2: SHDN1 -> /SHDN1
- C22 pad 1: N$10 -> /N$10
- C23 pad 2: SHDN2 -> /SHDN2
- C26 pad 1: -12V -> /-12V
- C27 pad 1: -12V -> /-12V
- C28 pad 2: +12V -> /+12V
- C29 pad 2: +12V -> /+12V
- C30 pad 1: +5V -> /+5V
- C31 pad 2: +12V -> /+12V
- C32 pad 2: -12V -> /-12V
- C33 pad 1: N$10 -> /N$10
- C35 pad 2: GT1 -> /GT1
- C5 pad 1: SUPPLY-BUZ -> /SUPPLY-BUZ
- C7 pad 1: +12V -> /+12V
- C8 pad 1: -12V -> /-12V
- D1 pad A: SUPPLY-BUZ -> /SUPPLY-BUZ
- D1 pad K: SUPPLY-BUZ-CPU -> /SUPPLY-BUZ-CPU
- D10 pad A: +5V -> /+5V
- D10 pad K: N$10 -> /N$10
- D11 pad A: SUPPLY-BUZ -> /SUPPLY-BUZ
- D11 pad K: N$10 -> /N$10
- D13 pad K: +12V -> /+12V
- D14 pad A: SUPPLY-BUZ -> /SUPPLY-BUZ
- D14 pad K: N$10 -> /N$10
- D15 pad 3: VCHARG -> /VCHARG
- D16 pad 1: +5V -> /+5V
- D16 pad 2: INHIB-STOP-INV -> /INHIB-STOP-INV
- D17 pad 1: +5V -> /+5V
- D17 pad 2: +5V -> /+5V
- D3 pad 3: N$31 -> /N$31
- D5 pad 3: BUZ-ACT -> /BUZ-ACT
- D7 pad 3: N$58 -> /N$58
- D8 pad K: VCHARG -> /VCHARG
- D9 pad 2: INHIB-STOP-INV -> /INHIB-STOP-INV
- D9 pad 3: GT1 -> /GT1
- FI1 pad L2A: STOP-INV -> /STOP-INV
- FI1 pad L4A: INHIB-STOP-INV -> /INHIB-STOP-INV
- IC1 pad 2: SUPPLY-BUZ -> /SUPPLY-BUZ
- IC2 pad 4: -12V -> /-12V
- IC2 pad 8: +12V -> /+12V
- IC3 pad 4: -12V -> /-12V
- IC3 pad 8: +12V -> /+12V
- IC4 pad 5: +5V -> /+5V
- IC5 pad 1: +12V -> /+12V
- IC6 pad 2: N$78 -> /N$78
- IC6 pad 6: N$58 -> /N$58
- IC7 pad 6: VCHARG -> /VCHARG
- IC8 pad 7: SHDN2 -> /SHDN2
- IC8 pad 8: N$10 -> /N$10
- IC8 pad 9: SHDN1 -> /SHDN1
- IC9 pad 6: N$10 -> /N$10
- J1 pad 6: SUPPLY-BUZ-CPU -> /SUPPLY-BUZ-CPU
- JP1 pad 2: GT1 -> /GT1
- L1 pad 2: +5V -> /+5V
- L2 pad 1: N$10 -> /N$10
- L3 pad 1: N$10 -> /N$10
- L4 pad 2: -12V -> /-12V
- LD1 pad K: N$78 -> /N$78
- R12 pad 2: N$19 -> /N$19
- R13 pad 1: N$19 -> /N$19
- R14 pad 2: N$19 -> /N$19
- R2 pad 2: SUPPLY-BUZ -> /SUPPLY-BUZ
- R20 pad 1: N$18 -> /N$18
- R23 pad 2: BUZ-ACT -> /BUZ-ACT
- R24 pad 2: BUZ-ACT -> /BUZ-ACT
- R25 pad 2: VBAT -> /VBAT
- R30 pad 1: BUZ-ACT -> /BUZ-ACT
- R31 pad 1: SUPPLY-BUZ -> /SUPPLY-BUZ
- R33 pad 1: N$58 -> /N$58
- R33 pad 2: +12V -> /+12V
- R34 pad 2: N$58 -> /N$58
- R38 pad 2: N$58 -> /N$58
- R40 pad 1: +12V -> /+12V
- R41 pad 1: VCHARG -> /VCHARG
- R43 pad 2: VCHARG -> /VCHARG
- R47 pad 2: VCHARG -> /VCHARG
- R48 pad 1: STOP-INV -> /STOP-INV
- R48 pad 2: GT1 -> /GT1
- R49 pad 2: GT1 -> /GT1
- R50 pad 1: VBAT -> /VBAT
- R50 pad 2: +5V -> /+5V
- R51 pad 2: VBAT -> /VBAT
- R52 pad 1: GT1 -> /GT1
- R52 pad 2: SUPPLY-BUZ -> /SUPPLY-BUZ
- R53 pad 1: N$10 -> /N$10
- R53 pad 2: SHDN2 -> /SHDN2
- R54 pad 1: N$10 -> /N$10
- R54 pad 2: SHDN1 -> /SHDN1
- R56 pad 2: -12V -> /-12V
- R57 pad 1: +12V -> /+12V
- R60 pad 1: STOP-INV -> /STOP-INV
- R60 pad 2: +5V -> /+5V
- R61 pad 2: N$10 -> /N$10
- R63 pad 2: SHDN1 -> /SHDN1
- R64 pad 2: SHDN2 -> /SHDN2
- R65 pad 2: SUPPLY-BUZ -> /SUPPLY-BUZ
- R66 pad 2: +12V -> /+12V
- R67 pad 2: BATTV -> /BATTV
- R69 pad 1: VCHARG -> /VCHARG
- R71 pad 2: BATTV -> /BATTV
- T1 pad C: +12V -> /+12V
- T10 pad D: SHDN1 -> /SHDN1
- T11 pad S: BATTV -> /BATTV
- T12 pad S: VCHARG -> /VCHARG
- T2 pad C: -12V -> /-12V
- T3 pad C: +12V -> /+12V
- T4 pad C: -12V -> /-12V
- T4 pad E: N$18 -> /N$18
- T6 pad D: VBAT -> /VBAT
- T6 pad S: VCHARG -> /VCHARG
- T7 pad G: GT1 -> /GT1
- T8 pad D: SUPPLY-BUZ -> /SUPPLY-BUZ
- T8 pad S: VBAT -> /VBAT
- T9 pad D: SHDN2 -> /SHDN2
Routing:
- net GND: track 787.5 -> 465.3 mm, vias 105 -> 0
- net +12V: track 195.6 -> 0.00 mm
- net /+12V: track 0.00 -> 195.6 mm
- net +5V: track 138.3 -> 0.00 mm
- net /+5V: track 0.00 -> 138.2 mm
- net /INHIB-STOP-INV: track 0.00 -> 131.1 mm
- net INHIB-STOP-INV: track 131.1 -> 0.00 mm
- net STOP-INV: track 116.7 -> 0.00 mm
- net /STOP-INV: track 0.00 -> 116.7 mm
- net N$10: track 110.3 -> 0.00 mm
- net /N$10: track 0.00 -> 98.6 mm
- net VCHARG: track 98.1 -> 0.00 mm
- net /VCHARG: track 0.00 -> 98.1 mm
- net SUPPLY-BUZ: track 97.1 -> 0.00 mm
- net /SUPPLY-BUZ: track 0.00 -> 97.0 mm
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- removed copper zone on F.Cu, net /N$42
- removed copper zone on F.Cu, net /N$46
- removed copper zone on In2.Cu, net N$10
Other:
- rule trace_min: 0.2 -> 0.1
- board text added: "(1)"
- board text added: "(1) Arraser les pattes des buzzers Respecter la cote de hauteur de cablage des buzzers. Voir plan 40966.E04.000. (1) Level off the buzzer's pins Respect the height dimension for buzzers assembling. Refer to drawing 40966.E04.000."
- board text added: "(1) Fabrique suivant IPC A610 classe III. (1) Manufactured according to IPC A610 class III."
- board text added: "(2)Le fabricant doit etre reconnu UL et doit apposer le marquage correspondant. (2) The manufacturer must be recognized UL and must affix corresponding marking."
- board text added: "+0.10 -0.10"
- board text added: "11.50"
- board text added: "15"
- board text added: "17.00"
- board text added: "18.55"
- board text added: "2.0"
- board text added: "21.00"
- board text added: "25.5"
- board text added: "3.68"
- board text added: "3.81"
- board text added: "31.15"
- board text added: "34.00"
- board text added: "58.00"
- board text added: "7 brins AWG 34 lg 60 +/-2mm"
- board text added: "7 fils blanc UL 1061 AWG26"
- board text added: "7 strands AWG 34 length 60 +/-2mm"
- board text added: "7 white wires UL 1061 AWG26"
- board text added: "7.5"
- board text added: "7.84"
- board text added: "76.00"
- board text added: "9.79"
- board text added: "ATTENTION: Le circuit imprime doit etre UL94V-0. WARNING: The printed circuit board must be UL94V-0."
- board text added: "BAT1"
- board text added: "BUZ1"
- board text added: "BUZ2"
- board text added: "C1"
- board text added: "C10"
- board text added: "C11"
- board text added: "C12"
- board text added: "C12 et BAT1 doivent etre colles. Voir plan 40966.E04.000. C12 and BAT1 must be glued. Refer to drawing 40966.E04.000."
- board text added: "C13"
- board text added: "C14"
- board text added: "C15"
- board text added: "C16"
- board text added: "C17"
- board text added: "C18"
- board text added: "C19"
- board text added: "C2"
- board text added: "C20"
- board text added: "C21"
- board text added: "C22"
- board text added: "C23"
- board text added: "C24"
- board text added: "C25"
- board text added: "C26"
- board text added: "C27"
- board text added: "C28"
- board text added: "C29"
- board text added: "C3"
- board text added: "C30"
- board text added: "C31"
- board text added: "C32"
- board text added: "C33"
- board text added: "C34"
- board text added: "C35"
- board text added: "C4"
- board text added: "C5"
- board text added: "C6"
- board text added: "C7"
- board text added: "C8"
- board text added: "C9"
- board text added: "Connecteur JST fem modele ZHR 7"
- board text added: "D1"
- board text added: "D10"
- board text added: "D11"
- board text added: "D12"
- board text added: "D13"
- board text added: "D14"
- board text added: "D15"
- board text added: "D16"
- board text added: "D17"
- board text added: "D2"
- board text added: "D3"
- board text added: "D4"
- board text added: "D5"
- board text added: "D6"
- board text added: "D7"
- board text added: "D8"
- board text added: "D9"
- board text added: "FI1"
- board text added: "FU1"
- board text added: "Fabrique suivant IPC A610 classe III. Manufactured according to IPC A610 class III."
- board text added: "Fabrique suivant IPC A610 classe III. Manufactured according to IPC A610 classe III."
- board text added: "Fils colle par colle Scotch Weld ref: 7838 B/A Wires stuck with Scotch Weld glue ref : 7838 B/A"
- board text added: "IC1"
- board text added: "IC2"
- board text added: "IC3"
- board text added: "IC4"
- board text added: "IC5"
- board text added: "IC6"
- board text added: "IC7"
- board text added: "IC8"
- board text added: "IC9"
- board text added: "J1"
- board text added: "J2"
- board text added: "J3"
- board text added: "JP1"
- board text added: "JST female connector model ZHR 7"
- board text added: "L1"
- board text added: "L2"
- board text added: "L2-2"
- board text added: "L3"
- board text added: "L3-2"
- board text added: "L4"
- board text added: "L4-2"
- board text added: "LD1"
- board text added: "R1"
- board text added: "R10"
- board text added: "R11"
- board text added: "R12"
- board text added: "R13"
- board text added: "R14"
- board text added: "R15"
- board text added: "R16"
- board text added: "R17"
- board text added: "R18"
- board text added: "R19"
- board text added: "R2"
- board text added: "R20"
- board text added: "R21"
- board text added: "R22"
- board text added: "R23"
- board text added: "R24"
- board text added: "R25"
- board text added: "R26"
- board text added: "R27"
- board text added: "R28"
- board text added: "R29"
- board text added: "R3"
- board text added: "R30"
- board text added: "R31"
- board text added: "R32"
- board text added: "R33"
- board text added: "R34"
- board text added: "R35"
- board text added: "R36"
- board text added: "R37"
- board text added: "R38"
- board text added: "R39"
- board text added: "R4"
- board text added: "R40"
- board text added: "R41"
- board text added: "R42"
- board text added: "R43"
- board text added: "R44"
- board text added: "R45"
- board text added: "R46"
- board text added: "R47"
- board text added: "R48"
- board text added: "R49"
- board text added: "R5"
- board text added: "R50"
- board text added: "R51"
- board text added: "R52"
- board text added: "R53"
- board text added: "R54"
- board text added: "R55"
- board text added: "R56"
- board text added: "R57"
- board text added: "R58"
- board text added: "R59"
- board text added: "R6"
- board text added: "R60"
- board text added: "R61"
- board text added: "R62"
- board text added: "R63"
- board text added: "R64"
- board text added: "R65"
- board text added: "R66"
- board text added: "R67"
- board text added: "R68"
- board text added: "R69"
- board text added: "R7"
- board text added: "R70"
- board text added: "R71"
- board text added: "R8"
- board text added: "R9"
- board text added: "SJ1"
- board text added: "SW1"
- board text added: "T1"
- board text added: "T10"
- board text added: "T11"
- board text added: "T12"
- board text added: "T13"
- board text added: "T2"
- board text added: "T3"
- board text added: "T4"
- board text added: "T5"
- board text added: "T6"
- board text added: "T7"
- board text added: "T8"
- board text added: "T9"
- board text added: "Toutes les dimensions sont en millimetre. All the dimensions are in millimeter."
- board text added: "Zone de positionnement de l'etiquette de tracabilite (12x25mm) Traceability label positionning zone (12x25mm)"
- board text added: "cam1"
- board text added: "cam14"
- board text added: "cam3"
- board text added: "cam5"
- board text added: "cam6"
- board text added: "cam7"
- board text added: "cam8"
- board text added: "cam9"
- board text added: "contact SZH-002T-P0.5"
