File: 10096510 Battery Connection/10096510 Battery Connection.sch (KiCad schematic (older format))
At the start: 12 parts, among them J1 09185107323, J3 811-S1-002-30-014101, J4 811-S1-002-30-014101, J5 811-S1-002-30-014101, J6 GKS-913-0024

Commit message: Updated symbol library. Changed MPN to Manufacturer_No, added "Item Number", and added "Documentation".
Parts:
- C1, C2: Documentation (none) -> ${KIPRJMOD}/Datasheets/YAGEO_CC0603KRX7R9BB103.pdf; Item Number (none) -> 10022508; MPN CC0603KRX7R9BB103 -> (none); Manufacturer_No (none) -> CC0603KRX7R9BB103
- C3, C4: Documentation (none) -> ${KIPRJMOD}/Datasheets/KEMET_C0402C470J5GAC.pdf; Item Number (none) -> 10022623; MPN C0402C470J5GAC -> (none); Manufacturer_No (none) -> C0402C470J5GAC
- FI1: Documentation (none) -> ${KIPRJMOD}/Datasheets/MURATA_BNX002-11.pdf; MPN BNX002-11 -> (none); Manufacturer_No (none) -> BNX002-11
- FI2, FI3: Documentation (none) -> ${KIPRJMOD}/Datasheets/WURTH_74279266.pdf; Item Number (none) -> 10022907; MPN 74279266 -> (none); Manufacturer_No (none) -> 74279266
- J1: Documentation (none) -> ${KIPRJMOD}/Datasheets/HARTING_09185107323.pdf; Item Number (none) -> 10023418; MPN 09185107323 -> (none); Manufacturer_No (none) -> 09185107323
- J3, J4, J5: Documentation (none) -> ${KIPRJMOD}/Datasheets/PRECI-DIP_811-S1-002-30-014101.pdf; Item Number (none) -> 10023420; MPN 811-S1-002-30-014101 -> (none); Manufacturer_No (none) -> 811-S1-002-30-014101
- J6: Documentation (none) -> ${KIPRJMOD}/Datasheets/INGUN_GKS-913 305 230 A 1502 S.pdf; Item Number (none) -> 10023419; MPN GKS-913 305 230 A 1502 S -> (none); Manufacturer_No (none) -> GKS-913 305 230 A 1502 S
Changed lines of the file:
@@
 F 1 "0402_47pF_C0402C470J5GAC" H 6950 3750 50  0001 L CNN
 F 2 "10096510_Battery_Connection:C_0402_1005Metric" H 7600 3850 50  0001 C CNN
-F 3 "${KIPRJMOD}/Datasheets/KEMET_C0402C470J5GAC.pdf" H 6600 3950 50  0001 C CNN
+F 3 "" H 6600 3950 50  0001 C CNN
 F 4 "Kemet" H 7070 4150 50  0001 C CNN "Manufacturer"
-F 5 "C0402C470J5GAC" H 7280 4050 50  0001 C CNN "MPN"
-F 6 "0402" H 7050 3950 50  0001 C CNN "Size"
-F 7 "50V" H 6715 3950 50  0000 L CNN "Voltage"
-F 8 "47pF" H 6715 3859 50  0000 L CNN "CAP_VAL"
+F 5 "0402" H 7050 3950 50  0001 C CNN "Size"
+F 6 "50V" H 6715 3950 50  0000 L CNN "Voltage"
+F 7 "47pF" H 6715 3859 50  0000 L CNN "CAP_VAL"
+F 8 "${KIPRJMOD}/Datasheets/KEMET_C0402C470J5GAC.pdf" H 0   0   50  0001 C CNN "Documentation"
+F 9 "10022623" H 0   0   50  0001 C CNN "Item Number"
+F 10 "C0402C470J5GAC" H 0   0   50  0001 C CNN "Manufacturer_No"
 	1    6600 3950
 	-1   0    0    -1
@@
 F 1 "0402_47pF_C0402C470J5GAC" H 6950 4600 50  0001 L CNN
 F 2 "10096510_Battery_Connection:C_0402_1005Metric" H 7600 4700 50  0001 C CNN
-F 3 "${KIPRJMOD}/Datasheets/KEMET_C0402C470J5GAC.pdf" H 6600 4800 50  0001 C CNN
+F 3 "" H 6600 4800 50  0001 C CNN
 F 4 "Kemet" H 7070 5000 50  0001 C CNN "Manufacturer"
-F 5 "C0402C470J5GAC" H 7280 4900 50  0001 C CNN "MPN"
-F 6 "0402" H 7050 4800 50  0001 C CNN "Size"
-F 7 "50V" H 6715 4800 50  0000 L CNN "Voltage"
-F 8 "47pF" H 6715 4709 50  0000 L CNN "CAP_VAL"
+F 5 "0402" H 7050 4800 50  0001 C CNN "Size"
+F 6 "50V" H 6715 4800 50  0000 L CNN "Voltage"
+F 7 "47pF" H 6715 4709 50  0000 L CNN "CAP_VAL"
+F 8 "${KIPRJMOD}/Datasheets/KEMET_C0402C470J5GAC.pdf" H 0   0   50  0001 C CNN "Documentation"
+F 9 "10022623" H 0   0   50  0001 C CNN "Item Number"
+F 10 "C0402C470J5GAC" H 0   0   50  0001 C CNN "Manufacturer_No"
 	1    6600 4800
 	1    0    0    -1
@@
 F 1 "09185107323" H 3000 4300 50  0000 R CNN
 F 2 "10096510_Battery_Connection:SHDRRA10W64P254_2X5_2050X890X930P" H 2700 4600 50  0001 C CNN
-F 3 "${KIPRJMOD}/Datasheets/HARTING_09185107323.pdf" H 2700 4600 50  0001 C CNN
+F 3 "" H 2700 4600 50  0001 C CNN
 F 4 "Harting" H 3450 4650 50  0001 C CNN "Manufacturer"
-F 5 "09185107323" H 3600 4550 50  0001 C CNN "MPN"
+F 5 "${KIPRJMOD}/Datasheets/HARTING_09185107323.pdf" H 0   0   50  0001 C CNN "Documentation"
+F 6 "10023418" H 0   0   50  0001 C CNN "Item Number"
+F 7 "09185107323" H 0   0   50  0001 C CNN "Manufacturer_No"
 	1    2700 4600
 	-1   0    0    1
@@
 F 1 "10nF" H 4736 2450 50  0000 R CNN
 F 2 "10096510_Battery_Connection:C_0603_1608Metric" H 5850 2250 50  0001 C CNN
-F 3 "${KIPRJMOD}/Datasheets/YAGEO_CC0603KRX7R9BB103.pdf" H 4850 2450 50  0001 C CNN
+F 3 "" H 4850 2450 50  0001 C CNN
 F 4 "Yageo" H 5300 2550 50  0001 C CNN "Manufacturer"
-F 5 "CC0603KRX7R9BB103" H 5600 2450 50  0001 C CNN "MPN"
-F 6 "0603" H 5300 2350 50  0001 C CNN "Size"
-F 7 "50V" H 4736 2541 50  0000 R CNN "Voltage"
-F 8 "10nF" H 4850 2450 50  0001 C CNN "CAP_VAL"
+F 5 "0603" H 5300 2350 50  0001 C CNN "Size"
+F 6 "50V" H 4736 2541 50  0000 R CNN "Voltage"
+F 7 "10nF" H 4850 2450 50  0000 C CNN "CAP_VAL"
+F 8 "${KIPRJMOD}/Datasheets/YAGEO_CC0603KRX7R9BB103.pdf" H 0   0   50  0001 C CNN "Documentation"
+F 9 "10022508" H 0   0   50  0001 C CNN "Item Number"
+F 10 "CC0603KRX7R9BB103" H 0   0   50  0001 C CNN "Manufacturer_No"
 	1    4850 2450
 	1    0    0    1
@@
 F 1 "BNX002-11" H 5575 2674 50  0000 C CNN
 F 2 "10096510_Battery_Connection:BNX002-011" H 5490 2370 50  0001 C CNN
-F 3 "${KIPRJMOD}/Datasheets/MURATA_BNX002-11.pdf" H 5490 2370 50  0001 C CNN
+F 3 "" H 5490 2370 50  0001 C CNN
 F 4 "10022532" H 5425 1975 50  0001 C CNN "Item Number"
 F 5 "Murata" H 5350 2050 50  0001 C CNN "Manufacturer"
-F 6 "BNX002-11" H 5450 1900 50  0001 C CNN "MPN"
+F 6 "${KIPRJMOD}/Datasheets/MURATA_BNX002-11.pdf" H 0   0   50  0001 C CNN "Documentation"
+F 7 "BNX002-11" H 0   0   50  0001 C CNN "Manufacturer_No"
 	1    5600 2350
 	1    0    0    -1
@@
 F 1 "811-S1-002-30-014101" H 8078 3630 50  0000 L CNN
 F 2 "10096510_Battery_Connection:CONN_811S100230014101" H 8100 3850 50  0001 L CNN
-F 3 "${KIPRJMOD}/Datasheets/PRECI-DIP_811-S1-002-30-014101.pdf" H 8100 3750 50  0001 L CNN
+F 3 "" H 8100 3750 50  0001 L CNN
 F 4 "CONN SPRING PISTON 2POS SMD" H 8100 3750 50  0001 L CNN "Description"
 F 5 "6mm" H 8100 3650 50  0001 L CNN "Height"
 F 6 "Preci-Dip" H 8100 3550 50  0001 L CNN "Manufacturer"
-F 7 "811-S1-002-30-014101" H 8100 3450 50  0001 L CNN "MPN"
+F 7 "${KIPRJMOD}/Datasheets/PRECI-DIP_811-S1-002-30-014101.pdf" H 0   0   50  0001 C CNN "Documentation"
+F 8 "10023420" H 0   0   50  0001 C CNN "Item Number"
+F 9 "811-S1-002-30-014101" H 0   0   50  0001 C CNN "Manufacturer_No"
 	1    7450 3750
 	1    0    0    -1
@@
 F 1 "811-S1-002-30-014101" H 8078 4480 50  0000 L CNN
 F 2 "10096510_Battery_Connection:CONN_811S100230014101" H 8100 4700 50  0001 L CNN
-F 3 "${KIPRJMOD}/Datasheets/PRECI-DIP_811-S1-002-30-014101.pdf" H 8100 4600 50  0001 L CNN
+F 3 "" H 8100 4600 50  0001 L CNN
 F 4 "CONN SPRING PISTON 2POS SMD" H 8100 4600 50  0001 L CNN "Description"
 F 5 "6mm" H 8100 4500 50  0001 L CNN "Height"
 F 6 "Preci-Dip" H 8100 4400 50  0001 L CNN "Manufacturer"
-F 7 "811-S1-002-30-014101" H 8100 4300 50  0001 L CNN "MPN"
+F 7 "${KIPRJMOD}/Datasheets/PRECI-DIP_811-S1-002-30-014101.pdf" H 0   0   50  0001 C CNN "Documentation"
+F 8 "10023420" H 0   0   50  0001 C CNN "Item Number"
+F 9 "811-S1-002-30-014101" H 0   0   50  0001 C CNN "Manufacturer_No"
 	1    7450 4600
 	1    0    0    -1
@@
 F 1 "GKS-913-0024" H 8400 5500 50  0000 C CNN
 F 2 "10096510_Battery_Connection:CONN_GKS-913-Z" H 7650 4950 50  0001 L CNN
-F 3 "${KIPRJMOD}/Datasheets/INGUN_GKS-913 305 230 A 1502 S" H 8100 5500 50  0001 L CNN
+F 3 "" H 8100 5500 50  0001 L CNN
 F 4 "Test probe" H 7650 5050 50  0001 L CNN "Description"
 F 5 "Ingun" H 7750 5250 50  0001 C CNN "Manufacturer"
-F 6 "GKS-913 305 230 A 1502 S" H 8200 5150 50  0001 C CNN "MPN"
+F 6 "${KIPRJMOD}/Datasheets/INGUN_GKS-913 305 230 A 1502 S.pdf" H 0   0   50  0001 C CNN "Documentation"
+F 7 "10023419" H 0   0   50  0001 C CNN "Item Number"
+F 8 "GKS-913 305 230 A 1502 S" H 0   0   50  0001 C CNN "Manufacturer_No"
 	1    7450 5500
 	1    0    0    -1
@@
 F 1 "74279266" H 3350 4783 50  0000 C CNN
 F 2 "10096510_Battery_Connection:L_0603_1608Metric" H 4750 4250 50  0001 C CNN
-F 3 "${KIPRJMOD}/Datasheets/WURTH_74279266.pdf" V 3350 4600 50  0001 C CNN
+F 3 "" V 3350 4600 50  0001 C CNN
 F 4 "Wurth Elektronik" H 4100 4850 50  0001 C CNN "Manufacturer"
-F 5 "74279266" H 4000 4750 50  0001 C CNN "MPN"
-F 6 "0603" H 3900 4550 50  0001 C CNN "Package"
-F 7 "1.00mm" H 3950 4450 50  0001 C CNN "Height"
-F 8 "200mA" H 3950 4350 50  0001 C CNN "Current Rating"
-F 9 "1kohm_at_100MHz" H 4150 4650 50  0001 C CNN "Impedance"
+F 5 "0603" H 3900 4550 50  0001 C CNN "Package"
+F 6 "1.00mm" H 3950 4450 50  0001 C CNN "Height"
+F 7 "200mA" H 3950 4350 50  0001 C CNN "Current Rating"
+F 8 "1kohm_at_100MHz" H 4150 4650 50  0001 C CNN "Impedance"
+F 9 "${KIPRJMOD}/Datasheets/WURTH_74279266.pdf" H 0   0   50  0001 C CNN "Documentation"
+F 10 "10022907" H 0   0   50  0001 C CNN "Item Number"
+F 11 "74279266" H 0   0   50  0001 C CNN "Manufacturer_No"
 	1    3350 4600
 	1    0    0    -1
@@
 F 1 "10nF" H 6665 2450 50  0000 L CNN
 F 2 "10096510_Battery_Connection:C_0603_1608Metric" H 7550 2250 50  0001 C CNN
-F 3 "${KIPRJMOD}/Datasheets/YAGEO_CC0603KRX7R9BB103.pdf" H 6550 2450 50  0001 C CNN
+F 3 "" H 6550 2450 50  0001 C CNN
 F 4 "Yageo" H 7000 2550 50  0001 C CNN "Manufacturer"
-F 5 "CC0603KRX7R9BB103" H 7300 2450 50  0001 C CNN "MPN"
-F 6 "0603" H 7000 2350 50  0001 C CNN "Size"
-F 7 "50V" H 6665 2359 50  0000 L CNN "Voltage"
-F 8 "10nF" H 6550 2450 50  0001 C CNN "CAP_VAL"
+F 5 "0603" H 7000 2350 50  0001 C CNN "Size"
+F 6 "50V" H 6665 2359 50  0000 L CNN "Voltage"
+F 7 "10nF" H 6550 2450 50  0000 C CNN "CAP_VAL"
+F 8 "${KIPRJMOD}/Datasheets/YAGEO_CC0603KRX7R9BB103.pdf" H 0   0   50  0001 C CNN "Documentation"
+F 9 "10022508" H 0   0   50  0001 C CNN "Item Number"
+F 10 "CC0603KRX7R9BB103" H 0   0   50  0001 C CNN "Manufacturer_No"
 	1    6550 2450
 	1    0    0    1
@@
 F 1 "74279266" H 1800 4783 50  0000 C CNN
 F 2 "10096510_Battery_Connection:L_0603_1608Metric" H 3200 4250 50  0001 C CNN
-F 3 "${KIPRJMOD}/Datasheets/WURTH_74279266.pdf" V 1800 4600 50  0001 C CNN
+F 3 "" V 1800 4600 50  0001 C CNN
 F 4 "Wurth Elektronik" H 2550 4850 50  0001 C CNN "Manufacturer"
-F 5 "74279266" H 2450 4750 50  0001 C CNN "MPN"
-F 6 "0603" H 2350 4550 50  0001 C CNN "Package"
-F 7 "1.00mm" H 2400 4450 50  0001 C CNN "Height"
-F 8 "200mA" H 2400 4350 50  0001 C CNN "Current Rating"
-F 9 "1kohm_at_100MHz" H 2600 4650 50  0001 C CNN "Impedance"
+F 5 "0603" H 2350 4550 50  0001 C CNN "Package"
+F 6 "1.00mm" H 2400 4450 50  0001 C CNN "Height"
+F 7 "200mA" H 2400 4350 50  0001 C CNN "Current Rating"
+F 8 "1kohm_at_100MHz" H 2600 4650 50  0001 C CNN "Impedance"
+F 9 "${KIPRJMOD}/Datasheets/WURTH_74279266.pdf" H 0   0   50  0001 C CNN "Documentation"
+F 10 "10022907" H 0   0   50  0001 C CNN "Item Number"
+F 11 "74279266" H 0   0   50  0001 C CNN "Manufacturer_No"
 	1    1800 4600
 	1    0    0    -1
@@
 F 1 "811-S1-002-30-014101" H 8078 2130 50  0000 L CNN
 F 2 "10096510_Battery_Connection:CONN_811S100230014101" H 8100 2350 50  0001 L CNN
-F 3 "${KIPRJMOD}/Datasheets/PRECI-DIP_811-S1-002-30-014101.pdf" H 8100 2250 50  0001 L CNN
+F 3 "" H 8100 2250 50  0001 L CNN
 F 4 "CONN SPRING PISTON 2POS SMD" H 8100 2250 50  0001 L CNN "Description"
 F 5 "6mm" H 8100 2150 50  0001 L CNN "Height"
 F 6 "Preci-Dip" H 8100 2050 50  0001 L CNN "Manufacturer"
-F 7 "811-S1-002-30-014101" H 8100 1950 50  0001 L CNN "MPN"
+F 7 "${KIPRJMOD}/Datasheets/PRECI-DIP_811-S1-002-30-014101.pdf" H 0   0   50  0001 C CNN "Documentation"
+F 8 "10023420" H 0   0   50  0001 C CNN "Item Number"
+F 9 "811-S1-002-30-014101" H 0   0   50  0001 C CNN "Manufacturer_No"
 	1    7450 2250
 	1    0    0    -1

Commit message: backannotate
Parts:
- C1: footprint 10096510_Battery_Connection:C_0603_1608Metric -> AllModules:C0603_4
- C2: footprint 10096510_Battery_Connection:C_0603_1608Metric -> AllModules:C0603_3
- C3: footprint 10096510_Battery_Connection:C_0402_1005Metric -> AllModules:C0402_2
- C4: footprint 10096510_Battery_Connection:C_0402_1005Metric -> AllModules:C0402_1
- FI1: footprint 10096510_Battery_Connection:BNX002-011 -> AllModules:BNX002_1
- FI2: footprint 10096510_Battery_Connection:L_0603_1608Metric -> AllModules:C0603_2
- FI3: footprint 10096510_Battery_Connection:L_0603_1608Metric -> AllModules:C0603_1
- J1: footprint 10096510_Battery_Connection:SHDRRA10W64P254_2X5_2050X890X930P -> AllModules:BP2X5C_1
- J3: footprint 10096510_Battery_Connection:CONN_811S100230014101 -> AllModules:811S1-02_3
- J4: footprint 10096510_Battery_Connection:CONN_811S100230014101 -> AllModules:811S1-02_2
- J5: footprint 10096510_Battery_Connection:CONN_811S100230014101 -> AllModules:811S1-02_1
- J6: footprint 10096510_Battery_Connection:CONN_GKS-913-Z -> AllModules:GKS913_1
Changed lines of the file:
@@
 F 0 "C3" H 6715 4041 50  0000 L CNN
 F 1 "0402_47pF_C0402C470J5GAC" H 6950 3750 50  0001 L CNN
-F 2 "10096510_Battery_Connection:C_0402_1005Metric" H 7600 3850 50  0001 C CNN
+F 2 "AllModules:C0402_2" H 7600 3850 50  0001 C CNN
 F 3 "" H 6600 3950 50  0001 C CNN
 F 4 "Kemet" H 7070 4150 50  0001 C CNN "Manufacturer"
@@
 F 0 "C4" H 6715 4891 50  0000 L CNN
 F 1 "0402_47pF_C0402C470J5GAC" H 6950 4600 50  0001 L CNN
-F 2 "10096510_Battery_Connection:C_0402_1005Metric" H 7600 4700 50  0001 C CNN
+F 2 "AllModules:C0402_1" H 7600 4700 50  0001 C CNN
 F 3 "" H 6600 4800 50  0001 C CNN
 F 4 "Kemet" H 7070 5000 50  0001 C CNN "Manufacturer"
@@
 F 0 "J1" H 2800 4200 50  0000 R CNN
 F 1 "09185107323" H 3000 4300 50  0000 R CNN
-F 2 "10096510_Battery_Connection:SHDRRA10W64P254_2X5_2050X890X930P" H 2700 4600 50  0001 C CNN
+F 2 "AllModules:BP2X5C_1" H 2700 4600 50  0001 C CNN
 F 3 "" H 2700 4600 50  0001 C CNN
 F 4 "Harting" H 3450 4650 50  0001 C CNN "Manufacturer"
@@
 F 0 "C1" H 4736 2359 50  0000 R CNN
 F 1 "10nF" H 4736 2450 50  0000 R CNN
-F 2 "10096510_Battery_Connection:C_0603_1608Metric" H 5850 2250 50  0001 C CNN
+F 2 "AllModules:C0603_4" H 5850 2250 50  0001 C CNN
 F 3 "" H 4850 2450 50  0001 C CNN
 F 4 "Yageo" H 5300 2550 50  0001 C CNN "Manufacturer"
@@
 F 0 "FI1" H 5575 2765 50  0000 C CNN
 F 1 "BNX002-11" H 5575 2674 50  0000 C CNN
-F 2 "10096510_Battery_Connection:BNX002-011" H 5490 2370 50  0001 C CNN
+F 2 "AllModules:BNX002_1" H 5490 2370 50  0001 C CNN
 F 3 "" H 5490 2370 50  0001 C CNN
 F 4 "10022532" H 5425 1975 50  0001 C CNN "Item Number"
@@
 F 0 "J4" H 8078 3721 50  0000 L CNN
 F 1 "811-S1-002-30-014101" H 8078 3630 50  0000 L CNN
-F 2 "10096510_Battery_Connection:CONN_811S100230014101" H 8100 3850 50  0001 L CNN
+F 2 "AllModules:811S1-02_2" H 8100 3850 50  0001 L CNN
 F 3 "" H 8100 3750 50  0001 L CNN
 F 4 "CONN SPRING PISTON 2POS SMD" H 8100 3750 50  0001 L CNN "Description"
@@
 F 0 "J5" H 8078 4571 50  0000 L CNN
 F 1 "811-S1-002-30-014101" H 8078 4480 50  0000 L CNN
-F 2 "10096510_Battery_Connection:CONN_811S100230014101" H 8100 4700 50  0001 L CNN
+F 2 "AllModules:811S1-02_1" H 8100 4700 50  0001 L CNN
 F 3 "" H 8100 4600 50  0001 L CNN
 F 4 "CONN SPRING PISTON 2POS SMD" H 8100 4600 50  0001 L CNN "Description"
@@
 F 0 "J6" H 8150 5600 50  0000 C CNN
 F 1 "GKS-913-0024" H 8400 5500 50  0000 C CNN
-F 2 "10096510_Battery_Connection:CONN_GKS-913-Z" H 7650 4950 50  0001 L CNN
+F 2 "AllModules:GKS913_1" H 7650 4950 50  0001 L CNN
 F 3 "" H 8100 5500 50  0001 L CNN
 F 4 "Test probe" H 7650 5050 50  0001 L CNN "Description"
@@
 F 0 "FI3" H 3350 4874 50  0000 C CNN
 F 1 "74279266" H 3350 4783 50  0000 C CNN
-F 2 "10096510_Battery_Connection:L_0603_1608Metric" H 4750 4250 50  0001 C CNN
+F 2 "AllModules:C0603_1" H 4750 4250 50  0001 C CNN
 F 3 "" V 3350 4600 50  0001 C CNN
 F 4 "Wurth Elektronik" H 4100 4850 50  0001 C CNN "Manufacturer"
@@
 F 0 "C2" H 6665 2541 50  0000 L CNN
 F 1 "10nF" H 6665 2450 50  0000 L CNN
-F 2 "10096510_Battery_Connection:C_0603_1608Metric" H 7550 2250 50  0001 C CNN
+F 2 "AllModules:C0603_3" H 7550 2250 50  0001 C CNN
 F 3 "" H 6550 2450 50  0001 C CNN
 F 4 "Yageo" H 7000 2550 50  0001 C CNN "Manufacturer"
@@
 F 0 "FI2" H 1800 4874 50  0000 C CNN
 F 1 "74279266" H 1800 4783 50  0000 C CNN
-F 2 "10096510_Battery_Connection:L_0603_1608Metric" H 3200 4250 50  0001 C CNN
+F 2 "AllModules:C0603_2" H 3200 4250 50  0001 C CNN
 F 3 "" V 1800 4600 50  0001 C CNN
 F 4 "Wurth Elektronik" H 2550 4850 50  0001 C CNN "Manufacturer"
@@
 F 0 "J3" H 8078 2221 50  0000 L CNN
 F 1 "811-S1-002-30-014101" H 8078 2130 50  0000 L CNN
-F 2 "10096510_Battery_Connection:CONN_811S100230014101" H 8100 2350 50  0001 L CNN
+F 2 "AllModules:811S1-02_3" H 8100 2350 50  0001 L CNN
 F 3 "" H 8100 2250 50  0001 L CNN
 F 4 "CONN SPRING PISTON 2POS SMD" H 8100 2250 50  0001 L CNN "Description"

Commit message: add cam as symbols
Parts:
- added CAM1: Fiducial, AllModules:FILM18_HORIZONTAL_1, symbol Mechanical:Fiducial
- added CAM10: Fiducial, AllModules:A3_PER_COVIDIEN_1, symbol Mechanical:Fiducial
- added CAM11: Fiducial, AllModules:FEE_COMP_2, symbol Mechanical:Fiducial
- added CAM12: Fiducial, AllModules:FABRICATION-FEE_1, symbol Mechanical:Fiducial
- added CAM14: Fiducial, AllModules:PERCAGE-MC_TABLEAU_1, symbol Mechanical:Fiducial
- added CAM16: Fiducial, AllModules:FEE_COMP_1, symbol Mechanical:Fiducial
- added CAM2: Fiducial, AllModules:A3_EQFC_COVIDIEN_1, symbol Mechanical:Fiducial
- added CAM3: Fiducial, AllModules:PER-COVIDIEN_TEXTE_1, symbol Mechanical:Fiducial
- added CAM4: Fiducial, AllModules:A3_EQFS_COVIDIEN_1, symbol Mechanical:Fiducial
- added CAM6, CAM7, CAM8, CAM9: Fiducial, AllModules:COIN_EXTERNE_1, symbol Mechanical:Fiducial
- added PT1, PT2: TestPoint, AllModules:MIRECMS_D-1.5_1, symbol Connector:TestPoint
Changed lines of the file:
@@
+	1    0    0    -1
+$EndComp
+$Comp
+L Connector:TestPoint PT1
+U 1 1 5E9E685B
+P 1650 6550
+F 0 "PT1" H 1708 6668 50  0000 L CNN
+F 1 "TestPoint" H 1708 6577 50  0000 L CNN
+F 2 "AllModules:MIRECMS_D-1.5_1" H 1850 6550 50  0001 C CNN
+F 3 "~" H 1850 6550 50  0001 C CNN
+	1    1650 6550
+	1    0    0    -1
+$EndComp
+$Comp
+L Connector:TestPoint PT2
+U 1 1 5E9E73E6
+P 1650 6850
+F 0 "PT2" H 1708 6968 50  0000 L CNN
+F 1 "TestPoint" H 1708 6877 50  0000 L CNN
+F 2 "AllModules:MIRECMS_D-1.5_1" H 1850 6850 50  0001 C CNN
+F 3 "~" H 1850 6850 50  0001 C CNN
+	1    1650 6850
+	1    0    0    -1
+$EndComp
+$Comp
+L Mechanical:Fiducial CAM1
+U 1 1 5E9EFCDE
+P 2700 6400
+F 0 "CAM1" H 2785 6400 50  0000 L CNN
+F 1 "Fiducial" H 2785 6355 50  0001 L CNN
+F 2 "AllModules:FILM18_HORIZONTAL_1" H 2700 6400 50  0001 C CNN
+F 3 "~" H 2700 6400 50  0001 C CNN
+	1    2700 6400
+	1    0    0    -1
+$EndComp
+$Comp
+L Mechanical:Fiducial CAM2
+U 1 1 5E9F043D
+P 2700 6550
+F 0 "CAM2" H 2785 6550 50  0000 L CNN
+F 1 "Fiducial" H 2785 6505 50  0001 L CNN
+F 2 "AllModules:A3_EQFC_COVIDIEN_1" H 2700 6550 50  0001 C CNN
+F 3 "~" H 2700 6550 50  0001 C CNN
+	1    2700 6550
+	1    0    0    -1
+$EndComp
+$Comp
+L Mechanical:Fiducial CAM3
+U 1 1 5E9F1828
+P 2700 6700
+F 0 "CAM3" H 2785 6700 50  0000 L CNN
+F 1 "Fiducial" H 2785 6655 50  0001 L CNN
+F 2 "AllModules:PER-COVIDIEN_TEXTE_1" H 2700 6700 50  0001 C CNN
+F 3 "~" H 2700 6700 50  0001 C CNN
+	1    2700 6700
+	1    0    0    -1
+$EndComp
+$Comp
+L Mechanical:Fiducial CAM4
+U 1 1 5E9F1832
+P 2700 6850
+F 0 "CAM4" H 2785 6850 50  0000 L CNN
+F 1 "Fiducial" H 2785 6805 50  0001 L CNN
+F 2 "AllModules:A3_EQFS_COVIDIEN_1" H 2700 6850 50  0001 C CNN
+F 3 "~" H 2700 6850 50  0001 C CNN
+	1    2700 6850
+	1    0    0    -1
+$EndComp
+$Comp
+L Mechanical:Fiducial CAM6
+U 1 1 5E9F54AD
+P 2700 7150
+F 0 "CAM6" H 2785 7150 50  0000 L CNN
+F 1 "Fiducial" H 2785 7105 50  0001 L CNN
+F 2 "AllModules:COIN_EXTERNE_1" H 2700 7150 50  0001 C CNN
+F 3 "~" H 2700 7150 50  0001 C CNN
+	1    2700 7150
+	1    0    0    -1
+$EndComp
+$Comp
+L Mechanical:Fiducial CAM7
+U 1 1 5E9F54B7
+P 2700 7300
+F 0 "CAM7" H 2785 7300 50  0000 L CNN
+F 1 "Fiducial" H 2785 7255 50  0001 L CNN
+F 2 "AllModules:COIN_EXTERNE_1" H 2700 7300 50  0001 C CNN
+F 3 "~" H 2700 7300 50  0001 C CNN
+	1    2700 7300
+	1    0    0    -1
+$EndComp
+$Comp
+L Mechanical:Fiducial CAM8
+U 1 1 5E9F54C1
+P 2700 7450
+F 0 "CAM8" H 2785 7450 50  0000 L CNN
+F 1 "Fiducial" H 2785 7405 50  0001 L CNN
+F 2 "AllModules:COIN_EXTERNE_1" H 2700 7450 50  0001 C CNN
+F 3 "~" H 2700 7450 50  0001 C CNN
+	1    2700 7450
+	1    0    0    -1
+$EndComp
+$Comp
+L Mechanical:Fiducial CAM9
+U 1 1 5E9FC9D9
+P 3150 6400
+F 0 "CAM9" H 3235 6400 50  0000 L CNN
+F 1 "Fiducial" H 3235 6355 50  0001 L CNN
+F 2 "AllModules:COIN_EXTERNE_1" H 3150 6400 50  0001 C CNN
+F 3 "~" H 3150 6400 50  0001 C CNN
+	1    3150 6400
+	1    0    0    -1
+$EndComp
+$Comp
+L Mechanical:Fiducial CAM10
+U 1 1 5E9FC9E3
+P 3150 6550
+F 0 "CAM10" H 3235 6550 50  0000 L CNN
+F 1 "Fiducial" H 3235 6505 50  0001 L CNN
+F 2 "AllModules:A3_PER_COVIDIEN_1" H 3150 6550 50  0001 C CNN
+F 3 "~" H 3150 6550 50  0001 C CNN
+	1    3150 6550
+	1    0    0    -1
+$EndComp
+$Comp
+L Mechanical:Fiducial CAM11
+U 1 1 5E9FC9ED
+P 3150 6700
+F 0 "CAM11" H 3235 6700 50  0000 L CNN
+F 1 "Fiducial" H 3235 6655 50  0001 L CNN
+F 2 "AllModules:FEE_COMP_2" H 3150 6700 50  0001 C CNN
+F 3 "~" H 3150 6700 50  0001 C CNN
+	1    3150 6700
+	1    0    0    -1
+$EndComp
+$Comp
+L Mechanical:Fiducial CAM12
+U 1 1 5E9FC9F7
+P 3150 6850
+F 0 "CAM12" H 3235 6850 50  0000 L CNN
+F 1 "Fiducial" H 3235 6805 50  0001 L CNN
+F 2 "AllModules:FABRICATION-FEE_1" H 3150 6850 50  0001 C CNN
+F 3 "~" H 3150 6850 50  0001 C CNN
+	1    3150 6850
+	1    0    0    -1
+$EndComp
+$Comp
+L Mechanical:Fiducial CAM14
+U 1 1 5E9FCA0B
+P 3150 7150
+F 0 "CAM14" H 3235 7150 50  0000 L CNN
+F 1 "Fiducial" H 3235 7105 50  0001 L CNN
+F 2 "AllModules:PERCAGE-MC_TABLEAU_1" H 3150 7150 50  0001 C CNN
+F 3 "~" H 3150 7150 50  0001 C CNN
+	1    3150 7150
+	1    0    0    -1
+$EndComp
+$Comp
+L Mechanical:Fiducial CAM16
+U 1 1 5E9FCA1F
+P 3150 7450
+F 0 "CAM16" H 3235 7450 50  0000 L CNN
+F 1 "Fiducial" H 3235 7405 50  0001 L CNN
+F 2 "AllModules:FEE_COMP_1" H 3150 7450 50  0001 C CNN
+F 3 "~" H 3150 7450 50  0001 C CNN
+	1    3150 7450
 	1    0    0    -1
 $EndComp

Commit message: repoint duplicated fp names
Parts:
- C1: footprint AllModules:C0603_4 -> AllModules:C0603_1
- C2: footprint AllModules:C0603_3 -> AllModules:C0603_1
- C3: footprint AllModules:C0402_2 -> AllModules:C0402_1
- FI2: footprint AllModules:C0603_2 -> AllModules:C0603_1
- J3: footprint AllModules:811S1-02_3 -> AllModules:811S1-02_1
- J4: footprint AllModules:811S1-02_2 -> AllModules:811S1-02_1
