File: 10096510 Battery Connection/10096510 Battery Connection.sch (KiCad schematic (older format))
At the start: 27 parts, among them J1 09185107323, J3 811-S1-002-30-014101, J4 811-S1-002-30-014101, J5 811-S1-002-30-014101, J6 GKS-913-0024

Commit message: migrate all to global library
Parts:
- C1, C2, FI2, FI3: footprint AllModules:C0603_1 -> AllModules:C0603_1b
- C3, C4: footprint AllModules:C0402_1 -> AllModules:C0402_1b
Changed lines of the file:
@@
 F 0 "C3" H 6715 4041 50  0000 L CNN
 F 1 "0402_47pF_C0402C470J5GAC" H 6950 3750 50  0001 L CNN
-F 2 "AllModules:C0402_1" H 7600 3850 50  0001 C CNN
+F 2 "AllModules:C0402_1b" H 7600 3850 50  0001 C CNN
 F 3 "" H 6600 3950 50  0001 C CNN
 F 4 "Kemet" H 7070 4150 50  0001 C CNN "Manufacturer"
@@
 F 0 "C4" H 6715 4891 50  0000 L CNN
 F 1 "0402_47pF_C0402C470J5GAC" H 6950 4600 50  0001 L CNN
-F 2 "AllModules:C0402_1" H 7600 4700 50  0001 C CNN
+F 2 "AllModules:C0402_1b" H 7600 4700 50  0001 C CNN
 F 3 "" H 6600 4800 50  0001 C CNN
 F 4 "Kemet" H 7070 5000 50  0001 C CNN "Manufacturer"
@@
 F 0 "C1" H 4736 2359 50  0000 R CNN
 F 1 "10nF" H 4736 2450 50  0000 R CNN
-F 2 "AllModules:C0603_1" H 5850 2250 50  0001 C CNN
+F 2 "AllModules:C0603_1b" H 5850 2250 50  0001 C CNN
 F 3 "" H 4850 2450 50  0001 C CNN
 F 4 "Yageo" H 5300 2550 50  0001 C CNN "Manufacturer"
@@
 F 0 "FI3" H 3350 4874 50  0000 C CNN
 F 1 "74279266" H 3350 4783 50  0000 C CNN
-F 2 "AllModules:C0603_1" H 4750 4250 50  0001 C CNN
+F 2 "AllModules:C0603_1b" H 4750 4250 50  0001 C CNN
 F 3 "" V 3350 4600 50  0001 C CNN
 F 4 "Wurth Elektronik" H 4100 4850 50  0001 C CNN "Manufacturer"
@@
 F 0 "C2" H 6665 2541 50  0000 L CNN
 F 1 "10nF" H 6665 2450 50  0000 L CNN
-F 2 "AllModules:C0603_1" H 7550 2250 50  0001 C CNN
+F 2 "AllModules:C0603_1b" H 7550 2250 50  0001 C CNN
 F 3 "" H 6550 2450 50  0001 C CNN
 F 4 "Yageo" H 7000 2550 50  0001 C CNN "Manufacturer"
@@
 F 0 "FI2" H 1800 4874 50  0000 C CNN
 F 1 "74279266" H 1800 4783 50  0000 C CNN
-F 2 "AllModules:C0603_1" H 3200 4250 50  0001 C CNN
+F 2 "AllModules:C0603_1b" H 3200 4250 50  0001 C CNN
 F 3 "" V 1800 4600 50  0001 C CNN
 F 4 "Wurth Elektronik" H 2550 4850 50  0001 C CNN "Manufacturer"

Commit message: ran renameSchSyms.py
Parts:
- C1, C2: symbol 10096510_Battery_Connection:0603_10nF_CC0603KRX7R9BB103 -> Capacitor:0603_10nF_CC0603KRX7R9BB103
- C3, C4: symbol 10096510_Battery_Connection:0402_47pF_C0402C470J5GAC -> Capacitor:0402_47pF_C0402C470J5GAC
- FI1: symbol 10096510_Battery_Connection:BNX002-11 -> Inductor:BNX002-11
- FI2, FI3: symbol 10096510_Battery_Connection:74279266 -> Inductor:74279266
- J1: symbol 10096510_Battery_Connection:09185107323 -> Connector:09185107323
- J3, J4, J5: symbol 10096510_Battery_Connection:811-S1-002-30-014101 -> Connector:811-S1-002-30-014101
- J6: symbol 10096510_Battery_Connection:GKS-913-0024 -> Connector:GKS-913-0024
Changed lines of the file:
@@
 	2250 4500 2250 4400
 $Comp
-L 10096510_Battery_Connection:0402_47pF_C0402C470J5GAC C3
+L Capacitor:0402_47pF_C0402C470J5GAC C3
 U 1 1 5E91F4F8
 P 6600 3950
@@
 $EndComp
 $Comp
-L 10096510_Battery_Connection:0402_47pF_C0402C470J5GAC C4
+L Capacitor:0402_47pF_C0402C470J5GAC C4
 U 1 1 5E9213A5
 P 6600 4800
@@
 	1150 3750 1150 4600
 $Comp
-L 10096510_Battery_Connection:09185107323 J1
+L Connector:09185107323 J1
 U 1 1 5E95772A
 P 2700 4600
@@
 	5050 2250 4850 2250
 $Comp
-L 10096510_Battery_Connection:0603_10nF_CC0603KRX7R9BB103 C1
+L Capacitor:0603_10nF_CC0603KRX7R9BB103 C1
 U 1 1 5E8FB3FB
 P 4850 2450
@@
 $EndComp
 $Comp
-L 10096510_Battery_Connection:BNX002-11 FI1
+L Inductor:BNX002-11 FI1
 U 1 1 5E8EDF96
 P 5600 2350
@@
 	7450 2250 7300 2250
 $Comp
-L 10096510_Battery_Connection:811-S1-002-30-014101 J4
+L Connector:811-S1-002-30-014101 J4
 U 1 1 5E99CA09
 P 7450 3750
@@
 $EndComp
 $Comp
-L 10096510_Battery_Connection:811-S1-002-30-014101 J5
+L Connector:811-S1-002-30-014101 J5
 U 1 1 5E99E657
 P 7450 4600
@@
 GND
 $Comp
-L 10096510_Battery_Connection:GKS-913-0024 J6
+L Connector:GKS-913-0024 J6
 U 1 1 5E9A6A5B
 P 7450 5500
@@
 	2250 4800 2400 4800
 $Comp
-L 10096510_Battery_Connection:74279266 FI3
+L Inductor:74279266 FI3
 U 1 1 5E9C95BC
 P 3350 4600
@@
 	1950 4600 2400 4600
 $Comp
-L 10096510_Battery_Connection:0603_10nF_CC0603KRX7R9BB103 C2
+L Capacitor:0603_10nF_CC0603KRX7R9BB103 C2
 U 1 1 5E90C557
 P 6550 2450
@@
 $EndComp
 $Comp
-L 10096510_Battery_Connection:74279266 FI2
+L Inductor:74279266 FI2
 U 1 1 5E9D0294
 P 1800 4600
@@
 $EndComp
 $Comp
-L 10096510_Battery_Connection:811-S1-002-30-014101 J3
+L Connector:811-S1-002-30-014101 J3
 U 1 1 5E99A69C
 P 7450 2250
